File: training-pcb/rgb-led.brd (EAGLE design)
At the start: 30 x 36 mm, 18 parts, among them J1 MICRO-USB, J2 AVR_SPI_PROG2PTH2, U1 ATTINY441/841SSU/SSUR, U2 TCA6507PW, U3 TPS78001DDCT

Commit message: New voltage regulator, route board, condense libraries
Parts:
- added C8: 100n, rcl:C0603
- C7: value 100n -> 1u
- D2: device SparkFun-LED:LED-RGB-THRU -> rgb-led:LED-RGB-THRU
- J1: device micro-usb-1:GS-14-2180 -> rgb-led:GS-14-2180
- J2: device SparkFun-Connectors:2X5-SHROUDED -> rgb-led:2X5-SHROUDED
- LED1: device RoboJackets-LEDs:5050 -> rgb-led:5050
- U1: device RoboJackets-ICs:SOIC-14 -> rgb-led:SOIC-14
- U2: device Texas Instruments_By_element14_Batch_1:SOP65P640X120-14N -> rgb-led:SOP65P640X120-14N
- U3: value TPS78001DDCT -> TLV70018DDCR; device Texas Instruments_By_element14_Batch_1:SOT95P280X110-5N -> rgb-led:SOT95P280X110-5N
- moved R2 51.1 mm to (5.70, 28.4), turned to 0 degrees
- moved C7 43.2 mm to (12.7, 23.9), turned to 90 degrees
- moved C6 39.6 mm to (15.6, 23.9), turned to 90 degrees
- moved R4 33.8 mm to (5.70, 33.1)
- moved U3 32.2 mm to (19.1, 22.9), turned to 180 degrees
- moved R3 26.1 mm to (5.70, 30.9)
- moved C5 25.8 mm to (18.1, 33.2), turned to 180 degrees
- moved J2 18.9 mm to (24.1, 10.8), flipped to the top
- moved C1 18.0 mm to (4.57, 5.28), turned to 270 degrees
- moved U1 14.7 mm to (6.86, 14.2), turned to 180 degrees
- moved J1 9.91 mm to (11.8, 2.52)
- moved U2 9.31 mm to (7.55, 23.9), turned to 180 degrees
- moved R1 8.12 mm to (25.8, 26.7)
- moved C2 8.00 mm to (12.2, 19.4), turned to 270 degrees
- moved D2 6.63 mm to (11.2, 31.3), turned to 270 degrees
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Connections:
- removed net N$6: C6.1, U3.5
- removed net VCC: U2.1
- new net +1.8V: C6.1, C7.1, U2.1, U3.5
- new net N$7: D2.3, R3.2
- new net N$8: D2.4, R4.2
- net +5V: now also C8.1, U3.3; no longer C7.1
- net GND: now also C8.2
Routing:
- net +5V: track 0.79 -> 83.1 mm, vias 0 -> 1
- net LED_CNTRL: track 0.00 -> 30.5 mm, vias 0 -> 2
- net MISO: track 0.18 -> 23.5 mm, vias 0 -> 1
- net SCK: track 0.00 -> 21.9 mm
- net MOSI: track 0.00 -> 21.3 mm
- net /RESET: track 5.37 -> 24.1 mm, vias 0 -> 2
- net N$5: track 0.00 -> 12.1 mm
- net EN: track 0.00 -> 10.5 mm
- net +1.8V: track 0.00 -> 9.40 mm
- net N$4: track 0.00 -> 8.28 mm
- net N$1: track 0.00 -> 8.21 mm
- net SDA: track 0.00 -> 8.16 mm
- net SCL: track 0.00 -> 7.01 mm
- net N$7: track 0.00 -> 5.05 mm
- net N$2: track 0.00 -> 5.04 mm
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- added copper zone on layer 16, net GND
