File: training-pcb/rgb-led.brd (EAGLE design)
At the start: 30 x 36 mm, 23 parts, among them J1 MICRO-USB, J2 AVR_SPI_PROG2PTH2, K1 SKQGADE010, U1 ATTINY441/841SSU/SSUR

Commit message: Fixed via overlap
Routing:
- net N$2: track 4.81 -> 5.97 mm
Changed lines of the file:
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@@
 <?xml version="1.0" encoding="utf-8"?>
 <!DOCTYPE eagle SYSTEM "eagle.dtd">
-<eagle version="7.6.0">
+<eagle version="7.5.0">
 <drawing>
 <settings>
@@
 <contactref element="R2" pad="1"/>
 <contactref element="K1" pad="2"/>
-<wire x1="4.3" y1="23.25" x2="3.75" y2="23.75" width="0.4064" layer="16"/>
-<wire x1="3.75" y1="23.75" x2="2.3" y2="25.2" width="0.4064" layer="1"/>
+<wire x1="4.3" y1="23.25" x2="4.25" y2="25.25" width="0.4064" layer="16"/>
+<wire x1="4.25" y1="25.25" x2="2.3" y2="25.2" width="0.4064" layer="1"/>
 <wire x1="2.3" y1="25.2" x2="2.3" y2="27.15" width="0.4064" layer="1"/>
 <wire x1="2.3" y1="27.15" x2="2.35" y2="27.2" width="0.4064" layer="1"/>
-<via x="3.75" y="23.75" extent="1-16" drill="0.6"/>
+<via x="4.25" y="25.25" extent="1-16" drill="0.6"/>
 </signal>
 <signal name="/BTN">

Commit message: PCB fixes for overlaps
Parts:
- moved C9 0.20 mm to (3.80, 28.9)
Changed lines of the file:
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@@
 <?xml version="1.0" encoding="utf-8"?>
 <!DOCTYPE eagle SYSTEM "eagle.dtd">
-<eagle version="7.5.0">
+<eagle version="7.6.0">
 <drawing>
 <settings>
@@
 </class>
 </classes>
-<designrules name="default">
+<designrules name="default *">
 <description language="de">&lt;b&gt;EAGLE Design Rules&lt;/b&gt;
 &lt;p&gt;
@@
 <param name="mdSmdStop" value="0mil"/>
 <param name="msWidth" value="10mil"/>
-<param name="msDrill" value="24mil"/>
+<param name="msDrill" value="20mil"/>
 <param name="msMicroVia" value="9.99mm"/>
 <param name="msBlindViaRatio" value="0.5"/>
-<param name="rvPadTop" value="0.25"/>
-<param name="rvPadInner" value="0.25"/>
-<param name="rvPadBottom" value="0.25"/>
+<param name="rvPadTop" value="0.15"/>
+<param name="rvPadInner" value="0.15"/>
+<param name="rvPadBottom" value="0.15"/>
 <param name="rvViaOuter" value="0.25"/>
 <param name="rvViaInner" value="0.25"/>
 <param name="rvMicroViaOuter" value="0.25"/>
 <param name="rvMicroViaInner" value="0.25"/>
-<param name="rlMinPadTop" value="10mil"/>
+<param name="rlMinPadTop" value="0mil"/>
 <param name="rlMaxPadTop" value="20mil"/>
-<param name="rlMinPadInner" value="10mil"/>
+<param name="rlMinPadInner" value="0mil"/>
 <param name="rlMaxPadInner" value="20mil"/>
-<param name="rlMinPadBottom" value="10mil"/>
+<param name="rlMinPadBottom" value="0mil"/>
 <param name="rlMaxPadBottom" value="20mil"/>
 <param name="rlMinViaOuter" value="8mil"/>
@@
 <element name="R6" library="resistor" package="R0805" value="" x="14.1" y="28.7" rot="MR90"/>
 <element name="R7" library="resistor" package="R0805" value="" x="7" y="33.4" rot="MR180"/>
-<element name="C9" library="rcl" package="C0603" value="100n" x="4" y="28.9" rot="MR90"/>
+<element name="C9" library="rcl" package="C0603" value="100n" x="3.8" y="28.9" rot="MR90"/>
 <element name="R9" library="resistor" package="R0805" value="10K" x="18.4" y="28.1" rot="R90"/>
 <element name="R8" library="resistor" package="R0805" value="10K" x="18.1" y="23.5"/>
@@
 <via x="10.7" y="19.255" extent="1-16" drill="0.6"/>
 <wire x1="10.7" y1="19.255" x2="10.7" y2="21.35" width="0.4064" layer="16"/>
-<wire x1="10.7" y1="21.35" x2="4" y2="28.05" width="0.4064" layer="16"/>
 <wire x1="4.3" y1="21.35" x2="7.05" y2="21.35" width="0.4064" layer="16"/>
 <wire x1="7.05" y1="21.35" x2="9.1" y2="19.3" width="0.4064" layer="16"/>
@@
 <wire x1="18.84" y1="32.87" x2="18.86" y2="32.85" width="0.4064" layer="1"/>
 <wire x1="18.86" y1="32.85" x2="21.79" y2="32.85" width="0.4064" layer="1"/>
+<wire x1="3.8" y1="28.05" x2="4" y2="28.05" width="0.4064" layer="16"/>
+<wire x1="4" y1="28.05" x2="10.7" y2="21.35" width="0.4064" layer="16"/>
 </signal>
 <signal name="MOSI">
@@
 <contactref element="U$1" pad="7"/>
 <contactref element="R8" pad="1"/>
-<wire x1="8.13" y1="16.77" x2="8.13" y2="19.33" width="0.4064" layer="1"/>
-<wire x1="8.13" y1="19.33" x2="12" y2="23.1" width="0.4064" layer="1"/>
-<wire x1="12" y1="23.1" x2="12.4" y2="28.135" width="0.4064" layer="1"/>
-<wire x1="12.4" y1="28.135" x2="16.054" y2="28.235" width="0.4064" layer="1"/>
-<via x="12" y="23.1" extent="1-16" drill="0.6"/>
-<wire x1="12" y1="23.1" x2="15" y2="23.1" width="0.4064" layer="16"/>
+<wire x1="8.13" y1="16.77" x2="8.13" y2="19.43" width="0.4064" layer="1"/>
+<via x="11.8" y="23.1" extent="1-16" drill="0.6"/>
+<wire x1="11.8" y1="23.1" x2="15" y2="23.1" width="0.4064" layer="16"/>
 <via x="15" y="23.1" extent="1-16" drill="0.6"/>
 <wire x1="15" y1="23.1" x2="16.75" y2="23.1" width="0.4064" layer="1"/>
 <wire x1="16.75" y1="23.1" x2="17.15" y2="23.5" width="0.4064" layer="1"/>
+<wire x1="11.8" y1="23.1" x2="8.13" y2="19.43" width="0.4064" layer="1"/>
+<wire x1="16.054" y1="28.235" x2="13.135" y2="28.235" width="0.4064" layer="1"/>
+<wire x1="13.135" y1="28.235" x2="11.8" y2="26.9" width="0.4064" layer="1"/>
+<wire x1="11.8" y1="26.9" x2="11.8" y2="23.1" width="0.4064" layer="1"/>
 </signal>
 <signal name="N$6">
@@
 <contactref element="R5" pad="1"/>
 <wire x1="9.746" y1="29.505" x2="9.741" y2="29.5" width="0.4064" layer="1"/>
-<wire x1="9.741" y1="29.5" x2="5.5" y2="29.5" width="0.4064" layer="1"/>
-<via x="5.5" y="29.5" extent="1-16" drill="0.6"/>
-<wire x1="5.5" y1="29.5" x2="5.5" y2="27.6" width="0.4064" layer="16"/>
-<wire x1="5.5" y1="27.6" x2="11.5" y2="21.6" width="0.4064" layer="16"/>
+<via x="5.4" y="29.5" extent="1-16" drill="0.6"/>
+<wire x1="5.4" y1="27.7" x2="11.5" y2="21.6" width="0.4064" layer="16"/>
 <wire x1="11.5" y1="21.6" x2="16.7" y2="21.6" width="0.4064" layer="16"/>
 <wire x1="16.7" y1="21.6" x2="16.7" y2="27.75" width="0.4064" layer="16"/>
+<wire x1="9.741" y1="29.5" x2="5.4" y2="29.5" width="0.4064" layer="1"/>
+<wire x1="5.4" y1="29.5" x2="5.4" y2="27.7" width="0.4064" layer="16"/>
 </signal>
 <signal name="N$12">

Commit message: Resize board to 30x30 then reroute
Parts:
- moved R7 11.3 mm to (7.90, 22.1), turned to 90 degrees
- moved U$1 9.52 mm to (11.4, 18.2)
- moved R6 7.47 mm to (10.6, 22.1)
- moved D1 7.42 mm to (13.3, 26.0)
- moved R5 7.38 mm to (13.4, 22.1)
- moved C2 6.08 mm to (14.8, 13.9), flipped to the bottom
- moved C3 6.08 mm to (17.1, 13.9), flipped to the bottom
- moved C4 6.08 mm to (19.4, 13.9), flipped to the bottom
- moved C9 5.82 mm to (8.60, 25.6), flipped to the top, turned to 180 degrees
- moved C5 5.55 mm to (19.3, 27.5)
- moved LED1 5.42 mm to (24.7, 25.8)
- moved R9 5.32 mm to (19.9, 23.0)
- moved R1 3.79 mm to (24.2, 22.1), turned to 180 degrees
- moved C6 3.45 mm to (4.70, 7.50), flipped to the bottom, turned to 270 degrees
- moved U1 1.79 mm to (8.46, 13.4), flipped to the bottom
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Routing:
- net N$11: track 26.1 -> 6.88 mm
- net +5V: track 95.3 -> 78.8 mm
- net MISO: track 23.1 -> 13.9 mm
- net SCK: track 21.9 -> 14.9 mm, vias 0 -> 1
- net /RESET: track 24.1 -> 18.6 mm, vias 2 -> 1
- net SDA: track 22.0 -> 16.8 mm, vias 2 -> 1
- net MOSI: track 21.7 -> 16.7 mm, vias 0 -> 1
- net N$12: track 9.22 -> 4.51 mm
- net LED_CNTRL: track 29.6 -> 25.2 mm, vias 2 -> 1
- net SCL: track 17.5 -> 21.6 mm, vias 0 -> 1
- net N$13: track 9.99 -> 6.02 mm
- net N$1: track 8.93 -> 6.23 mm
- net N$9: track 5.79 -> 3.81 mm
- net N$10: track 2.84 -> 4.72 mm
- net N$6: track 4.62 -> 3.70 mm
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Other:
- board size 30 x 36 mm -> 30 x 30 mm

Commit message: Clean up routing, fix silkscreen labels
Parts:
- moved C9 3.01 mm to (9.40, 22.7)
- moved C1 1.84 mm to (4.57, 5.28)
- moved C6 1.20 mm to (5.60, 6.70)
- moved C7 0.94 mm to (2.80, 6.70)
- moved R3 0.50 mm to (2.80, 15.0)
- moved K1 0.10 mm to (4.30, 24.1)
- renumbered U$1 to U2
Routing:
- net +5V: track 78.8 -> 75.0 mm
- net /BTN: track 13.9 -> 14.8 mm

Commit message: Added pullup on reset pin
Parts:
- added R4: 10k, resistor:R0805
Connections:
- net +5V: now also R4.2
- net /RESET: now also R4.1
Routing:
- net /RESET: track 18.6 -> 22.5 mm
- net +5V: track 75.0 -> 78.1 mm
Changed lines of the file:
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@@
 <attribute name="VALUE" x="5.34" y="15.635" size="1.27" layer="28" rot="MR270"/>
 </element>
+<element name="R4" library="resistor" package="R0805" value="10k" x="8.2" y="10.7" rot="R180"/>
 </elements>
 <signals>
@@
 <wire x1="9.744" y1="6.9" x2="4.79" y2="6.9" width="0.4064" layer="1"/>
 <wire x1="4.79" y1="6.9" x2="4.574" y2="6.684" width="0.4064" layer="1"/>
-<wire x1="4.79" y1="6.9" x2="4.79" y2="13.11" width="0.4064" layer="1"/>
+<wire x1="4.79" y1="6.9" x2="4.79" y2="9.2" width="0.4064" layer="1"/>
+<wire x1="4.79" y1="9.2" x2="4.79" y2="13.11" width="0.4064" layer="1"/>
 <wire x1="4.79" y1="13.11" x2="4.7" y2="13.5" width="0.4064" layer="1"/>
 <wire x1="4.65" y1="15.97" x2="4.65" y2="13.55" width="0.4064" layer="16"/>
@@
 <wire x1="12.7" y1="12.9" x2="13.5" y2="13.7" width="0.4064" layer="16"/>
 <wire x1="13.5" y1="13.7" x2="13.5" y2="14.3" width="0.4064" layer="16"/>
+<contactref element="R4" pad="2"/>
+<wire x1="7.25" y1="10.7" x2="6.29" y2="10.7" width="0.4064" layer="1"/>
+<wire x1="6.29" y1="10.7" x2="4.79" y2="9.2" width="0.4064" layer="1"/>
 </signal>
 <signal name="MOSI">
@@
 <wire x1="9" y1="14.1" x2="11" y2="14.1" width="0.4064" layer="16"/>
 <wire x1="11" y1="14.1" x2="11" y2="13.1" width="0.4064" layer="1"/>
-<wire x1="11" y1="13.1" x2="14.2" y2="9.9" width="0.4064" layer="1"/>
+<wire x1="11" y1="13.1" x2="12.7" y2="11.4" width="0.4064" layer="1"/>
+<wire x1="12.7" y1="11.4" x2="14.2" y2="9.9" width="0.4064" layer="1"/>
 <wire x1="14.2" y1="9.9" x2="22.023" y2="9.9" width="0.4064" layer="1"/>
 <wire x1="22.023" y1="9.9" x2="22.876" y2="10.753" width="0.4064" layer="1"/>
+<contactref element="R4" pad="1"/>
+<wire x1="9.15" y1="10.7" x2="12" y2="10.7" width="0.4064" layer="1"/>
+<wire x1="12" y1="10.7" x2="12.7" y2="11.4" width="0.4064" layer="1"/>
 </signal>
 <signal name="MISO">

Commit message: Minor PCB changes, change resistor sizes
Parts:
- added U$2: (no value), RoboJackets-Aesthetics:ROBOBUZZ_0.4X
- C1: value 100u -> 47u
- R2, R4, R5, R6, R7, R8, R9: device resistor:R0805 -> resistor:R0603
- moved C1 2.80 mm to (7.37, 5.42)
- moved J1 1.91 mm to (13.7, 2.52)
Connections:
- net GND: now also J1.5@1, J1.5@2, J1.5@3, J1.5@4, J1.5@6, J1.5@7
Routing:
- net +5V: track 78.1 -> 78.9 mm
Other:
- board text added: "25 Aug 2016"

Commit message: Minor pcb routing changes
Routing:
- net +5V: track 78.9 -> 79.6 mm

Commit message: Fix library files
Parts:
- K1: device Seeed-OPL-Button:SW4-SMD-5.2X5.2X1.5MM -> rgb-led:SW4-SMD-5.2X5.2X1.5MM
- U2: device adam - ics:SOIC8 -> rgb-led:SOIC8
Changed lines of the file:
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@@
 <attribute name="NAME" x="3.94" y="12.69" size="0.7" layer="26" rot="MR270"/>
 </element>
-<element name="U2" library="adam - ics" package="SOIC8" value="PCA9533" x="11.4" y="18.2" smashed="yes" rot="R270">
+<element name="U2" library="rgb-led" package="SOIC8" value="PCA9533" x="11.4" y="18.2" smashed="yes" rot="R270">
 <attribute name="NAME" x="10.941" y="14.6875" size="0.7" layer="25" ratio="10"/>
 <attribute name="VALUE" x="9.241" y="14.136" size="0.7" layer="27" ratio="10"/>
@@
 <attribute name="VALUE" x="20.04" y="22.365" size="0.7" layer="27" rot="R90"/>
 </element>
-<element name="K1" library="Seeed-OPL-Button" package="SW4-SMD-5.2X5.2X1.5MM" value="SKQGADE010" x="4.3" y="24.1" smashed="yes" rot="R90">
+<element name="K1" library="rgb-led" package="SW4-SMD-5.2X5.2X1.5MM" value="SKQGADE010" x="4.3" y="24.1" smashed="yes" rot="R90">
 <attribute name="MPN" value="SKQGADE010" x="4.3" y="24.1" size="1.778" layer="27" rot="R90" display="off"/>
 <attribute name="NAME" x="4.876" y="21.395" size="0.7" layer="25" ratio="11" rot="R180"/>
