File: training-pcb/rgb-led.sch (EAGLE design)
At the start: 23 parts, among them J1 MICRO-USB, J2 AVR_SPI_PROG2PTH2, K1 SKQGADE010, U1 ATTINY441/841SSU/SSUR

Commit message: Clean up routing, fix silkscreen labels
Parts:
- renumbered U$1 to U2
Changed lines of the file:
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@@
 <part name="C5" library="rcl" deviceset="C-US" device="C0603" value="100n"/>
 <part name="SUPPLY9" library="supply2" deviceset="GND" device=""/>
-<part name="U$1" library="adam - ics" deviceset="PCA9533" device=""/>
+<part name="U2" library="adam - ics" deviceset="PCA9533" device=""/>
 <part name="SUPPLY17" library="supply2" deviceset="GND" device=""/>
 <part name="D1" library="rgb-led" deviceset="LED-RGB-CA-THRU" device="CLEAR"/>
@@
 <instance part="C5" gate="G$1" x="20.32" y="60.96"/>
 <instance part="SUPPLY9" gate="GND" x="20.32" y="50.8"/>
-<instance part="U$1" gate="G$1" x="241.3" y="68.58"/>
+<instance part="U2" gate="G$1" x="241.3" y="68.58"/>
 <instance part="SUPPLY17" gate="GND" x="231.14" y="60.96"/>
 <instance part="D1" gate="G$1" x="261.62" y="101.6" smashed="yes" rot="R90">
@@
 </segment>
 <segment>
-<pinref part="U$1" gate="G$1" pin="VSS"/>
+<pinref part="U2" gate="G$1" pin="VSS"/>
 <pinref part="SUPPLY17" gate="GND" pin="GND"/>
 </segment>
@@
 </segment>
 <segment>
-<pinref part="U$1" gate="G$1" pin="VDD"/>
+<pinref part="U2" gate="G$1" pin="VDD"/>
 <wire x1="157.48" y1="93.98" x2="190.5" y2="93.98" width="0.1524" layer="91"/>
 <pinref part="C9" gate="G$1" pin="1"/>
@@
 </segment>
 <segment>
-<pinref part="U$1" gate="G$1" pin="SCL"/>
+<pinref part="U2" gate="G$1" pin="SCL"/>
 <wire x1="218.44" y1="81.28" x2="190.5" y2="81.28" width="0.1524" layer="91"/>
 <label x="170.18" y="81.28" size="1.778" layer="95"/>
@@
 </segment>
 <segment>
-<pinref part="U$1" gate="G$1" pin="SDA"/>
+<pinref part="U2" gate="G$1" pin="SDA"/>
 <label x="170.18" y="76.2" size="1.778" layer="95"/>
 <wire x1="218.44" y1="76.2" x2="200.66" y2="76.2" width="0.1524" layer="91"/>
@@
 <net name="N$11" class="0">
 <segment>
-<pinref part="U$1" gate="G$1" pin="LED0"/>
+<pinref part="U2" gate="G$1" pin="LED0"/>
 <pinref part="R5" gate="G$1" pin="1"/>
 <wire x1="246.38" y1="86.36" x2="256.54" y2="86.36" width="0.1524" layer="91"/>
@@
 <pinref part="R6" gate="G$1" pin="1"/>
 <wire x1="261.62" y1="86.36" x2="261.62" y2="81.28" width="0.1524" layer="91"/>
-<pinref part="U$1" gate="G$1" pin="LED1"/>
+<pinref part="U2" gate="G$1" pin="LED1"/>
 <wire x1="261.62" y1="81.28" x2="246.38" y2="81.28" width="0.1524" layer="91"/>
 </segment>
@@
 <pinref part="R7" gate="G$1" pin="1"/>
 <wire x1="266.7" y1="86.36" x2="266.7" y2="76.2" width="0.1524" layer="91"/>
-<pinref part="U$1" gate="G$1" pin="LED2"/>
+<pinref part="U2" gate="G$1" pin="LED2"/>
 <wire x1="266.7" y1="76.2" x2="246.38" y2="76.2" width="0.1524" layer="91"/>
 </segment>

Commit message: Added pullup on reset pin
Parts:
- added R4: 10k, resistor:R-US_R0805
Connections:
- net +5V: now also R4.2
- net /RESET: now also R4.1
Changed lines of the file:
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@@
 <part name="SUPPLY13" library="supply2" deviceset="+5V" device=""/>
 <part name="R3" library="resistor" deviceset="R-US_" device="R0805" value="39K"/>
+<part name="R4" library="resistor" deviceset="R-US_" device="R0805" value="10k"/>
+<part name="SUPPLY14" library="supply2" deviceset="+5V" device=""/>
 </parts>
 <sheets>
@@
 <attribute name="VALUE" x="119.38" y="88.392" size="1.778" layer="96" rot="R180"/>
 </instance>
+<instance part="R4" gate="G$1" x="259.08" y="147.32" smashed="yes" rot="R90">
+<attribute name="NAME" x="257.5814" y="143.51" size="1.778" layer="95" rot="R90"/>
+<attribute name="VALUE" x="262.382" y="143.51" size="1.778" layer="96" rot="R90"/>
+</instance>
+<instance part="SUPPLY14" gate="+5V" x="259.08" y="154.94"/>
 </instances>
 <busses>
@@
 <junction x="231.14" y="93.98"/>
 </segment>
+<segment>
+<pinref part="R4" gate="G$1" pin="2"/>
+<pinref part="SUPPLY14" gate="+5V" pin="+5V"/>
+</segment>
 </net>
 <net name="MOSI" class="0">
@@
 <segment>
 <pinref part="U1" gate="G$1" pin="PB3(PCINT11/ADC9/RESET'/DW)"/>
-<wire x1="226.06" y1="142.24" x2="251.46" y2="142.24" width="0.1524" layer="91"/>
+<wire x1="226.06" y1="142.24" x2="259.08" y2="142.24" width="0.1524" layer="91"/>
 <label x="241.3" y="142.24" size="1.778" layer="95"/>
-</segment>
-</net>
+<pinref part="R4" gate="G$1" pin="1"/>
+<wire x1="259.08" y1="142.24" x2="261.62" y2="142.24" width="0.1524" layer="91"/>
+<junction x="259.08" y="142.24"/>
+</segment>
+</net>

Commit message: Minor PCB changes, change resistor sizes
Parts:
- C1: value 100u -> 47u
- R2, R4, R5, R6, R7, R8, R9: device resistor:R-US_R0805 -> resistor:R-US_R0603
Changed lines of the file:
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@@
 </variantdefs>
 <classes>
-<class number="0" name="default" width="0" drill="0">
+<class number="0" name="default" width="0.2032" drill="0">
+</class>
+<class number="1" name="PWR" width="0.254" drill="0">
 </class>
 </classes>
@@
 </part>
 <part name="U1" library="rgb-led" deviceset="ATTINY441/841" device="SSU/SSUR"/>
-<part name="C1" library="rcl" deviceset="C-US" device="C1206" value="100u"/>
+<part name="C1" library="rcl" deviceset="C-US" device="C1206" value="47u"/>
 <part name="SUPPLY1" library="supply2" deviceset="+5V" device=""/>
 <part name="SUPPLY2" library="supply2" deviceset="GND" device=""/>
@@
 <part name="SUPPLY17" library="supply2" deviceset="GND" device=""/>
 <part name="D1" library="rgb-led" deviceset="LED-RGB-CA-THRU" device="CLEAR"/>
-<part name="R5" library="resistor" deviceset="R-US_" device="R0805"/>
-<part name="R6" library="resistor" deviceset="R-US_" device="R0805"/>
-<part name="R7" library="resistor" deviceset="R-US_" device="R0805"/>
+<part name="R5" library="resistor" deviceset="R-US_" device="R0603"/>
+<part name="R6" library="resistor" deviceset="R-US_" device="R0603"/>
+<part name="R7" library="resistor" deviceset="R-US_" device="R0603"/>
 <part name="SUPPLY19" library="supply2" deviceset="GND" device=""/>
 <part name="C9" library="rcl" deviceset="C-US" device="C0603" value="100n"/>
-<part name="R9" library="resistor" deviceset="R-US_" device="R0805" value="10K"/>
-<part name="R8" library="resistor" deviceset="R-US_" device="R0805" value="10K"/>
+<part name="R9" library="resistor" deviceset="R-US_" device="R0603" value="10K"/>
+<part name="R8" library="resistor" deviceset="R-US_" device="R0603" value="10K"/>
 <part name="K1" library="Seeed-OPL-Button" deviceset="SMD-SWITCH-TOP-260GF(4P-D5.2MM)" device="" value="SKQGADE010"/>
 <part name="SUPPLY10" library="supply2" deviceset="+5V" device=""/>
-<part name="R2" library="resistor" deviceset="R-US_" device="R0805" value="10K"/>
+<part name="R2" library="resistor" deviceset="R-US_" device="R0603" value="10K"/>
 <part name="SUPPLY11" library="supply2" deviceset="GND" device=""/>
 <part name="C6" library="rcl" deviceset="C-US" device="C0603" value="100n"/>
@@
 <part name="SUPPLY13" library="supply2" deviceset="+5V" device=""/>
 <part name="R3" library="resistor" deviceset="R-US_" device="R0805" value="39K"/>
-<part name="R4" library="resistor" deviceset="R-US_" device="R0805" value="10k"/>
+<part name="R4" library="resistor" deviceset="R-US_" device="R0603" value="10k"/>
 <part name="SUPPLY14" library="supply2" deviceset="+5V" device=""/>
 </parts>
@@
 </segment>
 </net>
-<net name="+5V" class="0">
+<net name="+5V" class="1">
 <segment>
 <pinref part="U1" gate="G$1" pin="VCC"/>

Commit message: Fix library files
Parts:
- K1: device Seeed-OPL-Button:SMD-SWITCH-TOP-260GF(4P-D5.2MM) -> rgb-led:SMD-SWITCH-TOP-260GF(4P-D5.2MM)
- U2: device adam - ics:PCA9533 -> rgb-led:PCA9533
Changed lines of the file:
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@@
 <part name="C5" library="rcl" deviceset="C-US" device="C0603" value="100n"/>
 <part name="SUPPLY9" library="supply2" deviceset="GND" device=""/>
-<part name="U2" library="adam - ics" deviceset="PCA9533" device=""/>
+<part name="U2" library="rgb-led" deviceset="PCA9533" device=""/>
 <part name="SUPPLY17" library="supply2" deviceset="GND" device=""/>
 <part name="D1" library="rgb-led" deviceset="LED-RGB-CA-THRU" device="CLEAR"/>
@@
 <part name="R9" library="resistor" deviceset="R-US_" device="R0603" value="10K"/>
 <part name="R8" library="resistor" deviceset="R-US_" device="R0603" value="10K"/>
-<part name="K1" library="Seeed-OPL-Button" deviceset="SMD-SWITCH-TOP-260GF(4P-D5.2MM)" device="" value="SKQGADE010"/>
+<part name="K1" library="rgb-led" deviceset="SMD-SWITCH-TOP-260GF(4P-D5.2MM)" device="" value="SKQGADE010"/>
 <part name="SUPPLY10" library="supply2" deviceset="+5V" device=""/>
 <part name="R2" library="resistor" deviceset="R-US_" device="R0603" value="10K"/>

Commit message: began arduino code directory
Parts:
- C1, C2, C3, C4, C5, C6, C7, C9, D1, J2, K1, LED1, R1, R3, R4, R5, R6, R7, U1: OC_NEWARK (none) -> unknown
- J1: MPN (none) -> 10104110-0001LF; OC_NEWARK (none) -> 82R7424
- R2, R8, R9: MF (none) -> FARNELL; MPN (none) -> MCF 0.25W 10K; OC_NEWARK (none) -> 38K0328
- U2: MPN (none) -> PCA9533DP/01,118; OC_NEWARK (none) -> 70R6524
