File: 2017-2018/lcd-buzzer.brd (EAGLE design)
At the start: 160 x 100 mm, 11 parts, among them J1 AVR_SPI_PROG2PTH2, U1 ATMEGA328P-MUR, U2 DRV2605YZFR, U3 74HC595PW, U4 74HC595PW, U5 74HC595PW, U6 74HC595PW

Commit message: First Version Completed
Added extra custom parts to the library, completed the schematics
Parts:
- removed J1: AVR_SPI_PROG2PTH2, rgb-led:2X5-SHROUDED
- added C3: 0.1uF, SparkFun-Capacitors:0603
- added SV1: (no value), con-lstb:MA03-2
- added U$2: LCD-S401C39TR, lcd-buzzer:S401C39TR
- added U$3: TC33X, lcd-buzzer:TC33X-2-103E
- added U$4: PS1240P02BT, lcd-buzzer:PS1240P02BT
- moved C2 73.9 mm to (-21.6, 63.5)
- moved U2 70.8 mm to (-15.2, 63.5)
- moved U3 44.9 mm to (-59.7, 34.3)
- moved U$1 39.8 mm to (-53.3, 57.1)
- moved C1 39.2 mm to (-62.2, 57.1)
- moved U4 31.8 mm to (-17.8, 57.1)
- moved U5 31.8 mm to (-26.7, 57.1)
- moved U1 31.0 mm to (-43.2, 58.4)
- moved U6 30.0 mm to (-35.6, 57.1)
- moved R1 22.6 mm to (-29.2, 63.5)
Connections:
- removed net AVCC: U1.18
- removed net GND_2: U1.3
- removed net GND_3: U1.5
- removed net VCC: U1.6
- removed net VCC_2: U1.4
- new net 1A: U$2.P$35, U3.1
- new net 1B: U$2.P$34, U3.2
- new net 1C: U$2.P$7, U3.3
- new net 1D: U$2.P$6, U3.4
- new net 1E: U$2.P$5, U3.5
- new net 1F: U$2.P$36, U3.6
- new net 1G: U$2.P$37, U3.7
- new net 2A: U$2.P$30, U4.1
- new net 2B: U$2.P$29, U4.2
- new net 2C: U$2.P$11, U4.3
- new net 2D: U$2.P$10, U4.4
- new net 2E: U$2.P$9, U4.5
- new net 2F: U$2.P$31, U4.6
- new net 2G: U$2.P$32, U4.7
- new net 3A: U$2.P$25, U5.1
- new net 3B: U$2.P$24, U5.2
- new net 3C: U$2.P$15, U5.3
- new net 3D: U$2.P$14, U5.4
- new net 3E: U$2.P$13, U5.5
- new net 3F: U$2.P$26, U5.6
- new net 3G: U$2.P$27, U5.7
- new net 4A: U$2.P$21, U6.1
- new net 4B: U$2.P$20, U6.2
- new net 4C: U$2.P$19, U6.3
- new net 4D: U$2.P$18, U6.4
- new net 4E: U$2.P$17, U6.5
- new net 4F: U$2.P$22, U6.6
- new net 4G: U$2.P$23, U6.7
- new net DIVIDED: U$2.P$1, U$2.P$40, U$3.WIPER
- new net LRA/ERM+: U$4.P$1, U2.A3
- new net LRA/ERM-: U$4.P$2, U2.C3
- net !RESET: now also SV1.5, U1.29; no longer J1.5
- net +5V: now also C3.1, SV1.2, U$3.CCW, U1.18, U1.4, U1.6; no longer J1.2
- net GND: now also C3.2, SV1.6, U$3.CW, U1.3, U1.5; no longer J1.10, J1.4, J1.6, J1.8
- net MISO: now also SV1.1, U1.16; no longer J1.9
- net MOSI: now also SV1.4, U1.15; no longer J1.1
- net SCK: now also SV1.3, U1.17; no longer J1.7
- net SCL: now also U1.28
- net SDA: now also U1.27
- net SFT1: now also U1.23
- net SFT2: now also U1.24
- net SFT3: now also U1.25
- net SFT4: now also U1.26
- net SHIFT_CLK: now also U1.31
- net STORAGE_CLK: now also U1.30

Commit message: Separate clocks for registers
Parts:
- renumbered U$3 to TC33X-2-103E, U$4 to PS1240P02BT
Connections:
- removed net SHIFT_CLK: U1.31, U3.12, U4.12, U5.12, U6.12
- removed net STORAGE_CLK: U1.30, U3.11, U4.11, U5.11, U6.11
- new net SHIFT_CLK1: U1.9, U3.12
- new net SHIFT_CLK2: U1.10, U4.12
- new net SHIFT_CLK3: U1.11, U5.12
- new net SHIFT_CLK4: U1.12, U6.12
- new net STORAGE_CLK1: U1.13, U3.11
- new net STORAGE_CLK2: U1.14, U4.11
- new net STORAGE_CLK3: U1.30, U5.11
- new net STORAGE_CLK4: U1.31, U6.11
Changed lines of the file:
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@@
 <element name="U$1" library="rgb-led" package="GS-14-2180" value="MICRO-USB" x="-53.34" y="57.15"/>
 <element name="U$2" library="lcd-buzzer" package="S401C39TR" value="LCD-S401C39TR" x="-63.5" y="1.27"/>
-<element name="U$3" library="lcd-buzzer" package="TC33X-2-103E" value="TC33X" x="-53.34" y="33.02"/>
-<element name="U$4" library="lcd-buzzer" package="PS1240P02BT" value="PS1240P02BT" x="-30.48" y="38.1"/>
+<element name="TC33X-2-103E" library="lcd-buzzer" package="TC33X-2-103E" value="TC33X" x="-53.34" y="33.02"/>
+<element name="PS1240P02BT" library="lcd-buzzer" package="PS1240P02BT" value="PS1240P02BT" x="-30.48" y="38.1"/>
 <element name="U1" library="lcd-buzzer" package="32M1-A" value="ATMEGA328P-MUR" x="-43.18" y="58.42">
 <attribute name="MANUFACTURER_PART_NUMBER" value="ATMEGA328PMUR" x="-43.18" y="58.42" size="1.778" layer="27" display="off"/>
@@
 <contactref element="U1" pad="4"/>
 <contactref element="U1" pad="18"/>
-<contactref element="U$3" pad="CCW"/>
+<contactref element="TC33X-2-103E" pad="CCW"/>
 <contactref element="SV1" pad="2"/>
 <wire x1="-15.24" y1="63" x2="-15.74" y2="64" width="0" layer="19" extent="1-1"/>
@@
 <contactref element="U1" pad="3"/>
 <contactref element="U1" pad="21"/>
-<contactref element="U$3" pad="CW"/>
+<contactref element="TC33X-2-103E" pad="CW"/>
 <contactref element="SV1" pad="6"/>
 <wire x1="-15.74" y1="63.5" x2="-14.74" y2="63.5" width="0" layer="19" extent="1-1"/>
@@
 <wire x1="-62.5094" y1="32.015" x2="-56.8706" y2="34.614996875" width="0" layer="19" extent="1-1"/>
 </signal>
-<signal name="SHIFT_CLK">
-<contactref element="U3" pad="12"/>
-<contactref element="U4" pad="12"/>
-<contactref element="U5" pad="12"/>
+<signal name="SHIFT_CLK4">
 <contactref element="U6" pad="12"/>
+<contactref element="U1" pad="12"/>
+<wire x1="-43.43" y1="56.0197" x2="-32.7406" y2="56.825" width="0" layer="19" extent="1-1"/>
+</signal>
+<signal name="STORAGE_CLK4">
+<contactref element="U6" pad="11"/>
 <contactref element="U1" pad="31"/>
-<wire x1="-23.8506" y1="56.825" x2="-14.9606" y2="56.825" width="0" layer="19" extent="1-1"/>
-<wire x1="-32.7406" y1="56.825" x2="-23.8506" y2="56.825" width="0" layer="19" extent="1-1"/>
-<wire x1="-44.43" y1="60.8203" x2="-32.7406" y2="56.825" width="0" layer="19" extent="1-1"/>
-<wire x1="-56.8706" y1="33.965" x2="-44.43" y2="60.8203" width="0" layer="19" extent="1-1"/>
-</signal>
-<signal name="STORAGE_CLK">
-<contactref element="U3" pad="11"/>
-<contactref element="U4" pad="11"/>
-<contactref element="U5" pad="11"/>
-<contactref element="U6" pad="11"/>
-<contactref element="U1" pad="30"/>
-<wire x1="-23.8506" y1="56.175" x2="-14.9606" y2="56.175" width="0" layer="19" extent="1-1"/>
-<wire x1="-32.7406" y1="56.175" x2="-23.8506" y2="56.175" width="0" layer="19" extent="1-1"/>
-<wire x1="-43.93" y1="60.8203" x2="-32.7406" y2="56.175" width="0" layer="19" extent="1-1"/>
-<wire x1="-56.8706" y1="33.315" x2="-43.93" y2="60.8203" width="0" layer="19" extent="1-1"/>
+<wire x1="-44.43" y1="60.8203" x2="-32.7406" y2="56.175" width="0" layer="19" extent="1-1"/>
 </signal>
 <signal name="SFT1">
@@
 <signal name="LRA/ERM+">
 <contactref element="U2" pad="A3"/>
-<contactref element="U$4" pad="P$1"/>
+<contactref element="PS1240P02BT" pad="P$1"/>
 <wire x1="-32.98" y1="38.1" x2="-14.74" y2="64" width="0" layer="19" extent="1-1"/>
 </signal>
 <signal name="LRA/ERM-">
 <contactref element="U2" pad="C3"/>
-<contactref element="U$4" pad="P$2"/>
+<contactref element="PS1240P02BT" pad="P$2"/>
 <wire x1="-27.98" y1="38.1" x2="-14.74" y2="63" width="0" layer="19" extent="1-1"/>
 </signal>
@@
 </signal>
 <signal name="DIVIDED">
-<contactref element="U$3" pad="WIPER"/>
+<contactref element="TC33X-2-103E" pad="WIPER"/>
 <contactref element="U$2" pad="P$1"/>
 <contactref element="U$2" pad="P$40"/>
@@
 <wire x1="-51.0794" y1="37.5412" x2="-63.5" y2="25.908" width="0" layer="19" extent="1-1"/>
 </signal>
+<signal name="SHIFT_CLK1">
+<contactref element="U3" pad="12"/>
+<contactref element="U1" pad="9"/>
+<wire x1="-44.93" y1="56.0197" x2="-56.8706" y2="33.965" width="0" layer="19" extent="1-1"/>
+</signal>
+<signal name="STORAGE_CLK1">
+<contactref element="U3" pad="11"/>
+<contactref element="U1" pad="13"/>
+<wire x1="-42.93" y1="56.0197" x2="-56.8706" y2="33.315" width="0" layer="19" extent="1-1"/>
+</signal>
+<signal name="STORAGE_CLK2">
+<contactref element="U4" pad="11"/>
+<contactref element="U1" pad="14"/>
+<wire x1="-42.43" y1="56.0197" x2="-14.9606" y2="56.175" width="0" layer="19" extent="1-1"/>
+</signal>
+<signal name="SHIFT_CLK2">
+<contactref element="U4" pad="12"/>
+<contactref element="U1" pad="10"/>
+<wire x1="-44.43" y1="56.0197" x2="-14.9606" y2="56.825" width="0" layer="19" extent="1-1"/>
+</signal>
+<signal name="STORAGE_CLK3">
+<contactref element="U5" pad="11"/>
+<contactref element="U1" pad="30"/>
+<wire x1="-43.93" y1="60.8203" x2="-23.8506" y2="56.175" width="0" layer="19" extent="1-1"/>
+</signal>
+<signal name="SHIFT_CLK3">
+<contactref element="U5" pad="12"/>
+<contactref element="U1" pad="11"/>
+<wire x1="-43.93" y1="56.0197" x2="-23.8506" y2="56.825" width="0" layer="19" extent="1-1"/>
+</signal>
 </signals>
