File: 2017-2018/lcd-buzzer.brd (EAGLE design)
At the start: 58.9 x 28.8 mm, 16 parts, among them U1 ATMEGA328P-MUR

Commit message: Button Added
Parts:
- added C4, C5: 100nF, resistor:C0603
- added K1: SKQGADE010, rgb-led:SW4-SMD-5.2X5.2X1.5MM
- added R2: 10k, resistor:R0603
- added R3: 39k, resistor:R0603
Connections:
- new net !BTN: C4.1, C5.1, R3.2, U1.2
- new net N$1: K1.1, R3.1
- net +5V: now also R2.2
- net GND: now also C4.2, C5.2, K1.2, K1.3, R2.1
- net SFT4: now also U1.1; no longer U1.2
- net SHIFT_CLK4: now also U1.32; no longer U1.1
- net STORAGE_CLK4: now also U1.31; no longer U1.32
Routing:
- net GND: track 74.5 -> 88.3 mm
- net !BTN: track 0.00 -> 11.3 mm
- net N$1: track 0.00 -> 2.44 mm
- net SFT4: track 14.6 -> 13.5 mm
- net SHIFT_CLK4: track 12.0 -> 11.2 mm
- net 2C: track 11.5 -> 11.4 mm, vias 0 -> 1
Other:
- board text added: "+"
- board text added: "_"
