File: 2017-2018/lcd-buzzer.sch (EAGLE design)
At the start: 12 parts, among them J1 AVR_SPI_PROG2PTH2, U1 ATMEGA328P-MUR, U2 DRV2605YZFR, U3 74HC595PW, U4 74HC595PW, U5 74HC595PW, U6 74HC595PW

Commit message: First Version Completed
Added extra custom parts to the library, completed the schematics
Parts:
- removed J1: AVR_SPI_PROG2PTH2, rgb-led:AVR_SPI_PROG2PTH2
- added SV1: (no value), con-lstb:MA03-2
- added U$2: LCD-S401C39TR, lcd-buzzer:LCD-S401C39TR
- added U$3: TC33X, lcd-buzzer:TC33X
- added U$4: PS1240P02BT, lcd-buzzer:PS1240P02BT
Connections:
- new net 1A: U$2.1A/P35, U3.Q1
- new net 1B: U$2.1B/P34, U3.Q2
- new net 1C: U$2.1C/P7, U3.Q3
- new net 1D: U$2.1D/P6, U3.Q4
- new net 1E: U$2.1E/P5, U3.Q5
- new net 1F: U$2.1F/P36, U3.Q6
- new net 1G: U$2.1G/P37, U3.Q7_2
- new net 2A: U$2.2A/P30, U4.Q1
- new net 2B: U$2.2B/P29, U4.Q2
- new net 2C: U$2.2C/P11, U4.Q3
- new net 2D: U$2.2D/P10, U4.Q4
- new net 2E: U$2.2E/P9, U4.Q5
- new net 2F: U$2.2F/P31, U4.Q6
- new net 2G: U$2.2G/P32, U4.Q7_2
- new net 3A: U$2.3A/P25, U5.Q1
- new net 3B: U$2.3B/P24, U5.Q2
- new net 3C: U$2.3C/P15, U5.Q3
- new net 3D: U$2.3D/P14, U5.Q4
- new net 3E: U$2.3E/P13, U5.Q5
- new net 3F: U$2.3F/P26, U5.Q6
- new net 3G: U$2.3G/P27, U5.Q7_2
- new net 4A: U$2.4A/P21, U6.Q1
- new net 4B: U$2.4B/P20, U6.Q2
- new net 4C: U$2.4C/P19, U6.Q3
- new net 4D: U$2.4D/P18, U6.Q4
- new net 4E: U$2.4E/P17, U6.Q5
- new net 4F: U$2.4F/P22, U6.Q6
- new net 4G: U$2.FG/P23, U6.Q7_2
- new net DIVIDED: U$2.COM/P1, U$2.COMP40, U$3.WIPER
- net !RESET: now also SV1.5, U1.PC6_(RESET/PCINT14); no longer J1.RESET
- net +5V: now also SV1.2, U$3.CCW, U1.AVCC, U1.VCC, U1.VCC_2; no longer J1.VCC
- net GND: now also SV1.6, U$3.CW, U1.GND, U1.GND_2, U1.GND_3; no longer J1.GND@1, J1.GND@2, J1.GND@3, J1.GND@4
- net LRA/ERM+: now also U$4.VCC
- net LRA/ERM-: now also U$4.P2
- net MISO: now also SV1.1, U1.(PCINT4/MISO)_PB4; no longer J1.MISO
- net MOSI: now also SV1.4, U1.(PCINT3/OC2A/MOSI)_PB3; no longer J1.MOSI
- net SCK: now also SV1.3, U1.PB5_(SCK/PCINT5); no longer J1.SCK
- net SCL: now also U1.PC5_(ADC5/SCL/PCINT13)
- net SDA: now also U1.PC4_(ADC4/SDA/PCINT12)
- net SFT1: now also U1.PC0_(ADC0/PCINT8)
- net SFT2: now also U1.PC1_(ADC1/PCINT9)
- net SFT3: now also U1.PC2_(ADC2/PCINT10)
- net SFT4: now also U1.PC3_(ADC3/PCINT11)
- net SHIFT_CLK: now also U1.PD1_(TXD/PCINT17)
- net STORAGE_CLK: now also U1.PD0_(RXD/PCINT16)
Other:
- note removed: "AVR Programming Port"
- moved on the sheet: C1, C2, C3, R1, U1, U2, U3, U4, U5, U6

Commit message: Separate clocks for registers
Parts:
- removed U$4: PS1240P02BT, lcd-buzzer:PS1240P02BT
- added PS1240P02BT: PS1240P02BT, lcd-buzzer:PS1240P02BT
- renumbered U$3 to TC33X-2-103E
Connections:
- removed net SHIFT_CLK: U1.PD1_(TXD/PCINT17), U3.ST_CP, U4.ST_CP, U5.ST_CP, U6.ST_CP
- removed net STORAGE_CLK: U1.PD0_(RXD/PCINT16), U3.SH_CP, U4.SH_CP, U5.SH_CP, U6.SH_CP
- new net SHIFT_CLK1: U1.(PCINT21/OC0B/T1)_PD5, U3.ST_CP
- new net SHIFT_CLK2: U1.(PCINT22/OC0A/AIN0)_PD6, U4.ST_CP
- new net SHIFT_CLK3: U1.(PCINT23/AIN1)_PD7, U5.ST_CP
- new net SHIFT_CLK4: U1.(PCINT0/CLKO/ICP1)_PB0, U6.ST_CP
- new net STORAGE_CLK1: U1.(PCINT1/OC1A)_PB1, U3.SH_CP
- new net STORAGE_CLK2: U1.(PCINT2/SS/OC1B)_PB2, U4.SH_CP
- new net STORAGE_CLK3: U1.PD0_(RXD/PCINT16), U5.SH_CP
- new net STORAGE_CLK4: U1.PD1_(TXD/PCINT17), U6.SH_CP
- net LRA/ERM+: now also PS1240P02BT.VCC; no longer U$4.VCC
- net LRA/ERM-: now also PS1240P02BT.P2; no longer U$4.P2
Changed lines of the file:
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@@
 <setting verticaltext="up"/>
 </settings>
-<grid distance="0.1" unitdist="inch" unit="inch" style="lines" multiple="1" display="no" altdistance="0.01" altunitdist="inch" altunit="inch"/>
+<grid distance="0.5" unitdist="mm" unit="mm" style="lines" multiple="1" display="no" altdistance="0.01" altunitdist="inch" altunit="inch"/>
 <layers>
 <layer number="1" name="Top" color="4" fill="1" visible="no" active="no"/>
@@
 <part name="C3" library="SparkFun-Capacitors" deviceset="0.1UF" device="-0603-25V-(+80/-20%)" value="0.1uF"/>
 <part name="U$2" library="lcd-buzzer" deviceset="LCD-S401C39TR" device=""/>
-<part name="U$3" library="lcd-buzzer" deviceset="TC33X" device=""/>
+<part name="TC33X-2-103E" library="lcd-buzzer" deviceset="TC33X" device=""/>
 <part name="SUPPLY33" library="supply2" library_urn="urn:adsk.eagle:library:372" deviceset="GND" device=""/>
 <part name="SUPPLY34" library="supply2" library_urn="urn:adsk.eagle:library:372" deviceset="+5V" device=""/>
-<part name="U$4" library="lcd-buzzer" deviceset="PS1240P02BT" device=""/>
+<part name="PS1240P02BT" library="lcd-buzzer" deviceset="PS1240P02BT" device=""/>
 <part name="SV1" library="con-lstb" library_urn="urn:adsk.eagle:library:162" deviceset="MA03-2" device=""/>
 <part name="SUPPLY31" library="supply2" library_urn="urn:adsk.eagle:library:372" deviceset="+5V" device=""/>
@@
 <instance part="C3" gate="G$1" x="261.62" y="120.65" rot="R90"/>
 <instance part="U$2" gate="G$1" x="220.98" y="73.66"/>
-<instance part="U$3" gate="G$1" x="182.88" y="105.41"/>
+<instance part="TC33X-2-103E" gate="G$1" x="182.88" y="105.41"/>
 <instance part="SUPPLY33" gate="GND" x="172.72" y="100.33"/>
 <instance part="SUPPLY34" gate="+5V" x="172.72" y="113.03"/>
-<instance part="U$4" gate="G$1" x="184.15" y="142.24"/>
+<instance part="PS1240P02BT" gate="G$1" x="191.77" y="147.32"/>
 <instance part="SV1" gate="1" x="269.24" y="99.06" rot="R180"/>
 <instance part="SUPPLY31" gate="+5V" x="280.67" y="106.68"/>
@@
 <segment>
 <pinref part="SUPPLY34" gate="+5V" pin="+5V"/>
-<pinref part="U$3" gate="G$1" pin="CCW"/>
+<pinref part="TC33X-2-103E" gate="G$1" pin="CCW"/>
 <wire x1="172.72" y1="110.49" x2="172.72" y2="105.41" width="0.1524" layer="91"/>
 <wire x1="172.72" y1="105.41" x2="177.8" y2="105.41" width="0.1524" layer="91"/>
@@
 <segment>
 <pinref part="SUPPLY33" gate="GND" pin="GND"/>
-<pinref part="U$3" gate="G$1" pin="CW"/>
+<pinref part="TC33X-2-103E" gate="G$1" pin="CW"/>
 <wire x1="172.72" y1="102.87" x2="177.8" y2="102.87" width="0.1524" layer="91"/>
 </segment>
@@
 </segment>
 </net>
-<net name="SHIFT_CLK" class="0">
-<segment>
-<pinref part="U3" gate="A" pin="ST_CP"/>
-<wire x1="55.02" y1="93.9" x2="67.72" y2="93.9" width="0.1524" layer="91"/>
-<label x="55.74" y="93.82" size="1.778" layer="95"/>
-</segment>
-<segment>
-<pinref part="U4" gate="A" pin="ST_CP"/>
-<wire x1="133.4" y1="93.9" x2="146.1" y2="93.9" width="0.1524" layer="91"/>
-<label x="134.12" y="93.82" size="1.778" layer="95"/>
-</segment>
-<segment>
-<pinref part="U5" gate="A" pin="ST_CP"/>
-<wire x1="54.46" y1="137.08" x2="67.16" y2="137.08" width="0.1524" layer="91"/>
-<label x="55.18" y="137" size="1.778" layer="95"/>
-</segment>
+<net name="SHIFT_CLK4" class="0">
 <segment>
 <pinref part="U6" gate="A" pin="ST_CP"/>
@@
 </segment>
 <segment>
-<pinref part="U1" gate="A" pin="PD1_(TXD/PCINT17)"/>
-<wire x1="166.7" y1="53.46" x2="166.7" y2="53.34" width="0.1524" layer="91"/>
-<wire x1="166.7" y1="53.34" x2="180.34" y2="53.34" width="0.1524" layer="91"/>
-<label x="167.64" y="53.34" size="1.778" layer="95"/>
-</segment>
-</net>
-<net name="STORAGE_CLK" class="0">
-<segment>
-<pinref part="U3" gate="A" pin="SH_CP"/>
-<wire x1="55.02" y1="91.36" x2="67.72" y2="91.36" width="0.1524" layer="91"/>
-<label x="55.74" y="91.32" size="1.778" layer="95"/>
-</segment>
-<segment>
-<pinref part="U4" gate="A" pin="SH_CP"/>
-<wire x1="133.4" y1="91.36" x2="146.1" y2="91.36" width="0.1524" layer="91"/>
-<label x="134.12" y="91.32" size="1.778" layer="95"/>
-</segment>
-<segment>
-<pinref part="U5" gate="A" pin="SH_CP"/>
-<wire x1="54.46" y1="134.54" x2="67.16" y2="134.54" width="0.1524" layer="91"/>
-<label x="55.18" y="134.5" size="1.778" layer="95"/>
-</segment>
+<pinref part="U1" gate="A" pin="(PCINT0/CLKO/ICP1)_PB0"/>
+<wire x1="29.54" y1="28.06" x2="17.78" y2="28.06" width="0.1524" layer="91"/>
+<wire x1="17.78" y1="28.06" x2="17.78" y2="27.94" width="0.1524" layer="91"/>
+<label x="9" y="28" size="1.778" layer="95"/>
+</segment>
+</net>
+<net name="STORAGE_CLK4" class="0">
 <segment>
 <pinref part="U6" gate="A" pin="SH_CP"/>
@@
 </segment>
 <segment>
-<pinref part="U1" gate="A" pin="PD0_(RXD/PCINT16)"/>
-<wire x1="166.7" y1="50.92" x2="166.7" y2="50.8" width="0.1524" layer="91"/>
-<wire x1="166.7" y1="50.8" x2="180.34" y2="50.8" width="0.1524" layer="91"/>
-<label x="167.64" y="50.8" size="1.778" layer="95"/>
+<pinref part="U1" gate="A" pin="PD1_(TXD/PCINT17)"/>
+<wire x1="166.7" y1="53.46" x2="180.34" y2="53.46" width="0.1524" layer="91"/>
+<wire x1="180.34" y1="53.46" x2="180.34" y2="53.34" width="0.1524" layer="91"/>
+<label x="167.64" y="53.34" size="1.778" layer="95"/>
 </segment>
 </net>
@@
 </segment>
 <segment>
-<pinref part="U$4" gate="G$1" pin="VCC"/>
-<wire x1="179.07" y1="137.16" x2="172.72" y2="137.16" width="0.1524" layer="91"/>
-<label x="170.18" y="137.16" size="1.778" layer="95"/>
+<pinref part="PS1240P02BT" gate="G$1" pin="VCC"/>
+<wire x1="186.69" y1="142.24" x2="180.34" y2="142.24" width="0.1524" layer="91"/>
+<label x="172.72" y="142.24" size="1.778" layer="95"/>
 </segment>
 </net>
@@
 </segment>
 <segment>
-<pinref part="U$4" gate="G$1" pin="P2"/>
-<wire x1="179.07" y1="129.54" x2="172.72" y2="129.54" width="0.1524" layer="91"/>
-<label x="170.18" y="129.54" size="1.778" layer="95"/>
+<pinref part="PS1240P02BT" gate="G$1" pin="P2"/>
+<wire x1="186.69" y1="134.62" x2="180.34" y2="134.62" width="0.1524" layer="91"/>
+<label x="172.72" y="134.62" size="1.778" layer="95"/>
 </segment>
 </net>
@@
 <net name="DIVIDED" class="0">
 <segment>
-<pinref part="U$3" gate="G$1" pin="WIPER"/>
+<pinref part="TC33X-2-103E" gate="G$1" pin="WIPER"/>
 <wire x1="204.47" y1="104.14" x2="215.9" y2="104.14" width="0.1524" layer="91"/>
 <label x="210.82" y="104.14" size="1.778" layer="95"/>
@@
 </segment>
 </net>
+<net name="SHIFT_CLK1" class="0">
+<segment>
+<pinref part="U3" gate="A" pin="ST_CP"/>
+<wire x1="55.02" y1="93.9" x2="67.72" y2="93.9" width="0.1524" layer="91"/>
+<label x="55.74" y="93.82" size="1.778" layer="95"/>
+</segment>
+<segment>
+<pinref part="U1" gate="A" pin="(PCINT21/OC0B/T1)_PD5"/>
+<wire x1="29.54" y1="35.68" x2="17.78" y2="35.68" width="0.1524" layer="91"/>
+<wire x1="17.78" y1="35.68" x2="17.78" y2="35.56" width="0.1524" layer="91"/>
+<label x="9" y="35.5" size="1.778" layer="95"/>
+</segment>
+</net>
+<net name="STORAGE_CLK1" class="0">
+<segment>
+<pinref part="U3" gate="A" pin="SH_CP"/>
+<wire x1="55.02" y1="91.36" x2="67.72" y2="91.36" width="0.1524" layer="91"/>
+<label x="55.74" y="91.32" size="1.778" layer="95"/>
+</segment>
+<segment>
+<pinref part="U1" gate="A" pin="(PCINT1/OC1A)_PB1"/>
+<wire x1="29.54" y1="25.52" x2="17.78" y2="25.52" width="0.1524" layer="91"/>
+<wire x1="17.78" y1="25.52" x2="17.78" y2="25.4" width="0.1524" layer="91"/>
+<label x="9" y="25.5" size="1.778" layer="95"/>
+</segment>
+</net>
+<net name="STORAGE_CLK2" class="0">
+<segment>
+<pinref part="U4" gate="A" pin="SH_CP"/>
+<wire x1="133.4" y1="91.36" x2="146.1" y2="91.36" width="0.1524" layer="91"/>
+<label x="134.12" y="91.32" size="1.778" layer="95"/>
+</segment>
+<segment>
+<pinref part="U1" gate="A" pin="(PCINT2/SS/OC1B)_PB2"/>
+<wire x1="29.54" y1="22.98" x2="17.78" y2="22.98" width="0.1524" layer="91"/>
+<wire x1="17.78" y1="22.98" x2="17.78" y2="22.86" width="0.1524" layer="91"/>
+<label x="9" y="23" size="1.778" layer="95"/>
+</segment>
+</net>
+<net name="SHIFT_CLK2" class="0">
+<segment>
+<pinref part="U4" gate="A" pin="ST_CP"/>
+<wire x1="133.4" y1="93.9" x2="146.1" y2="93.9" width="0.1524" layer="91"/>
+<label x="134.12" y="93.82" size="1.778" layer="95"/>
+</segment>
+<segment>
+<pinref part="U1" gate="A" pin="(PCINT22/OC0A/AIN0)_PD6"/>
+<wire x1="29.54" y1="33.14" x2="17.78" y2="33.14" width="0.1524" layer="91"/>
+<wire x1="17.78" y1="33.14" x2="17.78" y2="33.02" width="0.1524" layer="91"/>
+<label x="9" y="33" size="1.778" layer="95"/>
+</segment>
+</net>
+<net name="STORAGE_CLK3" class="0">
+<segment>
+<pinref part="U5" gate="A" pin="SH_CP"/>
+<wire x1="54.46" y1="134.54" x2="67.16" y2="134.54" width="0.1524" layer="91"/>
+<label x="55.18" y="134.5" size="1.778" layer="95"/>
+</segment>
+<segment>
+<pinref part="U1" gate="A" pin="PD0_(RXD/PCINT16)"/>
+<wire x1="166.7" y1="50.92" x2="180.34" y2="50.92" width="0.1524" layer="91"/>
+<wire x1="180.34" y1="50.92" x2="180.34" y2="50.8" width="0.1524" layer="91"/>
+<label x="167.64" y="50.8" size="1.778" layer="95"/>
+</segment>
+</net>
+<net name="SHIFT_CLK3" class="0">
+<segment>
+<pinref part="U5" gate="A" pin="ST_CP"/>
+<wire x1="54.46" y1="137.08" x2="67.16" y2="137.08" width="0.1524" layer="91"/>
+<label x="55.18" y="137" size="1.778" layer="95"/>
+</segment>
+<segment>
+<pinref part="U1" gate="A" pin="(PCINT23/AIN1)_PD7"/>
+<wire x1="29.54" y1="30.6" x2="17.78" y2="30.6" width="0.1524" layer="91"/>
+<wire x1="17.78" y1="30.6" x2="17.78" y2="30.48" width="0.1524" layer="91"/>
+<label x="9" y="30.5" size="1.778" layer="95"/>
+</segment>
+</net>

Commit message: Minor Changes based on Manipulation w/ LCD
Other:
- note added: "4 Shifters"
- note added: "Buzzer"
- note added: "LCD"
- note added: "SPI Programming Port"
- note added: "Trimmer Potentiometer"
- moved on the sheet: PS1240P02BT
Changed lines of the file:
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@@
 <setting verticaltext="up"/>
 </settings>
-<grid distance="0.5" unitdist="mm" unit="mm" style="lines" multiple="1" display="no" altdistance="0.01" altunitdist="inch" altunit="inch"/>
+<grid distance="0.1" unitdist="inch" unit="inch" style="lines" multiple="1" display="no" altdistance="0.01" altunitdist="inch" altunit="inch"/>
 <layers>
 <layer number="1" name="Top" color="4" fill="1" visible="no" active="no"/>
@@
 <text x="99.06" y="48.26" size="1.778" layer="91">Schematics shows here is !RESET</text>
 <text x="276.86" y="158.75" size="1.778" layer="91">Haptic Driver</text>
-<text x="217.17" y="86.36" size="1.778" layer="91">MicroUSB As Power</text>
+<text x="214.63" y="111.76" size="1.778" layer="91">MicroUSB As Power</text>
+<text x="195.58" y="157.48" size="1.778" layer="91">Buzzer</text>
+<text x="251.46" y="109.22" size="1.778" layer="91">SPI Programming Port</text>
+<text x="218.44" y="78.74" size="1.778" layer="91">LCD</text>
+<text x="55.88" y="162.56" size="1.778" layer="91">4 Shifters</text>
+<text x="185.42" y="116.84" size="1.778" layer="91">Trimmer Potentiometer</text>
 </plain>
 <instances>
@@
 <instance part="SUPPLY33" gate="GND" x="172.72" y="100.33"/>
 <instance part="SUPPLY34" gate="+5V" x="172.72" y="113.03"/>
-<instance part="PS1240P02BT" gate="G$1" x="191.77" y="147.32"/>
+<instance part="PS1240P02BT" gate="G$1" x="194.31" y="152.4"/>
 <instance part="SV1" gate="1" x="269.24" y="99.06" rot="R180"/>
 <instance part="SUPPLY31" gate="+5V" x="280.67" y="106.68"/>
@@
 <segment>
 <pinref part="PS1240P02BT" gate="G$1" pin="VCC"/>
-<wire x1="186.69" y1="142.24" x2="180.34" y2="142.24" width="0.1524" layer="91"/>
-<label x="172.72" y="142.24" size="1.778" layer="95"/>
+<wire x1="189.23" y1="147.32" x2="177.8" y2="147.32" width="0.1524" layer="91"/>
+<label x="172.72" y="147.32" size="1.778" layer="95"/>
 </segment>
 </net>
@@
 <segment>
 <pinref part="PS1240P02BT" gate="G$1" pin="P2"/>
-<wire x1="186.69" y1="134.62" x2="180.34" y2="134.62" width="0.1524" layer="91"/>
-<label x="172.72" y="134.62" size="1.778" layer="95"/>
-</segment>
-</net>
+<wire x1="189.23" y1="139.7" x2="177.8" y2="139.7" width="0.1524" layer="91"/>
+<label x="172.72" y="139.7" size="1.778" layer="95"/>
+</segment>
+</net>

Commit message: Haptic Drive Update
Parts:
- removed C2: 1.0uF, SparkFun-Capacitors:1.0UF-0603-16V-10%
- removed C3: 0.1uF, SparkFun-Capacitors:0.1UF-0603-25V-(+80/-20%)
- removed U2: DRV2605YZFR, lcd-buzzer:DRV2605YZFR
- added C4: 0.1uF, SparkFun-Capacitors:0.1UF-0603-25V-(+80/-20%)
- added C5: 1.0uF, SparkFun-Capacitors:1.0UF-0603-16V-10%
- added U7: DRV2605LDGSR, lcd-buzzer:DRV2605LDGSR
Connections:
- removed net N$2: C2.1, U2.VREG
- new net N$3: C5.2, U7.REG
- new net N$5: C4.1, U7.VDD
- net +5V: now also U7.EN; no longer C3.1, U2.EN, U2.VDD
- net GND: now also C4.2, C5.1, U7.GND, U7.IN/TRIG; no longer C2.2, C3.2, U2.GND, U2.IN/TRIG
- net LRA/ERM+: now also U7.OUT+; no longer U2.OUT+
- net LRA/ERM-: now also U7.OUT-; no longer U2.OUT-
- net SCL: now also U7.SCL; no longer U2.SCL
- net SDA: now also U7.SDA; no longer U2.SDA

Commit message: Board File Initial Commit
Library Updated. 328p pin configuration reassigned
Parts:
- renumbered C4 to C3, C5 to C2, U$2 to LCD, U3 to #1, U4 to #2, U5 to #3, U6 to #4, U7 to HAPTIC
Connections:
- removed net N$5: C3.1, HAPTIC.VDD
- net +5V: now also C3.1, HAPTIC.VDD
- net SFT1: now also U1.(PCINT22/OC0A/AIN0)_PD6; no longer U1.PC0_(ADC0/PCINT8)
- net SFT2: now also U1.(PCINT6/XTAL1/TOSC1)_PB6; no longer U1.PC1_(ADC1/PCINT9)
- net SFT4: now also U1.(PCINT20/XCK/T0)_PD4; no longer U1.PC3_(ADC3/PCINT11)
- net SHIFT_CLK1: now also U1.(PCINT23/AIN1)_PD7; no longer U1.(PCINT21/OC0B/T1)_PD5
- net SHIFT_CLK2: now also U1.(PCINT7/XTAL2/TOSC2)_PB7; no longer U1.(PCINT22/OC0A/AIN0)_PD6
- net SHIFT_CLK3: now also U1.PD0_(RXD/PCINT16); no longer U1.(PCINT23/AIN1)_PD7
- net SHIFT_CLK4: now also U1.(PCINT19/OC2B/INT1)_PD3; no longer U1.(PCINT0/CLKO/ICP1)_PB0
- net STORAGE_CLK1: now also U1.(PCINT0/CLKO/ICP1)_PB0; no longer U1.(PCINT1/OC1A)_PB1
- net STORAGE_CLK2: now also U1.(PCINT21/OC0B/T1)_PD5; no longer U1.(PCINT2/SS/OC1B)_PB2
- net STORAGE_CLK3: now also U1.PC3_(ADC3/PCINT11); no longer U1.PD0_(RXD/PCINT16)
- net STORAGE_CLK4: now also U1.PD2_(INT0/PCINT18); no longer U1.PD1_(TXD/PCINT17)
Other:
- moved on the sheet: R1
