File: 2017-2018/lcd-buzzer.sch (EAGLE design)
At the start: 15 parts, among them U1 ATMEGA328P-MUR

Commit message: Button Added
Parts:
- added C4, C5: 100nF, resistor:C-USC0603
- added K1: SKQGADE010, rgb-led:SMD-SWITCH-TOP-260GF(4P-D5.2MM)
- added R2: 10k, resistor:R-US_R0603
- added R3: 39k, resistor:R-US_R0603
Connections:
- new net !BTN: C4.1, C5.1, R3.2, U1.(PCINT20/XCK/T0)_PD4
- new net N$1: K1.A0, R3.1
- net +5V: now also R2.2
- net GND: now also C4.2, C5.2, K1.A1, K1.B1, R2.1
- net SFT4: now also U1.(PCINT19/OC2B/INT1)_PD3; no longer U1.(PCINT20/XCK/T0)_PD4
- net SHIFT_CLK4: now also U1.PD2_(INT0/PCINT18); no longer U1.(PCINT19/OC2B/INT1)_PD3
- net STORAGE_CLK4: now also U1.PD1_(TXD/PCINT17); no longer U1.PD2_(INT0/PCINT18)
Other:
- note added: "Datasheet shows here is !RESET"
- note removed: "Schematics shows here is !RESET"
Changed lines of the file:
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@@
 <part name="SUPPLY21" library="supply2" library_urn="urn:adsk.eagle:library:372" deviceset="+5V" device=""/>
 <part name="SUPPLY27" library="supply2" library_urn="urn:adsk.eagle:library:372" deviceset="+5V" device=""/>
+<part name="K1" library="rgb-led" deviceset="SMD-SWITCH-TOP-260GF(4P-D5.2MM)" device="" value="SKQGADE010"/>
+<part name="SUPPLY28" library="supply2" library_urn="urn:adsk.eagle:library:372" deviceset="+5V" device=""/>
+<part name="SUPPLY29" library="supply2" library_urn="urn:adsk.eagle:library:372" deviceset="GND" device=""/>
+<part name="R2" library="resistor" library_urn="urn:adsk.eagle:library:348" deviceset="R-US_" device="R0603" value="10k"/>
+<part name="R3" library="resistor" library_urn="urn:adsk.eagle:library:348" deviceset="R-US_" device="R0603" value="39k"/>
+<part name="C4" library="resistor" library_urn="urn:adsk.eagle:library:348" deviceset="C-US" device="C0603" value="100nF"/>
+<part name="C5" library="resistor" library_urn="urn:adsk.eagle:library:348" deviceset="C-US" device="C0603" value="100nF"/>
+<part name="SUPPLY30" library="supply2" library_urn="urn:adsk.eagle:library:372" deviceset="GND" device=""/>
 </parts>
 <sheets>
@@
 <plain>
 <text x="20.74" y="119.82" size="1.778" layer="91">pin 1 to 7 on Shifters will control LCD segments</text>
-<text x="99.06" y="48.26" size="1.778" layer="91">Schematics shows here is !RESET</text>
+<text x="99.06" y="48.26" size="1.778" layer="91">Datasheet shows here is !RESET</text>
 <text x="284.48" y="125.73" size="1.778" layer="91">Haptic Driver</text>
 <text x="214.63" y="111.76" size="1.778" layer="91">MicroUSB As Power</text>
@@
 <instance part="SUPPLY21" gate="+5V" x="-2.54" y="50.8"/>
 <instance part="SUPPLY27" gate="+5V" x="317.5" y="149.86"/>
+<instance part="K1" gate="G$1" x="320.04" y="48.26"/>
+<instance part="SUPPLY28" gate="+5V" x="332.74" y="68.58"/>
+<instance part="SUPPLY29" gate="GND" x="332.74" y="35.56"/>
+<instance part="R2" gate="G$1" x="332.74" y="58.42" rot="R90"/>
+<instance part="R3" gate="G$1" x="302.26" y="50.8" rot="R180"/>
+<instance part="C4" gate="G$1" x="294.64" y="43.18"/>
+<instance part="C5" gate="G$1" x="284.48" y="43.18"/>
+<instance part="SUPPLY30" gate="GND" x="289.56" y="30.48"/>
 </instances>
 <busses>
@@
 <pinref part="SUPPLY23" gate="+5V" pin="+5V"/>
 <wire x1="166.624" y1="20.32" x2="190.5" y2="20.32" width="0.1524" layer="91"/>
+<label x="167.64" y="20.32" size="1.778" layer="95"/>
 </segment>
 <segment>
@@
 <junction x="317.5" y="142.24"/>
 </segment>
+<segment>
+<pinref part="SUPPLY28" gate="+5V" pin="+5V"/>
+<pinref part="R2" gate="G$1" pin="2"/>
+<wire x1="332.74" y1="66.04" x2="332.74" y2="63.5" width="0.1524" layer="91"/>
+</segment>
 </net>
 <net name="GND" class="0">
@@
 <wire x1="185.42" y1="27.94" x2="185.42" y2="28.06" width="0.1524" layer="91"/>
 <wire x1="185.42" y1="28.06" x2="166.624" y2="27.94" width="0.1524" layer="91"/>
+<label x="167.64" y="27.94" size="1.778" layer="95"/>
 </segment>
 <segment>
@@
 <wire x1="19.05" y1="45.72" x2="18" y2="45.72" width="0.1524" layer="91"/>
 </segment>
+<segment>
+<pinref part="R2" gate="G$1" pin="1"/>
+<pinref part="SUPPLY29" gate="GND" pin="GND"/>
+<wire x1="332.74" y1="53.34" x2="332.74" y2="50.8" width="0.1524" layer="91"/>
+<pinref part="K1" gate="G$1" pin="B1"/>
+<wire x1="332.74" y1="50.8" x2="332.74" y2="45.72" width="0.1524" layer="91"/>
+<wire x1="332.74" y1="45.72" x2="332.74" y2="38.1" width="0.1524" layer="91"/>
+<wire x1="328.93" y1="45.72" x2="332.74" y2="45.72" width="0.1524" layer="91"/>
+<junction x="332.74" y="45.72"/>
+<pinref part="K1" gate="G$1" pin="A1"/>
+<wire x1="328.93" y1="50.8" x2="332.74" y2="50.8" width="0.1524" layer="91"/>
+<junction x="332.74" y="50.8"/>
+</segment>
+<segment>
+<pinref part="C5" gate="G$1" pin="2"/>
+<wire x1="284.48" y1="38.1" x2="284.48" y2="35.56" width="0.1524" layer="91"/>
+<pinref part="C4" gate="G$1" pin="2"/>
+<wire x1="284.48" y1="35.56" x2="289.56" y2="35.56" width="0.1524" layer="91"/>
+<wire x1="289.56" y1="35.56" x2="294.64" y2="35.56" width="0.1524" layer="91"/>
+<wire x1="294.64" y1="35.56" x2="294.64" y2="38.1" width="0.1524" layer="91"/>
+<pinref part="SUPPLY30" gate="GND" pin="GND"/>
+<wire x1="289.56" y1="33.02" x2="289.56" y2="35.56" width="0.1524" layer="91"/>
+<junction x="289.56" y="35.56"/>
+</segment>
 </net>
 <net name="SHIFT_CLK4" class="0">
@@
 </segment>
 <segment>
-<pinref part="U1" gate="A" pin="(PCINT19/OC2B/INT1)_PD3"/>
-<wire x1="29.464" y1="55.88" x2="12.7" y2="55.88" width="0.1524" layer="91"/>
-<label x="12.7" y="55.88" size="1.778" layer="95"/>
+<pinref part="U1" gate="A" pin="PD2_(INT0/PCINT18)"/>
+<wire x1="166.624" y1="55.88" x2="180.34" y2="55.88" width="0.1524" layer="91"/>
+<label x="167.64" y="55.88" size="1.778" layer="95"/>
 </segment>
 </net>
@@
 </segment>
 <segment>
-<pinref part="U1" gate="A" pin="PD2_(INT0/PCINT18)"/>
-<wire x1="166.624" y1="55.88" x2="180.34" y2="55.88" width="0.1524" layer="91"/>
-<label x="167.64" y="55.88" size="1.778" layer="95"/>
+<pinref part="U1" gate="A" pin="PD1_(TXD/PCINT17)"/>
+<wire x1="166.624" y1="53.34" x2="180.34" y2="53.34" width="0.1524" layer="91"/>
+<label x="167.64" y="53.34" size="1.778" layer="95"/>
 </segment>
 </net>
@@
 <pinref part="U1" gate="A" pin="PC2_(ADC2/PCINT10)"/>
 <wire x1="166.624" y1="38.1" x2="180.34" y2="38.1" width="0.1524" layer="91"/>
-<label x="172.72" y="38.1" size="1.778" layer="95"/>
+<label x="167.64" y="38.1" size="1.778" layer="95"/>
 </segment>
 </net>
@@
 </segment>
 <segment>
-<label x="12.7" y="53.34" size="1.778" layer="95"/>
-<pinref part="U1" gate="A" pin="(PCINT20/XCK/T0)_PD4"/>
-<wire x1="29.464" y1="53.34" x2="12.7" y2="53.34" width="0.1524" layer="91"/>
+<pinref part="U1" gate="A" pin="(PCINT19/OC2B/INT1)_PD3"/>
+<wire x1="29.464" y1="55.88" x2="12.7" y2="55.88" width="0.1524" layer="91"/>
+<label x="22.86" y="55.88" size="1.778" layer="95"/>
 </segment>
 </net>
@@
 <wire x1="193.04" y1="45.72" x2="203.2" y2="45.72" width="0.1524" layer="91"/>
 <wire x1="193.04" y1="45.72" x2="193.04" y2="48.26" width="0.1524" layer="91"/>
-<label x="193.04" y="48.26" size="1.778" layer="95"/>
+<label x="195.58" y="45.72" size="1.778" layer="95"/>
 <wire x1="193.04" y1="48.26" x2="193.04" y2="50.8" width="0.1524" layer="91"/>
 <junction x="193.04" y="48.26"/>
 <pinref part="U1" gate="A" pin="PC6_(RESET/PCINT14)"/>
 <wire x1="166.624" y1="48.26" x2="193.04" y2="48.26" width="0.1524" layer="91"/>
+<label x="167.64" y="48.26" size="1.778" layer="95"/>
 </segment>
 </net>
@@
 <pinref part="U1" gate="A" pin="PC5_(ADC5/SCL/PCINT13)"/>
 <wire x1="166.624" y1="45.72" x2="180" y2="45.72" width="0.1524" layer="91"/>
-<label x="172" y="46" size="1.778" layer="95"/>
+<label x="167.64" y="45.72" size="1.778" layer="95"/>
 </segment>
 <segment>
@@
 <pinref part="U1" gate="A" pin="PC4_(ADC4/SDA/PCINT12)"/>
 <wire x1="166.624" y1="43.18" x2="180" y2="43.18" width="0.1524" layer="91"/>
-<label x="172" y="43" size="1.778" layer="95"/>
+<label x="167.64" y="43.18" size="1.778" layer="95"/>
 </segment>
 <segment>
@@
 <pinref part="U1" gate="A" pin="PC3_(ADC3/PCINT11)"/>
 <wire x1="166.624" y1="40.64" x2="180.34" y2="40.64" width="0.1524" layer="91"/>
-<label x="172.72" y="40.64" size="1.778" layer="95"/>
+<label x="167.64" y="40.64" size="1.778" layer="95"/>
 </segment>
 </net>
@@
 </segment>
 </net>
+<net name="N$1" class="0">
+<segment>
+<pinref part="R3" gate="G$1" pin="1"/>
+<pinref part="K1" gate="G$1" pin="A0"/>
+<wire x1="307.34" y1="50.8" x2="311.15" y2="50.8" width="0.1524" layer="91"/>
+</segment>
+</net>
+<net name="!BTN" class="0">
+<segment>
+<pinref part="R3" gate="G$1" pin="2"/>
+<wire x1="297.18" y1="50.8" x2="294.64" y2="50.8" width="0.1524" layer="91"/>
+<pinref part="C5" gate="G$1" pin="1"/>
+<wire x1="294.64" y1="50.8" x2="284.48" y2="50.8" width="0.1524" layer="91"/>
+<wire x1="284.48" y1="50.8" x2="279.4" y2="50.8" width="0.1524" layer="91"/>
+<wire x1="284.48" y1="45.72" x2="284.48" y2="50.8" width="0.1524" layer="91"/>
+<junction x="284.48" y="50.8"/>
+<pinref part="C4" gate="G$1" pin="1"/>
+<wire x1="294.64" y1="45.72" x2="294.64" y2="50.8" width="0.1524" layer="91"/>
+<junction x="294.64" y="50.8"/>
+<label x="281.94" y="50.8" size="1.778" layer="95"/>
+</segment>
+<segment>
+<pinref part="U1" gate="A" pin="(PCINT20/XCK/T0)_PD4"/>
+<wire x1="29.464" y1="53.34" x2="12.7" y2="53.34" width="0.1524" layer="91"/>
+<label x="22.86" y="53.34" size="1.778" layer="95"/>
+</segment>
+</net>
