File: 2017-2018/lec-buzzer_alt.brd (EAGLE design)
At the start: 160 x 100 mm, 26 parts, among them K1 SKQGADE010, K2 SKQGADE010, K3 SKQGADE010, U1 ATMEGA328P-MUR

Commit message: 3 Button Board completed
LCD flipped, slight changes in shifter, Buzzer and SPI location
Parts:
- added U$2: (no value), RoboJackets-Aesthetics:ROBOBUZZ_0.4X
- moved LCD 47.5 mm to (67.8, 17.0), flipped to the bottom
- moved TC33X-2-103E 45.4 mm to (67.6, 25.1)
- moved #4 43.8 mm to (23.2, 35.4), turned to 0 degrees
- moved SV1 37.2 mm to (15.2, 37.3), turned to 90 degrees
- moved #3 32.5 mm to (23.4, 28.2)
- moved #1 30.0 mm to (58.3, 24.2), turned to 180 degrees
- moved R1 19.6 mm to (32.6, 30.2)
- moved R4 18.5 mm to (54.1, 31.8)
- moved C4 14.0 mm to (45.7, 31.8)
- moved C8 10.5 mm to (58.8, 31.8)
- moved PS1240P02BT 6.91 mm to (14.9, 22.4), turned to 270 degrees
- moved HAPTIC 6.76 mm to (25.2, 22.2), turned to 180 degrees
- moved R6 6.00 mm to (49.9, 31.8)
- moved C6 3.50 mm to (37.1, 31.8)
- moved U1 3.07 mm to (49.2, 24.5), turned to 180 degrees
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Connections:
- net !BTN2: now also U1.8; no longer U1.13
- net !BTN3: now also U1.1; no longer U1.14
- net SFT1: now also U1.30; no longer U1.10
- net SFT2: now also U1.24; no longer U1.7
- net SFT3: now also U1.11; no longer U1.25
- net SFT4: now also U1.12; no longer U1.1
- net SHIFT_CLK1: now also U1.31; no longer U1.11
- net SHIFT_CLK2: now also U1.25; no longer U1.8
- net SHIFT_CLK3: now also U1.10; no longer U1.30
- net SHIFT_CLK4: now also U1.13; no longer U1.32
- net STORAGE_CLK1: now also U1.32; no longer U1.12
- net STORAGE_CLK2: now also U1.26; no longer U1.9
- net STORAGE_CLK3: now also U1.9; no longer U1.26
- net STORAGE_CLK4: now also U1.14; no longer U1.31
Routing:
- net !RESET: track 0.00 -> 60.2 mm, vias 0 -> 5
- net STORAGE_CLK3: track 0.00 -> 51.5 mm, vias 0 -> 2
- net SCK: track 0.00 -> 49.1 mm, vias 0 -> 4
- net SHIFT_CLK3: track 0.00 -> 45.9 mm, vias 0 -> 2
- net MOSI: track 0.00 -> 43.8 mm, vias 0 -> 1
- net SFT3: track 0.00 -> 43.1 mm, vias 0 -> 2
- net MISO: track 0.00 -> 39.9 mm, vias 0 -> 1
- net 1A: track 0.00 -> 30.5 mm, vias 0 -> 2
- net !BTN2: track 0.00 -> 30.4 mm, vias 0 -> 2
- net SFT4: track 0.00 -> 30.3 mm, vias 0 -> 4
- net 1B: track 0.00 -> 29.8 mm, vias 0 -> 2
- net SHIFT_CLK4: track 0.00 -> 28.7 mm
- net DIVIDED: track 0.00 -> 27.3 mm, vias 0 -> 2
- net STORAGE_CLK4: track 0.00 -> 27.3 mm
- net 1F: track 0.00 -> 27.1 mm, vias 0 -> 2
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Other:
- board size 160 x 100 mm -> 60 x 29.5 mm
- board text added: "+"
- board text added: "-"
- board text added: "1"
- board text added: "20"
- board text added: "21"
- board text added: "40"

Commit message: Adds up!
Button Number changed, Parts Added
Parts:
- moved K1 11.2 mm to (37.6, 36.8)
- moved K2 11.2 mm to (48.8, 36.8)
Connections:
- net !BTN1: now also C6.1, R5.2, U1.8; no longer C4.1, R3.2, U1.2
- net !BTN2: now also C4.1, R3.2, U1.2; no longer C6.1, R5.2, U1.8
- net N$1: now also K2.1; no longer K1.1
- net N$2: now also K1.1; no longer K2.1
Routing:
- net !BTN2: track 30.4 -> 23.2 mm
- net !BTN1: track 23.2 -> 30.4 mm
Changed lines of the file:
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@@
 <attribute name="VENDOR" value="Texas Instruments" x="25.25" y="22.18" size="1.778" layer="27" rot="R180" display="off"/>
 </element>
-<element name="K1" library="rgb-led" package="SW4-SMD-5.2X5.2X1.5MM" value="SKQGADE010" x="48.76" y="36.83" smashed="yes">
+<element name="K2" library="rgb-led" package="SW4-SMD-5.2X5.2X1.5MM" value="SKQGADE010" x="48.76" y="36.83" smashed="yes">
 <attribute name="MPN" value="SKQGADE010" x="48.76" y="36.83" size="1.778" layer="27" display="off"/>
 <attribute name="NAME" x="46.855" y="39.624" size="0.889" layer="25" ratio="11"/>
 </element>
-<element name="K2" library="rgb-led" package="SW4-SMD-5.2X5.2X1.5MM" value="SKQGADE010" x="37.6" y="36.83" smashed="yes">
+<element name="K1" library="rgb-led" package="SW4-SMD-5.2X5.2X1.5MM" value="SKQGADE010" x="37.6" y="36.83" smashed="yes">
 <attribute name="MPN" value="SKQGADE010" x="37.6" y="36.83" size="1.778" layer="27" display="off"/>
 <attribute name="NAME" x="35.695" y="39.624" size="0.889" layer="25" ratio="11"/>
@@
 <contactref element="U1" pad="5"/>
 <contactref element="R2" pad="1"/>
+<contactref element="K2" pad="3"/>
+<contactref element="K2" pad="2"/>
+<contactref element="C4" pad="2"/>
+<contactref element="R4" pad="1"/>
 <contactref element="K1" pad="3"/>
 <contactref element="K1" pad="2"/>
-<contactref element="C4" pad="2"/>
-<contactref element="R4" pad="1"/>
-<contactref element="K2" pad="3"/>
-<contactref element="K2" pad="2"/>
 <contactref element="C6" pad="2"/>
 <contactref element="R6" pad="1"/>
@@
 <signal name="N$1">
 <contactref element="R3" pad="1"/>
-<contactref element="K1" pad="1"/>
+<contactref element="K2" pad="1"/>
 <wire x1="45.66" y1="38.68" x2="44.18" y2="38.68" width="0.254" layer="1"/>
 <wire x1="44.18" y1="38.68" x2="43.18" y2="37.68" width="0.254" layer="1"/>
@@
 <signal name="N$2">
 <contactref element="R5" pad="1"/>
-<contactref element="K2" pad="1"/>
+<contactref element="K1" pad="1"/>
 <wire x1="34.5" y1="38.68" x2="33.25" y2="38.68" width="0.254" layer="1"/>
 <wire x1="33.25" y1="38.68" x2="32.25" y2="37.68" width="0.254" layer="1"/>
@@
 </signal>
 <signal name="!BTN1">
-<contactref element="R3" pad="2"/>
-<contactref element="C4" pad="1"/>
-<contactref element="U1" pad="2"/>
-<wire x1="43.18" y1="35.32" x2="43.18" y2="35.98" width="0.254" layer="1"/>
-<wire x1="44.84" y1="33.66" x2="44.84" y2="31.75" width="0.254" layer="1"/>
-<wire x1="44.84" y1="33.66" x2="43.18" y2="35.32" width="0.254" layer="1"/>
-<wire x1="51.5703" y1="23.26" x2="52.26" y2="23.26" width="0.254" layer="1"/>
-<wire x1="52.26" y1="23.26" x2="52.7808" y2="23.7808" width="0.254" layer="1"/>
-<wire x1="52.7808" y1="23.7808" x2="52.7808" y2="24.5050125" width="0.254" layer="1"/>
-<wire x1="52.7808" y1="24.5050125" x2="53.38789375" y2="25.11210625" width="0.254" layer="1"/>
-<wire x1="53.38789375" y1="25.11210625" x2="53.38789375" y2="27.61210625" width="0.254" layer="1"/>
-<wire x1="53.38789375" y1="27.61210625" x2="53" y2="28" width="0.254" layer="1"/>
-<via x="53" y="28" extent="1-16" drill="0.35"/>
-<wire x1="53" y1="28" x2="53" y2="31" width="0.254" layer="16"/>
-<wire x1="53" y1="31" x2="51" y2="33" width="0.254" layer="16"/>
-<wire x1="51" y1="33" x2="45.5" y2="33" width="0.254" layer="16"/>
-<wire x1="45.5" y1="33" x2="44.84" y2="33.66" width="0.254" layer="16"/>
-<via x="44.84" y="33.66" extent="1-16" drill="0.35"/>
-</signal>
-<signal name="!BTN2">
 <contactref element="R5" pad="2"/>
 <contactref element="C6" pad="1"/>
@@
 <via x="55" y="34" extent="1-16" drill="0.35"/>
 </signal>
+<signal name="!BTN2">
+<contactref element="R3" pad="2"/>
+<contactref element="C4" pad="1"/>
+<contactref element="U1" pad="2"/>
+<wire x1="44.84" y1="33.66" x2="43.18" y2="35.32" width="0.254" layer="1"/>
+<wire x1="51.5703" y1="23.26" x2="52.26" y2="23.26" width="0.254" layer="1"/>
+<wire x1="52.26" y1="23.26" x2="52.7808" y2="23.7808" width="0.254" layer="1"/>
+<wire x1="52.7808" y1="23.7808" x2="52.7808" y2="24.5050125" width="0.254" layer="1"/>
+<wire x1="52.7808" y1="24.5050125" x2="53.38789375" y2="25.11210625" width="0.254" layer="1"/>
+<wire x1="53.38789375" y1="25.11210625" x2="53.38789375" y2="27.61210625" width="0.254" layer="1"/>
+<wire x1="53.38789375" y1="27.61210625" x2="53" y2="28" width="0.254" layer="1"/>
+<via x="53" y="28" extent="1-16" drill="0.35"/>
+<wire x1="53" y1="28" x2="53" y2="31" width="0.254" layer="16"/>
+<wire x1="53" y1="31" x2="51" y2="33" width="0.254" layer="16"/>
+<wire x1="51" y1="33" x2="45.5" y2="33" width="0.254" layer="16"/>
+<wire x1="45.5" y1="33" x2="44.84" y2="33.66" width="0.254" layer="16"/>
+<via x="44.84" y="33.66" extent="1-16" drill="0.35"/>
+<wire x1="43.18" y1="35.98" x2="43.18" y2="35.32" width="0.254" layer="1"/>
+<wire x1="44.84" y1="31.75" x2="44.84" y2="33.66" width="0.254" layer="1"/>
+</signal>
 </signals>

Commit message: Minor Updates
Board rearranged to fit in MINI USB port. MINI USB port used as plenty
of supply exists in the shop
Parts:
- removed U$1: MICRO-USB, rgb-led:GS-14-2180
- added X1: MINI-USB-32005-201, con-cypressindustries:32005-201
- moved U$2 33.0 mm to (29.0, 27.5)
- moved K3 3.50 mm to (55.9, 36.8)
- moved K2 3.00 mm to (45.8, 36.8)
- moved R7 3.00 mm to (50.8, 36.8)
- moved R3 2.50 mm to (40.7, 36.8)
- moved K1 2.00 mm to (35.6, 36.8)
- moved R5 2.00 mm to (30.2, 36.8)
- moved R1 0.75 mm to (33.2, 30.6), turned to 90 degrees
- moved R6 0.26 mm to (49.6, 31.8), turned to 0 degrees
- moved R4 0.12 mm to (53.9, 31.8), turned to 180 degrees
Connections:
- net +5V: now also X1.1; no longer U$1.1
- net GND: now also X1.5; no longer U$1.5, U$1.5@1, U$1.5@2, U$1.5@3, U$1.5@4, U$1.5@6, U$1.5@7
Routing:
- net GND: track 90.3 -> 66.9 mm, vias 21 -> 19
- net !BTN1: track 30.4 -> 50.6 mm, vias 2 -> 4
- net !BTN2: track 23.2 -> 34.7 mm, vias 2 -> 0
- net +5V: track 10.9 -> 18.6 mm, vias 4 -> 6
- net SFT4: track 30.3 -> 36.1 mm, vias 4 -> 0
- net !BTN3: track 20.3 -> 24.4 mm, vias 2 -> 0
- net DIVIDED: track 27.3 -> 30.7 mm, vias 2 -> 1
- net 1F: track 27.1 -> 24.9 mm, vias 2 -> 1
- net 1A: track 30.5 -> 28.8 mm, vias 2 -> 1
- net 1B: track 29.8 -> 28.3 mm, vias 2 -> 1
- net 1G: track 21.3 -> 19.9 mm, vias 2 -> 1
- net N$4: track 2.89 -> 2.39 mm
- net N$1: track 2.89 -> 2.39 mm

Commit message: Board Updated according to Design Review
Parts:
- removed R3, R5, R7: 7.8k, resistor:R0603
- added C3, C5: 0.1uF, rcl:C0603
- C1: value 47uF -> 10uF
- U1: value ATMEGA328P-MUR -> ATMEGA328P-AUR; device lcd-buzzer:32M1-A -> lcd-buzzer:32A
- moved R6 8.65 mm to (58.2, 32.3), turned to 270 degrees
- moved R4 7.71 mm to (46.2, 32.3), turned to 270 degrees
- moved C8 6.53 mm to (52.2, 32.3), turned to 270 degrees
- moved C4 2.50 mm to (43.2, 32.3), turned to 270 degrees
- moved X1 1.50 mm to (67.5, 35.0)
- moved R2 1.35 mm to (40.2, 32.4), turned to 270 degrees
- moved U1 1.28 mm to (48.0, 24.0)
- moved C6 0.62 mm to (37.2, 32.4), turned to 270 degrees
- moved #4 0.58 mm to (23.8, 35.4)
- moved #3 0.50 mm to (23.9, 28.2)
- moved #1 0.08 mm to (58.3, 24.2)
Connections:
- removed net N$1: K2.1, R3.1
- removed net N$2: K1.1, R5.1
- removed net N$4: K3.1, R7.1
- new net N$5: K2.2, R2.1
- new net N$6: K1.2, R4.1
- new net N$7: K3.2, R6.1
- net !BTN1: now also K1.1; no longer R5.2
- net !BTN2: now also K2.1; no longer R3.2
- net !BTN3: now also K3.1; no longer R7.2
- net +5V: now also C3.1, C5.1
- net GND: now also C3.2, C5.2; no longer K1.2, K2.2, K3.2, R2.1, R4.1, R6.1
- net SFT2: now also U1.23; no longer U1.24
- net SHIFT_CLK2: now also U1.24; no longer U1.25
- net STORAGE_CLK2: now also U1.25; no longer U1.26
Routing:
- net +5V: track 18.6 -> 2.96 mm, vias 6 -> 2
- net N$5: track 0.00 -> 15.0 mm, vias 0 -> 2
- net N$6: track 0.00 -> 14.6 mm, vias 0 -> 2
- net GND: track 66.9 -> 56.7 mm, vias 19 -> 21
- net !BTN1: track 50.6 -> 41.4 mm, vias 4 -> 5
- net N$7: track 0.00 -> 6.95 mm
- net !BTN2: track 34.7 -> 28.9 mm
- net SHIFT_CLK2: track 9.66 -> 4.17 mm
- net STORAGE_CLK3: track 51.5 -> 47.6 mm
- net !BTN3: track 24.4 -> 20.8 mm
- net MISO: track 39.9 -> 37.0 mm
- net N$2: track 2.66 -> 0.00 mm
- net N$4: track 2.39 -> 0.00 mm
- net N$1: track 2.39 -> 0.00 mm
- net SCL: track 26.8 -> 24.5 mm
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
Commit message: Board Revision
Reference Designator updated, wonky silkscreen fixed, Library updated
and 2x3 header replaced with shrouded version
Parts:
- removed #2, #3: 74HC595PW, lcd-buzzer:SOT403-1
- removed C8: 1uF, resistor:C0603
- removed PS1240P02BT: PS1240P02BT, lcd-buzzer:PS1240P02BT
- removed R6: 10k, resistor:R0603
- removed SV1: (no value), con-lstb:MA03-2
- added C7: 10uF, rcl:C0603
- added LS1: PS1240P02BT, lcd-buzzer:PS1240P02BT
- added R3: 10k, resistor:R0603
- added U3: ATMEGA328P-AUR, lcd-buzzer:32A
- added U5: 74HC595PW, lcd-buzzer:SOT403-1
- added X3: 2X3SHROUDED, lcd-buzzer:2X3SHROUDED
- C1: value 10uF -> 0.1uF
- C2: value 1.0uF -> 0.1uF
- C3: value 0.1uF -> 1.0uF
- C5: value 0.1uF -> 1uF; device rcl:C0603 -> resistor:C0603
- U1: value ATMEGA328P-AUR -> 74HC595PW; device lcd-buzzer:32A -> lcd-buzzer:SOT403-1
- moved C3 27.0 mm to (29.4, 24.6), turned to 90 degrees
- moved C2 26.0 mm to (55.2, 32.3), turned to 270 degrees
- moved U1 24.5 mm to (23.9, 28.2)
- moved C1 18.6 mm to (49.2, 32.3), turned to 270 degrees
- moved C6 15.0 mm to (52.2, 32.3)
- moved C5 12.0 mm to (37.2, 32.4)
- moved R4 12.0 mm to (58.2, 32.3)
- moved X1 1.14 mm to (66.4, 34.7)
- moved U$2 0.30 mm to (29.3, 27.5)
- renumbered #1 to U2, #4 to U4, HAPTIC to U6, K1 to S1, K2 to S2, K3 to S3, LCD to DS1, TC33X-2-103E to VR1
Connections:
- net !BTN1: now also C5.1, U3.8; no longer C6.1, U1.8
- net !BTN2: now also U3.2; no longer U1.2
- net !BTN3: now also C6.1, U3.1; no longer C8.1, U1.1
- net !RESET: now also U3.29, X3.!RESET; no longer SV1.5, U1.29
- net +5V: now also C2.1, C7.1, R3.2, U1.10, U1.16, U3.18, U3.4, U3.6, U5.10, U5.16, X3.+5V; no longer #2.10, #2.16, #3.10, #3.16, C3.1, C5.1, R6.2, SV1.2, U1.18, U1.4, U1.6
- net 2A: now also U5.1; no longer #2.1
- net 2B: now also U5.2; no longer #2.2
- net 2C: now also U5.3; no longer #2.3
- net 2D: now also U5.4; no longer #2.4
- net 2E: now also U5.5; no longer #2.5
- net 2F: now also U5.6; no longer #2.6
- net 2G: now also U5.7; no longer #2.7
- net 3A: now also U1.1; no longer #3.1
- net 3B: now also U1.2; no longer #3.2
- net 3C: now also U1.3; no longer #3.3
- net 3D: now also U1.4; no longer #3.4
- net 3E: now also U1.5; no longer #3.5
- net 3F: now also U1.6; no longer #3.6
- net 3G: now also U1.7; no longer #3.7
- net GND: now also C2.2, C3.1, C7.2, U1.13, U1.8, U3.21, U3.3, U3.5, U5.13, U5.8, X3.GND; no longer #2.13, #2.8, #3.13, #3.8, C2.1, C3.2, C8.2, SV1.6, U1.21, U1.3, U1.5
- net LRA/ERM+: now also LS1.P$1; no longer PS1240P02BT.P$1
- net LRA/ERM-: now also LS1.P$2; no longer PS1240P02BT.P$2
- net MISO: now also U3.16, X3.MISO; no longer SV1.1, U1.16
- net MOSI: now also U3.15, X3.MOSI; no longer SV1.4, U1.15
- net N$3: now also C3.2; no longer C2.2
- net N$6: now also R3.1; no longer R4.1
- net N$7: now also R4.1; no longer R6.1
- net SCK: now also U3.17, X3.SCK; no longer SV1.3, U1.17
- net SCL: now also U3.28; no longer U1.28
- net SDA: now also U3.27; no longer U1.27
- net SFT1: now also U3.30; no longer U1.30
- net SFT2: now also U3.23, U5.14; no longer #2.14, U1.23
- net SFT3: now also U1.14, U3.11; no longer #3.14, U1.11
- net SFT4: now also U3.12; no longer U1.12
- net SHIFT_CLK1: now also U3.31; no longer U1.31
- net SHIFT_CLK2: now also U3.24, U5.12; no longer #2.12, U1.24
- net SHIFT_CLK3: now also U1.12, U3.10; no longer #3.12, U1.10
- net SHIFT_CLK4: now also U3.13; no longer U1.13
- net STORAGE_CLK1: now also U3.32; no longer U1.32
- net STORAGE_CLK2: now also U3.25, U5.11; no longer #2.11, U1.25
- net STORAGE_CLK3: now also U1.11, U3.9; no longer #3.11, U1.9
- net STORAGE_CLK4: now also U3.14; no longer U1.14
Routing:
- net !RESET: track 61.1 -> 70.8 mm, vias 5 -> 6
- net MISO: track 37.0 -> 46.4 mm, vias 1 -> 3
- net SFT4: track 35.2 -> 29.1 mm
- net STORAGE_CLK2: track 12.8 -> 7.41 mm
- net GND: track 56.7 -> 60.4 mm, vias 21 -> 20
- net N$3: track 8.16 -> 11.7 mm
- net LRA/ERM-: track 9.08 -> 12.1 mm
- net SCK: track 49.7 -> 52.3 mm
- net 2A: track 19.6 -> 21.7 mm
- net 2G: track 26.0 -> 28.1 mm
- net 2B: track 18.9 -> 21.0 mm
- net MOSI: track 41.8 -> 40.0 mm
- net SFT2: track 4.78 -> 6.35 mm
- net SHIFT_CLK2: track 4.17 -> 5.67 mm
- net 2F: track 24.5 -> 25.5 mm
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Other:
- board size 60 x 29.5 mm -> 62 x 29.5 mm
- board text added: "U6"

Commit message: Keep updating
Changed to Class5, schematics alignment corrected.
Parts:
- moved U1 0.48 mm to (23.4, 28.2)
- moved U4 0.41 mm to (23.4, 35.4)
- moved U5 0.30 mm to (37.3, 24.2)
Routing:
- net GND: track 60.4 -> 56.7 mm
- net 4B: track 26.0 -> 25.0 mm
- net 2F: track 25.5 -> 26.5 mm
- net 1F: track 24.9 -> 24.0 mm
- net !RESET: track 70.8 -> 71.7 mm
- net 3A: track 24.7 -> 23.9 mm
- net 4G: track 10.5 -> 11.2 mm
- net N$3: track 11.7 -> 11.1 mm
