File: 2017-2018/lec-buzzer_alt.brd (EAGLE design)
At the start: 62 x 29.5 mm, 26 parts, among them U1 74HC595PW, U2 74HC595PW, U3 ATMEGA328P-AUR, U4 74HC595PW, U5 74HC595PW, U6 DRV2605LDGSR, X1 MINI-USB-32005-201, X3 2X3SHROUDED

Commit message: training board ver 1.5
Parts:
- added D1: Yellow, SparkFun-LED:LED-0603
- added R5: 150, resistor:R0603
- U3: value ATMEGA328P-AUR -> ATMEGA328P-SUR; device lcd-buzzer:32A -> lcd-buzzer:ATMEGA328P-AUR-REAL
- moved U3 4.30 mm to (50.8, 20.7)
- moved R1 0.66 mm to (33.1, 29.9)
- moved U$2 0.11 mm to (29.4, 27.6)
Connections:
- new net LED: D1.A, U3.7
- new net N$1: D1.C, R5.2
- net GND: now also R5.1
Routing:
- net LED: track 0.00 -> 6.82 mm, vias 0 -> 2
- net !BTN1: track 41.4 -> 38.4 mm
- net STORAGE_CLK4: track 26.4 -> 23.9 mm
- net MISO: track 46.4 -> 44.0 mm
- net N$1: track 0.00 -> 2.29 mm
- net MOSI: track 40.0 -> 37.7 mm
- net SHIFT_CLK4: track 27.9 -> 25.8 mm
- net SCK: track 52.4 -> 50.6 mm
- net SCL: track 24.7 -> 23.2 mm
- net +5V: track 2.50 -> 3.98 mm
- net SDA: track 23.3 -> 21.8 mm
- net SFT4: track 29.5 -> 28.2 mm
- net SHIFT_CLK3: track 44.6 -> 43.5 mm
- net STORAGE_CLK1: track 9.95 -> 8.99 mm
- net SFT3: track 41.5 -> 40.6 mm
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
Commit message: 2nd Version
Indicator LED added, ATMega328p package updated, schematics updated.
Parts:
- moved U3 4.74 mm to (47.4, 24.0)
- moved R5 1.50 mm to (60.5, 32.3)
- moved C1 0.70 mm to (48.5, 32.3)
- moved C2 0.70 mm to (54.5, 32.3)
- moved C4 0.70 mm to (42.5, 32.3)
- moved C6 0.70 mm to (51.5, 32.3)
- moved R2 0.70 mm to (39.5, 32.4)
- moved R3 0.70 mm to (45.5, 32.3)
- moved R4 0.70 mm to (57.5, 32.3)
- moved C5 0.60 mm to (36.6, 32.4)
- moved D1 0.54 mm to (58.5, 28.2)
- moved R1 0.50 mm to (32.6, 29.9)
Connections:
- new net LCD_RESET: U1.10, U2.10, U3.26, U4.10, U5.10
- net +5V: no longer U1.10, U2.10, U4.10, U5.10
Routing:
- net LCD_RESET: track 0.00 -> 65.2 mm, vias 0 -> 6
- net !BTN3: track 21.5 -> 27.0 mm, vias 0 -> 2
- net !BTN2: track 29.2 -> 33.2 mm, vias 0 -> 2
- net N$6: track 14.6 -> 11.3 mm
- net N$1: track 2.29 -> 4.49 mm
- net !BTN1: track 38.4 -> 36.9 mm
- net +5V: track 3.98 -> 2.50 mm
- net SCL: track 23.2 -> 24.5 mm
- net SDA: track 21.8 -> 22.7 mm
- net GND: track 57.2 -> 58.0 mm, vias 20 -> 19
- net N$5: track 15.1 -> 14.5 mm

Commit message: LCD Column pin grounded
Connections:
- net GND: now also DS1.P$12, DS1.P$16, DS1.P$28, DS1.P$8
Changed lines of the file:
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@@
 <wire x1="60.58" y1="34.98" x2="60.6" y2="35" width="0.2" layer="1"/>
 <via x="60.6" y="35" extent="1-16" drill="0.35"/>
+<contactref element="DS1" pad="P$28"/>
+<contactref element="DS1" pad="P$16"/>
+<contactref element="DS1" pad="P$12"/>
+<contactref element="DS1" pad="P$8"/>
 </signal>
 <signal name="SHIFT_CLK4">

Commit message: Training Board Updated
A list of changes:
1. LCD COM pin: Now connected to Arduino Pin 13
2. ^that also means the trimmer resistor is removed
3. LED added, connected to Arduino Pin 12, can be the first thing for trainees to play with
4. LCD_Reset connected to A3
5. One of the three buttons is now a RESETN Button
6. Libraries updated, all ICs now includes the tiny circle denoting its direction
7. Schematics beautified and a bigger RoboBuzz
Parts:
- removed R5: 150, resistor:R0603
- removed U$2: (no value), RoboJackets-Aesthetics:ROBOBUZZ_0.4X
- removed VR1: TC33X, lcd-buzzer:TC33X-2-103E
- removed X3: 2X3SHROUDED, lcd-buzzer:2X3SHROUDED
- added U$1: (no value), RoboJackets-Aesthetics:ROBOBUZZ_0.6X
- added X2: MINI-USB-32005-201, con-cypressindustries:32005-201
- C1: value 0.1uF -> 1.0uF
- C3: value 1.0uF -> 0.1uF
- R1: value 10k -> 150; device rcl:R0603 -> resistor:R0603
- R2: device resistor:R0603 -> rcl:R0603
- U3: value ATMEGA328P-SUR -> DRV2605LDGSR; device lcd-buzzer:ATMEGA328P-AUR-REAL -> lcd-buzzer:DGS10
- U4: value 74HC595PW -> ATMEGA328P-SUR; device lcd-buzzer:SOT403-1 -> lcd-buzzer:ATMEGA328P-AUR-REAL
- U6: value DRV2605LDGSR -> 74HC595PW; device lcd-buzzer:DGS10 -> lcd-buzzer:SOT403-1
- X1: value MINI-USB-32005-201 -> 2X3SHROUDED; device con-cypressindustries:32005-201 -> lcd-buzzer:2X3SHROUDED
- moved X1 52.3 mm to (14.1, 36.0), turned to 90 degrees
- moved R1 27.0 mm to (59.5, 32.3), turned to 270 degrees
- moved U4 26.5 mm to (47.4, 24.0), turned to 180 degrees
- moved C3 25.4 mm to (53.5, 32.3), turned to 270 degrees
- moved U3 22.2 mm to (25.2, 22.2)
- moved C1 20.7 mm to (29.4, 24.6), turned to 90 degrees
- moved S1 20.3 mm to (55.9, 36.8)
- moved S3 20.3 mm to (35.6, 36.8)
- moved R4 16.0 mm to (41.5, 32.4)
- moved U6 13.3 mm to (23.4, 35.4), turned to 0 degrees
- moved C6 13.0 mm to (38.5, 32.3), turned to 90 degrees
- moved R3 11.0 mm to (56.5, 32.3)
- moved C4 8.00 mm to (50.5, 32.3)
- moved C5 7.90 mm to (44.5, 32.3)
- moved C2 7.00 mm to (47.5, 32.3)
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Connections:
- removed net !BTN1: C5.1, S1.1, U3.8
- removed net DIVIDED: DS1.P$1, DS1.P$40, VR1.WIPER
- removed net LED: D1.A, U3.7
- removed net N$7 (its old number): R4.1, S3.2
- new net N$4: U4.19
- net !BTN2: now also C5.1, U4.2; no longer C4.1, U3.2
- net !BTN3: now also C4.1, S1.1, U4.1; no longer C6.1, S3.1, U3.1
- net !RESET: now also C6.1, R2.1, S3.1, U4.29, X1.!RESET; no longer R1.1, U3.29, X3.!RESET
- net +5V: now also C3.1, U3.10, U3.5, U4.18, U4.4, U4.6, U6.16, X1.+5V, X2.1; no longer C1.1, R1.2, U3.18, U3.4, U3.6, U4.16, U6.10, U6.5, VR1.CCW, X1.1, X3.+5V
- net 4A: now also U6.1; no longer U4.1
- net 4B: now also U6.2; no longer U4.2
- net 4C: now also U6.3; no longer U4.3
- net 4D: now also U6.4; no longer U4.4
- net 4E: now also U6.5; no longer U4.5
- net 4F: now also U6.6; no longer U4.6
- net 4G: now also U6.7; no longer U4.7
- net GND: now also C1.1, C3.2, R1.1, U3.4, U3.8, U4.21, U4.3, U4.5, U6.13, X1.GND, X2.5; no longer C1.2, C3.1, DS1.P$12, DS1.P$16, DS1.P$28, DS1.P$8, R5.1, U3.21, U3.3, U3.5, U4.13, U4.8, U6.4, VR1.CW, X1.5, X3.GND
- net LCD_RESET: now also U4.26, U6.10; no longer U3.26, U4.10
- net LRA/ERM+: now also U3.7; no longer U6.7
- net LRA/ERM-: now also U3.9; no longer U6.9
- net MISO: now also U4.16, X1.MISO; no longer U3.16, X3.MISO
- net MOSI: now also D1.A, U4.15, X1.MOSI; no longer U3.15, X3.MOSI
- net N$1: now also R1.2; no longer R5.2
- net N$3: now also C1.2, U3.1; no longer C3.2, U6.1
- net N$5: now also R4.1; no longer R2.1
- net SCK: now also DS1.P$1, DS1.P$12, DS1.P$16, DS1.P$28, DS1.P$40, DS1.P$8, U4.17, X1.SCK; no longer U3.17, X3.SCK
- net SCL: now also U3.2, U4.28; no longer U3.28, U6.2
- net SDA: now also U3.3, U4.27; no longer U3.27, U6.3
- net SFT1: now also U4.30; no longer U3.30
- net SFT2: now also U4.23; no longer U3.23
- net SFT3: now also U4.11; no longer U3.11
- net SFT4: now also U4.12, U6.14; no longer U3.12, U4.14
- net SHIFT_CLK1: now also U4.31; no longer U3.31
- net SHIFT_CLK2: now also U4.24; no longer U3.24
- net SHIFT_CLK3: now also U4.10; no longer U3.10
- net SHIFT_CLK4: now also U4.13, U6.12; no longer U3.13, U4.12
- net STORAGE_CLK1: now also U4.32; no longer U3.32
- net STORAGE_CLK2: now also U4.25; no longer U3.25
- net STORAGE_CLK3: now also U4.9; no longer U3.9
- net STORAGE_CLK4: now also U4.14, U6.11; no longer U3.14, U4.11
- net VDD/NC: now also U3.6; no longer U6.6
Routing:
- net SCK: track 50.6 -> 168.1 mm, vias 4 -> 7
- net MOSI: track 37.7 -> 103.0 mm, vias 1 -> 4
- net !BTN1: track 36.9 -> 0.00 mm, vias 5 -> 0
- net DIVIDED: track 30.7 -> 0.00 mm, vias 1 -> 0
- net !RESET: track 72.3 -> 84.5 mm, vias 6 -> 10
- net LED: track 7.26 -> 0.00 mm, vias 2 -> 0
- net N$7 (its old number): track 6.64 -> 0.00 mm
- net GND: track 58.0 -> 52.7 mm, vias 19 -> 18
- net N$7: track 11.3 -> 7.04 mm, vias 2 -> 0
- net !BTN3: track 27.0 -> 25.0 mm
- net N$1: track 4.49 -> 3.08 mm
- net SFT4: track 27.7 -> 26.8 mm
- net LCD_RESET: track 65.2 -> 65.7 mm

Commit message: training board v1.1
Parts:
- removed DS1: LCD-S401C39TR, lcd-buzzer:S401C39TR
- added D2: Green, SparkFun-LED:LED-0603
- added LCD1: LCD-S401C39TR, lcd-buzzer:S401C39TR
- added R5: 150, resistor:R0603
- D1: value Yellow -> Blue
- U4: value ATMEGA328P-SUR -> ATMEGA328P-AUR; device lcd-buzzer:ATMEGA328P-AUR-REAL -> lcd-buzzer:ATMEGA328P-AUR
- moved R1 37.9 mm to (25.5, 15.8), turned to 0 degrees
- moved C2 37.4 mm to (11.9, 20.9), turned to 90 degrees
- moved S3 34.8 mm to (55.5, 8.25)
- moved D1 34.2 mm to (25.5, 17.5)
- moved C3 30.4 mm to (25.1, 21.8)
- moved U$1 30.1 mm to (6.20, 7.00), flipped to the bottom
- moved U4 29.0 mm to (18.5, 21.0), turned to 0 degrees
- moved U1 28.5 mm to (44.5, 9.00), turned to 90 degrees
- moved C6 27.8 mm to (49.5, 6.75), turned to 270 degrees
- moved U2 27.4 mm to (35.5, 9.00), turned to 90 degrees
- moved U6 26.9 mm to (18.5, 9.00), turned to 90 degrees
- moved R2 24.6 mm to (50.8, 13.0)
- moved C5 20.7 mm to (32.5, 15.5), turned to 0 degrees
- moved R3 20.2 mm to (42.5, 17.8), turned to 0 degrees
- moved C1 20.0 mm to (12.0, 14.8), turned to 180 degrees
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Connections:
- removed net LCD_RESET: U1.10, U2.10, U4.26, U5.10, U6.10
- removed net N$4: U4.19
- removed net N$5: R4.1, S2.2
- removed net N$7: R3.1, S1.2
- removed net SFT1: U2.14, U4.30
- removed net SFT2: U4.23, U5.14
- removed net SFT3: U1.14, U4.11
- removed net SFT4: U4.12, U6.14
- removed net SHIFT_CLK1: U2.12, U4.31
- removed net SHIFT_CLK2: U4.24, U5.12
- removed net SHIFT_CLK3: U1.12, U4.10
- removed net SHIFT_CLK4: U4.13, U6.12
- removed net STORAGE_CLK1: U2.11, U4.32
- removed net STORAGE_CLK2: U4.25, U5.11
- removed net STORAGE_CLK3: U1.11, U4.9
- removed net STORAGE_CLK4: U4.14, U6.11
- removed net VDD/NC: U3.6
- new net COL: LCD1.28
- new net COM: LCD1.1, LCD1.40, U4.25
- new net DP1: LCD1.8
- new net DP2: LCD1.12
- new net DP3: LCD1.16
- new net LED1: D1.A, U4.14
- new net N$2: D2.C, R5.2
- new net SFT-!OE: U1.13, U2.13, U4.9, U5.13, U6.13
- new net SFT-!RESET: U1.10, U2.10, U4.12, U5.10, U6.10
- new net SFT-CLK: U1.11, U2.11, U4.11, U5.11, U6.11
- new net SFT-LATCH: U1.12, U2.12, U4.10, U5.12, U6.12
- new net SFT1-IN: U1.14, U4.13
- new net SFT2-IN: U1.9, U2.14
- new net SFT3-IN: U2.9, U5.14
- new net SFT4-IN: U5.9, U6.14
- net !BTN2: now also R4.1, S2.4; no longer S2.1, U4.2
- net !BTN3: now also R3.1, S1.4; no longer S1.1, U4.1
- net +5V: now also D2.A, S1.1, S2.1; no longer R3.2, R4.2
- net 1A: now also LCD1.35, U1.15; no longer DS1.P$35, U2.1
- net 1B: now also LCD1.34, U1.1; no longer DS1.P$34, U2.2
- net 1C: now also LCD1.7, U1.2; no longer DS1.P$7, U2.3
- net 1D: now also LCD1.6, U1.3; no longer DS1.P$6, U2.4
- net 1E: now also LCD1.5, U1.4; no longer DS1.P$5, U2.5
- net 1F: now also LCD1.36, U1.5; no longer DS1.P$36, U2.6
- net 1G: now also LCD1.37, U1.6; no longer DS1.P$37, U2.7
- net 2A: now also LCD1.30, U2.15; no longer DS1.P$30, U5.1
- net 2B: now also LCD1.29, U2.1; no longer DS1.P$29, U5.2
- net 2C: now also LCD1.11, U2.2; no longer DS1.P$11, U5.3
- net 2D: now also LCD1.10, U2.3; no longer DS1.P$10, U5.4
- net 2E: now also LCD1.9, U2.4; no longer DS1.P$9, U5.5
- net 2F: now also LCD1.31, U2.5; no longer DS1.P$31, U5.6
- net 2G: now also LCD1.32, U2.6; no longer DS1.P$32, U5.7
- net 3A: now also LCD1.25, U5.15; no longer DS1.P$25, U1.1
- net 3B: now also LCD1.24, U5.1; no longer DS1.P$24, U1.2
- net 3C: now also LCD1.15, U5.2; no longer DS1.P$15, U1.3
- net 3D: now also LCD1.14, U5.3; no longer DS1.P$14, U1.4
- net 3E: now also LCD1.13, U5.4; no longer DS1.P$13, U1.5
- net 3F: now also LCD1.26, U5.5; no longer DS1.P$26, U1.6
- net 3G: now also LCD1.27, U5.6; no longer DS1.P$27, U1.7
- net 4A: now also LCD1.21, U6.15; no longer DS1.P$21, U6.1
- net 4B: now also LCD1.20, U6.1; no longer DS1.P$20, U6.2
- net 4C: now also LCD1.19, U6.2; no longer DS1.P$19, U6.3
- net 4D: now also LCD1.18, U6.3; no longer DS1.P$18, U6.4
- net 4E: now also LCD1.17, U6.4; no longer DS1.P$17, U6.5
- net 4F: now also LCD1.22, U6.5; no longer DS1.P$22, U6.6
- net 4G: now also LCD1.23, U6.6; no longer DS1.P$23, U6.7
- net GND: now also C1.2, R3.2, R4.2, R5.1, S3.4; no longer C1.1, S1.3, S2.3, S3.3, U1.13, U2.13, U5.13, U6.13
- net LRA/ERM+: now also LS1.1; no longer LS1.P$1
- net LRA/ERM-: now also LS1.2; no longer LS1.P$2
- net MOSI: no longer D1.A
- net N$3: now also C1.1; no longer C1.2
- net SCK: no longer DS1.P$1, DS1.P$12, DS1.P$16, DS1.P$28, DS1.P$40, DS1.P$8
Routing:
- net SCK: track 168.1 -> 21.4 mm, vias 7 -> 1
- net MOSI: track 103.0 -> 17.6 mm, vias 4 -> 1
- net LCD_RESET: track 65.7 -> 0.00 mm, vias 6 -> 0
- net COM: track 0.00 -> 63.4 mm, vias 0 -> 1
- net STORAGE_CLK3: track 46.5 -> 0.00 mm, vias 2 -> 0
- net SFT-LATCH: track 0.00 -> 45.1 mm, vias 0 -> 4
- net SHIFT_CLK3: track 43.7 -> 0.00 mm, vias 2 -> 0
- net SFT-!OE: track 0.00 -> 42.1 mm, vias 0 -> 4
- net SFT3: track 40.7 -> 0.00 mm, vias 2 -> 0
- net SFT1-IN: track 0.00 -> 40.6 mm, vias 0 -> 2
- net SFT-!RESET: track 0.00 -> 39.0 mm, vias 0 -> 4
- net SFT-CLK: track 0.00 -> 36.5 mm, vias 0 -> 4
- net !BTN2: track 33.2 -> 6.08 mm, vias 2 -> 0
- net SFT4: track 26.8 -> 0.00 mm
- net SHIFT_CLK4: track 25.4 -> 0.00 mm
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Other:
- board text added: "RESET"
- board text added: "Training v1.1"
- board text removed: "+"
- board text removed: "-"
- board text removed: "1"
- board text removed: "20"
- board text removed: "21"
- board text removed: "U6"

Commit message: add lcd dots
Connections:
- net COL: now also U1.7
- net DP1: now also U2.7
- net DP2: now also U5.7
- net DP3: now also U6.7
Routing:
- net COL: track 0.00 -> 67.0 mm, vias 0 -> 2
- net DP1: track 0.00 -> 5.93 mm
- net DP2: track 0.00 -> 4.41 mm
- net DP3: track 0.00 -> 3.25 mm
Changed lines of the file:
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@@
 <wire x1="35.175" y1="6.1806" x2="35.175" y2="5.075" width="0.3" layer="1"/>
 <wire x1="35.175" y1="5.075" x2="35.5" y2="4.75" width="0.3" layer="1"/>
-<wire x1="35.5" y1="4.75" x2="37.18" y2="4.75" width="0.3" layer="1"/>
-<wire x1="37.18" y1="4.75" x2="38.68" y2="3.25" width="0.3" layer="1"/>
+<wire x1="35.5" y1="4.75" x2="36.75" y2="4.75" width="0.3" layer="1"/>
+<wire x1="36.75" y1="4.75" x2="37.25" y2="4.25" width="0.3" layer="1"/>
+<wire x1="37.25" y1="4.25" x2="37.68" y2="4.25" width="0.3" layer="1"/>
+<wire x1="37.68" y1="4.25" x2="38.68" y2="3.25" width="0.3" layer="1"/>
 </signal>
 <signal name="2F">
@@
 <signal name="COL">
 <contactref element="LCD1" pad="28"/>
+<wire x1="28.52" y1="27.888" x2="28.52" y2="26.48" width="0.3" layer="1"/>
+<wire x1="28.52" y1="26.48" x2="29" y2="26" width="0.3" layer="1"/>
+<via x="29" y="26" extent="1-16" drill="0.35"/>
+<wire x1="29" y1="26" x2="29.25" y2="26" width="0.3" layer="16"/>
+<wire x1="29.25" y1="26" x2="29.5" y2="26.25" width="0.3" layer="16"/>
+<wire x1="29.5" y1="26.25" x2="57.5" y2="26.25" width="0.3" layer="16"/>
+<wire x1="57.5" y1="26.25" x2="58.5" y2="25.25" width="0.3" layer="16"/>
+<wire x1="58.5" y1="25.25" x2="58.5" y2="5.5" width="0.3" layer="16"/>
+<wire x1="58.5" y1="5.5" x2="58" y2="5" width="0.3" layer="16"/>
+<wire x1="58" y1="5" x2="50.75" y2="5" width="0.3" layer="16"/>
+<wire x1="50.75" y1="5" x2="47.75" y2="8" width="0.3" layer="16"/>
+<via x="47.75" y="8" extent="1-16" drill="0.35"/>
+<contactref element="U1" pad="7"/>
+<wire x1="46.124996875" y1="6.1806" x2="46.124996875" y2="7.124996875" width="0.3" layer="1"/>
+<wire x1="46.124996875" y1="7.124996875" x2="47" y2="8" width="0.3" layer="1"/>
+<wire x1="47" y1="8" x2="47.75" y2="8" width="0.3" layer="1"/>
 </signal>
 <signal name="DP1">
 <contactref element="LCD1" pad="8"/>
+<contactref element="U2" pad="7"/>
+<wire x1="37.124996875" y1="6.1806" x2="37.124996875" y2="5.125003125" width="0.3" layer="1"/>
+<wire x1="37.124996875" y1="5.125003125" x2="37.5" y2="4.75" width="0.3" layer="1"/>
+<wire x1="37.5" y1="4.75" x2="39.72" y2="4.75" width="0.3" layer="1"/>
+<wire x1="39.72" y1="4.75" x2="41.22" y2="3.25" width="0.3" layer="1"/>
 </signal>
 <signal name="DP2">
 <contactref element="LCD1" pad="12"/>
+<contactref element="U5" pad="7"/>
+<wire x1="28.624996875" y1="6.1806" x2="28.624996875" y2="4.875003125" width="0.3" layer="1"/>
+<wire x1="28.624996875" y1="4.875003125" x2="29" y2="4.5" width="0.3" layer="1"/>
+<wire x1="29" y1="4.5" x2="29.81" y2="4.5" width="0.3" layer="1"/>
+<wire x1="29.81" y1="4.5" x2="31.06" y2="3.25" width="0.3" layer="1"/>
 </signal>
 <signal name="DP3">
 <contactref element="LCD1" pad="16"/>
+<contactref element="U6" pad="7"/>
+<wire x1="20.124996875" y1="6.1806" x2="20.124996875" y2="4.025003125" width="0.3" layer="1"/>
+<wire x1="20.124996875" y1="4.025003125" x2="20.9" y2="3.25" width="0.3" layer="1"/>
 </signal>
 <signal name="LED1">

Commit message: Button Connected
Connections:
- net !BTN2: now also U4.23
- net !BTN3: now also U4.24
Routing:
- net !BTN3: track 5.87 -> 26.7 mm, vias 0 -> 2
- net !BTN2: track 6.08 -> 16.4 mm, vias 0 -> 2
Changed lines of the file:
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@@
 <setting verticaltext="up"/>
 </settings>
-<grid distance="0.5" unitdist="mm" unit="mm" style="lines" multiple="1" display="yes" altdistance="0.25" altunitdist="mm" altunit="mm"/>
+<grid distance="0.1" unitdist="mm" unit="mm" style="lines" multiple="1" display="yes" altdistance="0.25" altunitdist="mm" altunit="mm"/>
 <layers>
 <layer number="1" name="Top" color="4" fill="1" visible="yes" active="yes"/>
@@
 <wire x1="41.65" y1="15.5" x2="41.65" y2="17.75" width="0.3" layer="1"/>
 <wire x1="41.65" y1="17.75" x2="41.65" y2="18.9" width="0.3" layer="1"/>
-<wire x1="41.65" y1="18.9" x2="39.9" y2="20.65" width="0.3" layer="1"/>
+<wire x1="39.9" y1="20.65" x2="41.65" y2="18.9" width="0.3" layer="1"/>
+<contactref element="U4" pad="24"/>
+<wire x1="22.5845" y1="23.603" x2="22.5845" y2="23.7845" width="0.3" layer="1"/>
+<wire x1="22.5845" y1="23.7845" x2="23.2" y2="24.4" width="0.3" layer="1"/>
+<via x="23.2" y="24.4" extent="1-16" drill="0.35"/>
+<wire x1="23.2" y1="24.4" x2="23.2" y2="23" width="0.3" layer="16"/>
+<wire x1="23.2" y1="23" x2="23.75" y2="22.45" width="0.3" layer="16"/>
+<wire x1="23.75" y1="22.45" x2="28.10146875" y2="22.45" width="0.3" layer="16"/>
+<wire x1="28.10146875" y1="22.45" x2="28.25146875" y2="22.6" width="0.3" layer="16"/>
+<wire x1="28.74853125" y1="22.6" x2="28.25146875" y2="22.6" width="0.3" layer="16"/>
+<via x="39.4" y="22" extent="1-16" drill="0.35"/>
+<wire x1="39.4" y1="22" x2="39.6" y2="22" width="0.3" layer="1"/>
+<wire x1="39.6" y1="22" x2="39.9" y2="21.7" width="0.3" layer="1"/>
+<wire x1="39.9" y1="21.7" x2="39.9" y2="20.65" width="0.3" layer="1"/>
+<wire x1="39.4" y1="22" x2="29.34853125" y2="22" width="0.3" layer="16"/>
+<wire x1="29.34853125" y1="22" x2="28.74853125" y2="22.6" width="0.3" layer="16"/>
 </signal>
 <signal name="!BTN2">
@@
 <wire x1="31.65" y1="15.5" x2="31.65" y2="17.75" width="0.3" layer="1"/>
 <wire x1="31.65" y1="17.75" x2="31.65" y2="18.4" width="0.3" layer="1"/>
-<wire x1="31.65" y1="18.4" x2="29.4" y2="20.65" width="0.3" layer="1"/>
+<wire x1="29.525" y1="20.525" x2="31.65" y2="18.4" width="0.3" layer="1"/>
+<contactref element="U4" pad="23"/>
+<wire x1="29.525" y1="20.525" x2="29.4" y2="20.65" width="0.3" layer="1"/>
+<wire x1="22.5845" y1="22.803" x2="21.803" y2="22.803" width="0.3" layer="1"/>
+<wire x1="21.803" y1="22.803" x2="21.5" y2="22.5" width="0.3" layer="1"/>
+<via x="21.5" y="22.5" extent="1-16" drill="0.35"/>
+<wire x1="21.5" y1="22.5" x2="22" y2="22" width="0.3" layer="16"/>
+<via x="28.5" y="22" extent="1-16" drill="0.35"/>
+<wire x1="28.5" y1="22" x2="29.525" y2="20.975" width="0.3" layer="1"/>
+<wire x1="29.525" y1="20.975" x2="29.525" y2="20.525" width="0.3" layer="1"/>
+<wire x1="22" y1="22" x2="28.5" y2="22" width="0.3" layer="16"/>
 </signal>
 <signal name="N$1">
