File: 2017-2018/lec-buzzer_alt.sch (EAGLE design)
At the start: 30 parts, among them K1 SKQGADE010, K2 SKQGADE010, K3 SKQGADE010, U1 ATMEGA328P-MUR

Commit message: begin 3 button board
Parts:
- removed C3: 0.1uF, SparkFun-Capacitors:0.1UF-0603-25V-(+80/-20%)
- removed C5, C7, C9: 100nF, resistor:C-USC0603
- C1: device SparkFun-Capacitors:47UF-POLAR-EIA3528-10V-10% -> rcl:C-USC0603
- C2: device SparkFun-Capacitors:1.0UF-0603-16V-10% -> rcl:C-USC0603
- C4, C6, C8: value 100nF -> 1uF
- R1: device SparkFun-Resistors:10KOHM-0603-1/10W-1% -> rcl:R-US_R0603
- R3, R5, R7: value 39k -> 7.8k
Connections:
- net !BTN1: no longer C5.1
- net !BTN2: no longer C7.1
- net !BTN3: no longer C9.1
- net +5V: now also C1.1; no longer C1.+, C3.1
- net GND: now also C1.2; no longer C1.-, C3.2, C5.2, C7.2, C9.2
Other:
- note added: "coupling capacitor?"

Commit message: 3 Button Board completed
LCD flipped, slight changes in shifter, Buzzer and SPI location
Connections:
- net !BTN2: now also U1.(PCINT7/XTAL2/TOSC2)_PB7; no longer U1.(PCINT1/OC1A)_PB1
- net !BTN3: now also U1.(PCINT19/OC2B/INT1)_PD3; no longer U1.(PCINT2/SS/OC1B)_PB2
- net SFT1: now also U1.PD0_(RXD/PCINT16); no longer U1.(PCINT22/OC0A/AIN0)_PD6
- net SFT2: now also U1.PC1_(ADC1/PCINT9); no longer U1.(PCINT6/XTAL1/TOSC1)_PB6
- net SFT3: now also U1.(PCINT23/AIN1)_PD7; no longer U1.PC2_(ADC2/PCINT10)
- net SFT4: now also U1.(PCINT0/CLKO/ICP1)_PB0; no longer U1.(PCINT19/OC2B/INT1)_PD3
- net SHIFT_CLK1: now also U1.PD1_(TXD/PCINT17); no longer U1.(PCINT23/AIN1)_PD7
- net SHIFT_CLK2: now also U1.PC2_(ADC2/PCINT10); no longer U1.(PCINT7/XTAL2/TOSC2)_PB7
- net SHIFT_CLK3: now also U1.(PCINT22/OC0A/AIN0)_PD6; no longer U1.PD0_(RXD/PCINT16)
- net SHIFT_CLK4: now also U1.(PCINT1/OC1A)_PB1; no longer U1.PD2_(INT0/PCINT18)
- net STORAGE_CLK1: now also U1.PD2_(INT0/PCINT18); no longer U1.(PCINT0/CLKO/ICP1)_PB0
- net STORAGE_CLK2: now also U1.PC3_(ADC3/PCINT11); no longer U1.(PCINT21/OC0B/T1)_PD5
- net STORAGE_CLK3: now also U1.(PCINT21/OC0B/T1)_PD5; no longer U1.PC3_(ADC3/PCINT11)
- net STORAGE_CLK4: now also U1.(PCINT2/SS/OC1B)_PB2; no longer U1.PD1_(TXD/PCINT17)
Changed lines of the file:
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@@
 <?xml version="1.0" encoding="utf-8"?>
 <!DOCTYPE eagle SYSTEM "eagle.dtd">
-<eagle version="8.3.0">
+<eagle version="8.3.1">
 <drawing>
 <settings>
@@
 </segment>
 <segment>
-<pinref part="U1" gate="A" pin="PD2_(INT0/PCINT18)"/>
-<wire x1="166.624" y1="55.88" x2="180.34" y2="55.88" width="0.1524" layer="91"/>
-<label x="167.64" y="55.88" size="1.778" layer="95"/>
+<pinref part="U1" gate="A" pin="(PCINT1/OC1A)_PB1"/>
+<wire x1="29.464" y1="25.4" x2="12.7" y2="25.4" width="0.1524" layer="91"/>
+<label x="12.7" y="25.4" size="1.778" layer="95"/>
 </segment>
 </net>
@@
 </segment>
 <segment>
-<pinref part="U1" gate="A" pin="PD1_(TXD/PCINT17)"/>
-<wire x1="166.624" y1="53.34" x2="180.34" y2="53.34" width="0.1524" layer="91"/>
-<label x="167.64" y="53.34" size="1.778" layer="95"/>
+<pinref part="U1" gate="A" pin="(PCINT2/SS/OC1B)_PB2"/>
+<wire x1="29.464" y1="22.86" x2="12.7" y2="22.86" width="0.1524" layer="91"/>
+<label x="12.7" y="22.86" size="1.778" layer="95"/>
 </segment>
 </net>
@@
 </segment>
 <segment>
-<pinref part="U1" gate="A" pin="(PCINT22/OC0A/AIN0)_PD6"/>
-<wire x1="29.464" y1="33.02" x2="12.7" y2="33.02" width="0.1524" layer="91"/>
-<label x="22.86" y="33.02" size="1.778" layer="95"/>
+<pinref part="U1" gate="A" pin="PD0_(RXD/PCINT16)"/>
+<wire x1="166.624" y1="50.8" x2="180.34" y2="50.8" width="0.1524" layer="91"/>
+<label x="167.64" y="50.8" size="1.778" layer="95"/>
 </segment>
 </net>
@@
 </segment>
 <segment>
-<pinref part="U1" gate="A" pin="PC2_(ADC2/PCINT10)"/>
-<wire x1="166.624" y1="38.1" x2="180.34" y2="38.1" width="0.1524" layer="91"/>
-<label x="167.64" y="38.1" size="1.778" layer="95"/>
+<pinref part="U1" gate="A" pin="(PCINT23/AIN1)_PD7"/>
+<wire x1="29.464" y1="30.48" x2="12.7" y2="30.48" width="0.1524" layer="91"/>
+<label x="12.7" y="30.48" size="1.778" layer="95"/>
 </segment>
 </net>
@@
 </segment>
 <segment>
-<pinref part="U1" gate="A" pin="(PCINT19/OC2B/INT1)_PD3"/>
-<wire x1="29.464" y1="55.88" x2="12.7" y2="55.88" width="0.1524" layer="91"/>
-<label x="22.86" y="55.88" size="1.778" layer="95"/>
+<pinref part="U1" gate="A" pin="(PCINT0/CLKO/ICP1)_PB0"/>
+<wire x1="29.464" y1="27.94" x2="12.7" y2="27.94" width="0.1524" layer="91"/>
+<label x="8.89" y="27.94" size="1.778" layer="95"/>
 </segment>
 </net>
@@
 </segment>
 <segment>
-<pinref part="U1" gate="A" pin="(PCINT6/XTAL1/TOSC1)_PB6"/>
-<wire x1="29.464" y1="40.64" x2="15.24" y2="40.64" width="0.1524" layer="91"/>
-<label x="22.86" y="40.64" size="1.778" layer="95"/>
+<pinref part="U1" gate="A" pin="PC1_(ADC1/PCINT9)"/>
+<wire x1="166.624" y1="35.56" x2="180.34" y2="35.56" width="0.1524" layer="91"/>
+<label x="167.64" y="35.56" size="1.778" layer="95"/>
 </segment>
 </net>
@@
 </segment>
 <segment>
-<pinref part="U1" gate="A" pin="(PCINT23/AIN1)_PD7"/>
-<wire x1="29.464" y1="30.48" x2="12.7" y2="30.48" width="0.1524" layer="91"/>
-<label x="12.7" y="30.48" size="1.778" layer="95"/>
+<pinref part="U1" gate="A" pin="PD1_(TXD/PCINT17)"/>
+<wire x1="166.624" y1="53.34" x2="180.34" y2="53.34" width="0.1524" layer="91"/>
+<label x="167.64" y="53.34" size="1.778" layer="95"/>
 </segment>
 </net>
@@
 </segment>
 <segment>
-<pinref part="U1" gate="A" pin="(PCINT0/CLKO/ICP1)_PB0"/>
-<wire x1="29.464" y1="27.94" x2="12.7" y2="27.94" width="0.1524" layer="91"/>
-<label x="8.89" y="27.94" size="1.778" layer="95"/>
+<pinref part="U1" gate="A" pin="PD2_(INT0/PCINT18)"/>
+<wire x1="166.624" y1="55.88" x2="180.34" y2="55.88" width="0.1524" layer="91"/>
+<label x="167.64" y="55.88" size="1.778" layer="95"/>
 </segment>
 </net>
@@
 </segment>
 <segment>
+<pinref part="U1" gate="A" pin="PC3_(ADC3/PCINT11)"/>
+<wire x1="166.624" y1="40.64" x2="180.34" y2="40.64" width="0.1524" layer="91"/>
+<label x="167.64" y="40.64" size="1.778" layer="95"/>
+</segment>
+</net>
+<net name="SHIFT_CLK2" class="0">
+<segment>
+<pinref part="#2" gate="A" pin="ST_CP"/>
+<wire x1="133.4" y1="93.9" x2="146.1" y2="93.9" width="0.1524" layer="91"/>
+<label x="134.12" y="93.82" size="1.778" layer="95"/>
+</segment>
+<segment>
+<pinref part="U1" gate="A" pin="PC2_(ADC2/PCINT10)"/>
+<wire x1="166.624" y1="38.1" x2="180.34" y2="38.1" width="0.1524" layer="91"/>
+<label x="167.64" y="38.1" size="1.778" layer="95"/>
+</segment>
+</net>
+<net name="STORAGE_CLK3" class="0">
+<segment>
+<pinref part="#3" gate="A" pin="SH_CP"/>
+<wire x1="54.46" y1="134.54" x2="67.16" y2="134.54" width="0.1524" layer="91"/>
+<label x="55.18" y="134.5" size="1.778" layer="95"/>
+</segment>
+<segment>
 <pinref part="U1" gate="A" pin="(PCINT21/OC0B/T1)_PD5"/>
 <wire x1="29.464" y1="35.56" x2="12.7" y2="35.56" width="0.1524" layer="91"/>
@@
 </segment>
 </net>
-<net name="SHIFT_CLK2" class="0">
-<segment>
-<pinref part="#2" gate="A" pin="ST_CP"/>
-<wire x1="133.4" y1="93.9" x2="146.1" y2="93.9" width="0.1524" layer="91"/>
-<label x="134.12" y="93.82" size="1.778" layer="95"/>
-</segment>
-<segment>
-<pinref part="U1" gate="A" pin="(PCINT7/XTAL2/TOSC2)_PB7"/>
-<wire x1="29.464" y1="38.1" x2="12.7" y2="38.1" width="0.1524" layer="91"/>
-<label x="12.7" y="38.1" size="1.778" layer="95"/>
-</segment>
-</net>
-<net name="STORAGE_CLK3" class="0">
-<segment>
-<pinref part="#3" gate="A" pin="SH_CP"/>
-<wire x1="54.46" y1="134.54" x2="67.16" y2="134.54" width="0.1524" layer="91"/>
-<label x="55.18" y="134.5" size="1.778" layer="95"/>
-</segment>
-<segment>
-<pinref part="U1" gate="A" pin="PC3_(ADC3/PCINT11)"/>
-<wire x1="166.624" y1="40.64" x2="180.34" y2="40.64" width="0.1524" layer="91"/>
-<label x="167.64" y="40.64" size="1.778" layer="95"/>
-</segment>
-</net>
 <net name="SHIFT_CLK3" class="0">
 <segment>
@@
 </segment>
 <segment>
-<pinref part="U1" gate="A" pin="PD0_(RXD/PCINT16)"/>
-<wire x1="166.624" y1="50.8" x2="180.34" y2="50.8" width="0.1524" layer="91"/>
-<label x="167.64" y="50.8" size="1.778" layer="95"/>
+<pinref part="U1" gate="A" pin="(PCINT22/OC0A/AIN0)_PD6"/>
+<wire x1="29.464" y1="33.02" x2="12.7" y2="33.02" width="0.1524" layer="91"/>
+<label x="10.16" y="33.02" size="1.778" layer="95"/>
 </segment>
 </net>
@@
 </segment>
 <segment>
-<pinref part="U1" gate="A" pin="(PCINT1/OC1A)_PB1"/>
-<wire x1="29.464" y1="25.4" x2="20.32" y2="25.4" width="0.1524" layer="91"/>
-<label x="20.32" y="25.4" size="1.778" layer="95"/>
+<pinref part="U1" gate="A" pin="(PCINT7/XTAL2/TOSC2)_PB7"/>
+<wire x1="29.464" y1="38.1" x2="12.7" y2="38.1" width="0.1524" layer="91"/>
+<label x="12.7" y="38.1" size="1.778" layer="95"/>
 </segment>
 </net>
@@
 </segment>
 <segment>
-<pinref part="U1" gate="A" pin="(PCINT2/SS/OC1B)_PB2"/>
-<wire x1="29.464" y1="22.86" x2="20.32" y2="22.86" width="0.1524" layer="91"/>
-<label x="20.32" y="22.86" size="1.778" layer="95"/>
-</segment>
-</net>
+<pinref part="U1" gate="A" pin="(PCINT19/OC2B/INT1)_PD3"/>
+<wire x1="29.464" y1="55.88" x2="12.7" y2="55.88" width="0.1524" layer="91"/>
+<label x="22.86" y="55.88" size="1.778" layer="95"/>
+</segment>
+</net>

Commit message: Adds up!
Button Number changed, Parts Added
Connections:
- net !BTN1: now also C6.1, R5.2, U1.(PCINT7/XTAL2/TOSC2)_PB7; no longer C4.1, R3.2, U1.(PCINT20/XCK/T0)_PD4
- net !BTN2: now also C4.1, R3.2, U1.(PCINT20/XCK/T0)_PD4; no longer C6.1, R5.2, U1.(PCINT7/XTAL2/TOSC2)_PB7
- net N$1: now also K2.A0; no longer K1.A0
- net N$2: now also K1.A0; no longer K2.A0
Other:
- moved on the sheet: K1, K2
Changed lines of the file:
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@@
 <part name="SUPPLY21" library="supply2" library_urn="urn:adsk.eagle:library:372" deviceset="+5V" device=""/>
 <part name="SUPPLY27" library="supply2" library_urn="urn:adsk.eagle:library:372" deviceset="+5V" device=""/>
-<part name="K1" library="rgb-led" deviceset="SMD-SWITCH-TOP-260GF(4P-D5.2MM)" device="" value="SKQGADE010"/>
+<part name="K2" library="rgb-led" deviceset="SMD-SWITCH-TOP-260GF(4P-D5.2MM)" device="" value="SKQGADE010"/>
 <part name="SUPPLY28" library="supply2" library_urn="urn:adsk.eagle:library:372" deviceset="+5V" device=""/>
 <part name="SUPPLY29" library="supply2" library_urn="urn:adsk.eagle:library:372" deviceset="GND" device=""/>
@@
 <part name="C4" library="resistor" library_urn="urn:adsk.eagle:library:348" deviceset="C-US" device="C0603" value="1uF"/>
 <part name="SUPPLY30" library="supply2" library_urn="urn:adsk.eagle:library:372" deviceset="GND" device=""/>
-<part name="K2" library="rgb-led" deviceset="SMD-SWITCH-TOP-260GF(4P-D5.2MM)" device="" value="SKQGADE010"/>
+<part name="K1" library="rgb-led" deviceset="SMD-SWITCH-TOP-260GF(4P-D5.2MM)" device="" value="SKQGADE010"/>
 <part name="SUPPLY36" library="supply2" library_urn="urn:adsk.eagle:library:372" deviceset="+5V" device=""/>
 <part name="SUPPLY37" library="supply2" library_urn="urn:adsk.eagle:library:372" deviceset="GND" device=""/>
@@
 <instance part="SUPPLY21" gate="+5V" x="-2.54" y="50.8"/>
 <instance part="SUPPLY27" gate="+5V" x="317.5" y="149.86"/>
-<instance part="K1" gate="G$1" x="320.04" y="48.26"/>
+<instance part="K2" gate="G$1" x="320.04" y="48.26"/>
 <instance part="SUPPLY28" gate="+5V" x="332.74" y="68.58"/>
 <instance part="SUPPLY29" gate="GND" x="332.74" y="35.56"/>
@@
 <instance part="C4" gate="G$1" x="294.64" y="43.18"/>
 <instance part="SUPPLY30" gate="GND" x="294.64" y="30.48"/>
-<instance part="K2" gate="G$1" x="320.04" y="5.08"/>
+<instance part="K1" gate="G$1" x="320.04" y="5.08"/>
 <instance part="SUPPLY36" gate="+5V" x="332.74" y="25.4"/>
 <instance part="SUPPLY37" gate="GND" x="332.74" y="-7.62"/>
@@
 <pinref part="SUPPLY29" gate="GND" pin="GND"/>
 <wire x1="332.74" y1="53.34" x2="332.74" y2="50.8" width="0.1524" layer="91"/>
-<pinref part="K1" gate="G$1" pin="B1"/>
+<pinref part="K2" gate="G$1" pin="B1"/>
 <wire x1="332.74" y1="50.8" x2="332.74" y2="45.72" width="0.1524" layer="91"/>
 <wire x1="332.74" y1="45.72" x2="332.74" y2="38.1" width="0.1524" layer="91"/>
 <wire x1="328.93" y1="45.72" x2="332.74" y2="45.72" width="0.1524" layer="91"/>
 <junction x="332.74" y="45.72"/>
-<pinref part="K1" gate="G$1" pin="A1"/>
+<pinref part="K2" gate="G$1" pin="A1"/>
 <wire x1="328.93" y1="50.8" x2="332.74" y2="50.8" width="0.1524" layer="91"/>
 <junction x="332.74" y="50.8"/>
@@
 <pinref part="SUPPLY37" gate="GND" pin="GND"/>
 <wire x1="332.74" y1="10.16" x2="332.74" y2="7.62" width="0.1524" layer="91"/>
-<pinref part="K2" gate="G$1" pin="B1"/>
+<pinref part="K1" gate="G$1" pin="B1"/>
 <wire x1="332.74" y1="7.62" x2="332.74" y2="2.54" width="0.1524" layer="91"/>
 <wire x1="332.74" y1="2.54" x2="332.74" y2="-5.08" width="0.1524" layer="91"/>
 <wire x1="328.93" y1="2.54" x2="332.74" y2="2.54" width="0.1524" layer="91"/>
 <junction x="332.74" y="2.54"/>
-<pinref part="K2" gate="G$1" pin="A1"/>
+<pinref part="K1" gate="G$1" pin="A1"/>
 <wire x1="328.93" y1="7.62" x2="332.74" y2="7.62" width="0.1524" layer="91"/>
 <junction x="332.74" y="7.62"/>
@@
 <segment>
 <pinref part="R3" gate="G$1" pin="1"/>
+<pinref part="K2" gate="G$1" pin="A0"/>
+<wire x1="307.34" y1="50.8" x2="311.15" y2="50.8" width="0.1524" layer="91"/>
+</segment>
+</net>
+<net name="N$2" class="0">
+<segment>
+<pinref part="R5" gate="G$1" pin="1"/>
 <pinref part="K1" gate="G$1" pin="A0"/>
-<wire x1="307.34" y1="50.8" x2="311.15" y2="50.8" width="0.1524" layer="91"/>
-</segment>
-</net>
-<net name="N$2" class="0">
-<segment>
-<pinref part="R5" gate="G$1" pin="1"/>
-<pinref part="K2" gate="G$1" pin="A0"/>
 <wire x1="307.34" y1="7.62" x2="311.15" y2="7.62" width="0.1524" layer="91"/>
 </segment>
@@
 </net>
 <net name="!BTN1" class="0">
+<segment>
+<pinref part="R5" gate="G$1" pin="2"/>
+<wire x1="297.18" y1="7.62" x2="294.64" y2="7.62" width="0.1524" layer="91"/>
+<wire x1="294.64" y1="7.62" x2="279.4" y2="7.62" width="0.1524" layer="91"/>
+<pinref part="C6" gate="G$1" pin="1"/>
+<wire x1="294.64" y1="2.54" x2="294.64" y2="7.62" width="0.1524" layer="91"/>
+<junction x="294.64" y="7.62"/>
+<label x="281.94" y="7.62" size="1.778" layer="95"/>
+</segment>
+<segment>
+<pinref part="U1" gate="A" pin="(PCINT7/XTAL2/TOSC2)_PB7"/>
+<wire x1="29.464" y1="38.1" x2="12.7" y2="38.1" width="0.1524" layer="91"/>
+<label x="12.7" y="38.1" size="1.778" layer="95"/>
+</segment>
+</net>
+<net name="!BTN3" class="0">
+<segment>
+<pinref part="R7" gate="G$1" pin="2"/>
+<wire x1="297.18" y1="-38.1" x2="294.64" y2="-38.1" width="0.1524" layer="91"/>
+<wire x1="294.64" y1="-38.1" x2="279.4" y2="-38.1" width="0.1524" layer="91"/>
+<pinref part="C8" gate="G$1" pin="1"/>
+<wire x1="294.64" y1="-43.18" x2="294.64" y2="-38.1" width="0.1524" layer="91"/>
+<junction x="294.64" y="-38.1"/>
+<label x="281.94" y="-38.1" size="1.778" layer="95"/>
+</segment>
+<segment>
+<pinref part="U1" gate="A" pin="(PCINT19/OC2B/INT1)_PD3"/>
+<wire x1="29.464" y1="55.88" x2="12.7" y2="55.88" width="0.1524" layer="91"/>
+<label x="22.86" y="55.88" size="1.778" layer="95"/>
+</segment>
+</net>
+<net name="!BTN2" class="0">
 <segment>
 <pinref part="R3" gate="G$1" pin="2"/>
@@
 </segment>
 </net>
-<net name="!BTN2" class="0">
-<segment>
-<pinref part="R5" gate="G$1" pin="2"/>
-<wire x1="297.18" y1="7.62" x2="294.64" y2="7.62" width="0.1524" layer="91"/>
-<wire x1="294.64" y1="7.62" x2="279.4" y2="7.62" width="0.1524" layer="91"/>
-<pinref part="C6" gate="G$1" pin="1"/>
-<wire x1="294.64" y1="2.54" x2="294.64" y2="7.62" width="0.1524" layer="91"/>
-<junction x="294.64" y="7.62"/>
-<label x="281.94" y="7.62" size="1.778" layer="95"/>
-</segment>
-<segment>
-<pinref part="U1" gate="A" pin="(PCINT7/XTAL2/TOSC2)_PB7"/>
-<wire x1="29.464" y1="38.1" x2="12.7" y2="38.1" width="0.1524" layer="91"/>
-<label x="12.7" y="38.1" size="1.778" layer="95"/>
-</segment>
-</net>
-<net name="!BTN3" class="0">
-<segment>
-<pinref part="R7" gate="G$1" pin="2"/>
-<wire x1="297.18" y1="-38.1" x2="294.64" y2="-38.1" width="0.1524" layer="91"/>
-<wire x1="294.64" y1="-38.1" x2="279.4" y2="-38.1" width="0.1524" layer="91"/>
-<pinref part="C8" gate="G$1" pin="1"/>
-<wire x1="294.64" y1="-43.18" x2="294.64" y2="-38.1" width="0.1524" layer="91"/>
-<junction x="294.64" y="-38.1"/>
-<label x="281.94" y="-38.1" size="1.778" layer="95"/>
-</segment>
-<segment>
-<pinref part="U1" gate="A" pin="(PCINT19/OC2B/INT1)_PD3"/>
-<wire x1="29.464" y1="55.88" x2="12.7" y2="55.88" width="0.1524" layer="91"/>
-<label x="22.86" y="55.88" size="1.778" layer="95"/>
-</segment>
-</net>
