File: 2017-2018/lec-buzzer_alt.sch (EAGLE design)
At the start: 26 parts, among them K1 SKQGADE010, K2 SKQGADE010, K3 SKQGADE010, U1 ATMEGA328P-MUR

Commit message: Minor Updates
Board rearranged to fit in MINI USB port. MINI USB port used as plenty
of supply exists in the shop
Parts:
- removed U$1: MICRO-USB, rgb-led:MICRO-USB
- added X1: MINI-USB-32005-201, con-cypressindustries:MINI-USB-32005-201
Connections:
- net +5V: now also X1.1; no longer U$1.1
- net GND: now also X1.5; no longer U$1.5
Other:
- note added: "MINI-USB As Power"
- note removed: "MicroUSB As Power"
- moved on the sheet: C1, SV1
Changed lines of the file:
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@@
 <part name="U1" library="lcd-buzzer" deviceset="ATMEGA328P-MUR" device=""/>
 <part name="#1" library="lcd-buzzer" deviceset="74HC595PW" device=""/>
-<part name="U$1" library="rgb-led" deviceset="MICRO-USB" device=""/>
 <part name="SUPPLY1" library="supply2" library_urn="urn:adsk.eagle:library:372" deviceset="+5V" device=""/>
 <part name="SUPPLY2" library="supply2" library_urn="urn:adsk.eagle:library:372" deviceset="GND" device=""/>
@@
 <part name="C8" library="resistor" library_urn="urn:adsk.eagle:library:348" deviceset="C-US" device="C0603" value="1uF"/>
 <part name="SUPPLY41" library="supply2" library_urn="urn:adsk.eagle:library:372" deviceset="GND" device=""/>
+<part name="X1" library="con-cypressindustries" library_urn="urn:adsk.eagle:library:138" deviceset="MINI-USB-" device="32005-201" package3d_urn="urn:adsk.eagle:package:6443/1"/>
 </parts>
 <sheets>
@@
 <text x="99.06" y="48.26" size="1.778" layer="91">Datasheet shows here is !RESET</text>
 <text x="284.48" y="125.73" size="1.778" layer="91">Haptic Driver</text>
-<text x="214.63" y="111.76" size="1.778" layer="91">MicroUSB As Power</text>
+<text x="278.13" y="116.84" size="1.778" layer="91">MINI-USB As Power</text>
 <text x="195.58" y="157.48" size="1.778" layer="91">Buzzer</text>
-<text x="251.46" y="109.22" size="1.778" layer="91">SPI Programming Port</text>
+<text x="226.06" y="111.76" size="1.778" layer="91">SPI Programming Port</text>
 <text x="218.44" y="78.74" size="1.778" layer="91">LCD</text>
 <text x="55.88" y="162.56" size="1.778" layer="91">4 Shifters</text>
@@
 <instance part="U1" gate="A" x="26.924" y="55.88"/>
 <instance part="#1" gate="A" x="16.92" y="104.06"/>
-<instance part="U$1" gate="G$1" x="228.6" y="99.06"/>
-<instance part="SUPPLY1" gate="+5V" x="241.3" y="111.76"/>
-<instance part="SUPPLY2" gate="GND" x="241.3" y="86.36"/>
+<instance part="SUPPLY1" gate="+5V" x="294.64" y="109.22"/>
+<instance part="SUPPLY2" gate="GND" x="294.64" y="83.82"/>
 <instance part="SUPPLY3" gate="+5V" x="76.8" y="106.6"/>
 <instance part="SUPPLY4" gate="GND" x="11.84" y="83.74"/>
@@
 <instance part="SUPPLY23" gate="+5V" x="190.5" y="22.86"/>
 <instance part="R1" gate="G$1" x="193.04" y="55.88" rot="R90"/>
-<instance part="C1" gate="G$1" x="241.3" y="101.6"/>
+<instance part="C1" gate="G$1" x="294.64" y="99.06"/>
 <instance part="SUPPLY26" gate="+5V" x="193.04" y="66.04"/>
 <instance part="LCD" gate="G$1" x="220.98" y="73.66"/>
@@
 <instance part="SUPPLY34" gate="+5V" x="172.72" y="113.03"/>
 <instance part="PS1240P02BT" gate="G$1" x="194.31" y="152.4"/>
-<instance part="SV1" gate="1" x="269.24" y="99.06" rot="R180"/>
-<instance part="SUPPLY31" gate="+5V" x="280.67" y="106.68"/>
-<instance part="SUPPLY32" gate="GND" x="280.67" y="91.44"/>
+<instance part="SV1" gate="1" x="243.84" y="101.6" rot="R180"/>
+<instance part="SUPPLY31" gate="+5V" x="255.27" y="109.22"/>
+<instance part="SUPPLY32" gate="GND" x="255.27" y="93.98"/>
 <instance part="HAPTIC" gate="A" x="246.38" y="142.24"/>
 <instance part="SUPPLY24" gate="GND" x="317.5" y="128.27"/>
@@
 <instance part="C8" gate="G$1" x="294.64" y="-45.72"/>
 <instance part="SUPPLY41" gate="GND" x="294.64" y="-58.42"/>
+<instance part="X1" gate="G$1" x="309.88" y="99.06"/>
 </instances>
 <busses>
@@
 <net name="+5V" class="0">
 <segment>
-<pinref part="U$1" gate="G$1" pin="1"/>
 <pinref part="SUPPLY1" gate="+5V" pin="+5V"/>
-<wire x1="233.68" y1="104.14" x2="241.3" y2="104.14" width="0.1524" layer="91"/>
-<wire x1="241.3" y1="104.14" x2="241.3" y2="109.22" width="0.1524" layer="91"/>
+<wire x1="294.64" y1="101.6" x2="294.64" y2="104.14" width="0.1524" layer="91"/>
 <pinref part="C1" gate="G$1" pin="1"/>
-<junction x="241.3" y="104.14"/>
+<pinref part="X1" gate="G$1" pin="1"/>
+<wire x1="294.64" y1="104.14" x2="294.64" y2="106.68" width="0.1524" layer="91"/>
+<wire x1="304.8" y1="104.14" x2="294.64" y2="104.14" width="0.1524" layer="91"/>
+<junction x="294.64" y="104.14"/>
 </segment>
 <segment>
@@
 <pinref part="SV1" gate="1" pin="2"/>
 <pinref part="SUPPLY31" gate="+5V" pin="+5V"/>
-<wire x1="276.86" y1="101.6" x2="280.67" y2="101.6" width="0.1524" layer="91"/>
-<wire x1="280.67" y1="101.6" x2="280.67" y2="104.14" width="0.1524" layer="91"/>
+<wire x1="251.46" y1="104.14" x2="255.27" y2="104.14" width="0.1524" layer="91"/>
+<wire x1="255.27" y1="104.14" x2="255.27" y2="106.68" width="0.1524" layer="91"/>
 </segment>
 <segment>
@@
 <segment>
 <pinref part="SUPPLY2" gate="GND" pin="GND"/>
-<wire x1="241.3" y1="96.52" x2="241.3" y2="93.98" width="0.1524" layer="91"/>
-<pinref part="U$1" gate="G$1" pin="5"/>
-<wire x1="241.3" y1="93.98" x2="241.3" y2="88.9" width="0.1524" layer="91"/>
-<wire x1="233.68" y1="93.98" x2="241.3" y2="93.98" width="0.1524" layer="91"/>
-<junction x="241.3" y="93.98"/>
+<wire x1="294.64" y1="93.98" x2="294.64" y2="91.44" width="0.1524" layer="91"/>
 <pinref part="C1" gate="G$1" pin="2"/>
+<pinref part="X1" gate="G$1" pin="5"/>
+<wire x1="294.64" y1="91.44" x2="294.64" y2="86.36" width="0.1524" layer="91"/>
+<wire x1="304.8" y1="93.98" x2="302.26" y2="93.98" width="0.1524" layer="91"/>
+<wire x1="302.26" y1="93.98" x2="302.26" y2="91.44" width="0.1524" layer="91"/>
+<wire x1="302.26" y1="91.44" x2="294.64" y2="91.44" width="0.1524" layer="91"/>
+<junction x="294.64" y="91.44"/>
 </segment>
 <segment>
@@
 <pinref part="SV1" gate="1" pin="6"/>
 <pinref part="SUPPLY32" gate="GND" pin="GND"/>
-<wire x1="276.86" y1="96.52" x2="280.67" y2="96.52" width="0.1524" layer="91"/>
-<wire x1="280.67" y1="96.52" x2="280.67" y2="93.98" width="0.1524" layer="91"/>
+<wire x1="251.46" y1="99.06" x2="255.27" y2="99.06" width="0.1524" layer="91"/>
+<wire x1="255.27" y1="99.06" x2="255.27" y2="96.52" width="0.1524" layer="91"/>
 </segment>
 <segment>
@@
 <segment>
 <pinref part="SV1" gate="1" pin="1"/>
-<wire x1="261.62" y1="101.6" x2="252.73" y2="101.6" width="0.1524" layer="91"/>
-<label x="254" y="101.6" size="1.778" layer="95"/>
+<wire x1="236.22" y1="104.14" x2="227.33" y2="104.14" width="0.1524" layer="91"/>
+<label x="228.6" y="104.14" size="1.778" layer="95"/>
 </segment>
 </net>
@@
 <segment>
 <pinref part="SV1" gate="1" pin="4"/>
-<wire x1="276.86" y1="99.06" x2="285.75" y2="99.06" width="0.1524" layer="91"/>
-<label x="278.13" y="99.06" size="1.778" layer="95"/>
+<wire x1="251.46" y1="101.6" x2="260.35" y2="101.6" width="0.1524" layer="91"/>
+<label x="252.73" y="101.6" size="1.778" layer="95"/>
 </segment>
 </net>
@@
 <segment>
 <pinref part="SV1" gate="1" pin="3"/>
-<wire x1="261.62" y1="99.06" x2="252.73" y2="99.06" width="0.1524" layer="91"/>
-<label x="254" y="99.06" size="1.778" layer="95"/>
+<wire x1="236.22" y1="101.6" x2="227.33" y2="101.6" width="0.1524" layer="91"/>
+<label x="228.6" y="101.6" size="1.778" layer="95"/>
 </segment>
 </net>
@@
 <segment>
 <pinref part="SV1" gate="1" pin="5"/>
-<wire x1="252.73" y1="96.52" x2="261.62" y2="96.52" width="0.1524" layer="91"/>
-<label x="254" y="96.52" size="1.778" layer="95"/>
-</segment>
-<segment>
+<wire x1="227.33" y1="99.06" x2="236.22" y2="99.06" width="0.1524" layer="91"/>
+<label x="228.6" y="99.06" size="1.778" layer="95"/>
+</segment>
+<segment>

Commit message: Board Updated according to Design Review
Parts:
- removed R3, R5, R7: 7.8k, resistor:R-US_R0603
- added C3, C5: 0.1uF, rcl:C-USC0603
- C1: value 47uF -> 10uF
- U1: value ATMEGA328P-MUR -> ATMEGA328P-AUR; device lcd-buzzer:ATMEGA328P-MUR -> lcd-buzzer:ATMEGA328P-AUR
Connections:
- removed net N$1: K2.A0, R3.1
- removed net N$2: K1.A0, R5.1
- removed net N$4: K3.A0, R7.1
- new net N$5: K2.A1, R2.1
- new net N$6: K1.A1, R4.1
- new net N$7: K3.A1, R6.1
- net !BTN1: now also K1.A0; no longer R5.2
- net !BTN2: now also K2.A0; no longer R3.2
- net !BTN3: now also K3.A0; no longer R7.2
- net +5V: now also C3.1, C5.1
- net GND: now also C3.2, C5.2; no longer K1.A1, K2.A1, K3.A1, R2.1, R4.1, R6.1
- net SFT2: now also U1.PC0_(ADC0/PCINT8); no longer U1.PC1_(ADC1/PCINT9)
- net SHIFT_CLK2: now also U1.PC1_(ADC1/PCINT9); no longer U1.PC2_(ADC2/PCINT10)
- net STORAGE_CLK2: now also U1.PC2_(ADC2/PCINT10); no longer U1.PC3_(ADC3/PCINT11)
Other:
- note added: "2x3 pin with walls"
- note added: "Get 50% more for chips, 4 times for Cs and Rs"
- note added: "Get connector that compatible with both AVR pocket and the 2x3, Ribbon cable"
- note added: "Verify Haptic Driver Info"
- note added: "Verify with datasheet"
- note removed: "Datasheet shows here is !RESET"
- moved on the sheet: C1, C4, C6, C8, K1, K2, K3, R2, R4, R6, X1

Commit message: Board Revision
Reference Designator updated, wonky silkscreen fixed, Library updated
and 2x3 header replaced with shrouded version
Parts:
- removed #3: 74HC595PW, lcd-buzzer:74HC595PW
- removed C8: 1uF, resistor:C-USC0603
- removed R6: 10k, resistor:R-US_R0603
- removed SV1: (no value), con-lstb:MA03-2
- added C7: 10uF, rcl:C-USC0603
- added R3: 10k, resistor:R-US_R0603
- added U3: ATMEGA328P-AUR, lcd-buzzer:ATMEGA328P-AUR
- added X3: 2X3SHROUDED, lcd-buzzer:2X3SHROUDED
- C1: value 10uF -> 0.1uF
- C2: value 1.0uF -> 0.1uF
- C3: value 0.1uF -> 1.0uF
- C5: value 0.1uF -> 1uF; device rcl:C-USC0603 -> resistor:C-USC0603
- U1: value ATMEGA328P-AUR -> 74HC595PW; device lcd-buzzer:ATMEGA328P-AUR -> lcd-buzzer:74HC595PW
- renumbered #1 to U2, #2 to U5, #4 to U4, HAPTIC to U6, K1 to S1, K2 to S2, K3 to S3, LCD to DS1, PS1240P02BT to LS1, TC33X-2-103E to VR1
Connections:
- net !BTN1: now also C5.1, U3.(PCINT7/XTAL2/TOSC2)_PB7; no longer C6.1, U1.(PCINT7/XTAL2/TOSC2)_PB7
- net !BTN2: now also U3.(PCINT20/XCK/T0)_PD4; no longer U1.(PCINT20/XCK/T0)_PD4
- net !BTN3: now also C6.1, U3.(PCINT19/OC2B/INT1)_PD3; no longer C8.1, U1.(PCINT19/OC2B/INT1)_PD3
- net !RESET: now also U3.PC6_(RESET/PCINT14), X3.5; no longer SV1.5, U1.PC6_(RESET/PCINT14)
- net +5V: now also C2.1, C7.1, R3.2, U1.!_2, U3.AVCC, U3.VCC, U3.VCC_2, X3.2; no longer #3.!_2, #3.VCC, C3.1, C5.1, R6.2, SV1.2, U1.AVCC, U1.VCC_2
- net 3A: now also U1.Q1; no longer #3.Q1
- net 3B: now also U1.Q2; no longer #3.Q2
- net 3C: now also U1.Q3; no longer #3.Q3
- net 3D: now also U1.Q4; no longer #3.Q4
- net 3E: now also U1.Q5; no longer #3.Q5
- net 3F: now also U1.Q6; no longer #3.Q6
- net 3G: now also U1.Q7_2; no longer #3.Q7_2
- net GND: now also C2.2, C3.1, C7.2, U1.!, U3.GND, U3.GND_2, U3.GND_3, X3.6; no longer #3.!, #3.GND, C2.1, C3.2, C8.2, SV1.6, U1.GND_2, U1.GND_3
- net MISO: now also U3.(PCINT4/MISO)_PB4, X3.1; no longer SV1.1, U1.(PCINT4/MISO)_PB4
- net MOSI: now also U3.(PCINT3/OC2A/MOSI)_PB3, X3.4; no longer SV1.4, U1.(PCINT3/OC2A/MOSI)_PB3
- net N$3: now also C3.2; no longer C2.2
- net N$6: now also R3.1; no longer R4.1
- net N$7: now also R4.1; no longer R6.1
- net SCK: now also U3.PB5_(SCK/PCINT5), X3.3; no longer SV1.3, U1.PB5_(SCK/PCINT5)
- net SCL: now also U3.PC5_(ADC5/SCL/PCINT13); no longer U1.PC5_(ADC5/SCL/PCINT13)
- net SDA: now also U3.PC4_(ADC4/SDA/PCINT12); no longer U1.PC4_(ADC4/SDA/PCINT12)
- net SFT1: now also U3.PD0_(RXD/PCINT16); no longer U1.PD0_(RXD/PCINT16)
- net SFT2: now also U3.PC0_(ADC0/PCINT8); no longer U1.PC0_(ADC0/PCINT8)
- net SFT3: now also U1.DS, U3.(PCINT23/AIN1)_PD7; no longer #3.DS, U1.(PCINT23/AIN1)_PD7
- net SFT4: now also U3.(PCINT0/CLKO/ICP1)_PB0; no longer U1.(PCINT0/CLKO/ICP1)_PB0
- net SHIFT_CLK1: now also U3.PD1_(TXD/PCINT17); no longer U1.PD1_(TXD/PCINT17)
- net SHIFT_CLK2: now also U3.PC1_(ADC1/PCINT9); no longer U1.PC1_(ADC1/PCINT9)
- net SHIFT_CLK3: now also U1.ST_CP, U3.(PCINT22/OC0A/AIN0)_PD6; no longer #3.ST_CP, U1.(PCINT22/OC0A/AIN0)_PD6
- net SHIFT_CLK4: now also U3.(PCINT1/OC1A)_PB1; no longer U1.(PCINT1/OC1A)_PB1
- net STORAGE_CLK1: now also U3.PD2_(INT0/PCINT18); no longer U1.PD2_(INT0/PCINT18)
- net STORAGE_CLK2: now also U3.PC2_(ADC2/PCINT10); no longer U1.PC2_(ADC2/PCINT10)
- net STORAGE_CLK3: now also U1.SH_CP, U3.(PCINT21/OC0B/T1)_PD5; no longer #3.SH_CP, U1.(PCINT21/OC0B/T1)_PD5
- net STORAGE_CLK4: now also U3.(PCINT2/SS/OC1B)_PB2; no longer U1.(PCINT2/SS/OC1B)_PB2
Other:
- note removed: "Get connector that compatible with both AVR pocket and the 2x3, Ribbon cable"
- moved on the sheet: C1, C2, C3, C5, C6, R4

Commit message: Keep updating
Changed to Class5, schematics alignment corrected.
Other:
- note added: "2x3 shrouded header pin"
- note removed: "2x3 pin with walls"
- moved on the sheet: C1, C2, C4, C5, C6, C7, R1, R2, R3, R4, S1, S2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

Commit message: training board ver 1.5
Parts:
- added D1: Yellow, SparkFun-LED:LED-YELLOW0603
- added R5: 150, resistor:R-US_R0603
- U3: value ATMEGA328P-AUR -> ATMEGA328P-SUR; device lcd-buzzer:ATMEGA328P-AUR -> lcd-buzzer:ATMEGA328P-SUR
Connections:
- new net LED: D1.A, U3.(PCINT6/XTAL1/TOSC1)_PB6
- new net N$1: D1.C, R5.2
- net GND: now also R5.1
Other:
- note removed: "Get 50% more for chips, 4 times for Cs and Rs"
- note removed: "Verify with datasheet"
