File: 2017-2018/lec-buzzer_alt.sch (EAGLE design)
At the start: 27 parts, among them U1 74HC595PW, U2 74HC595PW, U3 ATMEGA328P-SUR, U4 74HC595PW, U5 74HC595PW, U6 DRV2605LDGSR, X1 MINI-USB-32005-201, X3 2X3SHROUDED

Commit message: 2nd Version
Indicator LED added, ATMega328p package updated, schematics updated.
Connections:
- new net LCD_RESET: U1.!_2, U2.!_2, U3.PC3_(ADC3/PCINT11), U4.!_2, U5.!_2
- net +5V: no longer U1.!_2, U2.!_2, U4.!_2, U5.!_2
Other:
- note added: "Buttons"
- note added: "Indicator LED"
- note added: "Liquid Crystal Display"
- note added: "Microcontroller Unit"
- note added: "Mini-USB"
- note added: "Piezo Buzzer"
- note added: "Programming Port"
- note added: "Shift Registers"
- note removed: "4 Shifters"
- note removed: "Buzzer"
- note removed: "MINI-USB As Power"
- note removed: "SPI Programming Port"
- moved on the sheet: C1, C2, C3, C4, C5, C6, C7, D1, LS1, R1, R2, R3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

Commit message: LCD Column pin grounded
Connections:
- net GND: now also DS1.COL/P28, DS1.DP1/P8, DS1.DP2/P12, DS1.DP3/P16
Changed lines of the file:
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@@
 <part name="SUPPLY42" library="supply2" library_urn="urn:adsk.eagle:library:372" deviceset="GND" device=""/>
 <part name="FRAME2" library="RoboJackets-Frames" deviceset="FRAME_B_L" device=""/>
+<part name="SUPPLY6" library="supply2" library_urn="urn:adsk.eagle:library:372" deviceset="GND" device=""/>
+<part name="SUPPLY8" library="supply2" library_urn="urn:adsk.eagle:library:372" deviceset="GND" device=""/>
 </parts>
 <sheets>
@@
 <instance part="FRAME2" gate="G$1" x="0" y="0"/>
 <instance part="FRAME2" gate="G$2" x="325.12" y="0"/>
+<instance part="SUPPLY6" gate="GND" x="220.98" y="231.14"/>
+<instance part="SUPPLY8" gate="GND" x="294.64" y="243.84"/>
 </instances>
 <busses>
@@
 <wire x1="172.72" y1="118.11" x2="172.72" y2="121.92" width="0.1524" layer="91"/>
 </segment>
+<segment>
+<pinref part="DS1" gate="G$1" pin="COL/P28"/>
+<wire x1="241.3" y1="236.22" x2="226.06" y2="236.22" width="0.1524" layer="91"/>
+<pinref part="DS1" gate="G$1" pin="DP3/P16"/>
+<wire x1="241.3" y1="233.68" x2="226.06" y2="233.68" width="0.1524" layer="91"/>
+<wire x1="226.06" y1="236.22" x2="226.06" y2="233.68" width="0.1524" layer="91"/>
+<wire x1="226.06" y1="233.68" x2="220.98" y2="233.68" width="0.1524" layer="91"/>
+<junction x="226.06" y="233.68"/>
+<pinref part="SUPPLY6" gate="GND" pin="GND"/>
+</segment>
+<segment>
+<pinref part="DS1" gate="G$1" pin="DP2/P12"/>
+<wire x1="279.4" y1="246.38" x2="289.56" y2="246.38" width="0.1524" layer="91"/>
+<pinref part="DS1" gate="G$1" pin="DP1/P8"/>
+<wire x1="289.56" y1="246.38" x2="294.64" y2="246.38" width="0.1524" layer="91"/>
+<wire x1="279.4" y1="243.84" x2="289.56" y2="243.84" width="0.1524" layer="91"/>
+<wire x1="289.56" y1="243.84" x2="289.56" y2="246.38" width="0.1524" layer="91"/>
+<junction x="289.56" y="246.38"/>
+<pinref part="SUPPLY8" gate="GND" pin="GND"/>
+</segment>
 </net>

Commit message: Training Board Updated
A list of changes:
1. LCD COM pin: Now connected to Arduino Pin 13
2. ^that also means the trimmer resistor is removed
3. LED added, connected to Arduino Pin 12, can be the first thing for trainees to play with
4. LCD_Reset connected to A3
5. One of the three buttons is now a RESETN Button
6. Libraries updated, all ICs now includes the tiny circle denoting its direction
7. Schematics beautified and a bigger RoboBuzz
Parts:
- removed R5: 150, resistor:R-US_R0603
- removed VR1: TC33X, lcd-buzzer:TC33X
- removed X3: 2X3SHROUDED, lcd-buzzer:2X3SHROUDED
- added X2: MINI-USB-32005-201, con-cypressindustries:MINI-USB-32005-201
- C1: value 0.1uF -> 1.0uF
- C3: value 1.0uF -> 0.1uF
- R1: value 10k -> 150; device rcl:R-US_R0603 -> resistor:R-US_R0603
- R2: device resistor:R-US_R0603 -> rcl:R-US_R0603
- U3: value ATMEGA328P-SUR -> DRV2605LDGSR; device lcd-buzzer:ATMEGA328P-SUR -> lcd-buzzer:DRV2605LDGSR
- U4: value 74HC595PW -> ATMEGA328P-SUR; device lcd-buzzer:74HC595PW -> lcd-buzzer:ATMEGA328P-SUR
- U6: value DRV2605LDGSR -> 74HC595PW; device lcd-buzzer:DRV2605LDGSR -> lcd-buzzer:74HC595PW
- X1: value MINI-USB-32005-201 -> 2X3SHROUDED; device con-cypressindustries:MINI-USB-32005-201 -> lcd-buzzer:2X3SHROUDED
Connections:
- removed net !BTN1: C5.1, S1.A0, U3.(PCINT7/XTAL2/TOSC2)_PB7
- removed net DIVIDED: DS1.COM/P1, DS1.COMP40, VR1.WIPER
- removed net LED: D1.A, U3.(PCINT6/XTAL1/TOSC1)_PB6
- removed net N$7 (its old number): R4.1, S3.A1
- new net N$4: U4.ADC6
- net !BTN2: now also C5.1, U4.(PCINT20/XCK/T0)_PD4; no longer C4.1, U3.(PCINT20/XCK/T0)_PD4
- net !BTN3: now also C4.1, S1.A0, U4.(PCINT19/OC2B/INT1)_PD3; no longer C6.1, S3.A0, U3.(PCINT19/OC2B/INT1)_PD3
- net !RESET: now also C6.1, R2.1, S3.A0, U4.PC6_(RESET/PCINT14), X1.5; no longer R1.1, U3.PC6_(RESET/PCINT14), X3.5
- net +5V: now also C3.1, U3.EN, U3.VDD, U4.AVCC, U4.VCC_2, U6.VCC, X1.2, X2.1; no longer C1.1, R1.2, U3.AVCC, U3.VCC, U3.VCC_2, U6.EN, U6.VDD, VR1.CCW, X1.1, X3.2
- net 4A: now also U6.Q1; no longer U4.Q1
- net 4B: now also U6.Q2; no longer U4.Q2
- net 4C: now also U6.Q3; no longer U4.Q3
- net 4D: now also U6.Q4; no longer U4.Q4
- net 4E: now also U6.Q5; no longer U4.Q5
- net 4F: now also U6.Q6; no longer U4.Q6
- net 4G: now also U6.Q7_2; no longer U4.Q7_2
- net GND: now also C1.1, C3.2, R1.1, U3.IN/TRIG, U4.GND_2, U4.GND_3, U6.!, X1.6, X2.5; no longer C1.2, C3.1, DS1.COL/P28, DS1.DP1/P8, DS1.DP2/P12, DS1.DP3/P16, R5.1, U3.GND_2, U3.GND_3, U4.!, U6.IN/TRIG, VR1.CW, X1.5, X3.6
- net LCD_RESET: now also U4.PC3_(ADC3/PCINT11), U6.!_2; no longer U3.PC3_(ADC3/PCINT11), U4.!_2
- net LRA/ERM+: now also U3.OUT+; no longer U6.OUT+
- net LRA/ERM-: now also U3.OUT-; no longer U6.OUT-
- net MISO: now also U4.(PCINT4/MISO)_PB4, X1.1; no longer U3.(PCINT4/MISO)_PB4, X3.1
- net MOSI: now also D1.A, U4.(PCINT3/OC2A/MOSI)_PB3, X1.4; no longer U3.(PCINT3/OC2A/MOSI)_PB3, X3.4
- net N$1: now also R1.2; no longer R5.2
- net N$3: now also C1.2, U3.REG; no longer C3.2, U6.REG
- net N$5: now also R4.1; no longer R2.1
- net SCK: now also DS1.COL/P28, DS1.COM/P1, DS1.COMP40, DS1.DP1/P8, DS1.DP2/P12, DS1.DP3/P16, U4.PB5_(SCK/PCINT5), X1.3; no longer U3.PB5_(SCK/PCINT5), X3.3
- net SCL: now also U3.SCL, U4.PC5_(ADC5/SCL/PCINT13); no longer U3.PC5_(ADC5/SCL/PCINT13), U6.SCL
- net SDA: now also U3.SDA, U4.PC4_(ADC4/SDA/PCINT12); no longer U3.PC4_(ADC4/SDA/PCINT12), U6.SDA
- net SFT1: now also U4.PD0_(RXD/PCINT16); no longer U3.PD0_(RXD/PCINT16)
- net SFT2: now also U4.PC0_(ADC0/PCINT8); no longer U3.PC0_(ADC0/PCINT8)
- net SFT3: now also U4.(PCINT23/AIN1)_PD7; no longer U3.(PCINT23/AIN1)_PD7
- net SFT4: now also U4.(PCINT0/CLKO/ICP1)_PB0, U6.DS; no longer U3.(PCINT0/CLKO/ICP1)_PB0, U4.DS
- net SHIFT_CLK1: now also U4.PD1_(TXD/PCINT17); no longer U3.PD1_(TXD/PCINT17)
- net SHIFT_CLK2: now also U4.PC1_(ADC1/PCINT9); no longer U3.PC1_(ADC1/PCINT9)
- net SHIFT_CLK3: now also U4.(PCINT22/OC0A/AIN0)_PD6; no longer U3.(PCINT22/OC0A/AIN0)_PD6
- net SHIFT_CLK4: now also U4.(PCINT1/OC1A)_PB1, U6.ST_CP; no longer U3.(PCINT1/OC1A)_PB1, U4.ST_CP
- net STORAGE_CLK1: now also U4.PD2_(INT0/PCINT18); no longer U3.PD2_(INT0/PCINT18)
- net STORAGE_CLK2: now also U4.PC2_(ADC2/PCINT10); no longer U3.PC2_(ADC2/PCINT10)
- net STORAGE_CLK3: now also U4.(PCINT21/OC0B/T1)_PD5; no longer U3.(PCINT21/OC0B/T1)_PD5
- net STORAGE_CLK4: now also U4.(PCINT2/SS/OC1B)_PB2, U6.SH_CP; no longer U3.(PCINT2/SS/OC1B)_PB2, U4.SH_CP
Other:
- note removed: "LCD"
- note removed: "Trimmer Potentiometer"
- note removed: "Verify Haptic Driver Info"
- note removed: "coupling capacitor?"
- note removed: "pin 1 to 7 on Shifters will control LCD segments"
- moved on the sheet: C1, C2, C3, C4, C5, C6, C7, D1, LS1, R1, R2, R3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

Commit message: training board v1.1
Parts:
- removed DS1: LCD-S401C39TR, lcd-buzzer:LCD-S401C39TR
- added D2: Green, SparkFun-LED:LED-YELLOW0603
- added LCD1: LCD-S401C39TR, lcd-buzzer:LCD-S401C39TR
- added R5: 150, resistor:R-US_R0603
- D1: value Yellow -> Blue
- U4: value ATMEGA328P-SUR -> ATMEGA328P-AUR; device lcd-buzzer:ATMEGA328P-SUR -> lcd-buzzer:ATMEGA328P-AUR
Connections:
- removed net LCD_RESET: U1.!_2, U2.!_2, U4.PC3_(ADC3/PCINT11), U5.!_2, U6.!_2
- removed net N$4: U4.ADC6
- removed net N$5: R4.1, S2.A1
- removed net N$7: R3.1, S1.A1
- removed net SFT1: U2.DS, U4.PD0_(RXD/PCINT16)
- removed net SFT2: U4.PC0_(ADC0/PCINT8), U5.DS
- removed net SFT3: U1.DS, U4.(PCINT23/AIN1)_PD7
- removed net SFT4: U4.(PCINT0/CLKO/ICP1)_PB0, U6.DS
- removed net SHIFT_CLK1: U2.ST_CP, U4.PD1_(TXD/PCINT17)
- removed net SHIFT_CLK2: U4.PC1_(ADC1/PCINT9), U5.ST_CP
- removed net SHIFT_CLK3: U1.ST_CP, U4.(PCINT22/OC0A/AIN0)_PD6
- removed net SHIFT_CLK4: U4.(PCINT1/OC1A)_PB1, U6.ST_CP
- removed net STORAGE_CLK1: U2.SH_CP, U4.PD2_(INT0/PCINT18)
- removed net STORAGE_CLK2: U4.PC2_(ADC2/PCINT10), U5.SH_CP
- removed net STORAGE_CLK3: U1.SH_CP, U4.(PCINT21/OC0B/T1)_PD5
- removed net STORAGE_CLK4: U4.(PCINT2/SS/OC1B)_PB2, U6.SH_CP
- new net COL: LCD1.COL
- new net COM: LCD1.COM1, LCD1.COM2, U4.PC2_(ADC2/PCINT10)
- new net DP1: LCD1.DP1
- new net DP2: LCD1.DP2
- new net DP3: LCD1.DP3
- new net LED1: D1.A, U4.(PCINT2/SS/OC1B)_PB2
- new net N$2: D2.C, R5.2
- new net SFT-!OE: U1.!OE, U2.!OE, U4.(PCINT21/OC0B/T1)_PD5, U5.!OE, U6.!OE
- new net SFT-!RESET: U1.!MR, U2.!MR, U4.(PCINT0/CLKO/ICP1)_PB0, U5.!MR, U6.!MR
- new net SFT-CLK: U1.SHCP, U2.SHCP, U4.(PCINT23/AIN1)_PD7, U5.SHCP, U6.SHCP
- new net SFT-LATCH: U1.STCP, U2.STCP, U4.(PCINT22/OC0A/AIN0)_PD6, U5.STCP, U6.STCP
- new net SFT1-IN: U1.DS, U4.(PCINT1/OC1A)_PB1
- new net SFT2-IN: U1.Q7S, U2.DS
- new net SFT3-IN: U2.Q7S, U5.DS
- new net SFT4-IN: U5.Q7S, U6.DS
- net !BTN2: now also R4.1, S2.B0; no longer S2.A0, U4.(PCINT20/XCK/T0)_PD4
- net !BTN3: now also R3.1, S1.B0; no longer S1.A0, U4.(PCINT19/OC2B/INT1)_PD3
- net +5V: now also D2.A, S1.A0, S2.A0; no longer R3.2, R4.2
- net 1A: now also LCD1.1A, U1.Q0; no longer DS1.1A/P35, U2.Q1
- net 1B: now also LCD1.1B, U1.Q1; no longer DS1.1B/P34, U2.Q2
- net 1C: now also LCD1.1C, U1.Q2; no longer DS1.1C/P7, U2.Q3
- net 1D: now also LCD1.1D, U1.Q3; no longer DS1.1D/P6, U2.Q4
- net 1E: now also LCD1.1E, U1.Q4; no longer DS1.1E/P5, U2.Q5
- net 1F: now also LCD1.1F, U1.Q5; no longer DS1.1F/P36, U2.Q6
- net 1G: now also LCD1.1G, U1.Q6; no longer DS1.1G/P37, U2.Q7_2
- net 2A: now also LCD1.2A, U2.Q0; no longer DS1.2A/P30, U5.Q1
- net 2B: now also LCD1.2B, U2.Q1; no longer DS1.2B/P29, U5.Q2
- net 2C: now also LCD1.2C, U2.Q2; no longer DS1.2C/P11, U5.Q3
- net 2D: now also LCD1.2D, U2.Q3; no longer DS1.2D/P10, U5.Q4
- net 2E: now also LCD1.2E, U2.Q4; no longer DS1.2E/P9, U5.Q5
- net 2F: now also LCD1.2F, U2.Q5; no longer DS1.2F/P31, U5.Q6
- net 2G: now also LCD1.2G, U2.Q6; no longer DS1.2G/P32, U5.Q7_2
- net 3A: now also LCD1.3A, U5.Q0; no longer DS1.3A/P25, U1.Q1
- net 3B: now also LCD1.3B, U5.Q1; no longer DS1.3B/P24, U1.Q2
- net 3C: now also LCD1.3C, U5.Q2; no longer DS1.3C/P15, U1.Q3
- net 3D: now also LCD1.3D, U5.Q3; no longer DS1.3D/P14, U1.Q4
- net 3E: now also LCD1.3E, U5.Q4; no longer DS1.3E/P13, U1.Q5
- net 3F: now also LCD1.3F, U5.Q5; no longer DS1.3F/P26, U1.Q6
- net 3G: now also LCD1.3G, U5.Q6; no longer DS1.3G/P27, U1.Q7_2
- net 4A: now also LCD1.4A, U6.Q0; no longer DS1.4A/P21, U6.Q1
- net 4B: now also LCD1.4B, U6.Q1; no longer DS1.4B/P20, U6.Q2
- net 4C: now also LCD1.4C, U6.Q2; no longer DS1.4C/P19, U6.Q3
- net 4D: now also LCD1.4D, U6.Q3; no longer DS1.4D/P18, U6.Q4
- net 4E: now also LCD1.4E, U6.Q4; no longer DS1.4E/P17, U6.Q5
- net 4F: now also LCD1.4F, U6.Q5; no longer DS1.4F/P22, U6.Q6
- net 4G: now also LCD1.4G, U6.Q6; no longer DS1.FG/P23, U6.Q7_2
- net GND: now also C1.2, R3.2, R4.2, R5.1, S3.B0; no longer C1.1, S1.B1, S2.B1, S3.B1, U1.!, U2.!, U5.!, U6.!
- net LRA/ERM+: now also LS1.A; no longer LS1.VCC
- net LRA/ERM-: now also LS1.B; no longer LS1.P2
- net MOSI: no longer D1.A
- net N$3: now also C1.1; no longer C1.2
- net SCK: no longer DS1.COL/P28, DS1.COM/P1, DS1.COMP40, DS1.DP1/P8, DS1.DP2/P12, DS1.DP3/P16
Other:
- note added: "7 Segment LCD"
- note added: "Microcontroller"
- note added: "Power LED"
- note added: "Programming Connector"
- note added: "Reset Button"
- note removed: "2x3 shrouded header pin"
- note removed: "Liquid Crystal Display"
- note removed: "Microcontroller Unit"
- note removed: "Programming Port"
- moved on the sheet: C1, C2, C3, C4, C5, C6, C7, D1, R1, R2, R3, R4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

Commit message: add lcd dots
Connections:
- net COL: now also U1.Q7
- net DP1: now also U2.Q7
- net DP2: now also U5.Q7
- net DP3: now also U6.Q7
Changed lines of the file:
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@@
 <label x="226.06" y="226.06" size="1.27" layer="95" xref="yes"/>
+</segment>
+<segment>
+<pinref part="U1" gate="G$1" pin="Q7"/>
+<wire x1="33.02" y1="223.52" x2="30.48" y2="223.52" width="0.1524" layer="91"/>
+<label x="30.48" y="223.52" size="1.27" layer="95" rot="R180" xref="yes"/>
 </segment>
 </net>
@@
 <label x="226.06" y="228.6" size="1.27" layer="95" xref="yes"/>
 </segment>
+<segment>
+<pinref part="U2" gate="G$1" pin="Q7"/>
+<wire x1="91.44" y1="223.52" x2="88.9" y2="223.52" width="0.1524" layer="91"/>
+<label x="88.9" y="223.52" size="1.27" layer="95" rot="R180" xref="yes"/>
+</segment>
 </net>
 <net name="DP2" class="0">
@@
 <wire x1="218.44" y1="231.14" x2="226.06" y2="231.14" width="0.1524" layer="91"/>
 <label x="226.06" y="231.14" size="1.27" layer="95" xref="yes"/>
+</segment>
+<segment>
+<pinref part="U5" gate="G$1" pin="Q7"/>
+<wire x1="33.02" y1="180.34" x2="30.48" y2="180.34" width="0.1524" layer="91"/>
+<label x="30.48" y="180.34" size="1.27" layer="95" rot="R180" xref="yes"/>
 </segment>
 </net>
@@
 <label x="226.06" y="233.68" size="1.27" layer="95" xref="yes"/>
 </segment>
+<segment>
+<pinref part="U6" gate="G$1" pin="Q7"/>
+<wire x1="91.44" y1="180.34" x2="88.9" y2="180.34" width="0.1524" layer="91"/>
+<label x="88.9" y="180.34" size="1.27" layer="95" rot="R180" xref="yes"/>
+</segment>
 </net>

Commit message: Button Connected
Connections:
- net !BTN2: now also U4.PC0_(ADC0/PCINT8)
- net !BTN3: now also U4.PC1_(ADC1/PCINT9)
Changed lines of the file:
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@@
 <setting verticaltext="up"/>
 </settings>
-<grid distance="0.1" unitdist="inch" unit="inch" style="lines" multiple="1" display="no" altdistance="0.01" altunitdist="inch" altunit="inch"/>
+<grid distance="0.05" unitdist="inch" unit="inch" style="lines" multiple="1" display="no" altdistance="0.01" altunitdist="inch" altunit="inch"/>
 <layers>
 <layer number="1" name="Top" color="4" fill="1" visible="no" active="no"/>
@@
 <segment>
 <wire x1="220.98" y1="55.88" x2="224.79" y2="55.88" width="0.1524" layer="91"/>
-<label x="224.79" y="55.88" size="1.778" layer="95"/>
 <pinref part="X1" gate="G$1" pin="4"/>
+<label x="224.79" y="55.88" size="1.27" layer="95" xref="yes"/>
 </segment>
 </net>
@@
 <junction x="292.1" y="218.44"/>
 </segment>
+<segment>
+<pinref part="U4" gate="G$1" pin="PC1_(ADC1/PCINT9)"/>
+<wire x1="144.78" y1="45.72" x2="149.86" y2="45.72" width="0.1524" layer="91"/>
+<label x="149.86" y="45.72" size="1.27" layer="95" xref="yes"/>
+</segment>
 </net>
 <net name="!BTN2" class="0">
@@
 <junction x="365.76" y="218.44"/>
 </segment>
-</net>
+<segment>
+<pinref part="U4" gate="G$1" pin="PC0_(ADC0/PCINT8)"/>
+<wire x1="144.78" y1="43.18" x2="149.86" y2="43.18" width="0.1524" layer="91"/>
+<label x="149.86" y="43.18" size="1.27" layer="95" xref="yes"/>
+</segment>
+</net>
