File: 2018-2019/Training_Board.sch (EAGLE design)
At the start: 4 parts, among them IC1 ATMEGA328-20P

Commit message: <Relevant Commit Message>
Parts:
- added C2, C4: 10uF, rcl:C-USC0603
- added C3: 1uF, rcl:C-USC0603
- added JP1: (no value), pinhead:PINHD-1X12
- added JP2: (no value), pinhead:PINHD-1X16
- added PRGRM-HEADER: (no value), con-lstb:MA03-2
- added R2: 10k Ohm, resistor:R-US_R0603
- added U$2: AP2112SOT89-5, RoboJackets-PowerICs:AP2112SOT89-5
- added U$3: JST-PH2, Trainii:JST-PH2
Connections:
- removed net N$2: IC1.PC6(/RESET/PCI14), R1.2, U$1.2
- new net MISO: IC1.(PCI4/MISO)PB4, PRGRM-HEADER.6
- new net MOSI: IC1.(PCI3/MOSI/OC2A)PB3, PRGRM-HEADER.3
- new net N$1: R2.1, U$2.EN
- new net RST: IC1.PC6(/RESET/PCI14), PRGRM-HEADER.2, R1.2, U$1.2
- new net SCK: IC1.(PCI5/SCK)PB5, PRGRM-HEADER.4
- new net VBAT: C4.1, R2.2, U$2.VIN, U$3.2
- net GND: now also C2.2, C3.2, C4.2, PRGRM-HEADER.1, U$2.GND, U$3.1
- net VCC: now also C2.1, C3.1, PRGRM-HEADER.5, U$2.VOUT
Other:
- moved on the sheet: U$1

Commit message: Completed Schematic
Parts:
- removed U$2: AP2112SOT89-5, RoboJackets-PowerICs:AP2112SOT89-5
- added C5: 22 pF, resistor:C-USC0603
- added LD1117: R-78E5.0-0.5, RoboJackets-PowerICs:R-78E5.0-0.5
- added X1: CRYSTALS-NOGND-HC49/4H, IQD-Frequency-Products:CRYSTALS-NOGND-HC49/4H
- C3: value 1uF -> 22 pF; device rcl:C-USC0603 -> resistor:C-USC0603
- C4: value 10uF -> 100nF
Connections:
- new net ECHO_3V3: IC1.(PCI23/AIN1)PD7, JP2.12
- new net LEFT_A: IC1.(PCI0/ICP/CLKO)PB0, JP2.5
- new net LEFT_B: IC1.(PCI1/OC1A/OC1S)PB1, JP1.7
- new net LIFT_A: IC1.(PCI20/XCK/T0)PD4, JP1.4
- new net LIFT_B: IC1.(PCI21/T1/OC0B)PD5, JP1.3
- new net LINE_OUT_1: IC1.(PCI8/ADC0)PC0, JP2.6
- new net LINE_OUT_2: IC1.(PCI9/ADC1)PC1, JP2.7
- new net MOTOR_FAULT: IC1.(PCI2/SS/OC1B)PB2, JP2.16, R2.1
- new net N$2: IC1.(PCI10/ADC2)PC2
- new net N$26: JP2.10
- new net N$3: IC1.(PCI11/ADC3)PC3
- new net N$4: C5.1, IC1.PB7(XTAL2/TOSC2/PCI7), X1.1
- new net RIGHT_A: IC1.(PCI16/RXD)PD0, JP1.6
- new net RIGHT_B: IC1.(PCI17/TXD)PD1, JP1.5
- new net SCL: IC1.(PCI13/ADC5/SCL)PC5, JP1.2
- new net SDA: IC1.(PCI12/ADC4/SDA)PC4, JP1.1
- new net TICK_LEFT: IC1.(PCI18/INT0)PD2, JP2.8
- new net TICK_RIGHT: IC1.(PCI19/INT1/OC2B)PD3, JP2.9
- new net TRIG_3V3: IC1.(PCI22/AIN0OC0A)PD6, JP2.11
- net GND: now also C5.2, JP2.4, LD1117.GND; no longer U$2.GND
- net N$1: now also C3.1, IC1.PB6(XTAL1/TOSC1/PCI6), X1.2; no longer R2.1, U$2.EN
- net VBAT: now also LD1117.VIN; no longer R2.2, U$2.VIN
- net VCC: now also JP2.2, LD1117.VOUT, R2.2; no longer C3.1, IC1.VCC, U$2.VOUT
Other:
- moved on the sheet: C1, C3, C4, JP1, JP2, R2

Commit message: Fixed pins, added VCC, changed some names
Parts:
- removed R2: 10k Ohm, resistor:R-US_R0603
- removed U$3: JST-PH2, Trainii:JST-PH2
- added XO1: CRYSTALS-NOGND-HC49/4H, IQD-Frequency-Products:CRYSTALS-NOGND-HC49/4H
- X1: value CRYSTALS-NOGND-HC49/4H -> JST-PH2; device IQD-Frequency-Products:CRYSTALS-NOGND-HC49/4H -> Trainii:JST-PH2
- renumbered U$1 to S1
Connections:
- removed net N$2: IC1.(PCI10/ADC2)PC2
- removed net N$26: JP2.10
- removed net N$3: IC1.(PCI11/ADC3)PC3
- removed net VCC: C1.1, C2.1, IC1.AVCC, JP2.2, LD1117.VOUT, PRGRM-HEADER.5, R1.1, R2.2
- new net +3V3: C1.1, C2.1, IC1.AVCC, IC1.VCC, JP2.2, LD1117.VOUT, PRGRM-HEADER.5, R1.1
- net ECHO_3V3: now also JP2.13; no longer JP2.12
- net GND: now also X1.1; no longer U$3.1
- net LEFT_A: now also JP2.6; no longer JP2.5
- net LINE_OUT_1: now also JP2.7; no longer JP2.6
- net LINE_OUT_2: now also JP2.8; no longer JP2.7
- net MOTOR_FAULT: no longer R2.1
- net N$1: now also XO1.2; no longer X1.2
- net N$4: now also XO1.1; no longer X1.1
- net TICK_LEFT: now also JP2.9; no longer JP2.8
- net TICK_RIGHT: now also JP2.10; no longer JP2.9
- net TRIG_3V3: now also JP2.12; no longer JP2.11
- net VBAT: now also JP1.12, X1.2; no longer U$3.2
Other:
- moved on the sheet: C4
