File: 2018-2019/Training_Board.brd (EAGLE design)
At the start: 59 x 32 mm, 14 parts, among them IC1 ATMEGA328-20P, X1 JST-PH2

Commit message: Added LED, adjusted some routing
Parts:
- added D1: RED, led:CHIP-LED0603
- added D2: GREEN, led:CHIP-LED0603
- added R2, R3: 1k Ohm, rcl:M0805
- moved C2 0.20 mm to (49.9, 22.5), turned to 90 degrees
Connections:
- new net LED_1: IC1.3, R2.1
- new net LED_2: IC1.6, R3.1
- new net N$2: D2.A, R3.2
- new net N$3: D1.A, R2.2
- net GND: now also D1.C, D2.C
- net MOTOR_FAULT: now also IC1.2; no longer IC1.26
- net RIGHT_A: now also IC1.26; no longer IC1.2
- net RIGHT_B: now also IC1.25; no longer IC1.3
Routing:
- net +3V3: track 136.5 -> 98.1 mm, vias 0 -> 1
- net LED_2: track 0.00 -> 22.8 mm, vias 0 -> 1
- net RIGHT_A: track 27.9 -> 15.5 mm
- net RIGHT_B: track 27.4 -> 15.6 mm
- net LED_1: track 0.00 -> 11.2 mm
- net MOTOR_FAULT: track 42.8 -> 34.7 mm
- net RST: track 65.6 -> 62.1 mm
- net LEFT_A: track 34.6 -> 37.6 mm
- net SCK: track 30.2 -> 33.1 mm
- net GND: track 19.5 -> 22.4 mm, vias 2 -> 4
- net MOSI: track 61.9 -> 59.5 mm
- net N$3: track 0.00 -> 2.30 mm
- net N$2: track 0.00 -> 2.30 mm
- net MISO: track 60.4 -> 58.6 mm
- net SCL: track 30.2 -> 31.0 mm
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