File: 2018-2019/board/Training_Board.brd (EAGLE design)
At the start: 59 x 32 mm, 18 parts, among them IC1 ATMEGA328-20P, X1 JST-PH2

Commit message: Added filtering caps and re-spec of LDO
Parts:
- added C6: 100 nF, resistor:C0603
- added C7: 10 nF, resistor:C0603
- added R4: 10k Ohm, rcl:M0805
- LD1117: value R-78E5.0-0.5 -> AP2112SOT89-5; device RoboJackets-PowerICs:R-78E -> RoboJackets-PowerICs:SOT95P285X110-5
- moved C4 34.9 mm to (45.0, 25.4), turned to 180 degrees
- moved C2 4.88 mm to (45.0, 22.9), flipped to the top, turned to 180 degrees
- moved LD1117 2.56 mm to (48.9, 23.7), turned to 180 degrees
Connections:
- new net N$5: LD1117.3, R4.2
- new net N$6: C6.2, IC1.21
- net +3V3: now also LD1117.5; no longer LD1117.3
- net GND: now also C6.1, C7.1
- net VBAT: now also C7.2, LD1117.4, R4.1; no longer LD1117.1
Routing:
- net GND: track 22.4 -> 30.1 mm, vias 4 -> 6
- net VBAT: track 44.8 -> 51.4 mm, vias 0 -> 1
- net N$6: track 0.00 -> 3.27 mm
- net +3V3: track 98.1 -> 95.2 mm
- net N$5: track 0.00 -> 2.44 mm

Commit message: Added Aesthetics and extra smoothing capacitors
Parts:
- added C8: 1uF, rcl:C0603
- added U$1: (no value), RoboJackets-Aesthetics:ROBOBUZZ_0.4X
Connections:
- net GND: now also C8.2
- net VBAT: now also C8.1
Routing:
- net +3V3: track 95.2 -> 97.3 mm
- net VBAT: track 51.4 -> 52.0 mm
Other:
- board text added: "Electrical Training Board v1.0"
Changed lines of the file:
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@@
 <layer number="116" name="Patch_BOT" color="9" fill="4" visible="no" active="yes"/>
 <layer number="118" name="Rect_Pads" color="7" fill="1" visible="no" active="no"/>
-<layer number="121" name="_tsilk" color="7" fill="1" visible="no" active="yes"/>
+<layer number="121" name="_tsilk" color="7" fill="1" visible="yes" active="yes"/>
 <layer number="122" name="_bsilk" color="7" fill="1" visible="no" active="yes"/>
 <layer number="123" name="tTestmark" color="7" fill="1" visible="no" active="yes"/>
@@
 <wire x1="-1" y1="30" x2="-1" y2="-2" width="0" layer="20"/>
 <text x="46" y="0" size="1.016" layer="21" distance="40">RESET</text>
+<polygon width="0.3" layer="21">
+<vertex x="14" y="29"/>
+<vertex x="14" y="26"/>
+<vertex x="40" y="26"/>
+<vertex x="40" y="29"/>
+</polygon>
+<text x="9.5" y="5.5" size="1.4" layer="21">Electrical Training Board v1.0</text>
 </plain>
 <attributes>
@@
 <element name="C6" library="resistor" library_urn="urn:adsk.eagle:library:348" package="C0603" package3d_urn="urn:adsk.eagle:package:26138/1" value="100 nF" x="25" y="15" rot="MR180"/>
 <element name="C7" library="resistor" library_urn="urn:adsk.eagle:library:348" package="C0603" package3d_urn="urn:adsk.eagle:package:26138/1" value="10 nF" x="5.5" y="28" rot="MR180"/>
+<element name="C8" library="rcl" library_urn="urn:adsk.eagle:library:334" package="C0603" package3d_urn="urn:adsk.eagle:package:23616/2" value="1uF" x="45.5" y="25" rot="MR270">
+<attribute name="SPICEPREFIX" value="C" x="45.5" y="25" size="1.778" layer="28" rot="MR270" display="off"/>
+</element>
+<element name="U$1" library="RoboJackets-Aesthetics" package="ROBOBUZZ_0.4X" value="" x="54.5" y="21.5"/>
 </elements>
 <signals>
@@
 <wire x1="4.65" y1="28" x2="4.7" y2="27.95" width="0.3" layer="16"/>
 <wire x1="4.7" y1="27.95" x2="4.7" y2="26.19" width="0.3" layer="16"/>
-<wire x1="44.14" y1="22.86" x2="43.86" y2="22.86" width="0.3" layer="1"/>
-<wire x1="44.14" y1="22.86" x2="42.86" y2="22.86" width="0.3" layer="1"/>
-<wire x1="42.86" y1="22.86" x2="42" y2="22" width="0.3" layer="1"/>
+<wire x1="42" y1="22" x2="42.86" y2="22.86" width="0.3" layer="1"/>
 <via x="42" y="22" extent="1-16" drill="0.35"/>
+<contactref element="C8" pad="2"/>
+<wire x1="42.86" y1="22.86" x2="44.14" y2="22.86" width="0.3" layer="1"/>
 </signal>
 <signal name="VBAT">
@@
 <contactref element="C4" pad="1"/>
 <contactref element="JP1" pad="12"/>
-<wire x1="6.7" y1="26.19" x2="7.25" y2="25.64" width="0.3" layer="1"/>
-<wire x1="6.7" y1="26.19" x2="9.57" y2="23.32" width="0.3" layer="16"/>
 <wire x1="9.57" y1="23.32" x2="12.03" y2="23.32" width="0.3" layer="16"/>
 <contactref element="R4" pad="1"/>
@@
 <wire x1="6.35" y1="28" x2="6.35" y2="26.54" width="0.3" layer="16"/>
 <wire x1="6.35" y1="26.54" x2="6.7" y2="26.19" width="0.3" layer="16"/>
+<contactref element="C8" pad="1"/>
+<wire x1="6.7" y1="26.19" x2="9.57" y2="23.32" width="0.3" layer="16"/>
+<wire x1="45.5" y1="25.85" x2="46" y2="26.35" width="0.3" layer="16"/>
+<wire x1="46" y1="26.35" x2="46" y2="27" width="0.3" layer="16"/>
 </signal>
 <signal name="RST">
@@
 <contactref element="PRGRM-HEADER" pad="5"/>
 <wire x1="24.94" y1="12.51" x2="24.94" y2="9.97" width="0.3" layer="16"/>
-<wire x1="30.02" y1="15.3" x2="30.21" y2="15.11" width="0.3" layer="16"/>
 <wire x1="30.21" y1="15.11" x2="45" y2="15.11" width="0.3" layer="16"/>
-<wire x1="45.945" y1="16.055" x2="45" y2="15.11" width="0.3" layer="16"/>
+<wire x1="46" y1="16.11" x2="45" y2="15.11" width="0.3" layer="16"/>
 <wire x1="55.03" y1="5.32" x2="56.834" y2="7.124" width="0.3" layer="1"/>
 <wire x1="2.65" y1="8.33" x2="4.49" y2="6.49" width="0.3" layer="1"/>
@@
 <wire x1="25.8744" y1="1.79710625" x2="24.07729375" y2="0" width="0.3" layer="16"/>
 <wire x1="24.07729375" y1="0" x2="7.49" y2="0" width="0.3" layer="16"/>
-<wire x1="56.834" y1="7.124" x2="56.834" y2="14" width="0.3" layer="1"/>
+<wire x1="56.834" y1="7.124" x2="56.834" y2="15" width="0.3" layer="1"/>
 <contactref element="IC1" pad="20"/>
-<wire x1="56.834" y1="14" x2="56.834" y2="15" width="0.3" layer="1"/>
-<wire x1="46" y1="16.11" x2="45.945" y2="16.055" width="0.3" layer="16"/>
 <wire x1="56.834" y1="15" x2="51.834" y2="20" width="0.3" layer="1"/>
-<wire x1="50" y1="20" x2="51.834" y2="20" width="0.3" layer="1"/>
-<wire x1="45.84" y1="22.86" x2="45.98" y2="23" width="0.3" layer="1"/>
+<wire x1="49.1454" y1="20" x2="51.834" y2="20" width="0.3" layer="1"/>
 <wire x1="45.84" y1="22.86" x2="47.4527" y2="22.86" width="0.3" layer="1"/>
 <wire x1="47.4527" y1="22.86" x2="47.5727" y2="22.74" width="0.3" layer="1"/>
 <via x="46" y="20" extent="1-16" drill="0.35"/>
-<wire x1="45.945" y1="16.055" x2="46" y2="16.11" width="0.3" layer="16"/>
 <wire x1="46" y1="16.11" x2="46" y2="20" width="0.3" layer="16"/>
 <wire x1="46" y1="20" x2="47.5727" y2="21.5727" width="0.3" layer="1"/>
 <wire x1="47.5727" y1="21.5727" x2="47.5727" y2="22.74" width="0.3" layer="1"/>
 <wire x1="47.5727" y1="21.5727" x2="49.1454" y2="20" width="0.3" layer="1"/>
-<wire x1="49.1454" y1="20" x2="50" y2="20" width="0.3" layer="1"/>
-<wire x1="30.02" y1="15.3" x2="30.02" y2="17.59" width="0" layer="19" extent="16-16"/>
+<wire x1="30.02" y1="17.59" x2="30.02" y2="15.3" width="0.3" layer="16"/>
+<wire x1="30.02" y1="15.3" x2="30.21" y2="15.11" width="0.3" layer="16"/>
 </signal>
 <signal name="LED_1">
