File: 2018-2019/board/Training_Board.sch (EAGLE design)
At the start: 18 parts, among them IC1 ATMEGA328-20P, X1 JST-PH2

Commit message: Added filtering caps and re-spec of LDO
Parts:
- added C6: 100 nF, resistor:C-USC0603
- added C7: 10 nF, resistor:C-USC0603
- added R4: 10k Ohm, rcl:R-US_M0805
- LD1117: value R-78E5.0-0.5 -> AP2112SOT89-5; device RoboJackets-PowerICs:R-78E5.0-0.5 -> RoboJackets-PowerICs:AP2112SOT89-5
Connections:
- new net N$5: LD1117.EN, R4.2
- new net N$6: C6.2, IC1.AREF
- net GND: now also C6.1, C7.1
- net VBAT: now also C7.2, R4.1
Changed lines of the file:
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@@
 <part name="SUPPLY7" library="supply2" library_urn="urn:adsk.eagle:library:372" deviceset="GND" device=""/>
 <part name="SUPPLY8" library="supply2" library_urn="urn:adsk.eagle:library:372" deviceset="VCC" device="" value="+3V3"/>
-<part name="LD1117" library="RoboJackets-PowerICs" deviceset="R-78E5.0-0.5" device=""/>
+<part name="LD1117" library="RoboJackets-PowerICs" deviceset="AP2112" device="SOT89-5" package3d_urn="urn:adsk.eagle:package:4254535/1"/>
 <part name="C4" library="rcl" library_urn="urn:adsk.eagle:library:334" deviceset="C-US" device="C0603" package3d_urn="urn:adsk.eagle:package:23616/2" value="100nF"/>
 <part name="XO1" library="IQD-Frequency-Products" library_urn="urn:adsk.eagle:library:90" deviceset="CRYSTALS-NOGND" device="-HC49/4H" package3d_urn="urn:adsk.eagle:package:3356/1"/>
@@
 <part name="SUPPLY6" library="supply2" library_urn="urn:adsk.eagle:library:372" deviceset="GND" device=""/>
 <part name="SUPPLY10" library="supply2" library_urn="urn:adsk.eagle:library:372" deviceset="GND" device=""/>
+<part name="R4" library="rcl" library_urn="urn:adsk.eagle:library:334" deviceset="R-US_" device="M0805" package3d_urn="urn:adsk.eagle:package:23556/1" value="10k Ohm"/>
+<part name="C6" library="resistor" library_urn="urn:adsk.eagle:library:348" deviceset="C-US" device="C0603" package3d_urn="urn:adsk.eagle:package:26138/1" value="100 nF"/>
+<part name="C7" library="resistor" library_urn="urn:adsk.eagle:library:348" deviceset="C-US" device="C0603" package3d_urn="urn:adsk.eagle:package:26138/1" value="10 nF"/>
 </parts>
 <sheets>
@@
 <instance part="JP1" gate="G$1" x="167.64" y="55.88" rot="R180"/>
 <instance part="JP2" gate="A" x="129.54" y="53.34"/>
-<instance part="SUPPLY4" gate="GND" x="-53.34" y="63.5"/>
+<instance part="SUPPLY4" gate="GND" x="-66.04" y="63.5"/>
 <instance part="SUPPLY5" gate="G$1" x="-33.02" y="96.52"/>
 <instance part="X1" gate="G$1" x="-50.8" y="124.46"/>
@@
 <instance part="SUPPLY7" gate="GND" x="78.74" y="121.92"/>
 <instance part="SUPPLY8" gate="G$1" x="78.74" y="137.16"/>
-<instance part="LD1117" gate="G$1" x="-53.34" y="83.82"/>
+<instance part="LD1117" gate="G$1" x="-53.34" y="78.74"/>
 <instance part="C4" gate="G$1" x="-81.28" y="78.74"/>
 <instance part="XO1" gate="G$1" x="-4.064" y="58.42" rot="R180"/>
 <instance part="C3" gate="G$1" x="-10.16" y="50.8"/>
 <instance part="C5" gate="G$1" x="2.54" y="50.8"/>
-<instance part="SUPPLY9" gate="GND" x="7.62" y="73.66"/>
+<instance part="SUPPLY9" gate="GND" x="-10.16" y="73.66"/>
 <instance part="D1" gate="G$1" x="106.68" y="114.3" rot="R90"/>
 <instance part="D2" gate="G$1" x="147.32" y="114.3" rot="R90"/>
@@
 <instance part="SUPPLY6" gate="GND" x="152.4" y="106.68"/>
 <instance part="SUPPLY10" gate="GND" x="111.76" y="106.68"/>
+<instance part="R4" gate="G$1" x="-71.12" y="73.66" rot="R90"/>
+<instance part="C6" gate="G$1" x="4.318" y="68.58" rot="R90"/>
+<instance part="C7" gate="G$1" x="-40.64" y="127"/>
 </instances>
 <busses>
@@
 <segment>
 <pinref part="IC1" gate="G$1" pin="AGND"/>
-<wire x1="17.78" y1="76.2" x2="12.7" y2="76.2" width="0.1524" layer="91"/>
-<wire x1="12.7" y1="76.2" x2="7.62" y2="76.2" width="0.1524" layer="91"/>
+<wire x1="17.78" y1="76.2" x2="-2.54" y2="76.2" width="0.1524" layer="91"/>
 <pinref part="SUPPLY9" gate="GND" pin="GND"/>
+<pinref part="C6" gate="G$1" pin="1"/>
+<wire x1="-2.54" y1="76.2" x2="-10.16" y2="76.2" width="0.1524" layer="91"/>
+<wire x1="1.778" y1="68.58" x2="-2.54" y2="68.58" width="0.1524" layer="91"/>
+<wire x1="-2.54" y1="68.58" x2="-2.54" y2="76.2" width="0.1524" layer="91"/>
+<junction x="-2.54" y="76.2"/>
 </segment>
 <segment>
@@
 </segment>
 <segment>
-<pinref part="SUPPLY4" gate="GND" pin="GND"/>
-<pinref part="LD1117" gate="G$1" pin="GND"/>
-<wire x1="-53.34" y1="73.66" x2="-53.34" y2="66.04" width="0.1524" layer="91"/>
-<pinref part="C2" gate="G$1" pin="2"/>
-<wire x1="-33.02" y1="73.66" x2="-33.02" y2="66.04" width="0.1524" layer="91"/>
-<wire x1="-33.02" y1="66.04" x2="-53.34" y2="66.04" width="0.1524" layer="91"/>
-<junction x="-53.34" y="66.04"/>
-<pinref part="C4" gate="G$1" pin="2"/>
-<wire x1="-81.28" y1="73.66" x2="-81.28" y2="66.04" width="0.1524" layer="91"/>
-<wire x1="-81.28" y1="66.04" x2="-53.34" y2="66.04" width="0.1524" layer="91"/>
-</segment>
-<segment>
 <pinref part="X1" gate="G$1" pin="1"/>
-<wire x1="-53.34" y1="127" x2="-53.34" y2="137.16" width="0.1524" layer="91"/>
+<wire x1="-53.34" y1="127" x2="-53.34" y2="132.08" width="0.1524" layer="91"/>
 <label x="-53.34" y="137.16" size="1.778" layer="95" xref="yes"/>
+<pinref part="C7" gate="G$1" pin="1"/>
+<wire x1="-53.34" y1="132.08" x2="-53.34" y2="137.16" width="0.1524" layer="91"/>
+<wire x1="-40.64" y1="129.54" x2="-40.64" y2="132.08" width="0.1524" layer="91"/>
+<wire x1="-40.64" y1="132.08" x2="-53.34" y2="132.08" width="0.1524" layer="91"/>
+<junction x="-53.34" y="132.08"/>
 </segment>
 <segment>
@@
 <pinref part="SUPPLY10" gate="GND" pin="GND"/>
 </segment>
+<segment>
+<pinref part="C2" gate="G$1" pin="2"/>
+<wire x1="-33.02" y1="73.66" x2="-33.02" y2="66.04" width="0.1524" layer="91"/>
+<pinref part="SUPPLY4" gate="GND" pin="GND"/>
+<wire x1="-33.02" y1="66.04" x2="-66.04" y2="66.04" width="0.1524" layer="91"/>
+<pinref part="LD1117" gate="G$1" pin="GND"/>
+<wire x1="-66.04" y1="81.28" x2="-66.04" y2="66.04" width="0.1524" layer="91"/>
+<junction x="-66.04" y="66.04"/>
+<pinref part="C4" gate="G$1" pin="2"/>
+<wire x1="-81.28" y1="73.66" x2="-81.28" y2="66.04" width="0.1524" layer="91"/>
+<wire x1="-81.28" y1="66.04" x2="-66.04" y2="66.04" width="0.1524" layer="91"/>
+</segment>
 </net>
 <net name="VBAT" class="0">
 <segment>
 <pinref part="X1" gate="G$1" pin="2"/>
-<wire x1="-53.34" y1="124.46" x2="-53.34" y2="114.3" width="0.1524" layer="91"/>
+<wire x1="-53.34" y1="124.46" x2="-53.34" y2="116.84" width="0.1524" layer="91"/>
 <label x="-53.34" y="114.3" size="1.778" layer="95" xref="yes"/>
-</segment>
-<segment>
-<wire x1="-66.04" y1="86.36" x2="-81.28" y2="86.36" width="0.1524" layer="91"/>
+<pinref part="C7" gate="G$1" pin="2"/>
+<wire x1="-53.34" y1="116.84" x2="-53.34" y2="114.3" width="0.1524" layer="91"/>
+<wire x1="-40.64" y1="121.92" x2="-40.64" y2="116.84" width="0.1524" layer="91"/>
+<wire x1="-40.64" y1="116.84" x2="-53.34" y2="116.84" width="0.1524" layer="91"/>
+<junction x="-53.34" y="116.84"/>
+</segment>
+<segment>
+<wire x1="-66.04" y1="86.36" x2="-76.2" y2="86.36" width="0.1524" layer="91"/>
 <label x="-81.28" y="96.52" size="1.778" layer="95" xref="yes"/>
+<wire x1="-76.2" y1="86.36" x2="-81.28" y2="86.36" width="0.1524" layer="91"/>
 <wire x1="-81.28" y1="86.36" x2="-81.28" y2="96.52" width="0.1524" layer="91"/>
 <pinref part="LD1117" gate="G$1" pin="VIN"/>
@@
 <wire x1="-81.28" y1="81.28" x2="-81.28" y2="86.36" width="0.1524" layer="91"/>
 <junction x="-81.28" y="86.36"/>
+<pinref part="R4" gate="G$1" pin="1"/>
+<wire x1="-71.12" y1="68.58" x2="-76.2" y2="68.58" width="0.1524" layer="91"/>
+<wire x1="-76.2" y1="68.58" x2="-76.2" y2="86.36" width="0.1524" layer="91"/>
+<junction x="-76.2" y="86.36"/>
 </segment>
 <segment>
@@
 </segment>
 <segment>
-<pinref part="IC1" gate="G$1" pin="AVCC"/>
 <pinref part="SUPPLY1" gate="G$1" pin="VCC"/>
 <wire x1="-17.78" y1="83.82" x2="-17.78" y2="81.28" width="0.1524" layer="91"/>
-<junction x="-17.78" y="68.58"/>
-<wire x1="-17.78" y1="81.28" x2="-17.78" y2="68.58" width="0.1524" layer="91"/>
-<wire x1="-17.78" y1="68.58" x2="-17.78" y2="43.18" width="0.1524" layer="91"/>
+<junction x="-17.78" y="66.04"/>
+<wire x1="-17.78" y1="81.28" x2="-17.78" y2="66.04" width="0.1524" layer="91"/>
+<wire x1="-17.78" y1="66.04" x2="-17.78" y2="43.18" width="0.1524" layer="91"/>
 <pinref part="C1" gate="G$1" pin="1"/>
 <pinref part="R1" gate="G$1" pin="1"/>
 <wire x1="-5.08" y1="81.28" x2="-17.78" y2="81.28" width="0.1524" layer="91"/>
 <junction x="-17.78" y="81.28"/>
-<wire x1="17.78" y1="71.12" x2="17.78" y2="68.58" width="0.1524" layer="91"/>
-<wire x1="17.78" y1="68.58" x2="12.7" y2="68.58" width="0.1524" layer="91"/>
 <pinref part="IC1" gate="G$1" pin="VCC"/>
-<wire x1="12.7" y1="68.58" x2="-17.78" y2="68.58" width="0.1524" layer="91"/>
-<wire x1="12.7" y1="68.58" x2="12.7" y2="45.72" width="0.1524" layer="91"/>
+<wire x1="12.7" y1="66.04" x2="-17.78" y2="66.04" width="0.1524" layer="91"/>
+<wire x1="12.7" y1="66.04" x2="12.7" y2="45.72" width="0.1524" layer="91"/>
 <wire x1="12.7" y1="45.72" x2="17.78" y2="45.72" width="0.1524" layer="91"/>
-<junction x="12.7" y="68.58"/>
+<pinref part="IC1" gate="G$1" pin="AVCC"/>
+<wire x1="12.7" y1="66.04" x2="17.78" y2="66.04" width="0.1524" layer="91"/>
+<wire x1="17.78" y1="66.04" x2="17.78" y2="71.12" width="0.1524" layer="91"/>
+<junction x="12.7" y="66.04"/>
 </segment>
 <segment>
@@
 </segment>
 </net>
+<net name="N$5" class="0">
+<segment>
+<pinref part="LD1117" gate="G$1" pin="EN"/>
+<pinref part="R4" gate="G$1" pin="2"/>
+<wire x1="-66.04" y1="83.82" x2="-71.12" y2="83.82" width="0.1524" layer="91"/>
+<wire x1="-71.12" y1="83.82" x2="-71.12" y2="78.74" width="0.1524" layer="91"/>
+</segment>
+</net>
+<net name="N$6" class="0">
+<segment>
+<pinref part="C6" gate="G$1" pin="2"/>
+<wire x1="9.398" y1="68.58" x2="12.7" y2="68.58" width="0.1524" layer="91"/>
+<wire x1="12.7" y1="68.58" x2="12.7" y2="73.66" width="0.1524" layer="91"/>
+<pinref part="IC1" gate="G$1" pin="AREF"/>
+<wire x1="12.7" y1="73.66" x2="17.78" y2="73.66" width="0.1524" layer="91"/>
+</segment>
+</net>

Commit message: Added Aesthetics and extra smoothing capacitors
Parts:
- added C8: 1uF, rcl:C-USC0603
Connections:
- net GND: now also C8.2
- net VBAT: now also C8.1
Changed lines of the file:
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@@
 <part name="C6" library="resistor" library_urn="urn:adsk.eagle:library:348" deviceset="C-US" device="C0603" package3d_urn="urn:adsk.eagle:package:26138/1" value="100 nF"/>
 <part name="C7" library="resistor" library_urn="urn:adsk.eagle:library:348" deviceset="C-US" device="C0603" package3d_urn="urn:adsk.eagle:package:26138/1" value="10 nF"/>
+<part name="C8" library="rcl" library_urn="urn:adsk.eagle:library:334" deviceset="C-US" device="C0603" package3d_urn="urn:adsk.eagle:package:23616/2" value="1uF"/>
 </parts>
 <sheets>
@@
 <instance part="C6" gate="G$1" x="4.318" y="68.58" rot="R90"/>
 <instance part="C7" gate="G$1" x="-40.64" y="127"/>
+<instance part="C8" gate="G$1" x="-88.9" y="78.74"/>
 </instances>
 <busses>
@@
 <wire x1="-81.28" y1="73.66" x2="-81.28" y2="66.04" width="0.1524" layer="91"/>
 <wire x1="-81.28" y1="66.04" x2="-66.04" y2="66.04" width="0.1524" layer="91"/>
+<pinref part="C8" gate="G$1" pin="2"/>
+<wire x1="-88.9" y1="73.66" x2="-88.9" y2="66.04" width="0.1524" layer="91"/>
+<wire x1="-88.9" y1="66.04" x2="-81.28" y2="66.04" width="0.1524" layer="91"/>
+<junction x="-81.28" y="66.04"/>
 </segment>
 </net>
@@
 <wire x1="-76.2" y1="68.58" x2="-76.2" y2="86.36" width="0.1524" layer="91"/>
 <junction x="-76.2" y="86.36"/>
+<pinref part="C8" gate="G$1" pin="1"/>
+<wire x1="-81.28" y1="86.36" x2="-88.9" y2="86.36" width="0.1524" layer="91"/>
+<wire x1="-88.9" y1="86.36" x2="-88.9" y2="81.28" width="0.1524" layer="91"/>
 </segment>
 <segment>
