File: week_2_material/Hookup Schematic.sch (EAGLE design)
At the start: 5 parts, among them U1 ATMEGA328P_PDIP

Commit message: edited graphics and finished lab guide in LaTeX
Connections:
- new net PIN_2: Q1.B
- new net PIN_3: Q2.B
- new net PIN_5: Q3.B
- new net PIN_9: Q4.B
Changed lines of the file:
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@@
+</segment>
+</net>
+<net name="PIN_3" class="0">
+<segment>
+<pinref part="Q2" gate="G$1" pin="B"/>
+<wire x1="99.06" y1="76.2" x2="91.44" y2="76.2" width="0.1524" layer="91"/>
+<label x="91.44" y="76.2" size="1.778" layer="95" rot="R180" xref="yes"/>
+</segment>
+</net>
+<net name="PIN_5" class="0">
+<segment>
+<pinref part="Q3" gate="G$1" pin="B"/>
+<wire x1="160.02" y1="76.2" x2="167.64" y2="76.2" width="0.1524" layer="91"/>
+<label x="167.64" y="76.2" size="1.778" layer="95" xref="yes"/>
+</segment>
+</net>
+<net name="PIN_9" class="0">
+<segment>
+<pinref part="Q4" gate="G$1" pin="B"/>
+<wire x1="160.02" y1="45.72" x2="167.64" y2="45.72" width="0.1524" layer="91"/>
+<label x="167.64" y="45.72" size="1.778" layer="95" xref="yes"/>
+</segment>
+</net>
+<net name="PIN_2" class="0">
+<segment>
+<pinref part="Q1" gate="G$1" pin="B"/>
+<wire x1="99.06" y1="45.72" x2="91.44" y2="45.72" width="0.1524" layer="91"/>
+<label x="91.44" y="45.72" size="1.778" layer="95" rot="R180" xref="yes"/>
 </segment>
 </net>

Commit message: Cleaned up schematic
Parts:
- added U$1: MOTOR, motor:MOTOR
Connections:
- removed net N$2: Q3.C, Q4.C
- new net MOTOR_NEGATIVE: Q3.C, Q4.C, U$1.P$2
- net N$1: now also U$1.P$1
Changed lines of the file:
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@@
 <part name="SUPPLY1" library="supply2" library_urn="urn:adsk.eagle:library:372" deviceset="VCC" device=""/>
 <part name="SUPPLY2" library="supply2" library_urn="urn:adsk.eagle:library:372" deviceset="DGND" device=""/>
+<part name="U$1" library="motor" deviceset="MOTOR" device=""/>
 </parts>
 <sheets>
@@
 <instance part="SUPPLY1" gate="G$1" x="129.54" y="99.06"/>
 <instance part="SUPPLY2" gate="G$1" x="129.54" y="25.4"/>
+<instance part="U$1" gate="G$1" x="152.4" y="55.88"/>
 </instances>
 <busses>
@@
 <pinref part="Q2" gate="G$1" pin="C"/>
 <pinref part="Q1" gate="G$1" pin="C"/>
-<wire x1="109.22" y1="66.04" x2="109.22" y2="55.88" width="0.1524" layer="91"/>
+<wire x1="109.22" y1="66.04" x2="109.22" y2="60.96" width="0.1524" layer="91"/>
+<pinref part="U$1" gate="G$1" pin="P$1"/>
+<wire x1="109.22" y1="60.96" x2="109.22" y2="55.88" width="0.1524" layer="91"/>
+<wire x1="114.3" y1="60.96" x2="109.22" y2="60.96" width="0.1524" layer="91"/>
+<junction x="109.22" y="60.96"/>
 </segment>
 </net>
-<net name="N$2" class="0">
+<net name="MOTOR_NEGATIVE" class="0">
 <segment>
 <pinref part="Q3" gate="G$1" pin="C"/>
 <pinref part="Q4" gate="G$1" pin="C"/>
-<wire x1="149.86" y1="66.04" x2="149.86" y2="55.88" width="0.1524" layer="91"/>
+<wire x1="149.86" y1="66.04" x2="149.86" y2="60.96" width="0.1524" layer="91"/>
+<pinref part="U$1" gate="G$1" pin="P$2"/>
+<wire x1="149.86" y1="60.96" x2="149.86" y2="55.88" width="0.1524" layer="91"/>
+<wire x1="144.78" y1="60.96" x2="149.86" y2="60.96" width="0.1524" layer="91"/>
+<junction x="149.86" y="60.96"/>
 </segment>
 </net>
