File: board/Training_Board.brd (EAGLE design)
At the start: 59 x 32 mm, 23 parts, among them IC1 ATMEGA328-20P, X1 JST-PH2

Commit message: Board Changes
Made the name space bigger, remove thermal traces, rev board, round corner, move to origin
Parts:
- R1: device resistor:R0603 -> rcl:R0603
- R2, R3, R4: device rcl:M0805 -> rcl:R0603
- moved C1 2.24 mm to (31.2, 16.3)
- moved C2 2.24 mm to (46.0, 24.9)
- moved C3 2.24 mm to (55.0, 17.0)
- moved C4 2.24 mm to (46.0, 27.4)
- moved C5 2.24 mm to (55.0, 12.5)
- moved C6 2.24 mm to (26.0, 17.0)
- moved C7 2.24 mm to (6.50, 30.0)
- moved C8 2.24 mm to (46.5, 27.0)
- moved D1 2.24 mm to (7.50, 24.0)
- moved D2 2.24 mm to (4.50, 24.0)
- moved IC1 2.24 mm to (27.2, 15.8)
- moved JP1 2.24 mm to (27.0, 25.3)
- moved JP2 2.24 mm to (22.0, 5.00)
- moved LD1117 2.24 mm to (49.9, 25.7)
- moved PRGRM-HEADER 2.24 mm to (4.92, 12.9)
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Other:
- outline, holes or cut-outs redrawn
- board text added: "Electrical Training Board v1.1"
- board text removed: "Electrical Training Board v1.0"

Commit message: Updated packages of LDO and improved usability
Parts:
- removed LD1117: AP2112SOT89-5, RoboJackets-PowerICs:SOT95P285X110-5
- removed R4: 10k Ohm, rcl:R0603
- removed S1: PTS645PTS645_SMD1, RoboJackets-Switches:PTS645_SMD
- removed X1: JST-PH2, Trainii:JST-PH
- added U$2: PTS645PTS645_SMD1, RoboJackets-Switches:PTS645_SMD
- added U$3: LD1117ASOT223, RoboJackets-PowerICs:SOT230P700X180-4
- added U$4: JST-PH2, Trainii:JST-PH
- moved C4 11.6 mm to (57.5, 26.0), flipped to the bottom, turned to 270 degrees
- moved C8 10.3 mm to (56.5, 29.5), turned to 0 degrees
- moved C2 1.14 mm to (46.0, 26.0), flipped to the bottom, turned to 0 degrees
Connections:
- removed net N$5: LD1117.3, R4.2
- net +3V3: now also U$3.1, U$3.4; no longer LD1117.5
- net GND: now also U$2.P$1, U$2.P$2, U$3.2, U$4.1; no longer LD1117.2, S1.P$1, S1.P$2, X1.1
- net RST: now also U$2.P$3, U$2.P$4; no longer S1.P$3, S1.P$4
- net VBAT: now also U$3.3, U$4.2; no longer LD1117.4, R4.1, X1.2
Routing:
- net VBAT: track 52.2 -> 59.2 mm, vias 1 -> 0
- net GND: track 29.8 -> 25.3 mm, vias 6 -> 3
- net +3V3: track 97.3 -> 100.3 mm
- net N$5: track 2.52 -> 0.00 mm
- net RST: track 62.1 -> 63.2 mm

Commit message: Small DRC corrections and new gerbers
Parts:
- renumbered U$3 to U3
Routing:
- net +3V3: track 100.3 -> 107.3 mm
- net VBAT: track 59.2 -> 58.3 mm
- net GND: track 25.3 -> 24.6 mm
Changed lines of the file:
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@@
 <attribute name="VALUE" x="54.365" y="10.595" size="1.27" layer="27"/>
 </element>
-<element name="IC1" library="atmega328" package="DIL28-3" value="ATMEGA328-20P" x="27.21" y="15.78"/>
+<element name="IC1" library="atmega328" package="DIL28-3" value="ATMEGA328-20P" x="27.21" y="15.78" smashed="yes">
+<attribute name="NAME" x="15.303" y="23.24" size="1.778" layer="25" ratio="10" rot="R180"/>
+<attribute name="VALUE" x="11.462" y="14.8402" size="1.778" layer="27" ratio="10"/>
+</element>
 <element name="JP1" library="pinhead" library_urn="urn:adsk.eagle:library:325" package="1X12" package3d_urn="urn:adsk.eagle:package:22487/2" value="" x="27" y="25.32" rot="R180"/>
 <element name="JP2" library="pinhead" library_urn="urn:adsk.eagle:library:325" package="1X16" package3d_urn="urn:adsk.eagle:package:22432/2" value="" x="22" y="5"/>
@@
 <element name="U$1" library="RoboJackets-Aesthetics" package="ROBOBUZZ_0.4X" value="" x="55.5" y="23.5"/>
 <element name="U$2" library="RoboJackets-Switches" package="PTS645_SMD" value="PTS645PTS645_SMD1" x="49.5" y="4"/>
-<element name="U$3" library="RoboJackets-PowerICs" package="SOT230P700X180-4" package3d_urn="urn:adsk.eagle:package:5711203/1" value="LD1117ASOT223" x="52" y="24" rot="MR270"/>
+<element name="U3" library="RoboJackets-PowerICs" package="SOT230P700X180-4" package3d_urn="urn:adsk.eagle:package:5711203/1" value="LD1117ASOT223" x="52" y="24" rot="MR270"/>
 <element name="U$4" library="Trainii" package="JST-PH" value="JST-PH2" x="6.5" y="28"/>
 </elements>
@@
 <wire x1="55.85" y1="12.5" x2="56" y2="12.65" width="0.3" layer="1"/>
 <wire x1="56" y1="12.65" x2="56" y2="14.5" width="0.3" layer="1"/>
-<wire x1="55.85" y1="12.5" x2="55.85" y2="11" width="0.3" layer="1"/>
 <contactref element="D2" pad="C"/>
 <contactref element="D1" pad="C"/>
-<wire x1="55.85" y1="11" x2="55.85" y2="10.732" width="0.3" layer="1"/>
 <wire x1="4.5" y1="24.75" x2="5" y2="25.25" width="0.3" layer="1"/>
 <wire x1="5" y1="25.25" x2="5" y2="26" width="0.3" layer="1"/>
@@
 <contactref element="C6" pad="1"/>
 <contactref element="C7" pad="1"/>
-<wire x1="5.65" y1="30" x2="5.7" y2="29.95" width="0.3" layer="16"/>
 <contactref element="C8" pad="2"/>
 <contactref element="U$2" pad="P$1"/>
 <contactref element="U$2" pad="P$2"/>
 <wire x1="53.335" y1="6.25" x2="45.665" y2="6.25" width="0.3" layer="1"/>
-<wire x1="45.665" y1="6.25" x2="45.665" y2="6.665" width="0.3" layer="1"/>
-<wire x1="53.335" y1="6.25" x2="55.85" y2="8.765" width="0.3" layer="1"/>
-<wire x1="55.85" y1="8.765" x2="55.85" y2="11" width="0.3" layer="1"/>
-<contactref element="U$3" pad="2"/>
+<wire x1="55.85" y1="8.765" x2="53.335" y2="6.25" width="0.3" layer="1"/>
+<contactref element="U3" pad="2"/>
 <contactref element="U$4" pad="1"/>
 <wire x1="5.65" y1="30" x2="5.65" y2="28.15" width="0.3" layer="16"/>
 <wire x1="5.65" y1="28.15" x2="5.5" y2="28" width="0.3" layer="16"/>
+<wire x1="55.85" y1="12.5" x2="55.85" y2="8.765" width="0.3" layer="1"/>
 </signal>
 <signal name="VBAT">
 <contactref element="C4" pad="1"/>
 <contactref element="JP1" pad="12"/>
-<wire x1="10.57" y1="25.32" x2="11" y2="25.32" width="0.3" layer="16"/>
-<wire x1="11" y1="25.32" x2="13.03" y2="25.32" width="0.3" layer="16"/>
 <wire x1="16.71" y1="29" x2="13.03" y2="25.32" width="0.3" layer="16"/>
 <contactref element="C7" pad="2"/>
 <wire x1="7.35" y1="30" x2="7.35" y2="29" width="0.3" layer="16"/>
 <contactref element="C8" pad="1"/>
-<contactref element="U$3" pad="3"/>
-<wire x1="7.35" y1="29" x2="7.35" y2="28.54" width="0.3" layer="16"/>
+<contactref element="U3" pad="3"/>
 <wire x1="54.3" y1="27.0226" x2="52.3226" y2="29" width="0.3" layer="16"/>
 <wire x1="52.3226" y1="29" x2="16.71" y2="29" width="0.3" layer="16"/>
@@
 <wire x1="57.3274" y1="27.0226" x2="54.3" y2="27.0226" width="0.3" layer="16"/>
 <contactref element="U$4" pad="2"/>
+<wire x1="7.35" y1="28.15" x2="7.5" y2="28" width="0.3" layer="16"/>
+<wire x1="7.5" y1="28" x2="10.18" y2="25.32" width="0.3" layer="16"/>
 <wire x1="7.35" y1="29" x2="7.35" y2="28.15" width="0.3" layer="16"/>
-<wire x1="7.35" y1="28.15" x2="7.5" y2="28" width="0.3" layer="16"/>
-<wire x1="11" y1="25.32" x2="10.18" y2="25.32" width="0.3" layer="16"/>
-<wire x1="10.18" y1="25.32" x2="7.5" y2="28" width="0.3" layer="16"/>
+<wire x1="10.18" y1="25.32" x2="10.18" y2="25.32" width="0.3" layer="16"/>
+<wire x1="10.18" y1="25.32" x2="13.03" y2="25.32" width="0.3" layer="16"/>
 </signal>
 <signal name="RST">
@@
 <wire x1="10.7" y1="11.97" x2="12" y2="10.67" width="0.3" layer="1"/>
 <wire x1="12" y1="10.67" x2="12" y2="3" width="0.3" layer="1"/>
-<wire x1="13.834" y1="1.166" x2="12" y2="3" width="0.3" layer="1"/>
+<wire x1="12" y1="3" x2="13.834" y2="1.166" width="0.3" layer="1"/>
 <wire x1="6.19" y1="15.41" x2="9.63" y2="11.97" width="0.3" layer="1"/>
 <wire x1="9.63" y1="11.97" x2="10.7" y2="11.97" width="0.3" layer="1"/>
-<wire x1="42.448" y1="1.166" x2="42" y2="1.166" width="0.3" layer="1"/>
 <contactref element="U$2" pad="P$3"/>
 <contactref element="U$2" pad="P$4"/>
-<wire x1="42" y1="1.166" x2="13.834" y2="1.166" width="0.3" layer="1"/>
 <wire x1="53.335" y1="2.925" x2="53.335" y2="1.75" width="0.3" layer="1"/>
 <wire x1="56.03" y1="5.62" x2="53.335" y2="2.925" width="0.3" layer="1"/>
-<wire x1="42" y1="1.166" x2="45.081" y2="1.166" width="0.3" layer="1"/>
 <wire x1="45.081" y1="1.166" x2="45.665" y2="1.75" width="0.3" layer="1"/>
 <wire x1="53.335" y1="1.75" x2="45.665" y2="1.75" width="0.3" layer="1"/>
+<wire x1="13.834" y1="1.166" x2="45.081" y2="1.166" width="0.3" layer="1"/>
 </signal>
 <signal name="MISO">
@@
 <wire x1="36.1" y1="19.59" x2="32" y2="23.69" width="0.3" layer="1"/>
 <wire x1="6.19" y1="10.33" x2="4.7144" y2="11.8056" width="0.3" layer="1"/>
-<wire x1="4.7144" y1="15.8712" x2="2.7928" y2="17.7928" width="0.3" layer="1"/>
+<wire x1="2.7928" y1="17.7928" x2="4.7144" y2="15.8712" width="0.3" layer="1"/>
 <wire x1="4.7144" y1="11.8056" x2="4.7144" y2="15.8712" width="0.3" layer="1"/>
-<wire x1="2.7928" y1="26.4939375" x2="6.2988625" y2="30" width="0.3" layer="1"/>
-<wire x1="2.7928" y1="17.7928" x2="2.7928" y2="26.4939375" width="0.3" layer="1"/>
-<wire x1="6.2988625" y1="30" x2="29" y2="30" width="0.3" layer="1"/>
+<wire x1="29" y1="30" x2="6.2988625" y2="30" width="0.3" layer="1"/>
+<wire x1="6.2988625" y1="30" x2="5.1552625" y2="28.8564" width="0.3" layer="1"/>
+<wire x1="5.1552625" y1="28.8564" x2="5.1452625" y2="28.8564" width="0.3" layer="1"/>
+<wire x1="5.1452625" y1="28.8564" x2="2.7928" y2="26.5039375" width="0.3" layer="1"/>
+<wire x1="2.7928" y1="26.5039375" x2="2.7928" y2="17.7928" width="0.3" layer="1"/>
 </signal>
 <signal name="SCK">
@@
 <wire x1="31.02" y1="19.59" x2="31.02" y2="17.3" width="0.3" layer="16"/>
 <wire x1="31.02" y1="17.3" x2="31.21" y2="17.11" width="0.3" layer="16"/>
-<contactref element="U$3" pad="4"/>
-<contactref element="U$3" pad="1"/>
+<contactref element="U3" pad="4"/>
+<contactref element="U3" pad="1"/>
 <wire x1="49.7" y1="27.0226" x2="47.8726" y2="27.0226" width="0.3" layer="16"/>
 <wire x1="47.8726" y1="27.0226" x2="46.85" y2="26" width="0.3" layer="16"/>
@@
 <wire x1="47" y1="25.85" x2="46.85" y2="26" width="0.3" layer="16"/>
 <wire x1="47" y1="22" x2="52.834" y2="22" width="0.3" layer="1"/>
-<wire x1="52.834" y1="22" x2="52" y2="20.9774" width="0" layer="19" extent="1-16"/>
+<wire x1="49.7" y1="27.0226" x2="49.7" y2="23.2774" width="0.3" layer="16"/>
+<wire x1="49.7" y1="23.2774" x2="52" y2="20.9774" width="0.3" layer="16"/>
 </signal>
 <signal name="LED_1">
