File: board/training_board.brd (EAGLE design)
At the start: 160 x 100 mm, 0 parts

Commit message: Preliminary Schematic completed.  Components arranged and not routed on board.
Parts:
- added F1, F2: 350 mA, RoboJackets-Fuses:F1812
- added J1, J2: 1X2-3.5MM, adafruit:1X2-3.5MM
- added LED1, LED2: YELLOW, led:CHIP-LED0603
- added LED3: RED, led:CHIP-LED0603
- added Q1: ARDUINOR3-NOIOREF-NOTEXT, adafruit:ARDUINOR3-NOTEXT-NOIOREF
- added R2, R3: 1k O, rcl:R0603
- added R4: 10k O, rcl:R0603
- added R5: 240 O, rcl:R0603
- added U$1: PJ-037A, RoboJackets-Connectors:PJ-037A
- added U$2: PTS645, RoboJackets-Switches:PTS645
- added U1, U2: ZXBM5210-S-13, RoboJackets-ICs:SOIC-8
Connections:
- new net +12V: F1.1, F2.1, Q1.VIN, R5.2, U$1.P$2, U1.3, U1.6, U2.3, U2.6
- new net +5V: Q1.5V, R2.2, R3.2, R4.2
- new net 3V: Q1.3V
- new net GND: LED3.C, Q1.GND, Q1.GND1, Q1.GND2, U$1.P$1, U$2.P$1, U$2.P$2, U1.8, U2.8
- new net M1_FWD: Q1.D2, U1.4
- new net M1_REV: Q1.D3, U1.5
- new net M2_FWD: Q1.D4, U2.4
- new net M2_REV: Q1.D5, U2.5
- new net N$1: J1.1, U1.1
- new net N$12: LED1.C, Q1.D8
- new net N$13: LED2.C, Q1.D9
- new net N$14: LED1.A, R3.1
- new net N$15: LED2.A, R2.1
- new net N$16: LED3.A, R5.1
- new net N$2: J1.2, U1.7
- new net N$3: J2.1, U2.1
- new net N$4: J2.2, U2.7
- new net N$5: Q1.RESET, R4.1, U$2.P$3, U$2.P$4
- new net N$6: F1.2, U1.2
- new net N$7: F2.2, U2.2

Commit message: Added Preliminary Board layout
Parts:
- removed LED3: RED, led:CHIP-LED0603
- added 12V_OK: GREEN, led:CHIP-LED0603
- added F1_OK, F2_OK: (no value), led:CHIP-LED0603
- added R1, R6: 2.4K, rcl:R0603
- added SW1: 400AWMDP1R1M2, RoboJackets-Switches:400AWMDP1R1M2
- R2, R3: value 1k O -> 1K
- R4: value 10k O -> 10K
- R5: value 240 O -> 2.4K
- moved U$2 39.2 mm to (36.0, 12.0)
- moved LED1 25.3 mm to (31.0, 45.0), turned to 90 degrees
- moved R4 19.2 mm to (36.0, 7.00)
- moved LED2 19.1 mm to (31.0, 39.0), turned to 90 degrees
- moved R3 18.4 mm to (37.0, 45.0)
- moved R5 16.2 mm to (11.0, 49.0), turned to 0 degrees
- moved R2 10.6 mm to (37.0, 39.0)
- moved J1 7.00 mm to (3.00, 28.0), turned to 270 degrees
- moved F2 6.40 mm to (25.0, 13.0)
- moved U1 5.39 mm to (15.0, 24.0)
- moved F1 5.10 mm to (25.0, 27.0)
- moved U2 5.00 mm to (15.0, 11.0)
- moved J2 1.00 mm to (3.00, 9.00), turned to 270 degrees
Connections:
- removed net N$1: J1.1, U1.1
- removed net N$12: LED1.C, Q1.D8
- removed net N$13: LED2.C, Q1.D9
- removed net N$4: J2.2, U2.7
- new net M1+: SW1.P$4, U1.1
- new net M1+_SW: J1.1, SW1.P$5
- new net M2-: SW1.P$3, U2.7
- new net M2-_SW: J2.2, SW1.P$2
- new net N$10: Q1.D9, R3.2
- new net N$11: Q1.D8, R2.2
- new net N$8: F1_OK.A, R1.1
- new net N$9: F2_OK.A, R6.1
- net +5V: no longer R2.2, R3.2
- net GND: now also 12V_OK.C, F1_OK.C, F2_OK.C, LED1.C, LED2.C; no longer LED3.C
- net M1_FWD: now also Q1.D4; no longer Q1.D2
- net M1_REV: now also Q1.D5; no longer Q1.D3
- net M2_FWD: now also Q1.D2; no longer Q1.D4
- net M2_REV: now also Q1.D3; no longer Q1.D5
- net N$16: now also 12V_OK.A; no longer LED3.A
- net N$6: now also R1.2
- net N$7: now also R6.2
Routing:
- net +12V: track 0.00 -> 108.1 mm
- net M2_FWD: track 0.00 -> 63.6 mm, vias 0 -> 2
- net M2_REV: track 0.00 -> 57.2 mm, vias 0 -> 2
- net M1_FWD: track 0.00 -> 53.9 mm, vias 0 -> 2
- net M1_REV: track 0.00 -> 47.6 mm, vias 0 -> 2
- net GND: track 0.00 -> 38.3 mm, vias 0 -> 7
- net N$6: track 0.00 -> 33.8 mm
- net N$7: track 0.00 -> 21.1 mm
- net N$5: track 0.00 -> 16.4 mm
- net N$2: track 0.00 -> 14.1 mm
- net N$11: track 0.00 -> 13.4 mm
- net N$3: track 0.00 -> 11.9 mm
- net M2-: track 0.00 -> 9.20 mm
- net M1+: track 0.00 -> 6.82 mm
- net M2-_SW: track 0.00 -> 6.59 mm
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- added copper zone on layer 1, net GND
- added copper zone on layer 16, net GND
Other:
- board size 160 x 100 mm -> 68.7 x 53.3 mm

Commit message: Added Week 0 content to references folder
Parts:
- added C1, C3: 0.1uF, rcl:C0805
- added C2: 1uF, rcl:C0805
Connections:
- net +12V: now also C1.1, C2.1
- net GND: now also C1.2, C2.2, C3.2
- net N$5: now also C3.1
Routing:
- net +12V: track 108.1 -> 120.2 mm
- net GND: track 38.3 -> 47.3 mm, vias 7 -> 10
- net N$5: track 16.4 -> 19.6 mm
- net M2_FWD: track 63.6 -> 65.1 mm
Changed lines of the file:
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@@
 </element>
 <element name="U$1" library="RoboJackets-Connectors" package="PJ-037A" value="PJ-037A" x="4" y="42" smashed="yes"/>
-<element name="U$2" library="RoboJackets-Switches" package="PTS645" value="PTS645" x="36" y="12" smashed="yes"/>
+<element name="U$2" library="RoboJackets-Switches" package="PTS645" value="PTS645" x="36" y="12" smashed="yes">
+<attribute name="FUNCTION" value="RESET" x="36" y="12" size="1.778" layer="27" display="off"/>
+</element>
 <element name="F1" library="RoboJackets-Fuses" package="F1812" value="350 mA" x="25" y="27" smashed="yes" rot="R270">
 <attribute name="NAME" x="26.905" y="28.905" size="1.27" layer="25" rot="R270"/>
@@
 <attribute name="NAME" x="6" y="19.6" size="1" layer="25" font="vector" rot="R180"/>
 <attribute name="VALUE" x="10.4" y="15" size="1" layer="27" font="vector" rot="R90" display="off"/>
+</element>
+<element name="C1" library="rcl" library_urn="urn:adsk.eagle:library:334" package="C0805" package3d_urn="urn:adsk.eagle:package:23617/2" value="0.1uF" x="19" y="46" smashed="yes">
+<attribute name="NAME" x="17.73" y="47.27" size="1.27" layer="25"/>
+<attribute name="SPICEPREFIX" value="C" x="19" y="46" size="1.778" layer="27" display="off"/>
+<attribute name="VALUE" x="17.73" y="43.46" size="1.27" layer="27"/>
+</element>
+<element name="C2" library="rcl" library_urn="urn:adsk.eagle:library:334" package="C0805" package3d_urn="urn:adsk.eagle:package:23617/2" value="1uF" x="19" y="40" smashed="yes">
+<attribute name="NAME" x="17.73" y="41.27" size="1.27" layer="25"/>
+<attribute name="SPICEPREFIX" value="C" x="19" y="40" size="1.778" layer="27" display="off"/>
+<attribute name="VALUE" x="17.73" y="37.46" size="1.27" layer="27"/>
+</element>
+<element name="C3" library="rcl" library_urn="urn:adsk.eagle:library:334" package="C0805" package3d_urn="urn:adsk.eagle:package:23617/2" value="0.1uF" x="29" y="5" smashed="yes" rot="R180">
+<attribute name="NAME" x="30.27" y="3.73" size="1.27" layer="25" rot="R180"/>
+<attribute name="SPICEPREFIX" value="C" x="29" y="5" size="1.778" layer="27" rot="R180" display="off"/>
+<attribute name="VALUE" x="30.27" y="7.54" size="1.27" layer="27" rot="R180"/>
 </element>
 </elements>
@@
 <via x="11.9" y="28" extent="1-16" drill="0.35"/>
 <via x="10.9" y="26.9" extent="1-16" drill="0.35"/>
+<contactref element="C1" pad="2"/>
+<contactref element="C2" pad="2"/>
+<contactref element="C3" pad="2"/>
+<wire x1="19.95" y1="46" x2="19.95" y2="44" width="1" layer="1"/>
+<wire x1="19.95" y1="44" x2="19.95" y2="42" width="1" layer="1"/>
+<wire x1="19.95" y1="42" x2="19.95" y2="40" width="1" layer="1"/>
+<via x="19.95" y="42" extent="1-16" drill="0.35"/>
+<via x="19.95" y="44" extent="1-16" drill="0.35"/>
+<wire x1="28.05" y1="5" x2="28" y2="5.05" width="0.2" layer="1"/>
+<wire x1="28" y1="5.05" x2="28" y2="8" width="0.2" layer="1"/>
+<via x="28" y="8" extent="1-16" drill="0.35"/>
 </signal>
 <signal name="3V">
@@
 <wire x1="16" y1="16" x2="23.95" y2="16" width="0.5" layer="1"/>
 <wire x1="23.95" y1="16" x2="25" y2="14.95" width="0.5" layer="1"/>
-<wire x1="25" y1="28.95" x2="11.95" y2="42" width="1" layer="1"/>
+<wire x1="25" y1="28.95" x2="17.975" y2="35.975" width="1" layer="1"/>
+<wire x1="17.975" y1="35.975" x2="11.95" y2="42" width="1" layer="1"/>
 <wire x1="11.95" y1="42" x2="10" y2="42" width="1" layer="1"/>
 <wire x1="27.05" y1="28.95" x2="29" y2="27" width="1" layer="1"/>
@@
 <wire x1="11.85" y1="49" x2="11.95" y2="48.9" width="0.2" layer="1"/>
 <wire x1="11.95" y1="48.9" x2="11.95" y2="42" width="0.2" layer="1"/>
-<wire x1="27.05" y1="28.95" x2="25" y2="28.95" width="0" layer="19" extent="1-1"/>
+<contactref element="C1" pad="1"/>
+<contactref element="C2" pad="1"/>
+<wire x1="18.05" y1="46" x2="18.05" y2="40" width="1" layer="1"/>
+<wire x1="18.05" y1="40" x2="18.05" y2="36.05" width="1" layer="1"/>
+<wire x1="18.05" y1="36.05" x2="17.975" y2="35.975" width="1" layer="1"/>
+<wire x1="25" y1="28.95" x2="27.05" y2="28.95" width="1" layer="1"/>
 </signal>
 <signal name="+5V">
@@
 <wire x1="35.15" y1="7" x2="35.15" y2="8.9" width="0.5" layer="1"/>
 <wire x1="35.15" y1="8.9" x2="36" y2="9.75" width="0.5" layer="1"/>
+<contactref element="C3" pad="1"/>
+<wire x1="29.95" y1="5" x2="32.89" y2="5" width="0.2" layer="1"/>
+<wire x1="32.89" y1="5" x2="33.02" y2="4.87" width="0.2" layer="1"/>
 </signal>
 <signal name="M1_FWD">
@@
 <contactref element="U2" pad="4"/>
 <contactref element="Q1" pad="D2"/>
-<wire x1="16.905" y1="9.285" x2="16.905" y2="8.4" width="0.2" layer="1"/>
+<wire x1="16.905" y1="9.285" x2="16.905" y2="9" width="0.2" layer="1"/>
+<wire x1="16.905" y1="9" x2="16.905" y2="8.4" width="0.2" layer="1"/>
 <wire x1="58.42" y1="50.8" x2="58.2324" y2="50.6124" width="0.2" layer="1"/>
 <wire x1="58.2324" y1="50.6124" x2="58.2324" y2="44" width="0.2" layer="1"/>
 <wire x1="58.2324" y1="44" x2="58.2324" y2="43.677075" width="0.2" layer="1"/>
-<wire x1="58.2324" y1="44" x2="58.2324" y2="44" width="0.2" layer="1"/>
 <wire x1="58.2324" y1="44" x2="37.2324" y2="23" width="0.2" layer="1"/>
 <wire x1="37.2324" y1="23" x2="34" y2="23" width="0.2" layer="1"/>
@@
 <via x="21" y="11" extent="1-16" drill="0.35"/>
 <wire x1="21" y1="11" x2="20" y2="10" width="0.2" layer="1"/>
-<wire x1="20" y1="10" x2="18" y2="10" width="0.2" layer="1"/>
-<wire x1="16.905" y1="9.285" x2="18" y2="10" width="0" layer="19" extent="1-1"/>
+<wire x1="17.905" y1="10" x2="16.905" y2="9" width="0.2" layer="1"/>
+<wire x1="20" y1="10" x2="17.905" y2="10" width="0.2" layer="1"/>
 </signal>
 <signal name="M2_REV">

Commit message: Updated Routing, added decoupling capacitors, and added silkscreen
Parts:
- added U$3: (no value), RoboJackets-Aesthetics:ROBOJACKETS
- added U$4: (no value), RoboJackets-Aesthetics:ROBOBUZZ_0.8X
Routing:
- net M2_FWD: track 65.1 -> 64.5 mm
Other:
- board text added: "2019 Training Board V1.0"
Changed lines of the file:
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@@
 <layer number="110" name="fp0" color="7" fill="1" visible="no" active="yes"/>
 <layer number="111" name="LPC17xx" color="7" fill="1" visible="no" active="yes"/>
-<layer number="112" name="tSilk" color="7" fill="1" visible="no" active="yes"/>
+<layer number="112" name="tSilk" color="7" fill="1" visible="yes" active="yes"/>
 <layer number="113" name="ReferenceLS" color="7" fill="1" visible="no" active="no"/>
 <layer number="114" name="FRNTMAAT1" color="7" fill="1" visible="yes" active="yes"/>
@@
 <wire x1="68.7" y1="53.3" x2="0" y2="53.3" width="0" layer="20"/>
 <wire x1="0" y1="53.3" x2="0" y2="0" width="0" layer="20"/>
+<text x="37" y="22" size="1.5" layer="112">2019 Training Board
+V1.0</text>
+<polygon width="0.1524" layer="112">
+<vertex x="42" y="22"/>
+<vertex x="68" y="22"/>
+<vertex x="68" y="15"/>
+<vertex x="42" y="15"/>
+</polygon>
 </plain>
 <attributes>
@@
 <attribute name="VALUE" x="30.27" y="7.54" size="1.27" layer="27" rot="R180"/>
 </element>
+<element name="U$3" library="RoboJackets-Aesthetics" package="ROBOJACKETS" value="" x="37" y="27" smashed="yes"/>
+<element name="U$4" library="RoboJackets-Aesthetics" package="ROBOBUZZ_0.8X" value="" x="58" y="33" smashed="yes"/>
 </elements>
 <signals>
@@
 <wire x1="40" y1="18" x2="45.72" y2="12.28" width="0.5" layer="1"/>
 <wire x1="45.72" y1="12.28" x2="45.72" y2="2.54" width="0.5" layer="1"/>
-<wire x1="11.95" y1="42" x2="11.85" y2="42.1" width="0.2" layer="1"/>
 <wire x1="11.85" y1="49" x2="11.95" y2="48.9" width="0.2" layer="1"/>
 <wire x1="11.95" y1="48.9" x2="11.95" y2="42" width="0.2" layer="1"/>
@@
 <contactref element="U2" pad="4"/>
 <contactref element="Q1" pad="D2"/>
-<wire x1="16.905" y1="9.285" x2="16.905" y2="9" width="0.2" layer="1"/>
 <wire x1="16.905" y1="9" x2="16.905" y2="8.4" width="0.2" layer="1"/>
 <wire x1="58.42" y1="50.8" x2="58.2324" y2="50.6124" width="0.2" layer="1"/>
 <wire x1="58.2324" y1="50.6124" x2="58.2324" y2="44" width="0.2" layer="1"/>
-<wire x1="58.2324" y1="44" x2="58.2324" y2="43.677075" width="0.2" layer="1"/>
 <wire x1="58.2324" y1="44" x2="37.2324" y2="23" width="0.2" layer="1"/>
 <wire x1="37.2324" y1="23" x2="34" y2="23" width="0.2" layer="1"/>
@@
 <wire x1="55.88" y1="46.88" x2="55.88" y2="47.88" width="0.2" layer="1"/>
 </signal>
-<signal name="N$6">
-<contactref element="U1" pad="2"/>
-<contactref element="F1" pad="2"/>
-<contactref element="R1" pad="2"/>
-<wire x1="14.365" y1="21.4" x2="14.365" y2="21" width="0.5" layer="1"/>
-<wire x1="14.365" y1="21" x2="14.365" y2="18.635" width="0.5" layer="1"/>
-<wire x1="14.365" y1="18.635" x2="15" y2="18" width="0.5" layer="1"/>
-<wire x1="15" y1="18" x2="19" y2="18" width="0.5" layer="1"/>
-<wire x1="19" y1="18" x2="25" y2="24" width="0.5" layer="1"/>
-<wire x1="25" y1="24" x2="25" y2="25.05" width="0.5" layer="1"/>
-<wire x1="10.85" y1="34" x2="13.7812125" y2="34" width="0.2" layer="1"/>
-<wire x1="14.9174" y1="32.8638125" x2="13.7812125" y2="34" width="0.2" layer="1"/>
-<wire x1="14.9174" y1="32.8638125" x2="14.9174" y2="25.39545" width="0.2" layer="1"/>
-<wire x1="14.365" y1="24.84305" x2="14.365" y2="21" width="0.2" layer="1"/>
-<wire x1="14.9174" y1="25.39545" x2="14.365" y2="24.84305" width="0.2" layer="1"/>
-</signal>
 <signal name="N$7">
 <contactref element="U2" pad="2"/>
@@
 <wire x1="5" y1="12.7" x2="3" y2="10.7" width="0.6" layer="1"/>
 </signal>
+<signal name="N$1">
+<contactref element="U1" pad="2"/>
+<contactref element="F1" pad="2"/>
+<contactref element="R1" pad="2"/>
+<wire x1="14.365" y1="21" x2="14.365" y2="18.635" width="0.5" layer="1"/>
+<wire x1="14.365" y1="18.635" x2="15" y2="18" width="0.5" layer="1"/>
+<wire x1="15" y1="18" x2="19" y2="18" width="0.5" layer="1"/>
+<wire x1="19" y1="18" x2="25" y2="24" width="0.5" layer="1"/>
+<wire x1="25" y1="24" x2="25" y2="25.05" width="0.5" layer="1"/>
+<wire x1="10.85" y1="34" x2="13.7812125" y2="34" width="0.2" layer="1"/>
+<wire x1="14.9174" y1="32.8638125" x2="13.7812125" y2="34" width="0.2" layer="1"/>
+<wire x1="14.9174" y1="32.8638125" x2="14.9174" y2="25.39545" width="0.2" layer="1"/>
+<wire x1="14.365" y1="24.84305" x2="14.365" y2="21" width="0.2" layer="1"/>
+<wire x1="14.9174" y1="25.39545" x2="14.365" y2="24.84305" width="0.2" layer="1"/>
+<wire x1="14.365" y1="21.4" x2="14.365" y2="21" width="0.1524" layer="1"/>
+</signal>
 </signals>
 <mfgpreviewcolors>
@@
 </drawing>
 <compatibility>
+<note version="6.3" minversion="6.2.2" severity="warning">
+Since Version 6.2.2 text objects can contain more than one line,
+which will not be processed correctly with this version.
+</note>
 <note version="8.2" severity="warning">
 Since Version 8.2, EAGLE supports online libraries. The ids

Commit message: Fixed Stylistic issues and parts associations
Parts:
- removed U$1: PJ-037A, RoboJackets-Connectors:PJ-037A
- added J3: 1X2-3.5MM, adafruit:1X2-3.5MM
- C1: value 0.1uF -> 0.1uF 16V
- C2: value 1uF -> 1uF 16V
- C3: value 0.1uF -> 0.1uF 6V
- J1: value 1X2-3.5MM -> MAIN_PWR; device adafruit:1X2-3.5MM -> RoboJackets-Connectors:PJ-037A
- LED4, LED5: value (none) -> GREEN
- SW1: value 400AWMDP1R1M2 -> (none)
- moved J1 14.0 mm to (4.00, 42.0), turned to 0 degrees
- renumbered 12V_OK to LED3, F1_OK to LED4, F2_OK to LED5
Connections:
- removed net N$5: C3.1, Q1.RESET, R4.1, U$2.P$3, U$2.P$4
- new net N$4: C3.1, R4.1, U$2.P$3, U$2.P$4
- net +12V: now also J1.P$2; no longer U$1.P$2
- net GND: now also J1.P$1; no longer U$1.P$1
- net M1+: now also SW1.4; no longer SW1.P$4
- net M1+_SW: now also J3.1, SW1.5; no longer J1.1, SW1.P$5
- net M1_FWD: now also Q1.D10; no longer Q1.D4
- net M1_REV: now also Q1.D11; no longer Q1.D5
- net M2-: now also SW1.3; no longer SW1.P$3
- net M2-_SW: now also SW1.2; no longer SW1.P$2
- net M2_FWD: now also Q1.D5; no longer Q1.D2
- net M2_REV: now also Q1.D6; no longer Q1.D3
- net N$2: now also J3.2; no longer J1.2
Routing:
- net N$5: track 19.6 -> 0.00 mm
- net N$4: track 0.00 -> 17.1 mm
- net M1_REV: track 47.6 -> 31.3 mm, vias 2 -> 1
- net M1_FWD: track 53.9 -> 37.5 mm, vias 2 -> 1
- net GND: track 47.3 -> 39.6 mm, vias 10 -> 13
- net M2_REV: track 57.2 -> 54.0 mm
- net M2_FWD: track 64.5 -> 61.3 mm
- net N$1: track 33.8 -> 31.8 mm
Other:
- board size 68.7 x 53.3 mm -> 68.6 x 53.4 mm

Commit message: Added manufacturing files and Component list
Parts:
- renumbered U$2 to SW2
Other:
- board text added: "2019 Training Board V1.2"
- board text added: "Fuse Ok"
- board text added: "POWER"
- board text removed: "2019 Training Board V1.0"
Changed lines of the file:
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@@
 <drawing>
 <settings>
-<setting alwaysvectorfont="no"/>
+<setting alwaysvectorfont="yes"/>
 <setting verticaltext="up"/>
 </settings>
@@
 <wire x1="0" y1="53.4" x2="0" y2="0" width="0" layer="20"/>
 <text x="37" y="22" size="1.5" layer="112">2019 Training Board
-V1.0</text>
+V1.2</text>
 <polygon width="0.1524" layer="112">
 <vertex x="42" y="22"/>
@@
 <vertex x="42" y="15"/>
 </polygon>
+<text x="1.4" y="0.6" size="1" layer="21">Fuse Ok</text>
+<text x="4" y="32" size="1" layer="21">Fuse Ok</text>
+<text x="3" y="51" size="1.2" layer="21">POWER</text>
 </plain>
 <attributes>
@@
 </element>
 <element name="J1" library="RoboJackets-Connectors" package="PJ-037A" value="MAIN_PWR" x="4" y="42" smashed="yes"/>
-<element name="U$2" library="RoboJackets-Switches" package="PTS645" value="PTS645" x="36" y="12" smashed="yes">
+<element name="SW2" library="RoboJackets-Switches" package="PTS645" value="PTS645" x="36" y="12" smashed="yes">
 <attribute name="FUNCTION" value="RESET" x="36" y="12" size="1.778" layer="27" display="off"/>
 </element>
@@
 <contactref element="J1" pad="P$1"/>
 <contactref element="Q1" pad="GND1"/>
-<contactref element="U$2" pad="P$2"/>
-<contactref element="U$2" pad="P$1"/>
+<contactref element="SW2" pad="P$2"/>
+<contactref element="SW2" pad="P$1"/>
 <contactref element="U1" pad="8"/>
 <contactref element="LED3" pad="C"/>
@@
 </signal>
 <signal name="N$4">
-<contactref element="U$2" pad="P$3"/>
-<contactref element="U$2" pad="P$4"/>
+<contactref element="SW2" pad="P$3"/>
+<contactref element="SW2" pad="P$4"/>
 <contactref element="R4" pad="1"/>
 <contactref element="C3" pad="1"/>

Commit message: Removed 1 motor driver chip from training board
Parts:
- removed F2: 350 mA, RoboJackets-Fuses:F1812
- removed J2: 1X2-3.5MM, adafruit:1X2-3.5MM
- removed LED5: GREEN, led:CHIP-LED0603
- removed SW1: (no value), RoboJackets-Switches:400AWMDP1R1M2
- removed U2: ZXBM5210-S-13, RoboJackets-ICs:SOIC-8
- added Q2: DMN2056U, RoboJackets-Discrete:SOT-23-3
- added S1: (no value), adafruit:EG1218
- R6: value 2.4K -> 10K
- moved LED4 29.3 mm to (3.50, 4.81)
- moved R1 29.3 mm to (7.50, 4.81)
- moved C1 18.0 mm to (4.62, 35.2), turned to 90 degrees
- moved R6 15.6 mm to (12.3, 20.4), turned to 180 degrees
- moved J1 14.5 mm to (3.43, 27.5)
- moved U1 14.0 mm to (19.2, 10.7)
- moved J3 13.0 mm to (2.51, 15.0)
- moved C2 9.64 mm to (10.6, 35.2), turned to 90 degrees
- moved LED3 7.21 mm to (6.06, 41.9)
- moved R5 7.21 mm to (10.1, 41.9)
Connections:
- removed net M1+: SW1.4, U1.1
- removed net M2-: SW1.3, U2.7
- removed net M2-_SW: J2.2, SW1.2
- removed net N$7: F2.2, R6.2, U2.2
- removed net N$9: LED5.A, R6.1
- new net N$5: Q2.1, R6.1, S1.S
- net +12V: now also S1.P; no longer F2.1, U2.3, U2.6
- net GND: now also Q2.2, R6.2; no longer LED5.C, U1.8, U2.8
- net M1+_SW: now also U1.1; no longer SW1.5
- net M2_FWD: no longer U2.4
- net M2_REV: no longer U2.5
- net N$3: now also Q2.3, U1.8; no longer J2.1, U2.1
Routing:
- net M2_FWD: track 61.3 -> 0.00 mm, vias 2 -> 0
- net M2_REV: track 54.0 -> 0.00 mm, vias 2 -> 0
- net N$7: track 21.1 -> 0.00 mm
- net N$5: track 0.00 -> 13.9 mm, vias 0 -> 2
- net N$1: track 31.8 -> 43.9 mm
- net M1_FWD: track 37.5 -> 49.4 mm
- net M1_REV: track 31.3 -> 42.9 mm
- net M1+_SW: track 5.49 -> 16.9 mm
- net N$3: track 11.9 -> 1.94 mm
- net M2-: track 9.20 -> 0.00 mm
- net M1+: track 6.82 -> 0.00 mm
- net M2-_SW: track 6.59 -> 0.00 mm
- net +12V: track 120.0 -> 114.2 mm
- net N$2: track 14.1 -> 18.1 mm
- net N$9: track 2.81 -> 0.00 mm
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Other:
- board text added: "OFF"
- board text added: "ON"
