File: board/training_board.brd (EAGLE design)
At the start: 68.6 x 53.4 mm, 23 parts, among them J1 MAIN_PWR, J3 1X2-3.5MM, Q1 ARDUINOR3-NOIOREF-NOTEXT, Q2 DMN2056U, SW2 PTS645, U1 ZXBM5210-S-13

Commit message: Fixed reset issue and adjusted traces:
Parts:
- LED1, LED2: value YELLOW -> ORANGE
- moved R4 0.67 mm to (36.0, 6.33)
- renumbered J3 to OUT
Connections:
- removed net M2_FWD: Q1.D5
- removed net M2_REV: Q1.D6
- removed net N$4: C3.1, R4.1, SW2.P$3, SW2.P$4
- new net RESET: C3.1, Q1.RESET, R4.1, SW2.P$3, SW2.P$4
Routing:
- net RESET: track 0.00 -> 21.6 mm
- net N$4: track 17.1 -> 0.00 mm
- net +5V: track 4.98 -> 4.31 mm
Other:
- board text added: "2020 Training Board V1.3"
- board text added: "Reset"
- board text removed: "2019 Training Board V1.2"
Changed lines of the file:
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@@
 <?xml version="1.0" encoding="utf-8"?>
 <!DOCTYPE eagle SYSTEM "eagle.dtd">
-<eagle version="9.5.2">
+<eagle version="9.6.1">
 <drawing>
 <settings>
@@
 <wire x1="64.5" y1="53.4" x2="0" y2="53.4" width="0" layer="20"/>
 <wire x1="0" y1="53.4" x2="0" y2="0" width="0" layer="20"/>
-<text x="37" y="22" size="1.5" layer="112">2019 Training Board
-V1.2</text>
+<text x="37" y="22" size="1.5" layer="112">2020 Training Board
+V1.3</text>
 <polygon width="0.1524" layer="112">
 <vertex x="42" y="22"/>
@@
 <vertex x="42" y="15"/>
 </polygon>
-<text x="1.5" y="2.81" size="1" layer="21">Fuse Ok</text>
-<text x="2.06" y="43.85" size="1.2" layer="21">POWER</text>
+<text x="1.5" y="2.81" size="1.27" layer="25" font="vector">Fuse Ok</text>
+<text x="2.06" y="43.85" size="1.27" layer="25" font="vector">POWER</text>
 <text x="15.52" y="18.23" size="1.778" layer="21">ON</text>
 <text x="15.28" y="32.93" size="1.778" layer="21">OFF</text>
+<text x="33.5" y="15.25" size="1.27" layer="25" font="vector" align="bottom-center">Reset</text>
 </plain>
 <attributes>
@@
 <attribute name="VALUE" x="21.825" y="28.905" size="1.27" layer="27" rot="R270"/>
 </element>
-<element name="J3" library="adafruit" library_urn="urn:adsk.eagle:library:420" package="1X2-3.5MM" package3d_urn="urn:adsk.eagle:package:6240635/1" value="1X2-3.5MM" x="2.51" y="14.96" smashed="yes" rot="R270">
+<element name="OUT" library="adafruit" library_urn="urn:adsk.eagle:library:420" package="1X2-3.5MM" package3d_urn="urn:adsk.eagle:package:6240635/1" value="1X2-3.5MM" x="2.51" y="14.96" smashed="yes" rot="R270">
 <attribute name="NAME" x="7.51" y="11.96" size="1.27" layer="25" rot="R90" display="off"/>
 </element>
-<element name="LED1" library="led" library_urn="urn:adsk.eagle:library:259" package="CHIP-LED0603" package3d_urn="urn:adsk.eagle:package:15819/3" value="YELLOW" x="31" y="45" smashed="yes" rot="R90">
+<element name="LED1" library="led" library_urn="urn:adsk.eagle:library:259" package="CHIP-LED0603" package3d_urn="urn:adsk.eagle:package:15819/3" value="ORANGE" x="31" y="45" smashed="yes" rot="R90">
 <attribute name="NAME" x="31.635" y="44.365" size="1.27" layer="25" rot="R180"/>
 <attribute name="VALUE" x="31.635" y="46.905" size="1.27" layer="27" rot="R180" display="off"/>
 </element>
-<element name="LED2" library="led" library_urn="urn:adsk.eagle:library:259" package="CHIP-LED0603" package3d_urn="urn:adsk.eagle:package:15819/3" value="YELLOW" x="31" y="39" smashed="yes" rot="R90">
+<element name="LED2" library="led" library_urn="urn:adsk.eagle:library:259" package="CHIP-LED0603" package3d_urn="urn:adsk.eagle:package:15819/3" value="ORANGE" x="31" y="39" smashed="yes" rot="R90">
 <attribute name="NAME" x="31.635" y="38.365" size="1.27" layer="25" rot="R180"/>
 <attribute name="VALUE" x="31.635" y="40.905" size="1.27" layer="27" rot="R180" display="off"/>
@@
 <attribute name="VALUE" x="36.365" y="43.095" size="1.27" layer="27"/>
 </element>
-<element name="R4" library="rcl" library_urn="urn:adsk.eagle:library:334" package="R0603" package3d_urn="urn:adsk.eagle:package:23555/3" value="10K" x="36" y="7" smashed="yes">
-<attribute name="NAME" x="35.365" y="7.635" size="1.27" layer="25"/>
-<attribute name="SPICEPREFIX" value="R" x="36" y="7" size="1.778" layer="27" display="off"/>
-<attribute name="VALUE" x="35.365" y="5.095" size="1.27" layer="27"/>
+<element name="R4" library="rcl" library_urn="urn:adsk.eagle:library:334" package="R0603" package3d_urn="urn:adsk.eagle:package:23555/3" value="10K" x="36" y="6.33" smashed="yes">
+<attribute name="NAME" x="36" y="7" size="1.27" layer="25" align="bottom-center"/>
+<attribute name="SPICEPREFIX" value="R" x="36" y="6.33" size="1.778" layer="27" display="off"/>
+<attribute name="VALUE" x="36" y="5.66" size="1.27" layer="27" align="top-center"/>
 </element>
 <element name="R5" library="rcl" library_urn="urn:adsk.eagle:library:334" package="R0603" package3d_urn="urn:adsk.eagle:package:23555/3" value="2.4K" x="10.06" y="41.85" smashed="yes">
@@
 </element>
 <element name="C3" library="rcl" library_urn="urn:adsk.eagle:library:334" package="C0805" package3d_urn="urn:adsk.eagle:package:23617/2" value="0.1uF 6V" x="29" y="5" smashed="yes" rot="R180">
-<attribute name="NAME" x="30.27" y="3.73" size="1.27" layer="25" rot="R180"/>
+<attribute name="NAME" x="29" y="4" size="1.27" layer="27" font="vector" align="top-center"/>
 <attribute name="SPICEPREFIX" value="C" x="29" y="5" size="1.778" layer="27" rot="R180" display="off"/>
-<attribute name="VALUE" x="30.27" y="7.54" size="1.27" layer="27" rot="R180"/>
+<attribute name="VALUE" x="29" y="6" size="1.27" layer="25" font="vector" align="bottom-center"/>
 </element>
 <element name="U$3" library="RoboJackets-Aesthetics" package="ROBOJACKETS" value="" x="37" y="27" smashed="yes"/>
@@
 <signal name="+5V">
 <contactref element="R4" pad="2"/>
+<wire x1="36.85" y1="6.33" x2="38.1" y2="5.08" width="0.2" layer="1"/>
 <contactref element="Q1" pad="5V"/>
-<wire x1="38.1" y1="5.75" x2="38.1" y2="2.54" width="0.2" layer="1"/>
-<wire x1="36.85" y1="7" x2="38.1" y2="5.75" width="0.2" layer="1"/>
+<wire x1="38.1" y1="5.08" x2="38.1" y2="2.54" width="0.2" layer="1"/>
 </signal>
 <signal name="M1_FWD">
@@
 <wire x1="21.135" y1="13.625" x2="21.135" y2="13.25" width="0.2" layer="1"/>
 </signal>
-<signal name="M2_FWD">
-<contactref element="Q1" pad="D5"/>
-</signal>
-<signal name="M2_REV">
-<contactref element="Q1" pad="D6"/>
-</signal>
 <signal name="N$14">
 <contactref element="LED1" pad="A"/>
@@
 </signal>
 <signal name="N$2">
-<contactref element="J3" pad="2"/>
+<contactref element="OUT" pad="2"/>
 <contactref element="U1" pad="7"/>
 <wire x1="16.4" y1="16.4" x2="18.44" y2="14.36" width="0.6" layer="1"/>
@@
 </signal>
 <signal name="M1+_SW">
-<contactref element="J3" pad="1"/>
+<contactref element="OUT" pad="1"/>
 <contactref element="U1" pad="1"/>
 <wire x1="17.325" y1="8.05" x2="17.31" y2="8.05" width="0.6" layer="1"/>
@@
 <wire x1="18.615" y1="8.03" x2="18.615" y2="5.16" width="0.6" layer="1"/>
 </signal>
-<signal name="N$4">
-<contactref element="SW2" pad="P$3"/>
-<contactref element="SW2" pad="P$4"/>
-<contactref element="R4" pad="1"/>
-<contactref element="C3" pad="1"/>
-<wire x1="40.025" y1="9.75" x2="36" y2="9.75" width="0.5" layer="1"/>
-<wire x1="36" y1="9.75" x2="32.025" y2="9.75" width="0.5" layer="1"/>
-<wire x1="35.15" y1="7" x2="35.15" y2="8.9" width="0.5" layer="1"/>
-<wire x1="35.15" y1="8.9" x2="36" y2="9.75" width="0.5" layer="1"/>
-<wire x1="33.15" y1="5" x2="35.15" y2="7" width="0.2" layer="1"/>
-<wire x1="29.95" y1="5" x2="33.15" y2="5" width="0.2" layer="1"/>
-</signal>
 <signal name="N$3">
 <contactref element="U1" pad="8"/>
@@
 <wire x1="12.42" y1="14.57" x2="13.14" y2="14.57" width="0.2" layer="1"/>
 </signal>
+<signal name="RESET">
+<contactref element="Q1" pad="RESET"/>
+<contactref element="SW2" pad="P$3"/>
+<contactref element="SW2" pad="P$4"/>
+<contactref element="R4" pad="1"/>
+<contactref element="C3" pad="1"/>
+<wire x1="40.025" y1="9.75" x2="36" y2="9.75" width="0.5" layer="1"/>
+<wire x1="36" y1="9.75" x2="32.025" y2="9.75" width="0.5" layer="1"/>
+<wire x1="35.15" y1="6.33" x2="35.15" y2="8.9" width="0.5" layer="1"/>
+<wire x1="35.15" y1="8.9" x2="36" y2="9.75" width="0.5" layer="1"/>
+<wire x1="35.15" y1="6.33" x2="33.82" y2="5" width="0.5" layer="1"/>
+<wire x1="33.82" y1="5" x2="29.95" y2="5" width="0.5" layer="1"/>
+<wire x1="29.95" y1="5" x2="32.41" y2="2.54" width="0.5" layer="1"/>
+<wire x1="32.41" y1="2.54" x2="33.02" y2="2.54" width="0.5" layer="1"/>
+</signal>
 </signals>
