File: board/training_board.brd (EAGLE design)
At the start: 68.6 x 53.4 mm, 23 parts, among them J1 MAIN_PWR, Q1 ARDUINOR3-NOIOREF-NOTEXT, Q2 DMN2056U, SW2 PTS645, U1 ZXBM5210-S-13

Commit message: Updated board version and removed old image and gerbers
Changed lines of the file:
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@@
 <text x="1.5" y="2.81" size="1.27" layer="25" font="vector">Fuse Ok</text>
 <text x="2.06" y="43.85" size="1.27" layer="25" font="vector">POWER</text>
-<text x="15.52" y="18.23" size="1.778" layer="21">ON</text>
-<text x="15.28" y="32.93" size="1.778" layer="21">OFF</text>
-<text x="33.5" y="15.25" size="1.27" layer="25" font="vector" align="bottom-center">Reset</text>
+<text x="17.48" y="18.45" size="1.5" layer="112" font="vector" align="bottom-center">ON</text>
+<text x="17.48" y="34.45" size="1.5" layer="112" font="vector" align="top-center">OFF</text>
+<text x="36" y="15.5" size="1.27" layer="25" font="vector" align="bottom-center">Reset</text>
 </plain>
 <attributes>
@@
 </element>
 <element name="LED1" library="led" library_urn="urn:adsk.eagle:library:259" package="CHIP-LED0603" package3d_urn="urn:adsk.eagle:package:15819/3" value="ORANGE" x="31" y="45" smashed="yes" rot="R90">
-<attribute name="NAME" x="31.635" y="44.365" size="1.27" layer="25" rot="R180"/>
+<attribute name="NAME" x="31" y="44" size="1.27" layer="27" font="vector" align="top-center"/>
 <attribute name="VALUE" x="31.635" y="46.905" size="1.27" layer="27" rot="R180" display="off"/>
 </element>
 <element name="LED2" library="led" library_urn="urn:adsk.eagle:library:259" package="CHIP-LED0603" package3d_urn="urn:adsk.eagle:package:15819/3" value="ORANGE" x="31" y="39" smashed="yes" rot="R90">
-<attribute name="NAME" x="31.635" y="38.365" size="1.27" layer="25" rot="R180"/>
+<attribute name="NAME" x="31" y="38" size="1.27" layer="27" font="vector" align="top-center"/>
 <attribute name="VALUE" x="31.635" y="40.905" size="1.27" layer="27" rot="R180" display="off"/>
 </element>
@@
 </element>
 <element name="R2" library="rcl" library_urn="urn:adsk.eagle:library:334" package="R0603" package3d_urn="urn:adsk.eagle:package:23555/3" value="1K" x="37" y="39" smashed="yes">
-<attribute name="NAME" x="36.365" y="39.635" size="1.27" layer="25"/>
+<attribute name="NAME" x="37" y="40" size="1.27" layer="25" font="vector" align="bottom-center"/>
 <attribute name="SPICEPREFIX" value="R" x="37" y="39" size="1.778" layer="27" display="off"/>
-<attribute name="VALUE" x="36.365" y="37.095" size="1.27" layer="27"/>
+<attribute name="VALUE" x="37" y="38" size="1.27" layer="27" font="vector" align="top-center"/>
 </element>
 <element name="R3" library="rcl" library_urn="urn:adsk.eagle:library:334" package="R0603" package3d_urn="urn:adsk.eagle:package:23555/3" value="1K" x="37" y="45" smashed="yes">
-<attribute name="NAME" x="36.365" y="45.635" size="1.27" layer="25"/>
+<attribute name="NAME" x="37" y="46" size="1.27" layer="25" align="bottom-center"/>
 <attribute name="SPICEPREFIX" value="R" x="37" y="45" size="1.778" layer="27" display="off"/>
-<attribute name="VALUE" x="36.365" y="43.095" size="1.27" layer="27"/>
+<attribute name="VALUE" x="37" y="44" size="1.27" layer="27" font="vector" align="top-center"/>
 </element>
 <element name="R4" library="rcl" library_urn="urn:adsk.eagle:library:334" package="R0603" package3d_urn="urn:adsk.eagle:package:23555/3" value="10K" x="36" y="6.33" smashed="yes">
-<attribute name="NAME" x="36" y="7" size="1.27" layer="25" align="bottom-center"/>
+<attribute name="NAME" x="36" y="7.33" size="1.27" layer="25" align="bottom-center"/>
 <attribute name="SPICEPREFIX" value="R" x="36" y="6.33" size="1.778" layer="27" display="off"/>
-<attribute name="VALUE" x="36" y="5.66" size="1.27" layer="27" align="top-center"/>
+<attribute name="VALUE" x="36" y="5.33" size="1.27" layer="27" align="top-center"/>
 </element>
 <element name="R5" library="rcl" library_urn="urn:adsk.eagle:library:334" package="R0603" package3d_urn="urn:adsk.eagle:package:23555/3" value="2.4K" x="10.06" y="41.85" smashed="yes">
@@
 </element>
 <element name="R1" library="rcl" library_urn="urn:adsk.eagle:library:334" package="R0603" package3d_urn="urn:adsk.eagle:package:23555/3" value="2.4K" x="7.5" y="4.81" smashed="yes">
-<attribute name="NAME" x="6.865" y="5.445" size="1.27" layer="25"/>
+<attribute name="NAME" x="6.865" y="6" size="1.27" layer="25" font="vector" align="bottom-center"/>
 <attribute name="SPICEPREFIX" value="R" x="2.5" y="10.81" size="1.778" layer="27" display="off"/>
 <attribute name="VALUE" x="6.865" y="2.905" size="1.27" layer="27" display="off"/>

Commit message: Finished 1.3 rev silkscreen and layer fixes
Parts:
- moved R1 2.60 mm to (10.1, 4.78)
- moved J1 1.27 mm to (3.43, 26.2)
- moved R6 1.17 mm to (12.3, 19.2)
- moved R5 1.17 mm to (11.2, 41.9)
- moved LED4 0.50 mm to (4.00, 4.81)
Routing:
- net N$1: track 43.9 -> 39.9 mm
- net N$8: track 2.40 -> 5.44 mm
- net N$16: track 2.40 -> 3.57 mm
- net GND: track 40.6 -> 41.6 mm
- net +12V: track 114.2 -> 115.0 mm
Other:
- board text added: "FUSE OK"
- board text removed: "Fuse Ok"

Commit message: integrated DRV8871 into schematic and board
Parts:
- added R7: 128K, rcl:R0603
- U1: value ZXBM5210-S-13 -> DRV8871HSOP-8; device RoboJackets-ICs:SOIC-8 -> RoboJackets-ICs:SOIC127P600X170-9T240X310N
- moved U1 3.60 mm to (22.2, 12.7), turned to 180 degrees
- moved R6 3.57 mm to (8.78, 20.0)
- moved Q2 1.76 mm to (14.2, 11.9)
- moved SW2 1.24 mm to (37.1, 11.5)
- moved R1 0.99 mm to (10.6, 5.61)
- moved LED4 0.99 mm to (4.54, 5.64)
Connections:
- removed net M1+_SW: OUT.1, U1.1
- new net N$4: OUT.1, U1.8
- new net N$6: R7.1, U1.4
- net +12V: no longer U1.3, U1.6
- net GND: now also R7.2, SW2.1, SW2.2, U1.1, U1.9; no longer SW2.P$1, SW2.P$2
- net M1_FWD: now also U1.2; no longer U1.4
- net M1_REV: now also U1.3; no longer U1.5
- net N$1: now also U1.5; no longer U1.2
- net N$2: now also U1.6; no longer U1.7
- net N$3: now also U1.7; no longer U1.8
- net RESET: now also SW2.3, SW2.4; no longer SW2.P$3, SW2.P$4
Routing:
- net +12V: track 115.0 -> 92.6 mm
- net N$4: track 0.00 -> 20.3 mm
- net M1+_SW: track 16.9 -> 0.00 mm
- net N$1: track 39.9 -> 28.6 mm, vias 0 -> 2
- net N$5: track 13.4 -> 20.2 mm
- net GND: track 41.6 -> 46.1 mm, vias 11 -> 18
- net M1_FWD: track 49.4 -> 45.9 mm
- net N$6: track 0.00 -> 2.72 mm
- net N$3: track 1.94 -> 4.36 mm
- net M1_REV: track 42.9 -> 43.5 mm

Commit message: Library updates, slight routing changes
Parts:
- U1: device RoboJackets-ICs:SOIC127P600X170-9T240X310N -> RoboJackets-ICs:HSOP-8
Routing:
- net +12V: track 92.6 -> 91.1 mm
Changed lines of the file:
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@@
 <elements>
 <element name="Q1" library="adafruit" library_urn="urn:adsk.eagle:library:420" package="ARDUINOR3-NOTEXT-NOIOREF" package3d_urn="urn:adsk.eagle:package:6240888/1" value="ARDUINOR3-NOIOREF-NOTEXT" x="0" y="0" smashed="yes"/>
-<element name="U1" library="RoboJackets-ICs" package="SOIC127P600X170-9T240X310N" package3d_urn="urn:adsk.eagle:package:16996349/1" value="DRV8871HSOP-8" x="22.17" y="12.73" smashed="yes" rot="R180">
+<element name="U1" library="RoboJackets-ICs" package="HSOP-8" value="DRV8871HSOP-8" x="22.17" y="12.73" smashed="yes" rot="R180">
 <attribute name="DKPN" value="296-43024-1-ND" x="22.17" y="12.73" size="1.778" layer="27" rot="R180" display="off"/>
 <attribute name="NAME" x="25.17" y="12.73" size="1.27" layer="25" rot="R270" align="bottom-center"/>
@@
 <vertex x="21.04" y="16"/>
 </polygon>
-<wire x1="24.6434" y1="10.825" x2="24.5184" y2="10.7" width="0.3" layer="1"/>
-<wire x1="24.5184" y1="10.7" x2="22.89" y2="10.7" width="0.3" layer="1"/>
 <via x="20.85" y="8.93" extent="1-16" drill="0.35"/>
 <via x="22.1" y="8.93" extent="1-16" drill="0.35"/>
@@
 <via x="22.1" y="7.63" extent="1-16" drill="0.35"/>
 <via x="20.85" y="7.63" extent="1-16" drill="0.35"/>
+<wire x1="24.6434" y1="10.825" x2="23.105" y2="10.825" width="0.4" layer="1"/>
 </signal>
 <signal name="3V">
@@
 <wire x1="27.91" y1="27.04" x2="26" y2="28.95" width="0.4" layer="1"/>
 <wire x1="26" y1="28.95" x2="25" y2="28.95" width="0.4" layer="1"/>
-<wire x1="23.57" y1="28.95" x2="25" y2="28.95" width="0.6" layer="1"/>
 <wire x1="4.62" y1="34.28" x2="10.62" y2="34.28" width="0.8" layer="1"/>
 <wire x1="10.62" y1="34.28" x2="9.43" y2="33.09" width="0.8" layer="1"/>
@@
 <wire x1="10.62" y1="34.28" x2="19.67" y2="34.28" width="0.8" layer="1"/>
 <wire x1="19.67" y1="34.28" x2="25" y2="28.95" width="0.8" layer="1"/>
-<wire x1="25" y1="28.95" x2="19.98" y2="28.95" width="0.2" layer="1"/>
-<wire x1="19.98" y1="28.95" x2="17.48" y2="26.45" width="0.2" layer="1"/>
+<wire x1="17.48" y1="26.45" x2="19.98" y2="28.95" width="0.2" layer="1"/>
 <wire x1="13.63" y1="36.38" x2="11.53" y2="34.28" width="0.2" layer="1"/>
 <wire x1="11.53" y1="34.28" x2="10.62" y2="34.28" width="0.2" layer="1"/>
 <wire x1="12.08" y1="41.85" x2="13.63" y2="40.3" width="0.2" layer="1"/>
 <wire x1="13.63" y1="40.3" x2="13.63" y2="36.38" width="0.2" layer="1"/>
+<wire x1="19.98" y1="28.95" x2="25" y2="28.95" width="0.2" layer="1"/>
 </signal>
 <signal name="+5V">
@@
 <signal name="M1_FWD">
 <contactref element="Q1" pad="D10"/>
-<wire x1="36.576" y1="22.466" x2="36.576" y2="22.49" width="0.2" layer="16"/>
 <contactref element="U1" pad="2"/>
 <wire x1="36.576" y1="22.49" x2="36.576" y2="50.8" width="0.2" layer="16"/>
@@
 <mfgpreviewcolor name="substratecolor" color="0xFF786E46"/>
 </mfgpreviewcolors>
+<errors>
+</errors>
 </board>
 </drawing>

Commit message: Adjusted board to fix silkscreen overlapping pads
Parts:
- moved SW2 0.93 mm to (36.5, 12.2)
- moved R6 0.75 mm to (8.78, 19.2)
Routing:
- net RESET: track 21.5 -> 23.2 mm
- net N$5: track 20.2 -> 18.6 mm
- net GND: track 45.8 -> 46.7 mm
Other:
- board text added: "2020 Training Board V1.4"
- board text removed: "2020 Training Board V1.3"

Commit message: Fixed extra via and wire stub
Routing:
- net RESET: track 23.2 -> 22.3 mm
- net GND: vias 18 -> 17
