File: board/training_board.brd (EAGLE design)
At the start: 68.6 x 53.4 mm, 24 parts, among them J1 MAIN_PWR, Q1 DMN2056U, Q2 ARDUINOR3-NOIOREF-NOTEXT, SW1 PTS645, U1 DRV8871HSOP-8

Commit message: Changed DRV8871 for DRV8876
Parts:
- added C4, C5: 0.1 uF, Capacitor:CAPC1608X85
- added C6: 22 nF, Capacitor:CAPC1608X85
- added U2: DRV8876PWPRPWP0016J_NV, RoboJackets-ICs:PWP0016J_NV
- moved F1 75.7 mm to (-8.89, -40.6), turned to 0 degrees
- moved R7 63.7 mm to (-10.2, -54.6)
- moved LED4 58.3 mm to (-10.2, -50.8), turned to 0 degrees
Connections:
- new net N$12: C5.2, U2.12
- new net N$13: C6.1, U2.13
- new net N$17: C6.2, U2.14
- new net N$18: C4.1, C5.1, F1.2, U2.11
- new net N$7: R7.2
- new net N$9: Q1.3, U2.9
- new net PAD: U2.17
- net +5V: now also U2.16, U2.5
- net GND: now also C4.2, U2.15, U2.6, U2.7
- net M1_FWD: now also U2.2
- net M1_REV: now also U2.1
- net N$1: no longer F1.2, R7.2
- net N$2: now also U2.8; no longer U1.6
- net N$3: no longer Q1.3
- net N$4: now also U2.10; no longer U1.8
Routing:
- net N$4: track 20.3 -> 0.00 mm
- net N$2: track 18.6 -> 0.00 mm
- net +12V: track 91.1 -> 77.6 mm
- net N$8: track 5.44 -> 0.00 mm
- net N$1: track 29.8 -> 26.5 mm
- net GND: track 46.7 -> 44.9 mm, vias 17 -> 16

Commit message: Finished edits
Parts:
- removed Q1: DMN2056U, RoboJackets-Discrete:SOT-23-3
- removed R4: 10K, rcl:R0603
- removed R5: 120K, rcl:R0603
- removed U1: DRV8871HSOP-8, RoboJackets-ICs:HSOP-8
- added R8: 10k, rcl:R0603
- moved F1 80.1 mm to (25.4, 31.8)
- moved R7 61.3 mm to (3.81, 5.08), turned to 90 degrees
- moved LED4 57.4 mm to (7.62, 3.81), turned to 270 degrees
- moved C6 49.1 mm to (10.2, 12.7), turned to 270 degrees
- moved C5 38.6 mm to (10.2, 8.89), turned to 90 degrees
- moved C4 30.1 mm to (6.35, 8.89), turned to 270 degrees
- moved U2 27.4 mm to (16.5, 15.2), turned to 180 degrees
Connections:
- net N$12 renamed VCP
- net N$13 renamed CPH
- net N$17 renamed CPL
- net N$2 renamed OUT1
- net N$4 renamed OUT2
- removed net N$1: U1.5
- removed net N$18: C4.1, C5.1, F1.2, U2.11
- removed net N$3: U1.7
- removed net N$5: Q1.1, R4.1, S1.S
- removed net N$6: R5.1, U1.4
- removed net N$7: R7.2
- removed net N$9: Q1.3, U2.9
- removed net PAD: U2.17
- new net !SLEEP!: R8.1, S1.P, U2.3
- new net VM: C4.1, C5.1, F1.2, R7.2, U2.11
- net +12V: no longer S1.P
- net +5V: now also R8.2
- net GND: now also S1.S, U2.17, U2.9; no longer Q1.2, R4.2, R5.2, U1.1, U1.9
- net M1_FWD: no longer U1.2
- net M1_REV: no longer U1.3
Routing:
- net VM: track 0.00 -> 51.3 mm, vias 0 -> 2
- net +5V: track 4.31 -> 46.7 mm, vias 0 -> 2
- net N$1: track 26.5 -> 0.00 mm, vias 2 -> 0
- net !SLEEP!: track 0.00 -> 23.7 mm
- net N$5: track 18.6 -> 0.00 mm, vias 2 -> 0
- net OUT1: track 0.00 -> 18.4 mm
- net GND: track 44.9 -> 60.7 mm, vias 16 -> 17
- net OUT2: track 0.00 -> 12.6 mm
- net VCP: track 0.00 -> 10.7 mm
- net M1_REV: track 43.5 -> 50.0 mm
- net M1_FWD: track 46.3 -> 51.9 mm
- net +12V: track 77.6 -> 82.7 mm
- net CPL: track 0.00 -> 4.42 mm
- net CPH: track 0.00 -> 4.05 mm
- net N$3: track 4.03 -> 0.00 mm
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Other:
- board text added: "PON"

Commit message: Silkscreen edits
Other:
- board text added: "2022 Soldering Training Board"
- board text added: "RST"
- board text added: "v1.6"
- board text removed: "2020 Soldering Training Board"
- board text removed: ">VERSION"
Changed lines of the file:
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@@
 <drawing>
 <settings>
-<setting alwaysvectorfont="yes"/>
+<setting alwaysvectorfont="no"/>
 <setting verticaltext="up"/>
 </settings>
@@
 <layer number="25" name="tNames" color="7" fill="1" visible="yes" active="yes"/>
 <layer number="26" name="bNames" color="7" fill="1" visible="yes" active="yes"/>
-<layer number="27" name="tValues" color="7" fill="1" visible="no" active="yes"/>
+<layer number="27" name="tValues" color="7" fill="1" visible="yes" active="yes"/>
 <layer number="28" name="bValues" color="7" fill="1" visible="yes" active="yes"/>
 <layer number="29" name="tStop" color="7" fill="3" visible="no" active="yes"/>
@@
 <wire x1="64.5" y1="53.4" x2="0" y2="53.4" width="0" layer="20"/>
 <wire x1="0" y1="53.4" x2="0" y2="0" width="0" layer="20"/>
-<text x="37" y="22" size="1.5" layer="21" font="vector">2020 Soldering Training Board
+<text x="37" y="22" size="1.5" layer="21" font="vector">2022 Soldering Training Board
 </text>
 <text x="4.61" y="6.61" size="1" layer="27" font="vector" align="bottom-center">FUSE OK</text>
@@
 <text x="17.48" y="33.45" size="1" layer="51" font="vector" ratio="15" align="top-center">ON</text>
 <text x="36.5" y="15.65" size="1" layer="25" font="vector" align="bottom-center">Reset</text>
-<text x="37" y="22" size="1.5" layer="21" font="vector">&gt;VERSION</text>
+<text x="37" y="22" size="1.5" layer="21" font="vector">v1.6</text>
 <text x="6.223" y="1.778" size="1.27" layer="21" font="vector" ratio="15">PON</text>
+<text x="31.75" y="3.81" size="1" layer="21" font="vector" ratio="15">RST</text>
 </plain>
 <attributes>
