File: board/training_board.sch (EAGLE design)
At the start: 0 parts

Commit message: Preliminary Schematic completed.  Components arranged and not routed on board.
Parts:
- added F1, F2: 350 mA, RoboJackets-Fuses:CHIP_FUSE1812
- added J1, J2: 1X2-3.5MM, adafruit:1X2-3.5MM
- added LED1, LED2: YELLOW, led:LEDCHIP-LED0603
- added LED3: RED, led:LEDCHIP-LED0603
- added Q1: ARDUINOR3-NOIOREF-NOTEXT, adafruit:ARDUINOR3-NOIOREF-NOTEXT
- added R2, R3: 1k O, rcl:R-US_R0603
- added R4: 10k O, rcl:R-US_R0603
- added R5: 240 O, rcl:R-US_R0603
- added U$1: PJ-037A, RoboJackets-Connectors:PJ-037A
- added U$2: PTS645, RoboJackets-Switches:PTS645
- added U1, U2: ZXBM5210-S-13, RoboJackets-ICs:ZXBM5210-S-13
Connections:
- new net +12V: F1.1, F2.1, Q1.VIN, R5.2, U$1.1, U1.V_DD, U1.V_REF, U2.V_DD, U2.V_REF
- new net +5V: Q1.5V, R2.2, R3.2, R4.2
- new net GND: LED3.C, Q1.GND1, Q1.GND2, U$1.2, U$2.1, U1.GND, U2.GND
- new net M1_FWD: Q1.D2, U1.FWD
- new net M1_REV: Q1.D3, U1.REV
- new net M2_FWD: Q1.D4, U2.FWD
- new net M2_REV: Q1.D5, U2.REV
- new net N$1: J1.1, U1.OUT1
- new net N$12: LED1.C, Q1.D8
- new net N$13: LED2.C, Q1.D9
- new net N$14: LED1.A, R3.1
- new net N$15: LED2.A, R2.1
- new net N$16: LED3.A, R5.1
- new net N$2: J1.2, U1.OUT2
- new net N$3: J2.1, U2.OUT1
- new net N$4: J2.2, U2.OUT2
- new net N$5: Q1./RESET, R4.1, U$2.2
- new net N$6: F1.2, U1.V_M
- new net N$7: F2.2, U2.V_M
Other:
- note added: "350mA fuse specced for Sparkfun Gearmotors with .35A no-load current and 1.3A stall current"
- note added: "7-12V from the Barrel Jack is fed into the Vin pin on the Arduino Uno so the internal regulator provides 5V to power the logic levels in the circuit."
- note added: "Arduino Uno Microcontroller"
- note added: "Barrel Jack and 12V Power Indicator"
- note added: "From Adafruit Library"
- note added: "Microcontroller code resets when RESET pin is shorted to ground. This is accomplished with a momentary pushbutton. A 10k ohm pull-up resistor ensures the RESET pin is high when the pushbutton is an open circuit."
- note added: "Motor Driver Chips"
- note added: "Motor Driver chips are powered directly from the 12V supply. V_REF is connected to 12V so speed can be controlled by applying a PWM signal to the M2_FWD or M2_REV pins. The output of the internal H Bridge is applied across OUT1 and OUT2."
- note added: "Two user controlled LEDs are provided in common cathode configuration. Sending a logic '0' to these pins will cause the LED to turn on."

Commit message: Added Preliminary Board layout
Parts:
- added F1_OK, F2_OK: (no value), led:LEDCHIP-LED0603
- added R1, R6: 2.4K, rcl:R-US_R0603
- added SW1: 400AWMDP1R1M2, RoboJackets-Switches:400AWMDP1R1M2
- 12V_OK: value RED -> GREEN
- R2, R3: value 1k O -> 1K
- R4: value 10k O -> 10K
- R5: value 240 O -> 2.4K
- renumbered LED3 to 12V_OK
Connections:
- removed net N$1: J1.1, U1.OUT1
- removed net N$12: LED1.C, Q1.D8
- removed net N$13: LED2.C, Q1.D9
- removed net N$4: J2.2, U2.OUT2
- new net M1+: SW1.NO2, U1.OUT1
- new net M1+_SW: J1.1, SW1.C2
- new net M2-: SW1.NO1, U2.OUT2
- new net M2-_SW: J2.2, SW1.C1
- new net N$10: Q1.D9, R3.2
- new net N$11: Q1.D8, R2.2
- new net N$8: F1_OK.A, R1.1
- new net N$9: F2_OK.A, R6.1
- net +5V: no longer R2.2, R3.2
- net GND: now also F1_OK.C, F2_OK.C, LED1.C, LED2.C
- net M1_FWD: now also Q1.D4; no longer Q1.D2
- net M1_REV: now also Q1.D5; no longer Q1.D3
- net M2_FWD: now also Q1.D2; no longer Q1.D4
- net M2_REV: now also Q1.D3; no longer Q1.D5
- net N$6: now also R1.2
- net N$7: now also R6.2
Other:
- note added: "The top part of this symbol represents the pin inside the barrel jack (usually positive), while the bottom represents the spring-loaded tab that contacts the outside (usually negative)."
- note added: "Two user controlled LEDs are provided in common anode configuration. Sending a logic '1' to these pins will cause the LED to turn on."
- note removed: "Two user controlled LEDs are provided in common cathode configuration. Sending a logic '0' to these pins will cause the LED to turn on."
- moved on the sheet: LED1, LED2, R2, R3

Commit message: Added Week 0 content to references folder
Parts:
- added C1, C3: 0.1uF, rcl:C-USC0805
- added C2: 1uF, rcl:C-USC0805
- U$2: FUNCTION (none) -> RESET
Connections:
- net +12V: now also C1.1, C2.1
- net GND: now also C1.2, C2.2, C3.2
- net N$5: now also C3.1
Other:
- note added: "Decoupling capacitors help ensure a relatively constant output voltage even in the event of current spikes"
- moved on the sheet: 12V_OK, R5
Changed lines of the file:
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@@
 <part name="SUPPLY7" library="supply2" library_urn="urn:adsk.eagle:library:372" deviceset="GND" device=""/>
 <part name="SUPPLY9" library="supply2" library_urn="urn:adsk.eagle:library:372" deviceset="GND" device=""/>
-<part name="U$2" library="RoboJackets-Switches" deviceset="PTS645" device=""/>
+<part name="U$2" library="RoboJackets-Switches" deviceset="PTS645" device="">
+<attribute name="FUNCTION" value="RESET"/>
+</part>
 <part name="SUPPLY8" library="supply2" library_urn="urn:adsk.eagle:library:372" deviceset="GND" device=""/>
 <part name="SUPPLY10" library="supply2" library_urn="urn:adsk.eagle:library:372" deviceset="GND" device=""/>
@@
 <part name="SUPPLY4" library="supply2" library_urn="urn:adsk.eagle:library:372" deviceset="GND" device=""/>
 <part name="SW1" library="RoboJackets-Switches" deviceset="400AWMDP1R1M2" device=""/>
+<part name="C1" library="rcl" library_urn="urn:adsk.eagle:library:334" deviceset="C-US" device="C0805" package3d_urn="urn:adsk.eagle:package:23617/2" value="0.1uF"/>
+<part name="C2" library="rcl" library_urn="urn:adsk.eagle:library:334" deviceset="C-US" device="C0805" package3d_urn="urn:adsk.eagle:package:23617/2" value="1uF"/>
+<part name="C3" library="rcl" library_urn="urn:adsk.eagle:library:334" deviceset="C-US" device="C0805" package3d_urn="urn:adsk.eagle:package:23617/2" value="0.1uF"/>
 </parts>
 <sheets>
@@
 Gearmotors with .35A no-load current and
 1.3A stall current</text>
-<text x="12.7" y="142.24" size="1.778" layer="97">The top part of this symbol represents the pin inside the
+<text x="17.78" y="142.24" size="1.778" layer="97">The top part of this symbol represents the pin inside the
 barrel jack (usually positive), while the
 bottom represents the spring-loaded tab
 that contacts the outside (usually negative).  </text>
+<text x="73.66" y="187.96" size="1.778" layer="97">Decoupling capacitors help ensure a
+relatively constant output voltage even in
+the event of current spikes</text>
 </plain>
 <instances>
@@
 <attribute name="NAME" x="30.48" y="62.23" size="2.54" layer="95" font="vector"/>
 <attribute name="VALUE" x="35.56" y="57.15" size="2.54" layer="96" font="vector" ratio="15" align="top-center"/>
+<attribute name="FUNCTION" x="35.56" y="54.102" size="1.27" layer="97" ratio="10" align="top-center"/>
 </instance>
 <instance part="SUPPLY8" gate="GND" x="27.94" y="53.34" smashed="yes">
@@
 <attribute name="VALUE" x="146.812" y="59.055" size="1.778" layer="96" rot="R180"/>
 </instance>
-<instance part="12V_OK" gate="G$1" x="96.52" y="165.1" smashed="yes">
-<attribute name="NAME" x="100.076" y="157.988" size="1.778" layer="95" rot="R90"/>
+<instance part="12V_OK" gate="G$1" x="134.62" y="167.64" smashed="yes">
+<attribute name="NAME" x="138.176" y="160.528" size="1.778" layer="95" rot="R90"/>
 </instance>
 <instance part="R2" gate="G$1" x="132.08" y="53.34" smashed="yes" rot="R180">
@@
 <attribute name="VALUE" x="41.275" y="81.915" size="1.778" layer="96"/>
 </instance>
-<instance part="R5" gate="G$1" x="96.52" y="175.26" smashed="yes" rot="R90">
-<attribute name="NAME" x="95.0214" y="171.45" size="1.778" layer="95" rot="R90"/>
-<attribute name="VALUE" x="99.822" y="171.45" size="1.778" layer="96" rot="R90"/>
-</instance>
-<instance part="SUPPLY16" gate="GND" x="96.52" y="154.94" smashed="yes">
-<attribute name="VALUE" x="94.615" y="151.765" size="1.778" layer="96"/>
-</instance>
-<instance part="SUPPLY17" gate="+12V" x="96.52" y="185.42" smashed="yes">
-<attribute name="VALUE" x="93.98" y="188.595" size="1.778" layer="96"/>
+<instance part="R5" gate="G$1" x="134.62" y="177.8" smashed="yes" rot="R90">
+<attribute name="NAME" x="133.1214" y="173.99" size="1.778" layer="95" rot="R90"/>
+<attribute name="VALUE" x="137.922" y="173.99" size="1.778" layer="96" rot="R90"/>
+</instance>
+<instance part="SUPPLY16" gate="GND" x="134.62" y="157.48" smashed="yes">
+<attribute name="VALUE" x="132.715" y="154.305" size="1.778" layer="96"/>
+</instance>
+<instance part="SUPPLY17" gate="+12V" x="134.62" y="187.96" smashed="yes">
+<attribute name="VALUE" x="132.08" y="191.135" size="1.778" layer="96"/>
 </instance>
 <instance part="SUPPLY1" gate="+12V" x="45.72" y="40.64" smashed="yes">
@@
 <attribute name="VALUE" x="268.224" y="155.956" size="1.778" layer="96" font="vector" rot="R180"/>
 </instance>
+<instance part="C1" gate="G$1" x="93.98" y="172.72" smashed="yes">
+<attribute name="NAME" x="94.996" y="173.355" size="1.778" layer="95"/>
+<attribute name="VALUE" x="94.996" y="168.529" size="1.778" layer="96"/>
+</instance>
+<instance part="C2" gate="G$1" x="104.14" y="172.72" smashed="yes">
+<attribute name="NAME" x="105.156" y="173.355" size="1.778" layer="95"/>
+<attribute name="VALUE" x="105.156" y="168.529" size="1.778" layer="96"/>
+</instance>
+<instance part="C3" gate="G$1" x="43.18" y="55.88" smashed="yes">
+<attribute name="NAME" x="44.196" y="56.515" size="1.778" layer="95"/>
+<attribute name="VALUE" x="44.196" y="51.689" size="1.778" layer="96"/>
+</instance>
 </instances>
 <busses>
@@
 <wire x1="78.74" y1="167.64" x2="81.28" y2="167.64" width="0.1524" layer="91"/>
 <wire x1="81.28" y1="167.64" x2="81.28" y2="165.1" width="0.1524" layer="91"/>
+<pinref part="C1" gate="G$1" pin="2"/>
+<wire x1="93.98" y1="167.64" x2="93.98" y2="165.1" width="0.1524" layer="91"/>
+<wire x1="93.98" y1="165.1" x2="88.9" y2="165.1" width="0.1524" layer="91"/>
+<wire x1="88.9" y1="165.1" x2="88.9" y2="167.64" width="0.1524" layer="91"/>
+<wire x1="88.9" y1="167.64" x2="81.28" y2="167.64" width="0.1524" layer="91"/>
+<junction x="81.28" y="167.64"/>
+<pinref part="C2" gate="G$1" pin="2"/>
+<wire x1="104.14" y1="167.64" x2="104.14" y2="165.1" width="0.1524" layer="91"/>
+<wire x1="104.14" y1="165.1" x2="93.98" y2="165.1" width="0.1524" layer="91"/>
+<junction x="93.98" y="165.1"/>
 </segment>
 <segment>
 <pinref part="Q1" gate="G$1" pin="GND2"/>
-<wire x1="53.34" y1="50.8" x2="35.56" y2="50.8" width="0.1524" layer="91"/>
+<wire x1="53.34" y1="50.8" x2="43.18" y2="50.8" width="0.1524" layer="91"/>
 <pinref part="Q1" gate="G$1" pin="GND1"/>
+<wire x1="43.18" y1="50.8" x2="35.56" y2="50.8" width="0.1524" layer="91"/>
 <wire x1="35.56" y1="50.8" x2="35.56" y2="48.26" width="0.1524" layer="91"/>
 <wire x1="35.56" y1="48.26" x2="53.34" y2="48.26" width="0.1524" layer="91"/>
@@
 <wire x1="35.56" y1="48.26" x2="35.56" y2="45.72" width="0.1524" layer="91"/>
 <junction x="35.56" y="48.26"/>
+<pinref part="C3" gate="G$1" pin="2"/>
+<junction x="43.18" y="50.8"/>
 </segment>
 <segment>
@@
 <pinref part="12V_OK" gate="G$1" pin="C"/>
 <pinref part="SUPPLY16" gate="GND" pin="GND"/>
-<wire x1="96.52" y1="160.02" x2="96.52" y2="157.48" width="0.1524" layer="91"/>
+<wire x1="134.62" y1="162.56" x2="134.62" y2="160.02" width="0.1524" layer="91"/>
 </segment>
 <segment>
@@
 <wire x1="78.74" y1="175.26" x2="81.28" y2="175.26" width="0.1524" layer="91"/>
 <wire x1="81.28" y1="175.26" x2="81.28" y2="177.8" width="0.1524" layer="91"/>
+<pinref part="C1" gate="G$1" pin="1"/>
+<wire x1="93.98" y1="175.26" x2="93.98" y2="177.8" width="0.1524" layer="91"/>
+<wire x1="93.98" y1="177.8" x2="88.9" y2="177.8" width="0.1524" layer="91"/>
+<wire x1="88.9" y1="177.8" x2="88.9" y2="175.26" width="0.1524" layer="91"/>
+<wire x1="88.9" y1="175.26" x2="81.28" y2="175.26" width="0.1524" layer="91"/>
+<junction x="81.28" y="175.26"/>
+<pinref part="C2" gate="G$1" pin="1"/>
+<wire x1="104.14" y1="175.26" x2="104.14" y2="177.8" width="0.1524" layer="91"/>
+<wire x1="104.14" y1="177.8" x2="93.98" y2="177.8" width="0.1524" layer="91"/>
+<junction x="93.98" y="177.8"/>
 </segment>
 <segment>
@@
 <pinref part="SUPPLY17" gate="+12V" pin="+12V"/>
 <pinref part="R5" gate="G$1" pin="2"/>
-<wire x1="96.52" y1="182.88" x2="96.52" y2="180.34" width="0.1524" layer="91"/>
+<wire x1="134.62" y1="185.42" x2="134.62" y2="182.88" width="0.1524" layer="91"/>
 </segment>
 <segment>
@@
 <wire x1="43.18" y1="60.96" x2="43.18" y2="58.42" width="0.1524" layer="91"/>
 <junction x="43.18" y="58.42"/>
+<pinref part="C3" gate="G$1" pin="1"/>
 </segment>
 </net>
@@
 <pinref part="R5" gate="G$1" pin="1"/>
 <pinref part="12V_OK" gate="G$1" pin="A"/>
-<wire x1="96.52" y1="170.18" x2="96.52" y2="167.64" width="0.1524" layer="91"/>
-</segment>
-</net>
+<wire x1="134.62" y1="172.72" x2="134.62" y2="170.18" width="0.1524" layer="91"/>
+</segment>
+</net>

Commit message: Updated Routing, added decoupling capacitors, and added silkscreen
Changed lines of the file:
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@@
-</segment>
-</net>
-<net name="N$6" class="0">
-<segment>
-<wire x1="233.68" y1="170.18" x2="233.68" y2="177.8" width="0.1524" layer="91"/>
-<pinref part="U1" gate="G$1" pin="V_M"/>
-<wire x1="231.14" y1="170.18" x2="233.68" y2="170.18" width="0.1524" layer="91"/>
-<pinref part="F1" gate="G$1" pin="2"/>
-<wire x1="218.44" y1="177.8" x2="233.68" y2="177.8" width="0.1524" layer="91"/>
-<pinref part="R1" gate="G$1" pin="2"/>
-<wire x1="233.68" y1="177.8" x2="236.22" y2="177.8" width="0.1524" layer="91"/>
 </segment>
 </net>
@@
 </segment>
 </net>
+<net name="N$1" class="0">
+<segment>
+<pinref part="U1" gate="G$1" pin="V_M"/>
+<wire x1="231.14" y1="170.18" x2="233.68" y2="170.18" width="0.1524" layer="91"/>
+<pinref part="F1" gate="G$1" pin="2"/>
+<wire x1="218.44" y1="177.8" x2="233.68" y2="177.8" width="0.1524" layer="91"/>
+<pinref part="R1" gate="G$1" pin="2"/>
+<wire x1="233.68" y1="177.8" x2="236.22" y2="177.8" width="0.1524" layer="91"/>
+<wire x1="233.68" y1="170.18" x2="233.68" y2="177.8" width="0.1524" layer="91"/>
+<junction x="233.68" y="177.8"/>
+</segment>
+</net>

Commit message: Fixed Stylistic issues and parts associations
Parts:
- removed F1_OK, F2_OK: (no value), led:LEDCHIP-LED0603
- removed U$1: PJ-037A, RoboJackets-Connectors:PJ-037A
- added J3: 1X2-3.5MM, adafruit:1X2-3.5MM
- added LED4, LED5: GREEN, led:LEDCHIP-LED0603
- C1: value 0.1uF -> 0.1uF 16V
- C2: value 1uF -> 1uF 16V
- C3: value 0.1uF -> 0.1uF 6V
- J1: value 1X2-3.5MM -> MAIN_PWR; device adafruit:1X2-3.5MM -> RoboJackets-Connectors:PJ-037A
- SW1: value 400AWMDP1R1M2 -> (none)
- renumbered 12V_OK to LED3
Connections:
- removed net N$5: C3.1, Q1./RESET, R4.1, U$2.2
- new net N$4: C3.1, R4.1, U$2.2
- net +12V: now also J1.1; no longer U$1.1
- net GND: now also J1.2, LED4.C, LED5.C; no longer F1_OK.C, F2_OK.C, U$1.2
- net M1+_SW: now also J3.1; no longer J1.1
- net M1_FWD: now also Q1.D10; no longer Q1.D4
- net M1_REV: now also Q1.D11; no longer Q1.D5
- net M2_FWD: now also Q1.D5; no longer Q1.D2
- net M2_REV: now also Q1.D6; no longer Q1.D3
- net N$2: now also J3.2; no longer J1.2
- net N$8: now also LED4.A; no longer F1_OK.A
- net N$9: now also LED5.A; no longer F2_OK.A
Other:
- note added: "350mA fuse specced for Sparkfun Gearmotors with .35A no-load current and 1.3A stall current No intended mechanism for this motor so should be fine"
- note added: "Using DPDT switch as DPST"
- note removed: "350mA fuse specced for Sparkfun Gearmotors with .35A no-load current and 1.3A stall current"
- moved on the sheet: C2, C3, F1, F2, LED1, LED2, R1, R2, R3, R4, R6, U$2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

Commit message: Added manufacturing files and Component list
Parts:
- renumbered U$2 to SW2
Changed lines of the file:
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@@
 <part name="SUPPLY7" library="supply2" library_urn="urn:adsk.eagle:library:372" deviceset="GND" device=""/>
 <part name="SUPPLY9" library="supply2" library_urn="urn:adsk.eagle:library:372" deviceset="GND" device=""/>
-<part name="U$2" library="RoboJackets-Switches" deviceset="PTS645" device="">
+<part name="SW2" library="RoboJackets-Switches" deviceset="PTS645" device="">
 <attribute name="FUNCTION" value="RESET"/>
 </part>
@@
 <attribute name="VALUE" x="33.655" y="40.005" size="1.778" layer="96"/>
 </instance>
-<instance part="U$2" gate="G$1" x="22.86" y="58.42" smashed="yes">
+<instance part="SW2" gate="G$1" x="22.86" y="58.42" smashed="yes">
 <attribute name="NAME" x="17.78" y="62.23" size="2.54" layer="95" font="vector"/>
 <attribute name="VALUE" x="22.86" y="57.15" size="2.54" layer="96" font="vector" ratio="15" align="top-center"/>
@@
 </segment>
 <segment>
-<pinref part="U$2" gate="G$1" pin="1"/>
+<pinref part="SW2" gate="G$1" pin="1"/>
 <wire x1="17.78" y1="58.42" x2="15.24" y2="58.42" width="0.1524" layer="91"/>
 <wire x1="15.24" y1="58.42" x2="15.24" y2="55.88" width="0.1524" layer="91"/>
@@
 <net name="N$4" class="0">
 <segment>
-<pinref part="U$2" gate="G$1" pin="2"/>
+<pinref part="SW2" gate="G$1" pin="2"/>
 <wire x1="27.94" y1="58.42" x2="33.02" y2="58.42" width="0.1524" layer="91"/>
 <wire x1="33.02" y1="58.42" x2="33.02" y2="63.5" width="0.1524" layer="91"/>

Commit message: Removed 1 motor driver chip from training board
Parts:
- removed F2: 350 mA, RoboJackets-Fuses:CHIP_FUSE1812
- removed J2: 1X2-3.5MM, adafruit:1X2-3.5MM
- removed LED5: GREEN, led:LEDCHIP-LED0603
- removed SW1: (no value), RoboJackets-Switches:400AWMDP1R1M2
- removed U2: ZXBM5210-S-13, RoboJackets-ICs:ZXBM5210-S-13
- added Q2: DMN2056U, RoboJackets-Discrete:NMOSSOT-23-3
- added S1: (no value), adafruit:EG1218S
- R6: value 2.4K -> 10K
Connections:
- removed net M1+: SW1.NO2, U1.OUT1
- removed net M2-: SW1.NO1, U2.OUT2
- removed net M2-_SW: J2.2, SW1.C1
- removed net N$7: F2.2, R6.2, U2.V_M
- removed net N$9: LED5.A, R6.1
- new net N$5: Q2.G, R6.1, S1.S
- net +12V: now also S1.P; no longer F2.1, U2.V_DD, U2.V_REF
- net GND: now also Q2.S, R6.2; no longer LED5.C, U1.GND, U2.GND
- net M1+_SW: now also U1.OUT1; no longer SW1.C2
- net M2_FWD: no longer U2.FWD
- net M2_REV: no longer U2.REV
- net N$3: now also Q2.D, U1.GND; no longer J2.1, U2.OUT1
Other:
- note removed: "Using DPDT switch as DPST"
- moved on the sheet: F1, LED4, R1, R6, U1

Commit message: Fixed reset issue and adjusted traces:
Parts:
- LED1, LED2: value YELLOW -> ORANGE
- renumbered J3 to OUT
Connections:
- removed net M2_FWD: Q1.D5
- removed net M2_REV: Q1.D6
- removed net N$4: C3.1, R4.1, SW2.2
- new net RESET: C3.1, Q1./RESET, R4.1, SW2.2
Other:
- note added: "350mA fuse specced for Sparkfun Gearmotors with .35A no-load current and 1.3A stall current No intended mechanism for this motor so should be fine."
- note added: "Motor Driver chips are powered directly from the 12V supply. V_REF is connected to 12V so speed can be controlled by applying a PWM signal to the M1_FWD or M1_REV pins. The output of the internal H Bridge is applied across OUT1 and OUT2."
- note added: "Switch controls the gate of an N-MOSFET in a low-side switch configuration. When the switch is On and the gate is connected to 12V, the transistor conducts electricity and allows the motor driver chip to turn on. When the switch is off, the pulldown resistor discharges the transistor's gate and shuts the chip down."
- note removed: "350mA fuse specced for Sparkfun Gearmotors with .35A no-load current and 1.3A stall current No intended mechanism for this motor so should be fine"
- note removed: "Motor Driver chips are powered directly from the 12V supply. V_REF is connected to 12V so speed can be controlled by applying a PWM signal to the M2_FWD or M2_REV pins. The output of the internal H Bridge is applied across OUT1 and OUT2."
- moved on the sheet: C2
