File: board/training_board.sch (EAGLE design)
At the start: 21 parts, among them J1 MAIN_PWR, Q1 ARDUINOR3-NOIOREF-NOTEXT, Q2 DMN2056U, SW2 PTS645, U1 ZXBM5210-S-13

Commit message: integrated DRV8871 into schematic and board
Parts:
- added R7: 128K, rcl:R-US_R0603
- U1: value ZXBM5210-S-13 -> DRV8871HSOP-8; device RoboJackets-ICs:ZXBM5210-S-13 -> RoboJackets-ICs:DRV8871HSOP-8
Connections:
- removed net M1+_SW: OUT.1, U1.OUT1
- new net N$4: OUT.1, U1.OUT2
- new net N$6: R7.1, U1.ILIM
- net +12V: no longer U1.V_DD, U1.V_REF
- net GND: now also R7.2, U1.GND
- net M1_FWD: now also U1.IN2; no longer U1.FWD
- net M1_REV: now also U1.IN1; no longer U1.REV
- net N$1: now also U1.VM; no longer U1.V_M
- net N$2: now also U1.OUT1; no longer U1.OUT2
- net N$3: now also U1.PGND; no longer U1.GND
Other:
- note added: "Based on the formula on pg 9 of the datasheet, this limits current to 0.5A before enabling the internal current limit"
- note added: "Motor Driver chips are powered directly from the 12V supply. Speed can be controlled by applying a PWM signal to the M1_FWD or M1_REV pins. The output of the internal H Bridge is applied across OUT1 and OUT2."
- note removed: "Motor Driver chips are powered directly from the 12V supply. V_REF is connected to 12V so speed can be controlled by applying a PWM signal to the M1_FWD or M1_REV pins. The output of the internal H Bridge is applied across OUT1 and OUT2."
- moved on the sheet: F1, LED4, Q2, R1, R6, S1, U1
