File: board/training_board.sch (EAGLE design)
At the start: 22 parts, among them J1 MAIN_PWR, Q1 DMN2056U, Q2 ARDUINOR3-NOIOREF-NOTEXT, SW1 PTS645, U1 DRV8871HSOP-8

Commit message: Changed DRV8871 for DRV8876
Parts:
- added C4, C5: 0.1 uF, Capacitor:C-US_CHIP-0603(1608-METRIC)
- added C6: 22 nF, Capacitor:C-US_CHIP-0603(1608-METRIC)
- added U2: DRV8876PWPRPWP0016J_NV, RoboJackets-ICs:DRV8876PWPRPWP0016J_NV
Connections:
- new net N$12: C5.2, U2.VCP
- new net N$13: C6.1, U2.CPH
- new net N$17: C6.2, U2.CPL
- new net N$18: C4.1, C5.1, F1.2, U2.VM
- new net N$7: R7.2
- new net N$9: Q1.D, U2.PGND
- net +5V: now also U2.PMODE, U2.VREF
- net GND: now also C4.2, U2.IMODE, U2.IPROPI
- net M1_FWD: now also U2.PH_IN2
- net M1_REV: now also U2.EN_IN1
- net N$1: no longer F1.2, R7.2
- net N$2: now also U2.OUT1; no longer U1.OUT1
- net N$3: no longer Q1.D
- net N$4: now also U2.OUT2; no longer U1.OUT2
Other:
- note added: "Cap needs to be rated for VM acc. to datasheet"
- note added: "Datasheet recommends a low ESR, VM rated bypass capacitor between VM and GND. It also recommends a 16V capacitor between VCP and VM"
- note added: "From datasheet: "The internal current regulation can be disabled by tying IPROPI to GND and setting the VREF pin voltage greater than GND." Current regulation isn't necessary here, so we can go ahead and disable it."
- moved on the sheet: C3, F1, LED1, LED3, LED4, Q1, R1, R3, R4, R5, R6, R7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

Commit message: Finished edits
Parts:
- removed Q1: DMN2056U, RoboJackets-Discrete:NMOSSOT-23-3
- removed R4: 10K, rcl:R-US_R0603
- removed R5: 120K, rcl:R-US_R0603
- removed U1: DRV8871HSOP-8, RoboJackets-ICs:DRV8871HSOP-8
- added R8: 10k, rcl:R-US_R0603
Connections:
- net N$12 renamed VCP
- net N$13 renamed CPH
- net N$17 renamed CPL
- net N$2 renamed OUT1
- net N$4 renamed OUT2
- removed net N$1: U1.VM
- removed net N$18: C4.1, C5.1, F1.2, U2.VM
- removed net N$3: U1.PGND
- removed net N$5: Q1.G, R4.1, S1.S
- removed net N$6: R5.1, U1.ILIM
- removed net N$7: R7.2
- removed net N$9: Q1.D, U2.PGND
- new net !SLEEP!: R8.1, S1.P, U2.SLEEP_N
- new net VM: C4.1, C5.1, F1.2, R7.2, U2.VM
- net +12V: no longer S1.P
- net +5V: now also R8.2
- net GND: now also S1.S, U2.GND, U2.PAD, U2.PGND; no longer Q1.S, R4.2, R5.2, U1.GND
- net M1_FWD: no longer U1.IN2
- net M1_REV: no longer U1.IN1
Other:
- note added: "Device is disabled until nSleep input is pulled high"
- note added: "Motor Driver chips are powered directly from the 12V supply. Speed can be controlled by applying a PWM signal to the M1_FWD or M1_REV pins. The output of the internal H Bridge is applied across OUT1 and OUT2. PMode is configured in this way, but can be configured for other settings. Refer to datasheet to see other options."
- note removed: "Based on the formula on pg 9 of the datasheet, this limits current to 0.53A before enabling the internal current limit"
- note removed: "Motor Driver chips are powered directly from the 12V supply. Speed can be controlled by applying a PWM signal to the M1_FWD or M1_REV pins. The output of the internal H Bridge is applied across OUT1 and OUT2."
- note removed: "Switch controls the gate of an N-MOSFET in a low-side switch configuration. When the switch is On and the gate is connected to 12V, the transistor conducts electricity and allows the motor driver chip to turn on. When the switch is off, the pulldown resistor discharges the transistor's gate and shuts the chip down."
- moved on the sheet: S1
