File: board/week3_electrical_training.sch (EAGLE design)
At the start: 24 parts, among them J1 GY-521-MPU-6050, SW1 PTS645, SW2 PTS645, SW3 PTS645, U1 TLE493DA2B6HTSA1

Commit message: Updated week3 lab schematic
Parts:
- removed R8: 10K, rcl:R-US_R0603
- removed SW2: PTS645, RoboJackets-Switches:PTS645
Connections:
- removed net D2_CTRL: A1.D10, RN1.3
- net +5V: no longer R13.2
- net GND: no longer R8.2, SW2.1
- net N$1: no longer SW2.2
- net SW1_INT: no longer R8.1

Commit message: Updated week 3 schematic
Parts:
- removed C3: 0.1uF, rcl:C-USC0805
- removed R12, R7: 1.2K, rcl:R-US_R0603
- removed U1: TLE493DA2B6HTSA1, firmware_electrical_training_board:TLE493DA2B6HTSA1
Connections:
- net +3.3V: no longer C3.1, R12.2, R7.2, U1.VDD
- net GND: no longer C3.2, U1.GND
- net XCL: no longer R7.1, U1.SCL/INT
- net XDA: no longer R12.1, U1.SDA
