File: board/firmware_electrical_training/firmware_electrical_training_board.brd (EAGLE design)
At the start: 68.6 x 53.4 mm, 26 parts, among them J1 GY-521-MPU-6050, SW1 PTS645, SW2 PTS645, SW3 PTS645, U1 TLE493DA2B6HTSA1

Commit message: First draft of board
Parts:
- moved R7 157.9 mm to (36.5, 38.0), flipped to the bottom, turned to 90 degrees
- moved C3 157.6 mm to (48.0, 36.5), flipped to the bottom, turned to 270 degrees
- moved R12 156.4 mm to (36.6, 31.4), flipped to the bottom, turned to 270 degrees
- moved RN1 152.6 mm to (18.1, 31.0), flipped to the bottom, turned to 180 degrees
- moved D6 135.8 mm to (9.51, 11.6), turned to 90 degrees
- moved R9 135.2 mm to (49.0, 46.7), flipped to the bottom
- moved U1 132.1 mm to (42.5, 36.7), flipped to the bottom, turned to 90 degrees
- moved C2 128.1 mm to (48.9, 43.9), flipped to the bottom
- moved R13 126.2 mm to (35.0, 12.5), flipped to the bottom, turned to 180 degrees
- moved R10 122.1 mm to (49.0, 40.8), flipped to the bottom
- moved R8 119.2 mm to (55.5, 40.9), flipped to the bottom, turned to 180 degrees
- moved C4 119.0 mm to (35.5, 8.97), flipped to the bottom, turned to 180 degrees
- moved C1 117.0 mm to (55.6, 43.6), flipped to the bottom, turned to 180 degrees
- moved R6 114.1 mm to (53.7, 46.5), flipped to the bottom
- moved SW3 107.6 mm to (26.0, 10.8)
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Routing:
- net +5V: track 2.54 -> 135.8 mm, vias 0 -> 7
- net +3.3V: track 0.00 -> 69.0 mm, vias 0 -> 4
- net N$7: track 0.00 -> 52.4 mm, vias 0 -> 3
- net N$1: track 0.00 -> 52.3 mm, vias 0 -> 3
- net D1_CNTRL: track 0.00 -> 48.0 mm, vias 0 -> 1
- net SCL: track 0.00 -> 45.3 mm
- net SDA: track 0.00 -> 43.4 mm, vias 0 -> 1
- net D2_CNTRL: track 0.00 -> 41.4 mm, vias 0 -> 1
- net MPU_INT: track 0.00 -> 35.2 mm
- net D3_CNTRL: track 0.00 -> 32.3 mm, vias 0 -> 2
- net D4_CNTRL: track 0.00 -> 27.9 mm, vias 0 -> 2
- net D5_CNTRL: track 0.00 -> 27.1 mm, vias 0 -> 2
- net GND: track 9.16 -> 34.4 mm, vias 6 -> 5
- net !RESET: track 0.00 -> 24.0 mm, vias 0 -> 1
- net N$9: track 0.00 -> 21.0 mm, vias 0 -> 1
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- removed copper zone on layer 1, net GND
Other:
- board text added: "PWR OK"
- board text added: "RESET"
- board text removed: "FUSE OK"
- board text removed: "OFF"
- board text removed: "ON"
- board text removed: "POWER"
- board text removed: "Reset"

Commit message: Board aesthetic changes
Routing:
- net +3.3V: track 69.0 -> 72.4 mm
- net D1_CNTRL: track 48.0 -> 45.7 mm
- net GND: track 34.4 -> 36.5 mm
- net D2_CNTRL: track 41.4 -> 42.4 mm, vias 1 -> 2
- net N$5: track 12.3 -> 11.6 mm
- net SDA: track 43.4 -> 42.8 mm
- net N$4: track 11.4 -> 12.0 mm

Commit message: General Improvements
Debouce explain, button pins, MPU indicator
Other:
- board text added: "5V"
Changed lines of the file:
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@@
 <wire x1="64.5" y1="53.4" x2="0" y2="53.4" width="0" layer="20"/>
 <wire x1="0" y1="53.4" x2="0" y2="0" width="0" layer="20"/>
-<text x="37" y="22" size="1.5" layer="51" font="vector" ratio="15">2020 Training Board
+<text x="37" y="22" size="1.5" layer="21" font="vector" ratio="15">2020 Training Board
 V2.0</text>
-<polygon width="0.1524" layer="51">
+<polygon width="0.1524" layer="21">
 <vertex x="42" y="22"/>
 <vertex x="67" y="22"/>
@@
 <wire x1="14" y1="13" x2="5" y2="13" width="0.6" layer="21"/>
 <wire x1="14" y1="8" x2="5" y2="8" width="0.6" layer="21"/>
+<polygon width="0.1524" layer="21">
+<vertex x="32" y="21"/>
+<vertex x="33" y="22"/>
+<vertex x="33" y="20"/>
+</polygon>
+<text x="34" y="20" size="1.778" layer="21" font="vector" ratio="10">5V</text>
 </plain>
 <attributes>
@@
 <wire x1="30.025" y1="20.975" x2="30.11" y2="21.06" width="0.2" layer="1"/>
 <wire x1="38.1" y1="2.54" x2="38.1" y2="13" width="0.2" layer="1"/>
-<wire x1="38.1" y1="13" x2="38.1" y2="14.9" width="0.2" layer="1"/>
-<wire x1="32.025" y1="20.975" x2="30.025" y2="20.975" width="0.2" layer="1"/>
+<wire x1="38.1" y1="13" x2="38.1" y2="15.9" width="0.2" layer="1"/>
+<wire x1="33.025" y1="20.975" x2="30.025" y2="20.975" width="0.2" layer="1"/>
 <wire x1="30.025" y1="20.975" x2="28.425" y2="20.975" width="0.2" layer="1"/>
-<wire x1="38.1" y1="14.9" x2="33.5" y2="19.5" width="0.2" layer="1"/>
-<wire x1="33.5" y1="19.5" x2="32.025" y2="20.975" width="0.2" layer="1"/>
+<wire x1="38.1" y1="15.9" x2="35.5" y2="18.5" width="0.2" layer="1"/>
+<wire x1="35.5" y1="18.5" x2="33.025" y2="20.975" width="0.2" layer="1"/>
 <wire x1="35.85" y1="12.49" x2="37.59" y2="12.49" width="0.2" layer="16"/>
 <wire x1="37.59" y1="12.49" x2="38.1" y2="13" width="0.2" layer="16"/>
@@
 <via x="45" y="26" extent="1-16" drill="0.35"/>
 <wire x1="45" y1="26" x2="41" y2="26" width="0.2" layer="16"/>
-<wire x1="41" y1="26" x2="34.5" y2="19.5" width="0.2" layer="16"/>
-<wire x1="33.5" y1="19.5" x2="34.5" y2="19.5" width="0.2" layer="16"/>
-<via x="33.5" y="19.5" extent="1-16" drill="0.35"/>
+<wire x1="41" y1="26" x2="35.5" y2="20.5" width="0.2" layer="16"/>
+<wire x1="35.5" y1="18.5" x2="35.5" y2="20.5" width="0.2" layer="16"/>
+<via x="35.5" y="18.5" extent="1-16" drill="0.35"/>
 </signal>
 <signal name="D2_CNTRL">

Commit message: Fixed Resistor array part and changed orientation of LEDs.
Parts:
- RN1: device RoboJackets-Resistors:RA-8_2506 -> firmware_electrical_training_board:RA-8_2506
- moved SW3 39.6 mm to (7.44, 45.8)
- moved SW1 34.0 mm to (7.24, 9.88)
- moved SW2 29.3 mm to (23.2, 9.88), turned to 180 degrees
- moved D6 27.5 mm to (15.5, 38.4)
- moved D5 12.8 mm to (11.0, 19.5), turned to 90 degrees
- moved D4 9.08 mm to (11.0, 22.5), turned to 90 degrees
- moved D1 7.54 mm to (11.0, 31.5), turned to 90 degrees
- moved RN1 6.53 mm to (18.0, 24.4), turned to 270 degrees
- moved D3 6.16 mm to (11.0, 25.5), turned to 90 degrees
- moved D2 5.42 mm to (11.0, 28.5), turned to 90 degrees
Connections:
- removed net D1_CNTRL: A1.D5, RN1.1
- removed net D2_CNTRL: A1.D6, RN1.3
- removed net D3_CNTRL: A1.D9, RN1.5
- removed net D4_CNTRL: A1.D10, RN1.7
- removed net D5_CNTRL: A1.D11, RN1.10
- new net D1_CTRL: A1.D11, RN1.1
- new net D2_CTRL: A1.D10, RN1.2
- new net D3_CTRL: A1.D9, RN1.3
- new net D4_CTRL: A1.D6, RN1.4
- new net D5_CTRL: A1.D5, RN1.5
- net +5V: now also RN1.8; no longer RN1.16
- net N$2: now also RN1.16; no longer RN1.2
- net N$3: now also RN1.15; no longer RN1.4
- net N$4: now also RN1.14; no longer RN1.6
- net N$5: now also RN1.13; no longer RN1.8
- net N$6: now also RN1.12; no longer RN1.9
- net N$9: now also RN1.9; no longer RN1.15
Routing:
- net D5_CTRL: track 0.00 -> 50.6 mm
- net D4_CTRL: track 0.00 -> 47.7 mm
- net D1_CNTRL: track 45.7 -> 0.00 mm, vias 1 -> 0
- net D2_CNTRL: track 42.4 -> 0.00 mm, vias 2 -> 0
- net !RESET: track 24.0 -> 66.1 mm, vias 1 -> 2
- net +5V: track 136.0 -> 95.4 mm, vias 7 -> 5
- net D3_CTRL: track 0.00 -> 38.3 mm
- net D2_CTRL: track 0.00 -> 35.2 mm
- net D3_CNTRL: track 32.3 -> 0.00 mm, vias 2 -> 0
- net D1_CTRL: track 0.00 -> 32.1 mm
- net D4_CNTRL: track 27.9 -> 0.00 mm, vias 2 -> 0
- net D5_CNTRL: track 27.1 -> 0.00 mm, vias 2 -> 0
- net N$7: track 52.4 -> 76.1 mm
- net N$1: track 52.3 -> 61.2 mm
- net N$4: track 12.0 -> 5.45 mm
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
Commit message: Removed unnecessary resistors, cleaned up routing
Parts:
- removed R6, R9: 1K, rcl:R0603
Connections:
- removed net N$1: R9.2, SW2.3, SW2.4
- removed net N$7: R6.2, SW1.3, SW1.4
- net !SW2_INPUT: now also SW2.3, SW2.4; no longer R9.1
- net SW1_INT: now also SW1.3, SW1.4; no longer R6.1
Routing:
- net SW1_INT: track 10.6 -> 88.4 mm, vias 0 -> 3
- net N$7: track 76.1 -> 0.00 mm, vias 3 -> 0
- net N$1: track 61.2 -> 0.00 mm, vias 3 -> 0
- net !SW2_INPUT: track 11.4 -> 19.4 mm
Changed lines of the file:
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@@
 <?xml version="1.0" encoding="utf-8"?>
 <!DOCTYPE eagle SYSTEM "eagle.dtd">
-<eagle version="9.5.2">
+<eagle version="9.6.0">
 <drawing>
 <settings>
@@
 <attribute name="NAME" x="5.26" y="13.485" size="1.778" layer="25" font="vector" ratio="10"/>
 </element>
-<element name="R6" library="rcl" library_urn="urn:adsk.eagle:library:334" package="R0603" package3d_urn="urn:adsk.eagle:package:23555/3" value="1K" x="53.69" y="46.49" smashed="yes" rot="MR0">
-<attribute name="NAME" x="55.375" y="46.975" size="1" layer="26" font="vector" ratio="10" rot="MR180"/>
-<attribute name="POPULARITY" value="77" x="53.69" y="46.49" size="1.778" layer="28" rot="MR0" display="off"/>
-<attribute name="SPICEPREFIX" value="R" x="53.69" y="46.49" size="1.778" layer="28" rot="MR0" display="off"/>
-<attribute name="VALUE" x="54.325" y="44.585" size="1.27" layer="28" rot="MR0"/>
-</element>
 <element name="C1" library="rcl" library_urn="urn:adsk.eagle:library:334" package="C0805" package3d_urn="urn:adsk.eagle:package:23617/2" value="0.1uF" x="55.61" y="43.63" smashed="yes" rot="MR180">
 <attribute name="NAME" x="57.64" y="44.16" size="1" layer="26" font="vector" ratio="10" rot="MR180"/>
@@
 <attribute name="FUNCTION" value="!IN-2" x="23.2" y="9.875" size="1.778" layer="27" rot="R180" display="off"/>
 <attribute name="NAME" x="25.58" y="15.365" size="1.778" layer="25" font="vector" ratio="10" rot="R180"/>
-</element>
-<element name="R9" library="rcl" library_urn="urn:adsk.eagle:library:334" package="R0603" package3d_urn="urn:adsk.eagle:package:23555/3" value="1K" x="48.99" y="46.67" smashed="yes" rot="MR0">
-<attribute name="NAME" x="47.125" y="46.305" size="1" layer="26" font="vector" ratio="10" rot="MR0"/>
-<attribute name="POPULARITY" value="77" x="48.99" y="52.83" size="1.778" layer="28" rot="MR0" display="off"/>
-<attribute name="SPICEPREFIX" value="R" x="48.99" y="52.83" size="1.778" layer="28" rot="MR0" display="off"/>
-<attribute name="VALUE" x="49.625" y="44.765" size="1.27" layer="28" rot="MR0"/>
 </element>
 <element name="C2" library="rcl" library_urn="urn:adsk.eagle:library:334" package="C0805" package3d_urn="urn:adsk.eagle:package:23617/2" value="0.1uF" x="48.89" y="43.89" smashed="yes" rot="MR0">
@@
 <wire x1="23.7" y1="38.84" x2="23.7" y2="26.64" width="0.2" layer="16"/>
 <wire x1="18.8" y1="24.03" x2="21.76" y2="24.03" width="0.2" layer="16"/>
-<wire x1="23.7" y1="25.97" x2="23.7" y2="26.64" width="0.1524" layer="16"/>
+<wire x1="23.7" y1="25.97" x2="23.7" y2="26.64" width="0.2" layer="16"/>
 <wire x1="21.76" y1="24.03" x2="23.7" y2="25.97" width="0.2" layer="16"/>
 </signal>
@@
 <wire x1="58.42" y1="47.42" x2="53" y2="42" width="0.2" layer="1"/>
 </signal>
-<signal name="N$7">
+<signal name="SW1_INT">
+<contactref element="C1" pad="1"/>
+<contactref element="A1" pad="D3"/>
+<contactref element="R8" pad="1"/>
+<wire x1="54.54" y1="43.75" x2="54.66" y2="43.63" width="0.2" layer="16"/>
+<wire x1="54.66" y1="43.63" x2="54.66" y2="40.85" width="0.2" layer="16"/>
 <contactref element="SW1" pad="3"/>
 <contactref element="SW1" pad="4"/>
-<contactref element="R6" pad="2"/>
-<wire x1="52.84" y1="46.49" x2="51.65" y2="45.3" width="0.2" layer="16"/>
-<wire x1="51.65" y1="45.3" x2="51.5" y2="45.3" width="0.2" layer="16"/>
 <via x="51.5" y="45.3" extent="1-16" drill="0.35"/>
 <wire x1="49.7" y1="43.5" x2="51.5" y2="45.3" width="0.2" layer="1"/>
@@
 <wire x1="24.37" y1="38.4" x2="29.47" y2="43.5" width="0.2" layer="16"/>
 <wire x1="31.71" y1="43.5" x2="49.7" y2="43.5" width="0.2" layer="1"/>
-</signal>
-<signal name="SW1_INT">
-<contactref element="R6" pad="1"/>
-<contactref element="C1" pad="1"/>
-<contactref element="A1" pad="D3"/>
-<contactref element="R8" pad="1"/>
-<wire x1="55.88" y1="50.8" x2="54.54" y2="49.46" width="0.2" layer="16"/>
-<wire x1="54.54" y1="49.46" x2="54.54" y2="46.49" width="0.2" layer="16"/>
-<wire x1="54.54" y1="46.49" x2="54.54" y2="43.75" width="0.2" layer="16"/>
-<wire x1="54.54" y1="43.75" x2="54.66" y2="43.63" width="0.2" layer="16"/>
-<wire x1="54.66" y1="43.63" x2="54.66" y2="40.85" width="0.2" layer="16"/>
-</signal>
-<signal name="N$1">
-<contactref element="SW2" pad="3"/>
-<contactref element="SW2" pad="4"/>
-<contactref element="R9" pad="2"/>
-<wire x1="48.14" y1="46.67" x2="44.67" y2="46.67" width="0.2" layer="16"/>
-<wire x1="44.67" y1="46.67" x2="44" y2="46" width="0.2" layer="16"/>
-<via x="44" y="46" extent="1-16" drill="0.35"/>
-<wire x1="19.175" y1="12.125" x2="27.175" y2="12.125" width="0.2" layer="1"/>
-<wire x1="44" y1="46" x2="43.3" y2="45.3" width="0.2" layer="1"/>
-<wire x1="43.3" y1="45.3" x2="32.26" y2="45.3" width="0.2" layer="1"/>
-<wire x1="32.26" y1="45.3" x2="25.51" y2="38.55" width="0.2" layer="1"/>
-<wire x1="25.51" y1="38.55" x2="25.51" y2="37.76" width="0.2" layer="1"/>
-<wire x1="25.51" y1="37.76" x2="25.520903125" y2="37.770903125" width="0.2" layer="1"/>
-<wire x1="25.520903125" y1="37.770903125" x2="25.520903125" y2="37.830903125" width="0.2" layer="1"/>
-<via x="25.520903125" y="37.830903125" extent="1-16" drill="0.35"/>
-<wire x1="25.520903125" y1="37.830903125" x2="25.520903125" y2="16.479096875" width="0.2" layer="16"/>
-<wire x1="25.520903125" y1="16.479096875" x2="26.9" y2="15.1" width="0.2" layer="16"/>
-<via x="26.9" y="15.1" extent="1-16" drill="0.35"/>
-<wire x1="26.9" y1="15.1" x2="26.9" y2="12.4" width="0.2" layer="1"/>
-<wire x1="26.9" y1="12.4" x2="27.175" y2="12.125" width="0.2" layer="1"/>
+<wire x1="51.5" y1="46.42" x2="51.5" y2="45.3" width="0.2" layer="16"/>
+<wire x1="55.88" y1="50.8" x2="51.5" y2="46.42" width="0.2" layer="16"/>
+<wire x1="54.66" y1="43.63" x2="52.99" y2="45.3" width="0.2" layer="16"/>
+<wire x1="52.99" y1="45.3" x2="51.5" y2="45.3" width="0.2" layer="16"/>
 </signal>
 <signal name="!SW2_INPUT">
-<contactref element="R9" pad="1"/>
 <contactref element="C2" pad="1"/>
 <contactref element="R10" pad="1"/>
 <contactref element="A1" pad="D4"/>
 <wire x1="53.34" y1="50.8" x2="49.84" y2="47.3" width="0.2" layer="16"/>
-<wire x1="49.84" y1="47.3" x2="49.84" y2="46.67" width="0.2" layer="16"/>
 <wire x1="49.84" y1="43.89" x2="49.84" y2="40.84" width="0.2" layer="16"/>
 <wire x1="49.84" y1="40.84" x2="49.83" y2="40.83" width="0.2" layer="16"/>
-<wire x1="49.84" y1="46.67" x2="49.84" y2="43.89" width="0.2" layer="16"/>
+<contactref element="SW2" pad="3"/>
+<contactref element="SW2" pad="4"/>
+<wire x1="49.84" y1="47.3" x2="49.84" y2="43.89" width="0.2" layer="16"/>
+<wire x1="19.175" y1="12.125" x2="27.175" y2="12.125" width="0.2" layer="1"/>
+<wire x1="27.175" y1="12.125" x2="49.83" y2="40.83" width="0" layer="19" extent="1-16"/>
 </signal>
 <signal name="!RESET">

Commit message: Removed library, small changes
Parts:
- RN1: device firmware_electrical_training_board:RA-8_2506 -> RoboJackets-Resistors:RA-8_2506
Routing:
- net !SW2_INPUT: track 19.4 -> 65.5 mm, vias 0 -> 3
- net +3.3V: track 72.4 -> 62.1 mm, vias 4 -> 3
- net !RESET: track 66.1 -> 67.3 mm
- net SCL: track 45.3 -> 44.3 mm
- net +5V: track 95.4 -> 94.7 mm

Commit message: Fixed angled routing
Parts:
- U1: device firmware_electrical_training_board:SOT-23-6 -> RoboJackets-ICs:SOT-23-6
Routing:
- net SDA: track 42.8 -> 44.0 mm
Changed lines of the file:
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@@
 <drawing>
 <settings>
-<setting alwaysvectorfont="no"/>
+<setting alwaysvectorfont="yes"/>
 <setting verticaltext="up"/>
 </settings>
@@
 <attribute name="VALUE" x="49.615" y="38.925" size="1.27" layer="28" rot="MR0"/>
 </element>
-<element name="U1" library="firmware_electrical_training_board" package="SOT-23-6" value="TLE493DA2B6HTSA1" x="42.46" y="36.71" smashed="yes" rot="MR90">
+<element name="U1" library="RoboJackets-ICs" package="SOT-23-6" value="TLE493DA2B6HTSA1" x="42.46" y="36.71" smashed="yes" rot="MR90">
 <attribute name="DKPN" value="TLE493DA2B6HTSA1CT-ND" x="42.46" y="36.71" size="1.778" layer="28" rot="MR90" display="off"/>
 <attribute name="NAME" x="41.805" y="34.635" size="1" layer="26" font="vector" ratio="10" rot="MR180"/>
@@
 <contactref element="A1" pad="A5"/>
 <wire x1="30.11" y1="26.14" x2="41.86" y2="26.14" width="0.2" layer="1"/>
-<wire x1="41.86" y1="26.14" x2="63" y2="5" width="0.2" layer="1"/>
-<wire x1="63" y1="5" x2="63" y2="3.04" width="0.2" layer="1"/>
-<wire x1="63.5" y1="2.54" x2="63" y2="3.04" width="0.2" layer="1"/>
+<wire x1="63.5" y1="2.54" x2="63.5" y2="4.5" width="0.2" layer="1"/>
+<wire x1="63.5" y1="4.5" x2="41.86" y2="26.14" width="0.2" layer="1"/>
 </signal>
 <signal name="SDA">
 <contactref element="J1" pad="4"/>
 <contactref element="A1" pad="A4"/>
-<wire x1="60.96" y1="2.54" x2="38.5" y2="25" width="0.2" layer="1"/>
-<wire x1="38.5" y1="25" x2="34" y2="25" width="0.2" layer="1"/>
+<wire x1="60.96" y1="2.54" x2="60.96" y2="4.54" width="0.2" layer="1"/>
+<wire x1="60.96" y1="4.54" x2="40.5" y2="25" width="0.2" layer="1"/>
+<wire x1="40.5" y1="25" x2="34" y2="25" width="0.2" layer="1"/>
 <via x="34" y="25" extent="1-16" drill="0.35"/>
 <wire x1="33" y1="28" x2="33" y2="26" width="0.2" layer="16"/>
