File: board/firmware_electrical_training/firmware_electrical_training_board.sch (EAGLE design)
At the start: 24 parts, among them J1 GY-521-MPU-6050, SW1 PTS645, SW2 PTS645, SW3 PTS645, U1 TLE493DA2B6HTSA1

Commit message: General Improvements
Debouce explain, button pins, MPU indicator
Other:
- note added: "A RC circuit is present for all buttons to provide debouncing. Debouncing is so that the function will not be triggered more than once per press due to noise."
- note added: "Connects to Pin D3 of Arduino"
- note added: "Connects to Pin D4 of Arduino"
- note removed: "A RC circuit is present to provide debouncing."
Changed lines of the file:
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@@
 When you push on the button, the digital value will be a 0.
 When you do not push on the button, the digital value will be a 1.</text>
-<text x="198.12" y="154.94" size="1.27" layer="97" ratio="7">A RC circuit is present to provide debouncing.</text>
-<text x="180.34" y="121.92" size="1.27" layer="97" ratio="7">A RC circuit is present to provide debouncing.</text>
-<text x="180.34" y="73.66" size="1.27" layer="97" ratio="7">A RC circuit is present to provide debouncing.</text>
+<text x="236.22" y="190.5" size="1.27" layer="97" ratio="7">A RC circuit is present for all buttons to
+provide debouncing.
+Debouncing is so that the function will not
+be triggered more than once per press due
+to noise.</text>
 <text x="76.2" y="132.08" size="1.27" layer="97" ratio="7">GY-521-MPU-6050 has XDA and XCL.
 These are external I2C bus. This allows
@@
 <text x="10.16" y="165.1" size="3.81" layer="97" ratio="7">Magnetometer Sensor
 (DO NOT POPULATE)</text>
+<text x="248.92" y="170.18" size="1.27" layer="97" ratio="7">Connects to Pin D3 of Arduino</text>
+<text x="248.92" y="119.38" size="1.27" layer="97" ratio="7">Connects to Pin D4 of Arduino</text>
 </plain>
 <instances>
@@
 <wire x1="233.68" y1="165.1" x2="243.84" y2="165.1" width="0.1524" layer="91"/>
 <pinref part="C1" gate="G$1" pin="1"/>
-<label x="251.46" y="165.1" size="1.778" layer="95" xref="yes"/>
+<label x="248.92" y="165.1" size="1.778" layer="95" xref="yes"/>
 <pinref part="R8" gate="G$1" pin="1"/>
-<wire x1="243.84" y1="165.1" x2="251.46" y2="165.1" width="0.1524" layer="91"/>
+<wire x1="243.84" y1="165.1" x2="248.92" y2="165.1" width="0.1524" layer="91"/>
 <wire x1="243.84" y1="162.56" x2="243.84" y2="165.1" width="0.1524" layer="91"/>
 <junction x="243.84" y="165.1"/>
@@
 <junction x="233.68" y="114.3"/>
 <wire x1="233.68" y1="116.84" x2="233.68" y2="114.3" width="0.1524" layer="91"/>
-<wire x1="233.68" y1="114.3" x2="238.76" y2="114.3" width="0.1524" layer="91"/>
+<wire x1="233.68" y1="114.3" x2="248.92" y2="114.3" width="0.1524" layer="91"/>
 <pinref part="C2" gate="G$1" pin="1"/>
 <pinref part="R10" gate="G$1" pin="1"/>
-<label x="238.76" y="114.3" size="1.778" layer="95" xref="yes"/>
+<label x="248.92" y="114.3" size="1.778" layer="95" xref="yes"/>
 </segment>
 <segment>
@@
 <junction x="233.68" y="66.04"/>
 <wire x1="233.68" y1="68.58" x2="233.68" y2="66.04" width="0.1524" layer="91"/>
-<wire x1="233.68" y1="66.04" x2="238.76" y2="66.04" width="0.1524" layer="91"/>
+<wire x1="233.68" y1="66.04" x2="248.92" y2="66.04" width="0.1524" layer="91"/>
 <pinref part="C4" gate="G$1" pin="1"/>
 <pinref part="R13" gate="G$1" pin="1"/>
-<label x="238.76" y="66.04" size="1.778" layer="95" xref="yes"/>
+<label x="248.92" y="66.04" size="1.778" layer="95" xref="yes"/>
 <pinref part="SW3" gate="G$1" pin="2"/>
 <wire x1="210.82" y1="66.04" x2="233.68" y2="66.04" width="0.1524" layer="91"/>

Commit message: Fixed Resistor array part and changed orientation of LEDs.
Parts:
- RN1: device RoboJackets-Resistors:RA-82506 -> firmware_electrical_training_board:RA-82506
Connections:
- net D3_CNTRL renamed D3_CTRL
- removed net D1_CNTRL: A1.D5, RN1.1
- removed net D2_CNTRL: A1.D6, RN1.3
- removed net D4_CNTRL: A1.D10, RN1.7
- removed net D5_CNTRL: A1.D11, RN1.10
- new net D1_CTRL: A1.D11, RN1.1
- new net D2_CTRL: A1.D10, RN1.3
- new net D4_CTRL: A1.D6, RN1.7
- new net D5_CTRL: A1.D5, RN1.9
- net +5V: now also RN1.15; no longer RN1.16
- net N$6: now also RN1.10; no longer RN1.9
- net N$9: now also RN1.16; no longer RN1.15
Changed lines of the file:
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@@
 <?xml version="1.0" encoding="utf-8"?>
 <!DOCTYPE eagle SYSTEM "eagle.dtd">
-<eagle version="9.6.0">
+<eagle version="9.5.2">
 <drawing>
 <settings>
@@
 <part name="SUPPLY20" library="RoboJackets-Supplies" deviceset="+3.3V" device=""/>
 <part name="SUPPLY6" library="supply2" library_urn="urn:adsk.eagle:library:372" deviceset="GND" device=""/>
-<part name="RN1" library="RoboJackets-Resistors" deviceset="RA-8" device="2506" value="330">
+<part name="RN1" library="firmware_electrical_training_board" deviceset="RA-8" device="2506" value="330">
 <attribute name="DKPN" value="742C163331JPCT-ND"/>
 <attribute name="POWER" value="62.5mW"/>
@@
 </segment>
 <segment>
-<pinref part="RN1" gate="G$1" pin="16"/>
+<pinref part="RN1" gate="G$1" pin="15"/>
 <wire x1="142.24" y1="175.26" x2="134.62" y2="175.26" width="0.1524" layer="91"/>
 <pinref part="SUPPLY15" gate="+5V" pin="+5V"/>
 </segment>
 </net>
-<net name="D2_CNTRL" class="0">
-<segment>
-<pinref part="A1" gate="G$1" pin="D6"/>
-<wire x1="114.3" y1="45.72" x2="119.38" y2="45.72" width="0.1524" layer="91"/>
-<label x="119.38" y="45.72" size="1.778" layer="95" xref="yes"/>
-</segment>
+<net name="D2_CTRL" class="0">
 <segment>
 <pinref part="RN1" gate="G$1" pin="3"/>
@@
 <label x="139.7" y="190.5" size="1.778" layer="95" rot="R180" xref="yes"/>
 </segment>
-</net>
-<net name="D1_CNTRL" class="0">
-<segment>
-<wire x1="142.24" y1="193.04" x2="124.46" y2="193.04" width="0.1524" layer="91"/>
-<label x="124.46" y="193.04" size="1.778" layer="95" rot="R180" xref="yes"/>
-<pinref part="RN1" gate="G$1" pin="1"/>
-</segment>
+<segment>
+<pinref part="A1" gate="G$1" pin="D10"/>
+<wire x1="114.3" y1="58.42" x2="137.16" y2="58.42" width="0.1524" layer="91"/>
+<label x="137.16" y="58.42" size="1.778" layer="95" xref="yes"/>
+</segment>
+</net>
+<net name="D5_CTRL" class="0">
 <segment>
 <pinref part="A1" gate="G$1" pin="D5"/>
 <wire x1="114.3" y1="43.18" x2="137.16" y2="43.18" width="0.1524" layer="91"/>
 <label x="137.16" y="43.18" size="1.778" layer="95" xref="yes"/>
+</segment>
+<segment>
+<wire x1="142.24" y1="182.88" x2="124.46" y2="182.88" width="0.1524" layer="91"/>
+<label x="124.46" y="182.88" size="1.778" layer="95" rot="R180" xref="yes"/>
+<pinref part="RN1" gate="G$1" pin="9"/>
 </segment>
 </net>
@@
 </segment>
 </net>
-<net name="D3_CNTRL" class="0">
-<segment>
-<wire x1="142.24" y1="187.96" x2="124.46" y2="187.96" width="0.1524" layer="91"/>
-<label x="124.46" y="187.96" size="1.778" layer="95" rot="R180" xref="yes"/>
-<pinref part="RN1" gate="G$1" pin="5"/>
-</segment>
-<segment>
-<pinref part="A1" gate="G$1" pin="D9"/>
-<wire x1="114.3" y1="55.88" x2="119.38" y2="55.88" width="0.1524" layer="91"/>
-<label x="119.38" y="55.88" size="1.778" layer="95" xref="yes"/>
-</segment>
-</net>
-<net name="D4_CNTRL" class="0">
+<net name="D4_CTRL" class="0">
 <segment>
 <wire x1="142.24" y1="185.42" x2="139.7" y2="185.42" width="0.1524" layer="91"/>
@@
 </segment>
 <segment>
-<pinref part="A1" gate="G$1" pin="D10"/>
-<wire x1="114.3" y1="58.42" x2="137.16" y2="58.42" width="0.1524" layer="91"/>
-<label x="137.16" y="58.42" size="1.778" layer="95" xref="yes"/>
-</segment>
-</net>
-<net name="D5_CNTRL" class="0">
-<segment>
-<wire x1="142.24" y1="182.88" x2="124.46" y2="182.88" width="0.1524" layer="91"/>
-<label x="124.46" y="182.88" size="1.778" layer="95" rot="R180" xref="yes"/>
-<pinref part="RN1" gate="G$1" pin="10"/>
-</segment>
-<segment>
-<pinref part="A1" gate="G$1" pin="D11"/>
-<wire x1="114.3" y1="60.96" x2="119.38" y2="60.96" width="0.1524" layer="91"/>
-<label x="119.38" y="60.96" size="1.778" layer="95" xref="yes"/>
+<pinref part="A1" gate="G$1" pin="D6"/>
+<wire x1="114.3" y1="45.72" x2="119.38" y2="45.72" width="0.1524" layer="91"/>
+<label x="119.38" y="45.72" size="1.778" layer="95" xref="yes"/>
 </segment>
 </net>
@@
 <net name="N$6" class="0">
 <segment>
-<pinref part="RN1" gate="G$1" pin="9"/>
+<pinref part="RN1" gate="G$1" pin="10"/>
 <wire x1="152.4" y1="182.88" x2="154.94" y2="182.88" width="0.1524" layer="91"/>
 <wire x1="154.94" y1="182.88" x2="154.94" y2="152.4" width="0.1524" layer="91"/>
@@
 <net name="N$9" class="0">
 <segment>
-<pinref part="RN1" gate="G$1" pin="15"/>
+<pinref part="RN1" gate="G$1" pin="16"/>
 <wire x1="152.4" y1="175.26" x2="152.4" y2="142.24" width="0.1524" layer="91"/>
 <wire x1="152.4" y1="142.24" x2="162.56" y2="142.24" width="0.1524" layer="91"/>
@@
 </segment>
 </net>
+<net name="D1_CTRL" class="0">
+<segment>
+<pinref part="A1" gate="G$1" pin="D11"/>
+<wire x1="114.3" y1="60.96" x2="119.38" y2="60.96" width="0.1524" layer="91"/>
+<label x="119.38" y="60.96" size="1.778" layer="95" xref="yes"/>
+</segment>
+<segment>
+<wire x1="142.24" y1="193.04" x2="124.46" y2="193.04" width="0.1524" layer="91"/>
+<label x="124.46" y="193.04" size="1.778" layer="95" rot="R180" xref="yes"/>
+<pinref part="RN1" gate="G$1" pin="1"/>
+</segment>
+</net>
+<net name="D3_CTRL" class="0">
+<segment>
+<pinref part="A1" gate="G$1" pin="D9"/>
+<wire x1="114.3" y1="55.88" x2="119.38" y2="55.88" width="0.1524" layer="91"/>
+<label x="119.38" y="55.88" size="1.778" layer="95" xref="yes"/>
+</segment>
+<segment>
+<wire x1="142.24" y1="187.96" x2="124.46" y2="187.96" width="0.1524" layer="91"/>
+<label x="124.46" y="187.96" size="1.778" layer="95" rot="R180" xref="yes"/>
+<pinref part="RN1" gate="G$1" pin="5"/>
+</segment>
+</net>

Commit message: Removed unnecessary resistors, cleaned up routing
Parts:
- removed R6, R9: 1K, rcl:R-US_R0603
Connections:
- removed net N$1: R9.2, SW2.2
- removed net N$7: R6.2, SW1.2
- net !SW2_INPUT: now also SW2.2; no longer R9.1
- net SW1_INT: now also SW1.2; no longer R6.1
Changed lines of the file:
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@@
 <?xml version="1.0" encoding="utf-8"?>
 <!DOCTYPE eagle SYSTEM "eagle.dtd">
-<eagle version="9.5.2">
+<eagle version="9.6.0">
 <drawing>
 <settings>
@@
 <attribute name="FUNCTION" value="IN-1"/>
 </part>
-<part name="R6" library="rcl" library_urn="urn:adsk.eagle:library:334" deviceset="R-US_" device="R0603" package3d_urn="urn:adsk.eagle:package:23555/3" value="1K"/>
 <part name="SUPPLY3" library="supply2" library_urn="urn:adsk.eagle:library:372" deviceset="+5V" device=""/>
 <part name="C1" library="rcl" library_urn="urn:adsk.eagle:library:334" deviceset="C-US" device="C0805" package3d_urn="urn:adsk.eagle:package:23617/2" value="0.1uF"/>
@@
 <attribute name="FUNCTION" value="!IN-2"/>
 </part>
-<part name="R9" library="rcl" library_urn="urn:adsk.eagle:library:334" deviceset="R-US_" device="R0603" package3d_urn="urn:adsk.eagle:package:23555/3" value="1K"/>
 <part name="C2" library="rcl" library_urn="urn:adsk.eagle:library:334" deviceset="C-US" device="C0805" package3d_urn="urn:adsk.eagle:package:23617/2" value="0.1uF"/>
 <part name="R10" library="rcl" library_urn="urn:adsk.eagle:library:334" deviceset="R-US_" device="R0603" package3d_urn="urn:adsk.eagle:package:23555/3" value="10K"/>
@@
 <attribute name="FUNCTION" x="208.28" y="160.782" size="1.778" layer="96" align="top-center"/>
 </instance>
-<instance part="R6" gate="G$1" x="223.52" y="165.1" smashed="yes" rot="R180">
-<attribute name="NAME" x="224.79" y="168.6814" size="1.778" layer="95" rot="R180"/>
-<attribute name="VALUE" x="224.79" y="163.322" size="1.778" layer="96" rot="R180"/>
-</instance>
 <instance part="SUPPLY3" gate="+5V" x="198.12" y="182.88" smashed="yes">
 <attribute name="VALUE" x="196.215" y="186.055" size="1.778" layer="96"/>
@@
 <attribute name="VALUE" x="205.74" y="113.03" size="1.778" layer="96" align="top-center"/>
 <attribute name="FUNCTION" x="205.74" y="109.982" size="1.778" layer="96" align="top-center"/>
-</instance>
-<instance part="R9" gate="G$1" x="223.52" y="114.3" smashed="yes" rot="R180">
-<attribute name="NAME" x="224.79" y="117.8814" size="1.778" layer="95" rot="R180"/>
-<attribute name="VALUE" x="224.79" y="112.522" size="1.778" layer="96" rot="R180"/>
 </instance>
 <instance part="C2" gate="G$1" x="233.68" y="109.22" smashed="yes">
@@
 </segment>
 </net>
-<net name="N$7" class="0">
-<segment>
-<pinref part="SW1" gate="G$1" pin="2"/>
-<wire x1="213.36" y1="165.1" x2="218.44" y2="165.1" width="0.1524" layer="91"/>
-<pinref part="R6" gate="G$1" pin="2"/>
-</segment>
-</net>
 <net name="SW1_INT" class="0">
 <segment>
-<pinref part="R6" gate="G$1" pin="1"/>
-<wire x1="228.6" y1="165.1" x2="233.68" y2="165.1" width="0.1524" layer="91"/>
 <wire x1="233.68" y1="165.1" x2="233.68" y2="162.56" width="0.1524" layer="91"/>
-<junction x="233.68" y="165.1"/>
 <wire x1="233.68" y1="165.1" x2="243.84" y2="165.1" width="0.1524" layer="91"/>
 <pinref part="C1" gate="G$1" pin="1"/>
@@
 <wire x1="243.84" y1="162.56" x2="243.84" y2="165.1" width="0.1524" layer="91"/>
 <junction x="243.84" y="165.1"/>
+<pinref part="SW1" gate="G$1" pin="2"/>
+<wire x1="213.36" y1="165.1" x2="233.68" y2="165.1" width="0.1524" layer="91"/>
+<junction x="233.68" y="165.1"/>
 </segment>
 <segment>
@@
 </segment>
 </net>
-<net name="N$1" class="0">
-<segment>
-<pinref part="SW2" gate="G$1" pin="2"/>
-<wire x1="210.82" y1="114.3" x2="218.44" y2="114.3" width="0.1524" layer="91"/>
-<pinref part="R9" gate="G$1" pin="2"/>
-</segment>
-</net>
 <net name="!SW2_INPUT" class="0">
 <segment>
-<pinref part="R9" gate="G$1" pin="1"/>
-<wire x1="228.6" y1="114.3" x2="233.68" y2="114.3" width="0.1524" layer="91"/>
 <wire x1="233.68" y1="114.3" x2="233.68" y2="111.76" width="0.1524" layer="91"/>
 <junction x="233.68" y="114.3"/>
@@
 <pinref part="R10" gate="G$1" pin="1"/>
 <label x="248.92" y="114.3" size="1.778" layer="95" xref="yes"/>
-</segment>
-<segment>
+<pinref part="SW2" gate="G$1" pin="2"/>
+<wire x1="233.68" y1="114.3" x2="210.82" y2="114.3" width="0.1524" layer="91"/>
+</segment>
+<segment>

Commit message: Removed library, small changes
Parts:
- RN1: device firmware_electrical_training_board:RA-82506 -> RoboJackets-Resistors:RA-82506
Changed lines of the file:
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@@
 <part name="SUPPLY20" library="RoboJackets-Supplies" deviceset="+3.3V" device=""/>
 <part name="SUPPLY6" library="supply2" library_urn="urn:adsk.eagle:library:372" deviceset="GND" device=""/>
-<part name="RN1" library="firmware_electrical_training_board" deviceset="RA-8" device="2506" value="330">
+<part name="RN1" library="RoboJackets-Resistors" deviceset="RA-8" device="2506" value="330">
 <attribute name="DKPN" value="742C163331JPCT-ND"/>
 <attribute name="POWER" value="62.5mW"/>

Commit message: Fixed angled routing
Parts:
- U1: device firmware_electrical_training_board:TLE493DA2B6HTSA1 -> RoboJackets-ICs:TLE493DA2B6HTSA1
Changed lines of the file:
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@@
 <part name="SUPPLY10" library="supply2" library_urn="urn:adsk.eagle:library:372" deviceset="GND" device=""/>
 <part name="SUPPLY15" library="supply2" library_urn="urn:adsk.eagle:library:372" deviceset="+5V" device=""/>
-<part name="U1" library="firmware_electrical_training_board" deviceset="TLE493DA2B6HTSA1" device=""/>
+<part name="U1" library="RoboJackets-ICs" deviceset="TLE493DA2B6HTSA1" device=""/>
 <part name="SW3" library="RoboJackets-Switches" deviceset="PTS645" device="">
 <attribute name="FUNCTION" value="RESET"/>
