File: board/firmware_training/firmware_training_board.brd (EAGLE design)
At the start: 68.6 x 53.4 mm, 17 parts, among them J1 GY-521-MPU-6050, SW1 PTS645, SW2 PTS645

Commit message: Finished schematic, started board
Parts:
- removed D6: GRN, led:CHIP-LED0603
- A1: value ARDUINOR3-NOIOREF-NOTEXT -> NANO; device adafruit:ARDUINOR3-NOTEXT-NOIOREF -> firmware_training_board:NANO
- D1: device led:CHIP-LED0603 -> adafruit:LED5MM
- D2, D3, D4, D5: device led:CHIP-LED0603 -> firmware_training_board:LED5MM
- moved R8 41.8 mm to (14.0, 46.0), turned to 90 degrees
- moved D1 41.8 mm to (49.0, 49.0), turned to 0 degrees
- moved C1 41.6 mm to (14.0, 42.0)
- moved A1 41.0 mm to (28.0, 30.0)
- moved D2 40.0 mm to (49.0, 41.0), turned to 0 degrees
- moved D3 38.7 mm to (49.0, 33.0), turned to 0 degrees
- moved D5 38.0 mm to (49.0, 17.0), turned to 0 degrees
- moved D4 38.0 mm to (49.0, 25.0), turned to 0 degrees
- moved SW1 36.1 mm to (6.00, 46.0)
- moved R10 35.5 mm to (14.0, 35.0), turned to 270 degrees
- moved C2 35.2 mm to (14.0, 39.0), turned to 180 degrees
- moved U$4 33.4 mm to (37.0, 7.00), flipped to the bottom, turned to 90 degrees
- moved SW2 30.4 mm to (6.00, 35.0)
- moved RN1 25.6 mm to (40.0, 37.4), flipped to the top
- moved J1 24.2 mm to (8.11, 11.1)
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Connections:
- net N$2 renamed D1_LED
- net N$3 renamed D2_LED
- net N$4 renamed D3_LED
- net N$5 renamed D4_LED
- net N$6 renamed D5_LED
- removed net N$9: D6.A, RN1.9
- removed net VIN: A1.VIN
- net !RESET: now also A1.RST; no longer A1.RESET
- net +3.3V: now also A1.3.3V; no longer A1.3V
- net +5V: no longer RN1.8
- net GND: now also D1.K, D2.K, D3.K, D4.K, D5.K; no longer A1.GND2, D1.C, D2.C, D3.C, D4.C, D5.C, D6.C
- net MPU_INT: now also A1.D3; no longer A1.D2
- net SW1_INT: now also A1.D2; no longer A1.D3
Routing:
- net +5V: track 93.0 -> 0.00 mm, vias 5 -> 0
- net SW1_INT: track 88.3 -> 0.00 mm, vias 3 -> 0
- net !SW2_INPUT: track 65.5 -> 0.00 mm, vias 3 -> 0
- net +3.3V: track 48.5 -> 0.00 mm, vias 3 -> 0
- net D5_CTRL: track 50.6 -> 9.48 mm
- net D4_CTRL: track 47.7 -> 7.88 mm
- net MPU_INT: track 35.2 -> 0.00 mm
- net D3_CTRL: track 38.3 -> 3.99 mm
- net D2_CTRL: track 35.2 -> 5.48 mm
- net GND: track 29.1 -> 0.00 mm, vias 4 -> 0
- net SCL: track 44.3 -> 16.7 mm
- net SDA: track 44.0 -> 16.7 mm, vias 1 -> 0
- net D1_CTRL: track 32.1 -> 6.60 mm
- net N$9: track 20.2 -> 0.00 mm, vias 1 -> 0
- net D5_LED: track 8.60 -> 23.6 mm, vias 1 -> 0
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Other:
- board size 68.6 x 53.4 mm -> 63 x 51.4 mm
- board text removed: "PWR OK"
- board text removed: "RESET"

Commit message: First finished version
Parts:
- moved U$4 36.4 mm to (8.00, 29.0), turned to 0 degrees
- moved U$3 11.4 mm to (17.0, 2.00), flipped to the top
- moved A1 8.00 mm to (28.0, 22.0)
- moved C1 8.00 mm to (14.0, 34.0)
- moved C2 8.00 mm to (14.0, 31.0)
- moved D1 8.00 mm to (49.0, 41.0)
- moved D2 8.00 mm to (49.0, 33.0)
- moved D3 8.00 mm to (49.0, 25.0)
- moved D4 8.00 mm to (49.0, 17.0)
- moved D5 8.00 mm to (49.0, 9.00)
- moved J1 8.00 mm to (8.11, 3.06)
- moved R10 8.00 mm to (14.0, 27.0)
- moved R8 8.00 mm to (14.0, 38.0)
- moved RN1 8.00 mm to (40.0, 29.4)
- moved SW1 8.00 mm to (6.00, 38.0)
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Connections:
- removed net MPU_INT: A1.D3, J1.8
- net !SW2_INPUT: now also A1.D3; no longer A1.D4
Routing:
- net +5V: track 0.00 -> 79.0 mm, vias 0 -> 1
- net SW1_INT: track 0.00 -> 51.0 mm, vias 0 -> 2
- net !SW2_INPUT: track 0.00 -> 43.2 mm, vias 0 -> 1
- net GND: track 0.00 -> 12.3 mm, vias 0 -> 1
Other:
- board size 63 x 51.4 mm -> 54 x 45.4 mm

Commit message: Added curves to firmware board
Parts:
- moved J1 2.00 mm to (10.1, 3.06)
Routing:
- net GND: track 12.3 -> 0.00 mm, vias 1 -> 0
- net +5V: track 79.0 -> 77.0 mm
- net SDA: track 16.7 -> 15.0 mm
- net SCL: track 16.7 -> 15.0 mm
Other:
- board size 54 x 45.4 mm -> 54 x 45 mm
Changed lines of the file:
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@@
 <?xml version="1.0" encoding="utf-8"?>
 <!DOCTYPE eagle SYSTEM "eagle.dtd">
-<eagle version="9.5.1">
+<eagle version="9.6.2">
 <drawing>
 <settings>
@@
 <board>
 <plain>
-<wire x1="0" y1="0" x2="54" y2="0" width="0" layer="20"/>
-<wire x1="54" y1="45.4" x2="0" y2="45.4" width="0" layer="20"/>
-<wire x1="0" y1="45.4" x2="0" y2="0" width="0" layer="20"/>
+<wire x1="2" y1="0" x2="51" y2="0" width="0" layer="20"/>
 <text x="30" y="24" size="1.5" layer="22" font="vector" ratio="15" rot="MR270">2020 Training Board
 V2.0</text>
@@
 </polygon>
 <polygon width="0.1524" layer="21">
-<vertex x="6" y="3"/>
-<vertex x="5" y="2"/>
-<vertex x="5" y="4"/>
+<vertex x="8" y="3"/>
+<vertex x="7" y="2"/>
+<vertex x="7" y="4"/>
 </polygon>
-<text x="1" y="2" size="1.778" layer="21" font="vector" ratio="10">5V</text>
-<wire x1="54" y1="45.4" x2="54" y2="0" width="0" layer="20"/>
+<text x="4" y="2" size="1.778" layer="21" font="vector" ratio="10">5V</text>
+<wire x1="52" y1="45" x2="2" y2="45" width="0" layer="20"/>
+<wire x1="0" y1="43" x2="0" y2="2" width="0" layer="20"/>
+<wire x1="54" y1="43" x2="54" y2="3" width="0" layer="20"/>
+<wire x1="54" y1="3" x2="51" y2="0" width="0" layer="20" curve="-90"/>
+<wire x1="2" y1="45" x2="0" y2="43" width="0" layer="20" curve="90"/>
+<wire x1="0" y1="2" x2="2" y2="0" width="0" layer="20" curve="90"/>
+<wire x1="52" y1="45" x2="54" y2="43" width="0" layer="20" curve="-90"/>
 </plain>
 <attributes>
@@
 <element name="U$3" library="RoboJackets-Aesthetics" package="ROBOJACKETS" value="" x="17" y="2" smashed="yes" rot="R90"/>
 <element name="U$4" library="RoboJackets-Aesthetics" package="ROBOBUZZ_0.8X" value="" x="8" y="29" smashed="yes" rot="MR0"/>
-<element name="J1" library="SparkFun-Connectors" library_urn="urn:adsk.eagle:library:513" package="1X08" package3d_urn="urn:adsk.eagle:package:38138/1" value="GY-521-MPU-6050" x="8.11" y="3.06" smashed="yes" rot="R90">
-<attribute name="NAME" x="8.513" y="0.19" size="1" layer="25" font="vector" ratio="10" rot="R90"/>
-<attribute name="PROD_ID" value="CONN-08438" x="8.11" y="3.06" size="1.778" layer="27" rot="R90" display="off"/>
-<attribute name="VALUE" x="10.142" y="1.79" size="0.6096" layer="27" font="vector" ratio="20" rot="R90"/>
+<element name="J1" library="SparkFun-Connectors" library_urn="urn:adsk.eagle:library:513" package="1X08" package3d_urn="urn:adsk.eagle:package:38138/1" value="GY-521-MPU-6050" x="10.11" y="3.06" smashed="yes" rot="R90">
+<attribute name="NAME" x="8.133" y="20.27" size="1" layer="25" font="vector" ratio="10" rot="R90"/>
+<attribute name="PROD_ID" value="CONN-08438" x="10.11" y="3.06" size="1.778" layer="27" rot="R90" display="off"/>
+<attribute name="VALUE" x="12.142" y="1.79" size="0.6096" layer="27" font="vector" ratio="20" rot="R90"/>
 </element>
 <element name="D3" library="firmware_training_board" package="LED5MM" package3d_urn="urn:adsk.eagle:package:6240538/1" value="RED" x="49" y="25" smashed="yes">
@@
 </element>
 <element name="A1" library="firmware_training_board" package="NANO" value="NANO" x="28" y="22" smashed="yes">
-<attribute name="NAME" x="20" y="44" size="1" layer="25" font="vector" ratio="10"/>
+<attribute name="NAME" x="17" y="42" size="1" layer="25" font="vector" ratio="10"/>
 </element>
 </elements>
@@
 <polygon width="0.2" layer="16" thermals="no">
 <vertex x="0" y="0"/>
-<vertex x="54.201765625" y="0"/>
-<vertex x="54.201765625" y="45.4"/>
-<vertex x="0" y="45.4"/>
+<vertex x="54" y="0"/>
+<vertex x="54" y="45"/>
+<vertex x="0" y="45"/>
 </polygon>
 <contactref element="J1" pad="2"/>
@@
 <contactref element="A1" pad="GND"/>
 <contactref element="A1" pad="GND1"/>
-<wire x1="2.025" y1="24.75" x2="9.975" y2="24.75" width="0.2" layer="1"/>
-<wire x1="9.975" y1="24.75" x2="11" y2="23.725" width="0.2" layer="1"/>
-<wire x1="11" y1="23.725" x2="11" y2="23" width="0.2" layer="1"/>
-<wire x1="9.975" y1="24.75" x2="11" y2="23.725" width="0.2" layer="1"/>
-<wire x1="11" y1="23.725" x2="11" y2="23" width="0.2" layer="1"/>
-<via x="11" y="23" extent="1-16" drill="0.35"/>
+<wire x1="2.025" y1="24.75" x2="9.975" y2="24.75" width="0" layer="19" extent="1-1"/>
+<wire x1="14.95" y1="31" x2="9.975" y2="24.75" width="0" layer="19" extent="1-16"/>
 </signal>
 <signal name="+5V">
@@
 <contactref element="A1" pad="5V"/>
 <wire x1="2.025" y1="40.25" x2="9.975" y2="40.25" width="0.2" layer="1"/>
-<wire x1="8.11" y1="3.06" x2="11.06" y2="3.06" width="0.254" layer="1"/>
+<wire x1="10.11" y1="3.06" x2="11.06" y2="3.06" width="0.254" layer="1"/>
 <wire x1="19.3" y1="11.3" x2="20.38" y2="11.3" width="0.254" layer="1"/>
 <wire x1="11.06" y1="3.06" x2="19.3" y2="11.3" width="0.254" layer="1"/>
@@
 <contactref element="J1" pad="3"/>
 <contactref element="A1" pad="A5"/>
-<wire x1="8.11" y1="8.14" x2="18.89" y2="18.92" width="0.2" layer="1"/>
-<wire x1="18.89" y1="18.92" x2="20.38" y2="18.92" width="0.2" layer="1"/>
+<wire x1="20.38" y1="18.92" x2="20.38" y2="18.41" width="0.2" layer="1"/>
+<wire x1="20.38" y1="18.41" x2="10.11" y2="8.14" width="0.2" layer="1"/>
 </signal>
 <signal name="SDA">
 <contactref element="J1" pad="4"/>
 <contactref element="A1" pad="A4"/>
-<wire x1="8.11" y1="10.68" x2="18.89" y2="21.46" width="0.2" layer="1"/>
-<wire x1="18.89" y1="21.46" x2="20.38" y2="21.46" width="0.2" layer="1"/>
+<wire x1="20.38" y1="21.46" x2="20.38" y2="20.95" width="0.2" layer="1"/>
+<wire x1="20.38" y1="20.95" x2="10.11" y2="10.68" width="0.2" layer="1"/>
 </signal>
 <signal name="AD0">

Commit message: Moved parts to top
Parts:
- moved U$3 22.8 mm to (39.0, 8.00), flipped to the bottom
- moved U$4 22.2 mm to (5.00, 7.00), flipped to the top
- moved J1 3.00 mm to (13.1, 3.06)
- moved C1 1.00 mm to (15.0, 34.0), flipped to the top, turned to 0 degrees
- moved C2 1.00 mm to (15.0, 31.0), flipped to the top, turned to 0 degrees
- moved R10 1.00 mm to (15.0, 27.0), flipped to the top
- moved R8 1.00 mm to (15.0, 38.0), flipped to the top
Routing:
- net GND: track 0.00 -> 17.3 mm, vias 0 -> 4
- net +5V: track 77.0 -> 73.4 mm, vias 1 -> 0
- net SDA: track 15.0 -> 13.8 mm
- net SCL: track 15.0 -> 13.8 mm
- net !SW2_INPUT: track 43.2 -> 44.3 mm, vias 1 -> 2
- net SW1_INT: track 51.0 -> 50.2 mm

Commit message: Cleaned up silk screen
Parts:
- moved U$3 4.00 mm to (39.0, 4.00)
- moved U$4 1.00 mm to (5.00, 6.00)
Other:
- board text added: "INT"
- board text added: "VCC"
- board text removed: "5V"
Changed lines of the file:
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@@
 </polygon>
 <polygon width="0.1524" layer="21">
-<vertex x="8" y="3"/>
-<vertex x="7" y="2"/>
-<vertex x="7" y="4"/>
+<vertex x="11" y="3"/>
+<vertex x="10" y="2"/>
+<vertex x="10" y="4"/>
 </polygon>
-<text x="4" y="2" size="1.778" layer="21" font="vector" ratio="10">5V</text>
+<text x="7" y="3" size="1.778" layer="21" font="vector" ratio="10" align="center">VCC</text>
 <wire x1="52" y1="45" x2="2" y2="45" width="0" layer="20"/>
 <wire x1="0" y1="43" x2="0" y2="2" width="0" layer="20"/>
@@
 <wire x1="0" y1="2" x2="2" y2="0" width="0" layer="20" curve="90"/>
 <wire x1="52" y1="45" x2="54" y2="43" width="0" layer="20" curve="-90"/>
+<text x="7" y="21" size="1.778" layer="21" font="vector" ratio="10" align="center">INT</text>
+<polygon width="0.1524" layer="21">
+<vertex x="11" y="21"/>
+<vertex x="10" y="20"/>
+<vertex x="10" y="22"/>
+</polygon>
 </plain>
 <attributes>
@@
 </autorouter>
 <elements>
-<element name="U$3" library="RoboJackets-Aesthetics" package="ROBOJACKETS" value="" x="39" y="8" smashed="yes" rot="MR90"/>
-<element name="U$4" library="RoboJackets-Aesthetics" package="ROBOBUZZ_0.8X" value="" x="5" y="7" smashed="yes"/>
+<element name="U$3" library="RoboJackets-Aesthetics" package="ROBOJACKETS" value="" x="39" y="4" smashed="yes" rot="MR90"/>
+<element name="U$4" library="RoboJackets-Aesthetics" package="ROBOBUZZ_0.8X" value="" x="5" y="6" smashed="yes"/>
 <element name="J1" library="SparkFun-Connectors" library_urn="urn:adsk.eagle:library:513" package="1X08" package3d_urn="urn:adsk.eagle:package:38138/1" value="GY-521-MPU-6050" x="13.11" y="3.06" smashed="yes" rot="R90">
-<attribute name="NAME" x="11.133" y="20.27" size="1" layer="25" font="vector" ratio="10" rot="R90"/>
+<attribute name="NAME" x="16.133" y="2.27" size="1" layer="25" font="vector" ratio="10" rot="R90"/>
 <attribute name="PROD_ID" value="CONN-08438" x="13.11" y="3.06" size="1.778" layer="27" rot="R90" display="off"/>
 <attribute name="VALUE" x="15.142" y="1.79" size="0.6096" layer="27" font="vector" ratio="20" rot="R90"/>
 </element>
 <element name="D3" library="firmware_training_board" package="LED5MM" package3d_urn="urn:adsk.eagle:package:6240538/1" value="RED" x="49" y="25" smashed="yes">
-<attribute name="NAME" x="45" y="25" size="1.27" layer="25" font="vector" ratio="10" align="center-right"/>
+<attribute name="NAME" x="45" y="25" size="1.6764" layer="25" font="vector" ratio="15" align="center-right"/>
 <attribute name="VALUE" x="50.905" y="24.365" size="1.27" layer="27" rot="R90"/>
 </element>
 <element name="D4" library="firmware_training_board" package="LED5MM" package3d_urn="urn:adsk.eagle:package:6240538/1" value="RED" x="49" y="17" smashed="yes">
-<attribute name="NAME" x="45" y="17" size="1.27" layer="25" font="vector" ratio="10" align="center-right"/>
+<attribute name="NAME" x="45" y="17" size="1.6764" layer="25" font="vector" ratio="15" align="center-right"/>
 <attribute name="VALUE" x="50.905" y="16.365" size="1.27" layer="27" rot="R90"/>
 </element>
 <element name="D5" library="firmware_training_board" package="LED5MM" package3d_urn="urn:adsk.eagle:package:6240538/1" value="RED" x="49" y="9" smashed="yes">
-<attribute name="NAME" x="45" y="9" size="1.27" layer="25" font="vector" ratio="10" align="center-right"/>
+<attribute name="NAME" x="45" y="9" size="1.6764" layer="25" font="vector" ratio="15" align="center-right"/>
 <attribute name="VALUE" x="50.905" y="8.365" size="1.27" layer="27" rot="R90"/>
 </element>
 <element name="D1" library="adafruit" library_urn="urn:adsk.eagle:library:420" package="LED5MM" package3d_urn="urn:adsk.eagle:package:6240538/1" value="RED" x="49" y="41" smashed="yes">
-<attribute name="NAME" x="45" y="41" size="1.27" layer="25" font="vector" ratio="10" align="center-right"/>
+<attribute name="NAME" x="45" y="41" size="1.6764" layer="25" font="vector" ratio="15" align="center-right"/>
 <attribute name="VALUE" x="50.905" y="40.365" size="1.27" layer="27" rot="R90"/>
 </element>
 <element name="D2" library="firmware_training_board" package="LED5MM" package3d_urn="urn:adsk.eagle:package:6240538/1" value="RED" x="49" y="33" smashed="yes">
-<attribute name="NAME" x="45" y="33" size="1.27" layer="25" font="vector" ratio="10" align="center-right"/>
+<attribute name="NAME" x="45" y="33" size="1.6764" layer="25" font="vector" ratio="15" align="center-right"/>
 <attribute name="VALUE" x="50.905" y="32.365" size="1.27" layer="27" rot="R90"/>
 </element>
 <element name="SW1" library="RoboJackets-Switches" package="PTS645" value="PTS645" x="6" y="38" smashed="yes">
 <attribute name="FUNCTION" value="IN-1" x="6" y="38" size="1.778" layer="27" display="off"/>
-<attribute name="NAME" x="4.02" y="41.61" size="1.778" layer="25" font="vector" ratio="10"/>
+<attribute name="NAME" x="6" y="42" size="1.778" layer="25" font="vector" ratio="15" align="bottom-center"/>
 </element>
 <element name="C1" library="rcl" library_urn="urn:adsk.eagle:library:334" package="C0805" package3d_urn="urn:adsk.eagle:package:23617/2" value="0.1uF" x="15" y="34" smashed="yes">
@@
 <element name="SW2" library="RoboJackets-Switches" package="PTS645" value="PTS645" x="6" y="27" smashed="yes" rot="R180">
 <attribute name="FUNCTION" value="!IN-2" x="6" y="27" size="1.778" layer="27" rot="R180" display="off"/>
-<attribute name="NAME" x="8.38" y="32.49" size="1.778" layer="25" font="vector" ratio="10" rot="R180"/>
+<attribute name="NAME" x="6" y="31" size="1.778" layer="25" font="vector" ratio="15" align="bottom-center"/>
 </element>
 <element name="C2" library="rcl" library_urn="urn:adsk.eagle:library:334" package="C0805" package3d_urn="urn:adsk.eagle:package:23617/2" value="0.1uF" x="15" y="31" smashed="yes">
@@
 <element name="RN1" library="RoboJackets-Resistors" package="RA-8_2506" value="330" x="40" y="29.43" smashed="yes" rot="R270">
 <attribute name="DKPN" value="742C163331JPCT-ND" x="40" y="29.43" size="1.778" layer="27" rot="R270" display="off"/>
-<attribute name="NAME" x="38.62" y="24.37" size="1.27" layer="25" font="vector" ratio="10"/>
+<attribute name="NAME" x="40.63" y="33.62" size="1.27" layer="25" font="vector" ratio="10" rot="R90"/>
 <attribute name="POWER" value="62.5mW" x="40" y="29.43" size="1.778" layer="27" rot="R270" display="off"/>
 <attribute name="TOLERANCE" value="5%" x="40" y="29.43" size="1.778" layer="27" rot="R270" display="off"/>

Commit message: Fixed minor schematic notes, board silkscreen, and trace widths
Parts:
- renumbered R10 to R2, R8 to R1
Connections:
- net SW1_INT renamed SW1_INPUT
- removed net +3.3V: A1.3.3V
- removed net AD0: J1.7
Other:
- board text added: "2020 Firmware Training Board V2.0"
- board text removed: "2020 Training Board V2.0"
