File: board/firmware_training/firmware_training_board.brd (EAGLE design)
At the start: 54 x 45 mm, 16 parts, among them J1 GY-521-MPU-6050, SW1 PTS645, SW2 PTS645

Commit message: Removed extra net
Connections:
- removed net !RESET: A1.RST
Changed lines of the file:
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@@
 <drawing>
 <settings>
-<setting alwaysvectorfont="yes"/>
+<setting alwaysvectorfont="no"/>
 <setting verticaltext="up"/>
 </settings>
-<grid distance="50" unitdist="mil" unit="mm" style="lines" multiple="1" display="no" altdistance="5" altunitdist="mil" altunit="mm"/>
+<grid distance="50" unitdist="mil" unit="mil" style="lines" multiple="1" display="no" altdistance="5" altunitdist="mil" altunit="mil"/>
 <layers>
 <layer number="1" name="Top" color="4" fill="1" visible="yes" active="yes"/>
@@
 <wire x1="37.02" y1="31.62" x2="38.01" y2="30.63" width="0.2" layer="1"/>
 </signal>
-<signal name="!RESET">
-<contactref element="A1" pad="RST"/>
-</signal>
 </signals>
