File: board/firmware_training/firmware_training_board.sch (EAGLE design)
At the start: 15 parts, among them J1 GY-521-MPU-6050, SW1 PTS645, SW2 PTS645

Commit message: Finished schematic, started board
Parts:
- removed D6: GRN, led:LEDCHIP-LED0603
- A1: value ARDUINOR3-NOIOREF-NOTEXT -> NANO; device adafruit:ARDUINOR3-NOIOREF-NOTEXT -> firmware_training_board:NANO
- D1: device led:LEDCHIP-LED0603 -> adafruit:LED5MM
- D2, D3, D4, D5: device led:LEDCHIP-LED0603 -> firmware_training_board:LED5MM
Connections:
- net N$2 renamed D1_LED
- net N$3 renamed D2_LED
- net N$4 renamed D3_LED
- net N$5 renamed D4_LED
- net N$6 renamed D5_LED
- removed net N$9: D6.A, RN1.16
- net !RESET: now also A1.RST; no longer A1./RESET
- net +3.3V: now also A1.3.3V; no longer A1.3V
- net +5V: no longer RN1.15
- net GND: now also A1.GND; no longer A1.GND1, D6.C
- net MPU_INT: now also A1.D3; no longer A1.D2
- net SCL: now also A1.A5; no longer A1.A5/SCL
- net SDA: now also A1.A4; no longer A1.A4/SDA
- net SW1_INT: now also A1.D2; no longer A1.D3
Other:
- note added: "Arduino Nano Microcontroller"
- note added: "SCL and SDA - main I2C bus to MCU AD0 - sets I2C address. (Not Connected) MPU_INT - interrupt for new packet"
- note removed: "Arduino Uno Microcontroller"
- note removed: "From Adafruit Library"
- note removed: "SCL and SDA - main I2C bus to MCU. XCL and XDA - external I2C bus. This allows for an external magnetometer. AD0 - sets I2C address. (Not Connected) MPU_INT - interrupt for new packet"
- note removed: "Shows 5V Power"
- moved on the sheet: C1, C2, J1, R10, R8, RN1, SW1, SW2

Commit message: First finished version
Connections:
- removed net MPU_INT: A1.D3, J1.8
- net !SW2_INPUT: now also A1.D3; no longer A1.D4
Other:
- note added: "SCL and SDA - main I2C bus to MCU AD0 - sets I2C address. (Not Connected)"
- note removed: "SCL and SDA - main I2C bus to MCU AD0 - sets I2C address. (Not Connected) MPU_INT - interrupt for new packet"
Changed lines of the file:
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@@
 <?xml version="1.0" encoding="utf-8"?>
 <!DOCTYPE eagle SYSTEM "eagle.dtd">
-<eagle version="9.6.2">
+<eagle version="9.5.1">
 <drawing>
 <settings>
@@
 to noise.</text>
 <text x="185.42" y="248.92" size="1.27" layer="97" ratio="7">SCL and SDA - main I2C bus to MCU
-AD0 - sets I2C address. (Not Connected)
-MPU_INT - interrupt for new packet</text>
+AD0 - sets I2C address. (Not Connected)</text>
 <text x="81.28" y="152.4" size="1.27" layer="97" ratio="7">Connects to Pin D3 of Arduino</text>
 <text x="81.28" y="96.52" size="1.27" layer="97" ratio="7">Connects to Pin D4 of Arduino</text>
@@
 </segment>
 </net>
-<net name="MPU_INT" class="0">
-<segment>
-<pinref part="J1" gate="G$1" pin="8"/>
-<wire x1="152.4" y1="254" x2="167.64" y2="254" width="0.1524" layer="91"/>
-<label x="167.64" y="254" size="1.778" layer="95" xref="yes"/>
-</segment>
-<segment>
-<pinref part="A1" gate="G$1" pin="D3"/>
-<wire x1="76.2" y1="223.52" x2="99.06" y2="223.52" width="0.1524" layer="91"/>
-<label x="99.06" y="223.52" size="1.778" layer="95" xref="yes"/>
-</segment>
-</net>
 <net name="SW1_INT" class="0">
 <segment>
@@
 </segment>
 <segment>
-<pinref part="A1" gate="G$1" pin="D4"/>
-<wire x1="76.2" y1="226.06" x2="81.28" y2="226.06" width="0.1524" layer="91"/>
-<label x="81.28" y="226.06" size="1.778" layer="95" xref="yes"/>
-</segment>
-</net>
+<label x="99.06" y="223.52" size="1.778" layer="95" xref="yes"/>
+<wire x1="76.2" y1="223.52" x2="99.06" y2="223.52" width="0.1524" layer="91"/>
+<pinref part="A1" gate="G$1" pin="D3"/>
+</segment>
+</net>

Commit message: Changed tag size, edited descriptions in schematic
Other:
- note added: "A RC circuit is present for all buttons to provide debouncing. Debouncing is so that the signal will not change more than once per press due to an imperfect connection in the switch."
- note added: "Five user controlled LEDs are provided in common cathode configuration. Sending a logic '1' to these pins will cause the LED to turn on. All pins PWM capable."
- note removed: "A RC circuit is present for all buttons to provide debouncing. Debouncing is so that the function will not be triggered more than once per press due to noise."
- note removed: "Five user controlled LEDs are provided in common anode configuration. Sending a logic '1' to these pins will cause the LED to turn on. All pins PWM capable."
Changed lines of the file:
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@@
 <?xml version="1.0" encoding="utf-8"?>
 <!DOCTYPE eagle SYSTEM "eagle.dtd">
-<eagle version="9.5.1">
+<eagle version="9.6.2">
 <drawing>
 <settings>
@@
 <text x="12.7" y="261.62" size="6.4516" layer="97" ratio="7">Arduino Nano Microcontroller</text>
 <text x="231.14" y="187.96" size="1.27" layer="97" ratio="7">Five user controlled LEDs are provided in
-common anode configuration. Sending a
+common cathode configuration. Sending a
 logic '1' to these pins will cause the LED to
 turn on. All pins PWM capable.</text>
@@
 <text x="68.58" y="172.72" size="1.27" layer="97" ratio="7">A RC circuit is present for all buttons to
 provide debouncing.
-Debouncing is so that the function will not
-be triggered more than once per press due
-to noise.</text>
+Debouncing is so that the signal will not
+change more than once per press due
+to an imperfect connection in the switch.</text>
 <text x="185.42" y="248.92" size="1.27" layer="97" ratio="7">SCL and SDA - main I2C bus to MCU
 AD0 - sets I2C address. (Not Connected)</text>
@@
 <attribute name="NAME" x="142.24" y="257.048" size="1.778" layer="95"/>
 </instance>
-<instance part="SUPPLY1" gate="+5V" x="160.02" y="236.22" smashed="yes" rot="R270">
-<attribute name="VALUE" x="163.195" y="238.125" size="1.778" layer="96" rot="R270"/>
-</instance>
-<instance part="SUPPLY2" gate="GND" x="170.18" y="238.76" smashed="yes" rot="R90">
-<attribute name="VALUE" x="173.355" y="236.855" size="1.778" layer="96" rot="R90"/>
+<instance part="SUPPLY1" gate="+5V" x="167.64" y="236.22" smashed="yes" rot="R270">
+<attribute name="VALUE" x="170.815" y="238.125" size="1.778" layer="96" rot="R270"/>
+</instance>
+<instance part="SUPPLY2" gate="GND" x="175.26" y="238.76" smashed="yes" rot="R90">
+<attribute name="VALUE" x="178.435" y="236.855" size="1.778" layer="96" rot="R90"/>
 </instance>
 <instance part="D3" gate="G$1" x="287.02" y="231.14" smashed="yes" rot="R90">
@@
 <segment>
 <pinref part="J1" gate="G$1" pin="2"/>
-<wire x1="152.4" y1="238.76" x2="167.64" y2="238.76" width="0.1524" layer="91"/>
+<wire x1="152.4" y1="238.76" x2="172.72" y2="238.76" width="0.1524" layer="91"/>
 <pinref part="SUPPLY2" gate="GND" pin="GND"/>
 </segment>
@@
 <segment>
 <pinref part="J1" gate="G$1" pin="1"/>
-<wire x1="152.4" y1="236.22" x2="157.48" y2="236.22" width="0.1524" layer="91"/>
+<wire x1="152.4" y1="236.22" x2="165.1" y2="236.22" width="0.1524" layer="91"/>
 <pinref part="SUPPLY1" gate="+5V" pin="+5V"/>
 </segment>
@@
 <pinref part="RN1" gate="G$1" pin="3"/>
 <wire x1="264.16" y1="248.92" x2="261.62" y2="248.92" width="0.1524" layer="91"/>
-<label x="261.62" y="248.92" size="1.778" layer="95" rot="R180" xref="yes"/>
-</segment>
-<segment>
-<wire x1="76.2" y1="241.3" x2="99.06" y2="241.3" width="0.1524" layer="91"/>
-<label x="99.06" y="241.3" size="1.778" layer="95" xref="yes"/>
+<label x="261.62" y="248.92" size="1.27" layer="95" rot="R180" xref="yes"/>
+</segment>
+<segment>
+<wire x1="76.2" y1="241.3" x2="81.28" y2="241.3" width="0.1524" layer="91"/>
+<label x="81.28" y="241.3" size="1.27" layer="95" xref="yes"/>
 <pinref part="A1" gate="G$1" pin="D10"/>
 </segment>
@@
 <net name="D5_CTRL" class="0">
 <segment>
-<wire x1="76.2" y1="228.6" x2="99.06" y2="228.6" width="0.1524" layer="91"/>
-<label x="99.06" y="228.6" size="1.778" layer="95" xref="yes"/>
+<wire x1="76.2" y1="228.6" x2="81.28" y2="228.6" width="0.1524" layer="91"/>
+<label x="81.28" y="228.6" size="1.27" layer="95" xref="yes"/>
 <pinref part="A1" gate="G$1" pin="D5"/>
 </segment>
 <segment>
-<wire x1="264.16" y1="241.3" x2="246.38" y2="241.3" width="0.1524" layer="91"/>
-<label x="246.38" y="241.3" size="1.778" layer="95" rot="R180" xref="yes"/>
+<wire x1="264.16" y1="241.3" x2="261.62" y2="241.3" width="0.1524" layer="91"/>
+<label x="261.62" y="241.3" size="1.27" layer="95" rot="R180" xref="yes"/>
 <pinref part="RN1" gate="G$1" pin="9"/>
 </segment>
@@
 <pinref part="J1" gate="G$1" pin="3"/>
 <wire x1="152.4" y1="241.3" x2="157.48" y2="241.3" width="0.1524" layer="91"/>
-<label x="157.48" y="241.3" size="1.778" layer="95" xref="yes"/>
+<label x="157.48" y="241.3" size="1.27" layer="95" xref="yes"/>
 </segment>
 <segment>
 <wire x1="43.18" y1="226.06" x2="38.1" y2="226.06" width="0.1524" layer="91"/>
-<label x="38.1" y="226.06" size="1.778" layer="95" rot="R180" xref="yes"/>
+<label x="38.1" y="226.06" size="1.27" layer="95" rot="R180" xref="yes"/>
 <pinref part="A1" gate="G$1" pin="A5"/>
 </segment>
@@
 <segment>
 <pinref part="J1" gate="G$1" pin="4"/>
-<wire x1="152.4" y1="243.84" x2="167.64" y2="243.84" width="0.1524" layer="91"/>
-<label x="167.64" y="243.84" size="1.778" layer="95" xref="yes"/>
+<wire x1="152.4" y1="243.84" x2="157.48" y2="243.84" width="0.1524" layer="91"/>
+<label x="157.48" y="243.84" size="1.27" layer="95" xref="yes"/>
 </segment>
 <segment>
 <wire x1="43.18" y1="228.6" x2="38.1" y2="228.6" width="0.1524" layer="91"/>
-<wire x1="38.1" y1="228.6" x2="38.1" y2="231.14" width="0.1524" layer="91"/>
-<label x="38.1" y="231.14" size="1.778" layer="95" rot="R180" xref="yes"/>
+<label x="38.1" y="228.6" size="1.27" layer="95" rot="R180" xref="yes"/>
 <pinref part="A1" gate="G$1" pin="A4"/>
 </segment>
@@
 <pinref part="J1" gate="G$1" pin="7"/>
 <wire x1="152.4" y1="251.46" x2="157.48" y2="251.46" width="0.1524" layer="91"/>
-<label x="157.48" y="251.46" size="1.778" layer="95" xref="yes"/>
+<label x="157.48" y="251.46" size="1.27" layer="95" xref="yes"/>
 </segment>
 </net>
@@
 <segment>
 <wire x1="264.16" y1="243.84" x2="261.62" y2="243.84" width="0.1524" layer="91"/>
-<label x="261.62" y="243.84" size="1.778" layer="95" rot="R180" xref="yes"/>
+<label x="261.62" y="243.84" size="1.27" layer="95" rot="R180" xref="yes"/>
 <pinref part="RN1" gate="G$1" pin="7"/>
 </segment>
 <segment>
 <wire x1="76.2" y1="231.14" x2="81.28" y2="231.14" width="0.1524" layer="91"/>
-<label x="81.28" y="231.14" size="1.778" layer="95" xref="yes"/>
+<label x="81.28" y="231.14" size="1.27" layer="95" xref="yes"/>
 <pinref part="A1" gate="G$1" pin="D6"/>
 </segment>
@@
 <wire x1="66.04" y1="147.32" x2="76.2" y2="147.32" width="0.1524" layer="91"/>
 <pinref part="C1" gate="G$1" pin="1"/>
-<label x="81.28" y="147.32" size="1.778" layer="95" xref="yes"/>
+<label x="81.28" y="147.32" size="1.27" layer="95" xref="yes"/>
 <pinref part="R8" gate="G$1" pin="1"/>
 <wire x1="76.2" y1="147.32" x2="81.28" y2="147.32" width="0.1524" layer="91"/>
@@
 <segment>
 <wire x1="76.2" y1="220.98" x2="81.28" y2="220.98" width="0.1524" layer="91"/>
-<label x="81.28" y="220.98" size="1.778" layer="95" xref="yes"/>
+<label x="81.28" y="220.98" size="1.27" layer="95" xref="yes"/>
 <pinref part="A1" gate="G$1" pin="D2"/>
 </segment>
@@
 <pinref part="C2" gate="G$1" pin="1"/>
 <pinref part="R10" gate="G$1" pin="1"/>
-<label x="81.28" y="91.44" size="1.778" layer="95" xref="yes"/>
+<label x="81.28" y="91.44" size="1.27" layer="95" xref="yes"/>
 <pinref part="SW2" gate="G$1" pin="2"/>
 <wire x1="66.04" y1="91.44" x2="43.18" y2="91.44" width="0.1524" layer="91"/>
 </segment>
 <segment>
-<label x="99.06" y="223.52" size="1.778" layer="95" xref="yes"/>
-<wire x1="76.2" y1="223.52" x2="99.06" y2="223.52" width="0.1524" layer="91"/>
+<label x="81.28" y="223.52" size="1.27" layer="95" xref="yes"/>
+<wire x1="76.2" y1="223.52" x2="81.28" y2="223.52" width="0.1524" layer="91"/>
 <pinref part="A1" gate="G$1" pin="D3"/>
 </segment>
@@
 <net name="!RESET" class="0">
 <segment>
-<wire x1="43.18" y1="215.9" x2="35.56" y2="215.9" width="0.1524" layer="91"/>
-<label x="35.56" y="215.9" size="1.778" layer="95" rot="R180" xref="yes"/>
+<wire x1="43.18" y1="215.9" x2="38.1" y2="215.9" width="0.1524" layer="91"/>
+<label x="38.1" y="215.9" size="1.27" layer="95" rot="R180" xref="yes"/>
 <pinref part="A1" gate="G$1" pin="RST"/>
 </segment>
@@
 <segment>
 <wire x1="76.2" y1="243.84" x2="81.28" y2="243.84" width="0.1524" layer="91"/>
-<label x="81.28" y="243.84" size="1.778" layer="95" xref="yes"/>
+<label x="81.28" y="243.84" size="1.27" layer="95" xref="yes"/>
 <pinref part="A1" gate="G$1" pin="D11"/>
 </segment>
 <segment>
-<wire x1="264.16" y1="251.46" x2="246.38" y2="251.46" width="0.1524" layer="91"/>
-<label x="246.38" y="251.46" size="1.778" layer="95" rot="R180" xref="yes"/>
+<wire x1="264.16" y1="251.46" x2="261.62" y2="251.46" width="0.1524" layer="91"/>
+<label x="261.62" y="251.46" size="1.27" layer="95" rot="R180" xref="yes"/>
 <pinref part="RN1" gate="G$1" pin="1"/>
 </segment>
@@
 <segment>
 <wire x1="76.2" y1="238.76" x2="81.28" y2="238.76" width="0.1524" layer="91"/>
-<label x="81.28" y="238.76" size="1.778" layer="95" xref="yes"/>
+<label x="81.28" y="238.76" size="1.27" layer="95" xref="yes"/>
 <pinref part="A1" gate="G$1" pin="D9"/>
 </segment>
 <segment>
-<wire x1="264.16" y1="246.38" x2="246.38" y2="246.38" width="0.1524" layer="91"/>
-<label x="246.38" y="246.38" size="1.778" layer="95" rot="R180" xref="yes"/>
+<wire x1="264.16" y1="246.38" x2="261.62" y2="246.38" width="0.1524" layer="91"/>
+<label x="261.62" y="246.38" size="1.27" layer="95" rot="R180" xref="yes"/>
 <pinref part="RN1" gate="G$1" pin="5"/>
 </segment>

Commit message: Fixed minor schematic notes, board silkscreen, and trace widths
Parts:
- renumbered R10 to R2, R8 to R1
Connections:
- net SW1_INT renamed SW1_INPUT
- removed net +3.3V: A1.3.3V
- removed net AD0: J1.7
Other:
- note added: "Connects to Pin D2 of Arduino"
- note added: "SW2 is pulled low with a normally open momentary pushbutton. When you push on the button, the digital value will be a 0. When you do not push on the button, the digital value will be a 1. SW2 is also connected to an interrupt pin."
- note removed: "Connects to Pin D4 of Arduino"
- note removed: "SW2 is pulled low with a normally open momentary pushbutton. When you push on the button, the digital value will be a 0. When you do not push on the button, the digital value will be a 1."
Changed lines of the file:
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@@
 <part name="SUPPLY3" library="supply2" library_urn="urn:adsk.eagle:library:372" deviceset="+5V" device=""/>
 <part name="C1" library="rcl" library_urn="urn:adsk.eagle:library:334" deviceset="C-US" device="C0805" package3d_urn="urn:adsk.eagle:package:23617/2" value="0.1uF"/>
-<part name="R8" library="rcl" library_urn="urn:adsk.eagle:library:334" deviceset="R-US_" device="R0603" package3d_urn="urn:adsk.eagle:package:23555/3" value="10K"/>
+<part name="R1" library="rcl" library_urn="urn:adsk.eagle:library:334" deviceset="R-US_" device="R0603" package3d_urn="urn:adsk.eagle:package:23555/3" value="10K"/>
 <part name="SUPPLY7" library="supply2" library_urn="urn:adsk.eagle:library:372" deviceset="GND" device=""/>
 <part name="SW2" library="RoboJackets-Switches" deviceset="PTS645" device="">
@@
 </part>
 <part name="C2" library="rcl" library_urn="urn:adsk.eagle:library:334" deviceset="C-US" device="C0805" package3d_urn="urn:adsk.eagle:package:23617/2" value="0.1uF"/>
-<part name="R10" library="rcl" library_urn="urn:adsk.eagle:library:334" deviceset="R-US_" device="R0603" package3d_urn="urn:adsk.eagle:package:23555/3" value="10K"/>
+<part name="R2" library="rcl" library_urn="urn:adsk.eagle:library:334" deviceset="R-US_" device="R0603" package3d_urn="urn:adsk.eagle:package:23555/3" value="10K"/>
 <part name="SUPPLY11" library="supply2" library_urn="urn:adsk.eagle:library:372" deviceset="+5V" device=""/>
 <part name="SUPPLY12" library="supply2" library_urn="urn:adsk.eagle:library:372" deviceset="GND" device=""/>
 <part name="SUPPLY10" library="supply2" library_urn="urn:adsk.eagle:library:372" deviceset="GND" device=""/>
-<part name="SUPPLY8" library="RoboJackets-Supplies" deviceset="+3.3V" device=""/>
 <part name="SUPPLY6" library="supply2" library_urn="urn:adsk.eagle:library:372" deviceset="GND" device=""/>
 <part name="RN1" library="RoboJackets-Resistors" deviceset="RA-8" device="2506" value="330">
@@
 <text x="12.7" y="185.42" size="6.4516" layer="97" ratio="7">Buttons</text>
 <text x="228.6" y="261.62" size="6.4516" layer="97" ratio="7">LEDs</text>
-<text x="12.7" y="104.14" size="1.27" layer="97" ratio="7">SW2 is pulled low with a normally open momentary pushbutton.
+<text x="12.7" y="101.6" size="1.27" layer="97" ratio="7">SW2 is pulled low with a normally open momentary pushbutton.
 When you push on the button, the digital value will be a 0.
-When you do not push on the button, the digital value will be a 1.</text>
+When you do not push on the button, the digital value will be a 1.
+SW2 is also connected to an interrupt pin.</text>
 <text x="68.58" y="172.72" size="1.27" layer="97" ratio="7">A RC circuit is present for all buttons to
 provide debouncing.
@@
 <text x="185.42" y="248.92" size="1.27" layer="97" ratio="7">SCL and SDA - main I2C bus to MCU
 AD0 - sets I2C address. (Not Connected)</text>
-<text x="81.28" y="152.4" size="1.27" layer="97" ratio="7">Connects to Pin D3 of Arduino</text>
-<text x="81.28" y="96.52" size="1.27" layer="97" ratio="7">Connects to Pin D4 of Arduino</text>
+<text x="81.28" y="152.4" size="1.27" layer="97" ratio="7">Connects to Pin D2 of Arduino</text>
+<text x="81.28" y="96.52" size="1.27" layer="97" ratio="7">Connects to Pin D3 of Arduino</text>
 <wire x1="298.45" y1="180.594" x2="298.45" y2="271.78" width="0.1524" layer="97" style="shortdash"/>
 <wire x1="224.79" y1="180.594" x2="224.79" y2="271.78" width="0.1524" layer="97" style="shortdash"/>
@@
 <attribute name="VALUE" x="67.056" y="138.049" size="1.778" layer="96"/>
 </instance>
-<instance part="R8" gate="G$1" x="76.2" y="139.7" smashed="yes" rot="R270">
+<instance part="R1" gate="G$1" x="76.2" y="139.7" smashed="yes" rot="R270">
 <attribute name="NAME" x="77.978" y="140.6906" size="1.778" layer="95"/>
 <attribute name="VALUE" x="77.978" y="137.922" size="1.778" layer="96"/>
@@
 <attribute name="VALUE" x="67.056" y="82.169" size="1.778" layer="96"/>
 </instance>
-<instance part="R10" gate="G$1" x="66.04" y="99.06" smashed="yes" rot="R90">
+<instance part="R2" gate="G$1" x="66.04" y="99.06" smashed="yes" rot="R90">
 <attribute name="NAME" x="67.818" y="100.0506" size="1.778" layer="95"/>
 <attribute name="VALUE" x="67.818" y="97.536" size="1.778" layer="96"/>
@@
 <instance part="SUPPLY10" gate="GND" x="30.48" y="76.2" smashed="yes">
 <attribute name="VALUE" x="28.575" y="73.025" size="1.778" layer="96"/>
-</instance>
-<instance part="SUPPLY8" gate="P" x="25.4" y="248.92" smashed="yes">
-<attribute name="VALUE" x="23.495" y="252.095" size="1.778" layer="96"/>
 </instance>
 <instance part="SUPPLY6" gate="GND" x="76.2" y="129.54" smashed="yes">
@@
 </segment>
 <segment>
-<pinref part="R8" gate="G$1" pin="2"/>
+<pinref part="R1" gate="G$1" pin="2"/>
 <wire x1="76.2" y1="134.62" x2="76.2" y2="132.08" width="0.1524" layer="91"/>
 <pinref part="SUPPLY6" gate="GND" pin="GND"/>
@@
 </segment>
 <segment>
-<pinref part="R10" gate="G$1" pin="2"/>
+<pinref part="R2" gate="G$1" pin="2"/>
 <wire x1="66.04" y1="104.14" x2="66.04" y2="106.68" width="0.1524" layer="91"/>
 <pinref part="SUPPLY11" gate="+5V" pin="+5V"/>
@@
 </segment>
 </net>
-<net name="AD0" class="0">
-<segment>
-<pinref part="J1" gate="G$1" pin="7"/>
-<wire x1="152.4" y1="251.46" x2="157.48" y2="251.46" width="0.1524" layer="91"/>
-<label x="157.48" y="251.46" size="1.27" layer="95" xref="yes"/>
-</segment>
-</net>
 <net name="D4_CTRL" class="0">
 <segment>
@@
 </segment>
 </net>
-<net name="SW1_INT" class="0">
+<net name="SW1_INPUT" class="0">
 <segment>
 <wire x1="66.04" y1="147.32" x2="66.04" y2="144.78" width="0.1524" layer="91"/>
@@
 <pinref part="C1" gate="G$1" pin="1"/>
 <label x="81.28" y="147.32" size="1.27" layer="95" xref="yes"/>
-<pinref part="R8" gate="G$1" pin="1"/>
+<pinref part="R1" gate="G$1" pin="1"/>
 <wire x1="76.2" y1="147.32" x2="81.28" y2="147.32" width="0.1524" layer="91"/>
 <wire x1="76.2" y1="144.78" x2="76.2" y2="147.32" width="0.1524" layer="91"/>
@@
 <wire x1="66.04" y1="91.44" x2="81.28" y2="91.44" width="0.1524" layer="91"/>
 <pinref part="C2" gate="G$1" pin="1"/>
-<pinref part="R10" gate="G$1" pin="1"/>
+<pinref part="R2" gate="G$1" pin="1"/>
 <label x="81.28" y="91.44" size="1.27" layer="95" xref="yes"/>
 <pinref part="SW2" gate="G$1" pin="2"/>
@@
 </segment>
 </net>
-<net name="+3.3V" class="0">
-<segment>
-<wire x1="43.18" y1="243.84" x2="25.4" y2="243.84" width="0.1524" layer="91"/>
-<wire x1="25.4" y1="243.84" x2="25.4" y2="246.38" width="0.1524" layer="91"/>
-<pinref part="SUPPLY8" gate="P" pin="+3.3V"/>
-<pinref part="A1" gate="G$1" pin="3.3V"/>
-</segment>
-</net>

Commit message: Removed extra net
Connections:
- removed net !RESET: A1.RST
Changed lines of the file:
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@@
-</segment>
-</net>
-<net name="!RESET" class="0">
-<segment>
-<wire x1="43.18" y1="215.9" x2="38.1" y2="215.9" width="0.1524" layer="91"/>
-<label x="38.1" y="215.9" size="1.27" layer="95" rot="R180" xref="yes"/>
-<pinref part="A1" gate="G$1" pin="RST"/>
 </segment>
 </net>
