File: board/soldering_training/training_board.sch (EAGLE design)
At the start: 22 parts, among them J1 MAIN_PWR, Q1 ARDUINOR3-NOIOREF-NOTEXT, Q2 DMN2056U, SW2 PTS645, U1 DRV8871HSOP-8

Commit message: Fixed soldering training board resistor to common value
Parts:
- R7: value 128K -> 120K
Other:
- note added: "Based on the formula on pg 9 of the datasheet, this limits current to 0.53A before enabling the internal current limit"
- note removed: "Based on the formula on pg 9 of the datasheet, this limits current to 0.5A before enabling the internal current limit"
Changed lines of the file:
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@@
 <?xml version="1.0" encoding="utf-8"?>
 <!DOCTYPE eagle SYSTEM "eagle.dtd">
-<eagle version="9.5.2">
+<eagle version="9.6.2">
 <drawing>
 <settings>
@@
 <part name="SUPPLY3" library="supply2" library_urn="urn:adsk.eagle:library:372" deviceset="+12V" device=""/>
 <part name="SUPPLY5" library="supply2" library_urn="urn:adsk.eagle:library:372" deviceset="+5V" device=""/>
-<part name="R7" library="rcl" library_urn="urn:adsk.eagle:library:334" deviceset="R-US_" device="R0603" package3d_urn="urn:adsk.eagle:package:23555/3" value="128K"/>
+<part name="R7" library="rcl" library_urn="urn:adsk.eagle:library:334" deviceset="R-US_" device="R0603" package3d_urn="urn:adsk.eagle:package:23555/3" value="120K"/>
 <part name="SUPPLY12" library="supply2" library_urn="urn:adsk.eagle:library:372" deviceset="GND" device=""/>
 <part name="SUPPLY13" library="supply2" library_urn="urn:adsk.eagle:library:372" deviceset="GND" device=""/>
@@
 the transistor's gate and shuts the chip down.</text>
 <text x="238.76" y="142.24" size="1.27" layer="97" ratio="7">Based on the formula on pg 9 of the
-datasheet, this limits current to 0.5A
+datasheet, this limits current to 0.53A
 before enabling the internal current limit</text>
 <wire x1="149.86" y1="127.254" x2="149.86" y2="211.328" width="0.1524" layer="97"/>

Commit message: Fixed font and ERC
Parts:
- S1: value (none) -> EG1903-ND
Changed lines of the file:
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@@
 <part name="FRAME1" library="RoboJackets-Frames" deviceset="FRAME_A_L" device="">
 <attribute name="AUTHOR" value="Varun Madabushi"/>
-<attribute name="REVISION" value="1.3"/>
+<attribute name="REVISION" value="1.5"/>
 <attribute name="SCH_DESC" value="Arduino Motor Control Shield"/>
 <attribute name="TEAM" value="Electrical Training"/>
@@
 <part name="Q2" library="RoboJackets-Discrete" deviceset="NMOS" device="SOT-23-3" value="DMN2056U"/>
 <part name="R6" library="rcl" library_urn="urn:adsk.eagle:library:334" deviceset="R-US_" device="R0603" package3d_urn="urn:adsk.eagle:package:23555/3" value="10K"/>
-<part name="S1" library="adafruit" library_urn="urn:adsk.eagle:library:420" deviceset="EG1218" device="S" package3d_urn="urn:adsk.eagle:package:6240649/1"/>
+<part name="S1" library="adafruit" library_urn="urn:adsk.eagle:library:420" deviceset="EG1218" device="S" package3d_urn="urn:adsk.eagle:package:6240649/1" value="EG1903-ND"/>
 <part name="SUPPLY3" library="supply2" library_urn="urn:adsk.eagle:library:372" deviceset="+12V" device=""/>
 <part name="SUPPLY5" library="supply2" library_urn="urn:adsk.eagle:library:372" deviceset="+5V" device=""/>
@@
 <sheet>
 <plain>
-<text x="58.42" y="86.36" size="1.27" layer="97" font="vector" ratio="7">From Adafruit Library</text>
+<text x="58.42" y="86.36" size="1.27" layer="97" ratio="7">From Adafruit Library</text>
 <wire x1="173.99" y1="43.18" x2="173.99" y2="127.254" width="0.1524" layer="97"/>
 <wire x1="-6.096" y1="127.254" x2="173.99" y2="127.254" width="0.1524" layer="97"/>
@@
 with .35A no-load current and 1.3A stall current
 No intended mechanism for this motor so should be fine.</text>
-<text x="27.94" y="154.94" size="1.27" layer="97" font="vector" ratio="7">The top part of this symbol represents the pin inside the
+<text x="27.94" y="154.94" size="1.27" layer="97" ratio="7">The top part of this symbol represents the pin inside the
 barrel jack (usually positive), while the
 bottom represents the spring-loaded tab
 that contacts the outside (usually negative).  </text>
-<text x="88.9" y="182.88" size="1.27" layer="97" font="vector" ratio="7">Decoupling capacitors help ensure a
+<text x="88.9" y="182.88" size="1.27" layer="97" ratio="7">Decoupling capacitors help ensure a
 relatively constant output voltage even in
 the event of current spikes</text>
@@
 </instance>
 <instance part="J1" gate="G$1" x="68.58" y="170.18" smashed="yes">
-<attribute name="NAME" x="58.42" y="177.8" size="1.778" layer="96" font="vector"/>
-<attribute name="VALUE" x="58.42" y="165.1" size="1.778" layer="96" font="vector"/>
+<attribute name="NAME" x="58.42" y="177.8" size="1.778" layer="96"/>
+<attribute name="VALUE" x="58.42" y="165.1" size="1.778" layer="96"/>
 </instance>
 <instance part="SUPPLY6" gate="+12V" x="81.28" y="180.34" smashed="yes">
@@
 </instance>
 <instance part="SUPPLY7" gate="GND" x="81.28" y="162.56" smashed="yes">
-<attribute name="VALUE" x="79.375" y="159.385" size="1.778" layer="96" font="vector"/>
+<attribute name="VALUE" x="79.375" y="159.385" size="1.778" layer="96"/>
 </instance>
 <instance part="SUPPLY9" gate="GND" x="35.56" y="43.18" smashed="yes">
@@
 </instance>
 <instance part="SW2" gate="G$1" x="22.86" y="58.42" smashed="yes">
-<attribute name="NAME" x="20.32" y="62.23" size="1.778" layer="96" font="vector"/>
-<attribute name="VALUE" x="22.86" y="57.15" size="1.778" layer="96" font="vector" align="top-center"/>
-<attribute name="FUNCTION" x="22.86" y="54.102" size="1.778" layer="96" font="vector" align="top-center"/>
+<attribute name="NAME" x="20.32" y="62.23" size="1.778" layer="96"/>
+<attribute name="VALUE" x="22.86" y="57.15" size="1.778" layer="96" align="top-center"/>
+<attribute name="FUNCTION" x="22.86" y="54.102" size="1.778" layer="96" align="top-center"/>
 </instance>
 <instance part="SUPPLY8" gate="GND" x="15.24" y="53.34" smashed="yes">
 <attribute name="VALUE" x="13.335" y="50.165" size="1.778" layer="96"/>
 </instance>
-<instance part="SUPPLY10" gate="GND" x="226.06" y="96.52" smashed="yes">
-<attribute name="VALUE" x="224.155" y="93.345" size="1.778" layer="96"/>
+<instance part="SUPPLY10" gate="GND" x="226.06" y="93.98" smashed="yes">
+<attribute name="VALUE" x="224.155" y="90.805" size="1.778" layer="96"/>
 </instance>
 <instance part="SUPPLY11" gate="+12V" x="180.34" y="177.8" smashed="yes">
@@
 <instance part="FRAME1" gate="G$1" x="0" y="0" smashed="yes"/>
 <instance part="FRAME1" gate="G$2" x="173.99" y="0" smashed="yes">
-<attribute name="LAST_DATE_TIME" x="186.69" y="1.27" size="2.54" layer="94" font="vector"/>
-<attribute name="SHEET" x="260.35" y="1.27" size="2.54" layer="94" font="vector"/>
-<attribute name="DRAWING_NAME" x="186.69" y="19.05" size="2.54" layer="94" font="vector"/>
+<attribute name="LAST_DATE_TIME" x="186.69" y="1.27" size="2.54" layer="94"/>
+<attribute name="SHEET" x="260.35" y="1.27" size="2.54" layer="94"/>
+<attribute name="DRAWING_NAME" x="186.69" y="19.05" size="2.54" layer="94"/>
 <attribute name="SCH_DESC" x="175.26" y="6.35" size="2.54" layer="94"/>
 <attribute name="TEAM" x="175.26" y="31.75" size="3.048" layer="94" ratio="10" align="top-left"/>
@@
 <instance part="C1" gate="G$1" x="93.98" y="172.72" smashed="yes">
 <attribute name="NAME" x="94.996" y="173.355" size="1.778" layer="95"/>
-<attribute name="VALUE" x="94.996" y="168.529" size="1.778" layer="96" font="vector"/>
+<attribute name="VALUE" x="94.996" y="168.529" size="1.778" layer="96"/>
 </instance>
 <instance part="C2" gate="G$1" x="109.22" y="172.72" smashed="yes">
 <attribute name="NAME" x="110.236" y="173.355" size="1.778" layer="95"/>
-<attribute name="VALUE" x="110.236" y="168.529" size="1.778" layer="96" font="vector"/>
+<attribute name="VALUE" x="110.236" y="168.529" size="1.778" layer="96"/>
 </instance>
 <instance part="C3" gate="G$1" x="43.18" y="58.42" smashed="yes">
@@
 </instance>
 <instance part="Q2" gate="G$1" x="226.06" y="119.38" smashed="yes">
-<attribute name="VALUE" x="228.6" y="119.38" size="1.778" layer="95" font="vector"/>
-<attribute name="NAME" x="228.6" y="121.92" size="1.778" layer="95" font="vector"/>
+<attribute name="VALUE" x="228.6" y="119.38" size="1.778" layer="95"/>
+<attribute name="NAME" x="228.6" y="121.92" size="1.778" layer="95"/>
 </instance>
 <instance part="R6" gate="G$1" x="218.44" y="109.22" smashed="yes" rot="R270">
@@
 <instance part="S1" gate="1" x="208.28" y="121.92" smashed="yes" rot="R270">
 <attribute name="NAME" x="206.375" y="115.57" size="1.778" layer="95"/>
-<attribute name="VALUE" x="211.455" y="125.73" size="1.778" layer="96"/>
 </instance>
 <instance part="SUPPLY3" gate="+12V" x="200.66" y="124.46" smashed="yes">
@@
 <wire x1="226.06" y1="114.3" x2="226.06" y2="101.6" width="0.1524" layer="91"/>
 <wire x1="226.06" y1="101.6" x2="226.06" y2="96.52" width="0.1524" layer="91"/>
-<wire x1="226.06" y1="96.52" x2="226.06" y2="99.06" width="0.1524" layer="91"/>
 <pinref part="R6" gate="G$1" pin="2"/>
 <wire x1="218.44" y1="104.14" x2="218.44" y2="101.6" width="0.1524" layer="91"/>

Commit message: Renamed SW2 to SW1
Parts:
- renumbered SW2 to SW1
Changed lines of the file:
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@@
 <part name="SUPPLY7" library="supply2" library_urn="urn:adsk.eagle:library:372" deviceset="GND" device=""/>
 <part name="SUPPLY9" library="supply2" library_urn="urn:adsk.eagle:library:372" deviceset="GND" device=""/>
-<part name="SW2" library="RoboJackets-Switches" deviceset="PTS645" device="">
+<part name="SW1" library="RoboJackets-Switches" deviceset="PTS645" device="">
 <attribute name="FUNCTION" value="RESET"/>
 </part>
@@
 <attribute name="VALUE" x="33.655" y="40.005" size="1.778" layer="96"/>
 </instance>
-<instance part="SW2" gate="G$1" x="22.86" y="58.42" smashed="yes">
+<instance part="SW1" gate="G$1" x="22.86" y="58.42" smashed="yes">
 <attribute name="NAME" x="20.32" y="62.23" size="1.778" layer="96"/>
 <attribute name="VALUE" x="22.86" y="57.15" size="1.778" layer="96" align="top-center"/>
@@
 </segment>
 <segment>
-<pinref part="SW2" gate="G$1" pin="1"/>
+<pinref part="SW1" gate="G$1" pin="1"/>
 <wire x1="17.78" y1="58.42" x2="15.24" y2="58.42" width="0.1524" layer="91"/>
 <wire x1="15.24" y1="58.42" x2="15.24" y2="55.88" width="0.1524" layer="91"/>
@@
 <wire x1="48.26" y1="58.42" x2="53.34" y2="58.42" width="0.1524" layer="91"/>
 <wire x1="48.26" y1="58.42" x2="48.26" y2="63.5" width="0.1524" layer="91"/>
-<pinref part="SW2" gate="G$1" pin="2"/>
+<pinref part="SW1" gate="G$1" pin="2"/>
 <wire x1="27.94" y1="58.42" x2="33.02" y2="58.42" width="0.1524" layer="91"/>
 <wire x1="33.02" y1="58.42" x2="33.02" y2="63.5" width="0.1524" layer="91"/>

Commit message: Fixed minor issues and made roboBuzz bigger
Parts:
- C3: value 0.1uF 6V -> 0.1uF 16V
- LED2: value ORANGE -> GREEN
- LED3: value GREEN -> ORANGE
- Q1: value ARDUINOR3-NOIOREF-NOTEXT -> DMN2056U; device adafruit:ARDUINOR3-NOIOREF-NOTEXT -> RoboJackets-Discrete:NMOSSOT-23-3
- Q2: value DMN2056U -> ARDUINOR3-NOIOREF-NOTEXT; device RoboJackets-Discrete:NMOSSOT-23-3 -> adafruit:ARDUINOR3-NOIOREF-NOTEXT
- R1: value 2.4K -> 1K
- R2: value 1K -> 2.4K
- R5: value 2.4K -> 120K
- R7: value 120K -> 2.4K
Connections:
- removed net N$16 (its old number): LED3.A, R5.1
- new net N$15: LED3.A, R3.1
- net +12V: now also Q2.VIN, R2.2; no longer Q1.VIN, R5.2
- net +5V: now also Q2.5V, R6.2; no longer Q1.5V, R4.2
- net GND: now also Q1.S, Q2.GND1, Q2.GND2, R4.2, R5.2; no longer Q1.GND1, Q1.GND2, Q2.S, R6.2, R7.2
- net M1_FWD: now also Q2.D10; no longer Q1.D10
- net M1_REV: now also Q2.D11; no longer Q1.D11
- net N$1: now also R7.2; no longer R1.2
- net N$10: now also Q2.D9, R1.2; no longer Q1.D9, R3.2
- net N$11: now also Q2.D8, R3.2; no longer Q1.D8, R2.2
- net N$14: now also R1.1; no longer R3.1
- net N$3: now also Q1.D; no longer Q2.D
- net N$5: now also Q1.G, R4.1; no longer Q2.G, R6.1
- net N$6: now also R5.1; no longer R7.1
- net N$8: now also R7.1; no longer R1.1
- net RESET: now also Q2./RESET, R6.1; no longer Q1./RESET, R4.1
Other:
- moved on the sheet: LED2, LED3, R1, R2, R3, R4, R5, R6, R7
