File: labs/week-4-schematic.kicad_sch (KiCad schematic)
At the start: 24 parts, among them J1 GY-521-MPU-6050, SW1 PTS645, SW2 PTS645, SW3 PTS645, U1 TLE493DA2B6HTSA1

Commit message: Add lab files for Week 4
Parts:
- C1, C2, C3, C4: footprint (none) -> Capacitor_SMD:C_0805_2012Metric_Pad1.18x1.45mm_HandSolder
- D1, D2, D3, D4, D5, D6: footprint (none) -> LED_SMD:LED_0603_1608Metric_Pad1.05x0.95mm_HandSolder
- J1: footprint (none) -> SparkFun-Connector:1X08
- MOD1: footprint ARDUINO-UNO-R3:ARDUINO-UNO-R3 -> RoboJackets:ARDUINO_UNO_R3
- R1, R2, R3, R4, R5, R6, R7: footprint (none) -> Resistor_SMD:R_0603_1608Metric_Pad0.98x0.95mm_HandSolder
- RN1: footprint (none) -> RoboJackets:742C163331JP
- SW1, SW2, SW3: footprint (none) -> RoboJackets:PTS645SM43SMTR
- U1: footprint (none) -> RoboJackets:TLE493DA2B6HTSA1
