File: labs/week-4.kicad_sch (KiCad schematic)
At the start: 24 parts, among them J1 GY-521-MPU-6050, SW1 PTS645, SW2 PTS645, SW3 PTS645, U1 TLE493DA2B6HTSA1

Commit message: Fix schematic with fixed symbol
Parts:
- RN1: value 330 -> R_Pack8_US; footprint RoboJackets:742C163331JP -> (none)
Connections:
- net +5V: now also RN1.8; no longer RN1.15
- net D2_CTRL: now also RN1.2; no longer RN1.3
- net D3_CTRL: now also RN1.3; no longer RN1.5
- net D4_CTRL: now also RN1.4; no longer RN1.7
- net D5_CTRL: now also RN1.5; no longer RN1.9
- net at D1.2 (A): now also RN1.16; no longer RN1.2
- net at D4.2 (A): now also RN1.13; no longer RN1.8
- net at D5.2 (A): now also RN1.12; no longer RN1.10
- net at D2.2 (A): now also RN1.15; no longer RN1.4
- net at D6.2 (A): now also RN1.9; no longer RN1.16
- net at D3.2 (A): now also RN1.14; no longer RN1.6

Commit message: Convert soldering training board from EAGLE to KiCad
Parts:
- RN1: footprint (none) -> RoboJackets:742C163331JP
Changed lines of the file:
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@@
       (effects (font (size 1.27 1.27)))
     )
-    (property "Footprint" "" (at 133.4135 22.9235 0)
+    (property "Footprint" "RoboJackets:742C163331JP" (at 133.4135 22.9235 0)
       (effects (font (size 1.27 1.27)) hide)
     )
